File: fuse-board/fuse-board.kicad_sch (KiCad schematic)
At the start: 27 parts, among them J1 FTSH-107-01-F-DV-K-P-TR, J2 74651173R, J3 74651173R, J4 ATM15-12PA-BM04, J5 1053141106, SW1 Y97KT23B5NAFP, U1 STM32G491KCUx, U2 AP63205WU, U3 MIC5504-3.3YM5, Y1 ECS-240-8-37B-CKY-TR

Commit message: add efuses and sheets
Parts:
- removed C1, C2: 6.8pF, Capacitor_SMD:C_0603_1608Metric_Pad1.08x0.95mm_HandSolder, symbol Device:C
- removed C3, C5, C6, C8: 100nF, Capacitor_SMD:C_0603_1608Metric_Pad1.08x0.95mm_HandSolder, symbol Device:C
- removed C4: 10uF, Capacitor_SMD:C_0603_1608Metric_Pad1.08x0.95mm_HandSolder, symbol Device:C
- removed C7: 1uF, Capacitor_SMD:C_0603_1608Metric_Pad1.08x0.95mm_HandSolder, symbol Device:C
- removed FB1: FCM 1608KF-601T03, Inductor_SMD:L_0603_1608Metric_Pad1.05x0.95mm_HandSolder, symbol Device:FerriteBead
- removed J1: FTSH-107-01-F-DV-K-P-TR, Connector_PinHeader_1.27mm:PinHeader_2x07_P1.27mm_Vertical_SMD, symbol Connector_Generic:Conn_02x07_Odd_Even
- removed R1: 10k, Resistor_SMD:R_0603_1608Metric_Pad0.98x0.95mm_HandSolder, symbol Device:R
- removed SW1: Y97KT23B5NAFP, Button_Switch_SMD:SW_SPST_PTS647_Sx38, symbol Switch:SW_Push
- removed U1: STM32G491KCUx, Package_DFN_QFN:QFN-32-1EP_5x5mm_P0.5mm_EP3.45x3.45mm, symbol MCU_ST_STM32G4:STM32G491KCUx
- removed Y1: ECS-240-8-37B-CKY-TR, Crystal:Crystal_SMD_2016-4Pin_2.0x1.6mm, symbol Device:Crystal_GND24
Connections:
- net 12V_In renamed 12V_IN
- no-connect marks 4 -> 0
Other:
- added sheet Efuses (efuses.kicad_sch)
- added sheet Efuses Fans (efuses-fans.kicad_sch)
- added sheet MCU (mcu.kicad_sch)
- note removed: "24MHz"
- note removed: "Decoupling 100nF capacitors need to be placed as close to respective Vdd/Vss as possible. Note that VSS contains all VSS mcu pins for each VDD/VSS pair."
- note removed: "ST-Link Programming/Debugging Connector"
- note removed: "STM32G491KCU6 MCU"
- moved on the sheet: C10, C11, C12, C13, C9, L1, U2, U3

Commit message: prot components
Parts:
- added C23, C47: 47uF, symbol Device:C
- added C48, C49: 10uF, symbol Device:C
- added D1: SMCJ18A, symbol Device:D_Zener
- added D2, D3, D4: SS34, symbol Device:D_Schottky
Connections:
- net 12V_IN: now also C23.1, C47.1, C48.1, C49.1, D1.1 (K)
- net GND: now also C23.2, C47.2, C48.2, C49.2, D1.2 (A), D2.2 (A), D3.2 (A), D4.2 (A)
- net TB_Fan_A: now also D2.1 (K)
- net TB_Fan_C: now also D4.1 (K)
- new net Efuses Fans/FANB_OUT: D3.1 (K)

Commit message: add sheet pins and status LEDs
Other:
- note added: "Fused Circuits + MCU"
- note added: "Pwr-in, bulk caps, protection"
- moved on the sheet: C23, C47, C48, C49, D1, D2, D3, D4, F1, J2, J3, J4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

Commit message: fix weird unconnected wire
Connections:
- net Efuses Fans/FANB_OUT is gone; now on net TB_Fan_B: D3.1 (K)

Commit message: add LEDs (1 gpio)
Parts:
- added C54, C55: 100nF, Capacitor_SMD:C_0805_2012Metric_Pad1.18x1.45mm_HandSolder, symbol Device:C
- added U14: ISO1044BD, Package_SO:SOIC-8_3.9x4.9mm_P1.27mm, symbol Interface_CAN_LIN:ISO1044BD
Connections:
- net +3V3: now also C54.1, U14.1 (VCC1)
- net +5V: now also C55.1, U14.8 (VCC2)
- net GND: now also C54.2, C55.2, U14.4 (GND1), U14.7 (GND2)
- new net CANRX: U14.3 (RXD)
- new net CANTX: U14.2 (TXD)
Other:
- sheet MCU ports: added CANRX, CANTX; removed none
- note added: "CAN Transceiver"

Commit message: combine similar components
Parts:
- C10: Digikey Part Number (none) -> 311-1140-1-ND; Manufacturer Part Number (none) -> CC0805KRX7R9BB104; PN CC0805KRX7R9BB104 -> (none)
- C11: Manufacturer Part Number (none) -> CL21A476MQYNNNE; PN CL21A476MQYNNNE -> (none)
- C12, C13: Manufacturer Part Number (none) -> CL21B105KBFNNNE; PN CL21B105KBFNNNE -> (none)
- C23, C47: footprint (none) -> Capacitor_SMD:C_0805_2012Metric_Pad1.18x1.45mm_HandSolder; Manufacturer (none) -> Samsung Electro-Mechanics; Manufacturer Part Number (none) -> CL21A476MQYNNNE
- C48, C49: footprint (none) -> Capacitor_SMD:C_0603_1608Metric_Pad1.08x0.95mm_HandSolder; Digikey Part Number (none) -> 1276-CL10A106KO8NQNCCT-ND; Digikey URL (none) -> https://www.digikey.com/en/products/detail/samsung-electro-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; Manufacturer (none) -> Samsung Electro-Mechanics; Manufacturer Part Number (none) -> CL10A106KO8NQNC
- C54, C55: Digi PN 311-1140-1-ND -> (none); Digikey Part Number (none) -> 311-1140-1-ND; MFG Yageo -> (none); MFG PN CC0805KRX7R9BB104 -> (none); Manufacturer (none) -> Yageo; Manufacturer Part Number (none) -> CC0805KRX7R9BB104
- C9: Manufacturer Part Number (none) -> CL21A106KOQNNNG; PN CL21A106KOQNNNG -> (none)
- J2, J3: Digi PN 732-74651173RCT-ND -> (none); Digi URL https://www.digikey.com/en/products/detail/w%C3%BCrth-elekt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 -> (none); Digikey Part Number (none) -> 732-74651173RCT-ND; Digikey URL (none) -> https://www.digikey.com/en/products/detail/w%C3%BCrth-elekt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; MFG Würth Elektronik -> (none); MFG PN 74651173R -> (none); Manufacturer (none) -> Würth Elektronik; Manufacturer Part Number (none) -> 74651173R
- J4: Digi PN 889-3307-ND -> (none); Digi URL https://www.digikey.com/en/products/detail/amphenol-sine-sy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 -> (none); Digikey Part Number (none) -> 889-3307-ND; Digikey URL (none) -> https://www.digikey.com/en/products/detail/amphenol-sine-sy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; MFG Amphenol Sine Systems Corp -> (none); MFG PN ATM15-12PA-BM04 -> (none); Manufacturer (none) -> Amphenol Sine Systems Corp; Manufacturer Part Number (none) -> ATM15-12PA-BM04
- J5: Digi PN WM16908-ND -> (none); Digi URL https://www.digikey.com/en/products/detail/molex/1053141106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 -> (none); Digikey Part Number (none) -> WM16908-ND; Digikey URL (none) -> https://www.digikey.com/en/products/detail/molex/1053141106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; MFG Molex -> (none); MFG PN 1053141106 -> (none); Manufacturer (none) -> Molex; Manufacturer Part Number (none) -> 1053141106
- L1: Manufacturer Part Number (none) -> SRP5030TA-4R7M; PN SRP5030TA-4R7M -> (none)
- U14: Digi PN 296-ISO1044BDRCT-ND -> (none); Digikey Part Number (none) -> 296-ISO1044BDRCT-ND; MFG Texas Instruments -> (none); MFG PN ISO1044BDR -> (none); Manufacturer (none) -> Texas Instruments; Manufacturer Part Number (none) -> ISO1044BDR

Commit message: source except remaining passives
Parts:
- C10, C54, C55: Digikey URL (none) -> https://www.digikey.com/en/products/detail/yageo/CC0805KRX7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
- C11, C23, C47: Digikey Part Number (none) -> 1276-1852-1-ND; Digikey URL (none) -> https://www.digikey.com/en/products/detail/samsung-electro-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
- C12, C13: Digikey Part Number (none) -> 1276-1029-1-ND; Digikey URL (none) -> https://www.digikey.com/en/products/detail/samsung-electro-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
- C9: Digikey Part Number (none) -> 1276-6455-1-ND; Digikey URL (none) -> https://www.digikey.com/en/products/detail/samsung-electro-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
- D1: footprint (none) -> Diode_SMD:D_SMB-SMC_Universal_Handsoldering; Digikey Part Number (none) -> SMCJ18ALFCT-ND; Digikey URL (none) -> https://www.digikey.com/en/products/detail/littelfuse-inc/S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; Manufacturer (none) -> Littelfuse Inc.; Manufacturer Part Number (none) -> SMCJ18A
- D2, D3, D4: footprint (none) -> Diode_SMD:D_SMB-SMC_Universal_Handsoldering; Digikey Part Number (none) -> SS34FSCT-ND; Digikey URL (none) -> https://www.digikey.com/en/products/detail/onsemi/SS34/1052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; Manufacturer (none) -> onsemi; Manufacturer Part Number (none) -> SS34
- L1: Digikey Part Number (none) -> SRP5030TA-4R7MCT-ND; Digikey URL (none) -> https://www.digikey.com/en/products/detail/bourns-inc/SRP50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
- U14: Digikey URL (none) -> https://www.digikey.com/en/products/detail/texas-instrument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
- U2: Digikey Part Number (none) -> AP63205WU-7DICT-ND; Digikey URL (none) -> https://www.digikey.com/en/products/detail/diodes-incorpora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; Manufacturer (none) -> Diodes Incorporated; Manufacturer Part Number (none) -> AP63205WU-7
- U3: Digikey Part Number (none) -> 576-4764-1-ND; Digikey URL (none) -> https://www.digikey.com/en/products/detail/microchip-techno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; Manufacturer (none) -> Microchip Technology; Manufacturer Part Number (none) -> MIC5504-3.3YM5-TR

Commit message: src and fix some issues
Parts:
- F1: footprint (none) -> Fuse:Fuse_1812_4532Metric_Pad1.30x3.40mm_HandSolder; Digikey Part Number (none) -> F5632CT-ND; Digikey URL (none) -> https://www.digikey.com/en/products/detail/littelfuse-inc/1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; Manufacturer (none) -> Littelfuse Inc.; Manufacturer Part Number (none) -> 1812L110/24DR
Changed lines of the file:
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@@
 			)
 		)
-		(property "Footprint" ""
+		(property "Footprint" "Fuse:Fuse_1812_4532Metric_Pad1.30x3.40mm_HandSolder"
 			(at 49.53 38.1 0)
 			(hide yes)
@@
 			)
 		)
-		(property "Datasheet" ""
+		(property "Datasheet" "https://www.littelfuse.com/assetdocs/resettable-ptcs-1812l-datasheet?assetguid=ca5c80cb-504e-4a8a-8e74-0107520a1717"
 			(at 48.26 33.02 0)
 			(hide yes)
@@
 			(at 48.26 33.02 0)
 			(hide yes)
+			(show_name no)
+			(do_not_autoplace no)
+			(effects
+				(font
+					(size 1.27 1.27)
+				)
+			)
+		)
+		(property "Digikey Part Number" "F5632CT-ND"
+			(at 48.26 33.02 0)
+			(hide yes)
+			(show_name no)
+			(do_not_autoplace no)
+			(effects
+				(font
+					(size 1.27 1.27)
+				)
+			)
+		)
+		(property "Digikey URL" "https://www.digikey.com/en/products/detail/littelfuse-inc/1812L110-24DR/2520731?s=N4IgTCBcDaIIwA45gDZzgBgPRgCwBMAnEAXQF8g"
+			(at 48.26 33.02 0)
+			(hide yes)
+			(show_name no)
+			(do_not_autoplace no)
+			(effects
+				(font
+					(size 1.27 1.27)
+				)
+			)
+		)
+		(property "Manufacturer" "Littelfuse Inc."
+			(at 48.26 33.02 0)
+			(hide yes)
+			(show_name no)
+			(do_not_autoplace no)
+			(effects
+				(font
+					(size 1.27 1.27)
+				)
+			)
+		)
+		(property "Manufacturer Part Number" "1812L110/24DR"
+			(at 48.26 33.02 0)
+			(hide yes)
