File: fuse-board/fuse-board.kicad_sch (KiCad schematic)
At the start: 24 parts, among them J2 74651173R, J3 74651173R, J4 ATM15-12PA-BM04, J5 1053141106, U14 ISO1044BD, U2 AP63205WU, U3 MIC5504-3.3YM5

Commit message: get rid of LEDs and add LED_SIGNAL
Other:
- sheet MCU ports: added LED_SIGNAL; removed none
Changed lines of the file:
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@@
 	(wire
 		(pts
-			(xy 31.75 148.59) (xy 34.29 148.59)
+			(xy 31.75 151.13) (xy 34.29 151.13)
 		)
 		(stroke
@@
 	(wire
 		(pts
-			(xy 34.29 146.05) (xy 29.21 146.05)
+			(xy 34.29 148.59) (xy 29.21 148.59)
 		)
 		(stroke
@@
 	(wire
 		(pts
-			(xy 63.5 148.59) (xy 60.96 148.59)
+			(xy 63.5 151.13) (xy 60.96 151.13)
 		)
 		(stroke
@@
 	(wire
 		(pts
-			(xy 68.58 143.51) (xy 60.96 143.51)
+			(xy 68.58 146.05) (xy 60.96 146.05)
 		)
 		(stroke
@@
 	(wire
 		(pts
-			(xy 26.67 166.37) (xy 26.67 143.51)
+			(xy 26.67 166.37) (xy 26.67 146.05)
 		)
 		(stroke
@@
 	(wire
 		(pts
-			(xy 63.5 161.29) (xy 63.5 148.59)
+			(xy 63.5 161.29) (xy 63.5 151.13)
 		)
 		(stroke
@@
 	(wire
 		(pts
-			(xy 68.58 166.37) (xy 68.58 143.51)
+			(xy 68.58 166.37) (xy 68.58 146.05)
 		)
 		(stroke
@@
 	(wire
 		(pts
-			(xy 66.04 163.83) (xy 66.04 146.05)
+			(xy 66.04 163.83) (xy 66.04 148.59)
 		)
 		(stroke
@@
 	(wire
 		(pts
-			(xy 31.75 161.29) (xy 31.75 148.59)
+			(xy 31.75 161.29) (xy 31.75 151.13)
 		)
 		(stroke
@@
 	(wire
 		(pts
-			(xy 29.21 146.05) (xy 29.21 163.83)
+			(xy 29.21 148.59) (xy 29.21 163.83)
 		)
 		(stroke
@@
 	(wire
 		(pts
-			(xy 66.04 146.05) (xy 60.96 146.05)
+			(xy 66.04 148.59) (xy 60.96 148.59)
 		)
 		(stroke
@@
 	(wire
 		(pts
-			(xy 26.67 143.51) (xy 34.29 143.51)
+			(xy 26.67 146.05) (xy 34.29 146.05)
 		)
 		(stroke
@@
 	(sheet
 		(at 34.29 118.11)
-		(size 26.67 33.02)
+		(size 26.67 35.56)
 		(exclude_from_sim no)
 		(in_bom yes)
@@
 		)
 		(property "Sheetfile" "mcu.kicad_sch"
-			(at 34.29 151.7146 0)
+			(at 34.29 154.2546 0)
 			(show_name no)
 			(do_not_autoplace no)
@@
 		)
 		(pin "FANA_IMON" input
-			(at 60.96 143.51 0)
+			(at 60.96 146.05 0)
 			(effects
 				(font
@@
 		)
 		(pin "FANB_IMON" input
-			(at 60.96 146.05 0)
+			(at 60.96 148.59 0)
 			(effects
 				(font
@@
 		)
 		(pin "FANC_IMON" input
-			(at 60.96 148.59 0)
+			(at 60.96 151.13 0)
 			(effects
 				(font
@@
 		)
 		(pin "FANA_EN" output
-			(at 34.29 148.59 180)
+			(at 34.29 151.13 180)
 			(effects
 				(font
@@
 		)
 		(pin "FANB_EN" output
-			(at 34.29 146.05 180)
+			(at 34.29 148.59 180)
 			(effects
 				(font
@@
 		)
 		(pin "FANC_EN" output
-			(at 34.29 143.51 180)
+			(at 34.29 146.05 180)
 			(effects
 				(font
@@
 			(effects
 				(font
+					(size 1.27 1.27)
+				)
+				(justify right)
+			)
+		)
+		(pin "LED_SIGNAL" output
+			(at 60.96 142.24 0)
+			(effects
+				(font

Commit message: switch efuse config and symbol
passives still need to be sourced
Other:
- removed sheet Efuses Fans
- sheet Efuses ports: added FANA_EN, FANA_IMON, FANA_OUT, FANB_EN, FANB_IMON, FANB_OUT, FANC_EN, FANC_IMON, FANC_OUT; removed none
- moved on the sheet: C54, C55, U14

Commit message: add connectors and source components
Parts:
- added J6: 1053131102, Connector_Molex:Molex_Nano-Fit_105313-xx02_1x02_P2.50mm_Horizontal, symbol Connector_Generic:Conn_01x02
- added J7: 1053131203, Connector_Molex:Molex_Nano-Fit_105313-xx03_1x03_P2.50mm_Horizontal, symbol Connector_Generic:Conn_01x03
Connections:
- net +5V: now also J7.2 (Pin_2)
- net GND: now also J7.3 (Pin_3)
- net MCU/LED_SIGNAL: now also J7.1 (Pin_1)
- net at U14.5 (CANL): now also J6.2 (Pin_2)
- net at U14.6 (CANH): now also J6.1 (Pin_1)
Other:
- moved on the sheet: C54, C55, D2, D4, U14, U2

Commit message: combine pins, 9 adc pins, notes
Other:
- note added: "bigger capacitor, ferrite bead from 5v supply"
- note added: "net lines for power and board setup"
Changed lines of the file:
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@@
+		)
+	)
+	(text "bigger capacitor, ferrite bead from 5v supply"
+		(exclude_from_sim no)
+		(at 231.648 106.426 0)
+		(effects
+			(font
+				(size 1.27 1.27)
+			)
 		)
 	)
@@
 		)
 	)
+	(text "net lines for power and board setup"
+		(exclude_from_sim no)
+		(at 202.438 119.888 0)
+		(effects
+			(font
+				(size 1.27 1.27)
+			)
+		)
+	)
