File: fuse-board/efuses-fans.kicad_sch (KiCad schematic)
At the start: 21 parts, among them U10 PTPS259830LNRGER, U11 PTPS259830LNRGER, U12 PTPS259830LNRGER

Commit message: combine similar components
Parts:
- C20, C21, C22: Digi PN 311-3484-1-ND -> (none); Digi URL https://www.digikey.com/en/products/detail/yageo/CC0603JRX7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 -> (none); Digikey Part Number (none) -> 1276-CL10B105KB9VPJCCT-ND; Digikey URL (none) -> https://www.digikey.com/en/products/detail/samsung-electro-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; MFG Yageo -> (none); MFG PN CC0603JRX7R6BB105 -> (none); Manufacturer (none) -> Samsung Electro-Mechanics; Manufacturer Part Number (none) -> CL10B105KB9VPJC
- R14, R16, R18: value 280 -> 113
- R15, R17, R19: value 6.04k -> 1.05k
Other:
- note added: "U10 / U11 / U12 Fans (13A to emulate 10A blade): R_ILIM = 113 Ω → I_LIM = 13.0 A R_IMON = 1.05 kΩ → V_IMON @ 13 A ≈ 3.26 V C_ITIMER = 10 nF → t_ITIMER = 4.67 ms C_dVdt = 10 nF → SR ≈ 0.46 V/ms (turn-on ~26 ms @ 12 V)"
Changed lines of the file:
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@@
 	(generator_version "10.0")
 	(paper "A4")
+	(text "U10 / U11 / U12 Fans (13A to emulate 10A blade):\nR_ILIM = 113 Ω → I_LIM = 13.0 A\nR_IMON = 1.05 kΩ → V_IMON @ 13 A ≈ 3.26 V\nC_ITIMER = 10 nF → t_ITIMER = 4.67 ms\nC_dVdt = 10 nF → SR ≈ 0.46 V/ms (turn-on ~26 ms @ 12 V)"
+		(exclude_from_sim no)
+		(at 188.976 32.258 0)
+		(effects
+			(font
+				(size 1.27 1.27)
+			)
+			(justify left)
+		)
+	)
 	(junction
 		(at 38.1 138.43)
@@
 			)
 		)
-		(property "Value" "280"
+		(property "Value" "113"
 			(at 199.39 69.8499 0)
 			(show_name no)
@@
 			)
 		)
-		(property "Datasheet" "https://mm.digikey.com/Volume0/opasdata/d220001/medias/docus/3584/CL10B105KP8NNNC_Spec.pdf"
+		(property "Datasheet" "https://mm.digikey.com/Volume0/opasdata/d220001/medias/docus/5458/CL10B105KB9VPJC_Spec.pdf"
 			(at 250.19 86.36 0)
 			(hide yes)
@@
 			)
 		)
-		(property "Digi PN" "311-3484-1-ND"
+		(property "Digi PN" ""
 			(at 250.19 86.36 0)
 			(hide yes)
@@
 			)
 		)
-		(property "MFG" "Yageo"
+		(property "MFG" ""
 			(at 250.19 86.36 0)
 			(hide yes)
@@
 			)
 		)
-		(property "MFG PN" "CC0603JRX7R6BB105"
+		(property "MFG PN" ""
 			(at 250.19 86.36 0)
 			(hide yes)
@@
 			)
 		)
-		(property "Digi URL" "https://www.digikey.com/en/products/detail/yageo/CC0603JRX7R6BB105/7164368"
+		(property "Digi URL" ""
 			(at 250.19 86.36 0)
 			(hide yes)
@@
 			)
 		)
-		(property "Manufacturer" ""
+		(property "Manufacturer" "Samsung Electro-Mechanics"
 			(at 250.19 86.36 0)
 			(hide yes)
@@
 			)
 		)
-		(property "Digikey Part Number" ""
+		(property "Digikey Part Number" "1276-CL10B105KB9VPJCCT-ND"
 			(at 250.19 86.36 0)
 			(hide yes)
@@
 			)
 		)
-		(property "Digikey URL" ""
+		(property "Digikey URL" "https://www.digikey.com/en/products/detail/samsung-electro-mechanics/cl10b105kb9vpjc/20498526"
 			(at 250.19 86.36 0)
 			(hide yes)
@@
 			)
 		)
-		(property "Manufacturer Part Number" ""
+		(property "Manufacturer Part Number" "CL10B105KB9VPJC"
 			(at 250.19 86.36 0)
 			(hide yes)
@@
 			)
 		)
-		(property "Value" "6.04k"
+		(property "Value" "1.05k"
 			(at 99.06 34.2899 0)
 			(show_name no)
@@
 			)
 		)
-		(property "Value" "280"
+		(property "Value" "113"
 			(at 88.9 109.2199 0)
 			(show_name no)
@@
 			)
 		)
-		(property "Value" "280"
+		(property "Value" "113"
 			(at 88.9 34.2899 0)
 			(show_name no)
@@
 			)
 		)
-		(property "Value" "6.04k"
+		(property "Value" "1.05k"
 			(at 99.06 109.2199 0)
 			(show_name no)
@@
 			)
 		)
-		(property "Value" "6.04k"
+		(property "Value" "1.05k"
 			(at 209.55 69.8499 0)
 			(show_name no)
@@
 			)
 		)
-		(property "Datasheet" "https://mm.digikey.com/Volume0/opasdata/d220001/medias/docus/3584/CL10B105KP8NNNC_Spec.pdf"
+		(property "Datasheet" "https://mm.digikey.com/Volume0/opasdata/d220001/medias/docus/5458/CL10B105KB9VPJC_Spec.pdf"
 			(at 256.54 86.36 0)
 			(hide yes)
@@
 			)
 		)
-		(property "Digi PN" "311-3484-1-ND"
+		(property "Digi PN" ""
 			(at 256.54 86.36 0)
 			(hide yes)
@@
 			)
 		)
-		(property "MFG" "Yageo"
+		(property "MFG" ""
 			(at 256.54 86.36 0)
 			(hide yes)
@@
 			)
 		)
-		(property "MFG PN" "CC0603JRX7R6BB105"
+		(property "MFG PN" ""
 			(at 256.54 86.36 0)
 			(hide yes)
@@
 			)
 		)
-		(property "Digi URL" "https://www.digikey.com/en/products/detail/yageo/CC0603JRX7R6BB105/7164368"
+		(property "Digi URL" ""
 			(at 256.54 86.36 0)
 			(hide yes)
@@
 			)
 		)
-		(property "Manufacturer" ""
+		(property "Manufacturer" "Samsung Electro-Mechanics"
 			(at 256.54 86.36 0)
 			(hide yes)
@@
 			)
 		)
-		(property "Digikey Part Number" ""
+		(property "Digikey Part Number" "1276-CL10B105KB9VPJCCT-ND"
 			(at 256.54 86.36 0)
 			(hide yes)
@@
 			)
 		)
-		(property "Digikey URL" ""
+		(property "Digikey URL" "https://www.digikey.com/en/products/detail/samsung-electro-mechanics/cl10b105kb9vpjc/20498526"
 			(at 256.54 86.36 0)
 			(hide yes)
@@
 			)
 		)
-		(property "Manufacturer Part Number" ""
+		(property "Manufacturer Part Number" "CL10B105KB9VPJC"
 			(at 256.54 86.36 0)
 			(hide yes)
@@
 			)
 		)
-		(property "Datasheet" "https://mm.digikey.com/Volume0/opasdata/d220001/medias/docus/3584/CL10B105KP8NNNC_Spec.pdf"
+		(property "Datasheet" "https://mm.digikey.com/Volume0/opasdata/d220001/medias/docus/5458/CL10B105KB9VPJC_Spec.pdf"
 			(at 262.89 86.36 0)
 			(hide yes)
@@
 			)
 		)
-		(property "Digi PN" "311-3484-1-ND"
+		(property "Digi PN" ""
 			(at 262.89 86.36 0)
 			(hide yes)
@@
 			)
 		)
-		(property "MFG" "Yageo"
+		(property "MFG" ""
 			(at 262.89 86.36 0)
 			(hide yes)
@@
 			)
 		)
-		(property "MFG PN" "CC0603JRX7R6BB105"
+		(property "MFG PN" ""
 			(at 262.89 86.36 0)
 			(hide yes)
@@
 			)
 		)
-		(property "Digi URL" "https://www.digikey.com/en/products/detail/yageo/CC0603JRX7R6BB105/7164368"
+		(property "Digi URL" ""
 			(at 262.89 86.36 0)
 			(hide yes)
@@
 			)
 		)
-		(property "Manufacturer" ""
+		(property "Manufacturer" "Samsung Electro-Mechanics"
 			(at 262.89 86.36 0)
 			(hide yes)
@@
 			)
 		)
-		(property "Digikey Part Number" ""
+		(property "Digikey Part Number" "1276-CL10B105KB9VPJCCT-ND"
 			(at 262.89 86.36 0)
 			(hide yes)
@@
 			)
 		)
-		(property "Digikey URL" ""
+		(property "Digikey URL" "https://www.digikey.com/en/products/detail/samsung-electro-mechanics/cl10b105kb9vpjc/20498526"
 			(at 262.89 86.36 0)
 			(hide yes)
@@
 			)
 		)
-		(property "Manufacturer Part Number" ""
+		(property "Manufacturer Part Number" "CL10B105KB9VPJC"
 			(at 262.89 86.36 0)
 			(hide yes)

Commit message: source except remaining passives
Parts:
- U10, U11, U12: Digikey Part Number (none) -> 296-TPS259830LNRGERCT-ND; Digikey URL (none) -> https://www.digikey.com/en/products/detail/texas-instrument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; Manufacturer (none) -> Texas Instruments; Manufacturer Part Number (none) -> TPS259830LNRGER
Other:
- note added: "U10 / U11 / U12 Fans (13A to emulate 10A blade): R_ILIM = 113 Ω → I_LIM = 13.0 A R_IMON = 1.05 kΩ → V_IMON @ 13 A ≈ 3.32 V C_ITIMER = 10 nF → t_ITIMER = 4.67 ms C_dVdt = 10 nF → SR ≈ 0.46 V/ms (turn-on ~26 ms @ 12 V)"
- note removed: "U10 / U11 / U12 Fans (13A to emulate 10A blade): R_ILIM = 113 Ω → I_LIM = 13.0 A R_IMON = 1.05 kΩ → V_IMON @ 13 A ≈ 3.26 V C_ITIMER = 10 nF → t_ITIMER = 4.67 ms C_dVdt = 10 nF → SR ≈ 0.46 V/ms (turn-on ~26 ms @ 12 V)"
Changed lines of the file:
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@@
 	(generator_version "10.0")
 	(paper "A4")
-	(text "U10 / U11 / U12 Fans (13A to emulate 10A blade):\nR_ILIM = 113 Ω → I_LIM = 13.0 A\nR_IMON = 1.05 kΩ → V_IMON @ 13 A ≈ 3.26 V\nC_ITIMER = 10 nF → t_ITIMER = 4.67 ms\nC_dVdt = 10 nF → SR ≈ 0.46 V/ms (turn-on ~26 ms @ 12 V)"
+	(text "U10 / U11 / U12 Fans (13A to emulate 10A blade):\nR_ILIM = 113 Ω → I_LIM = 13.0 A\nR_IMON = 1.05 kΩ → V_IMON @ 13 A ≈ 3.32 V\nC_ITIMER = 10 nF → t_ITIMER = 4.67 ms\nC_dVdt = 10 nF → SR ≈ 0.46 V/ms (turn-on ~26 ms @ 12 V)"
 		(exclude_from_sim no)
 		(at 188.976 32.258 0)
@@
 			)
 		)
+		(property "Digikey Part Number" "296-TPS259830LNRGERCT-ND"
+			(at 167.64 88.9 0)
+			(hide yes)
+			(show_name no)
+			(do_not_autoplace no)
+			(effects
+				(font
+					(size 1.27 1.27)
+				)
+			)
+		)
+		(property "Digikey URL" "https://www.digikey.com/en/products/detail/texas-instruments/TPS259830LNRGER/22106807"
+			(at 167.64 88.9 0)
+			(hide yes)
+			(show_name no)
+			(do_not_autoplace no)
+			(effects
+				(font
+					(size 1.27 1.27)
+				)
+			)
+		)
+		(property "Manufacturer" "Texas Instruments"
+			(at 167.64 88.9 0)
+			(hide yes)
+			(show_name no)
+			(do_not_autoplace no)
+			(effects
+				(font
+					(size 1.27 1.27)
+				)
+			)
+		)
+		(property "Manufacturer Part Number" "TPS259830LNRGER"
+			(at 167.64 88.9 0)
+			(hide yes)
+			(show_name no)
+			(do_not_autoplace no)
+			(effects
+				(font
+					(size 1.27 1.27)
+				)
+			)
+		)
 		(pin "9"
 		)
@@
 			)
 		)
+		(property "Digikey Part Number" "296-TPS259830LNRGERCT-ND"
+			(at 57.15 128.27 0)
+			(hide yes)
+			(show_name no)
+			(do_not_autoplace no)
+			(effects
+				(font
+					(size 1.27 1.27)
+				)
+			)
+		)
+		(property "Digikey URL" "https://www.digikey.com/en/products/detail/texas-instruments/TPS259830LNRGER/22106807"
+			(at 57.15 128.27 0)
+			(hide yes)
+			(show_name no)
+			(do_not_autoplace no)
+			(effects
+				(font
+					(size 1.27 1.27)
+				)
+			)
+		)
+		(property "Manufacturer" "Texas Instruments"
+			(at 57.15 128.27 0)
+			(hide yes)
+			(show_name no)
+			(do_not_autoplace no)
+			(effects
+				(font
+					(size 1.27 1.27)
+				)
+			)
+		)
+		(property "Manufacturer Part Number" "TPS259830LNRGER"
+			(at 57.15 128.27 0)
+			(hide yes)
+			(show_name no)
+			(do_not_autoplace no)
+			(effects
+				(font
+					(size 1.27 1.27)
+				)
+			)
+		)
 		(pin "9"
 		)
@@
 			(at 57.15 53.34 0)
 			(hide yes)
+			(show_name no)
+			(do_not_autoplace no)
+			(effects
+				(font
+					(size 1.27 1.27)
+				)
+			)
+		)
+		(property "Digikey Part Number" "296-TPS259830LNRGERCT-ND"
+			(at 57.15 53.34 0)
+			(hide yes)
+			(show_name no)
+			(do_not_autoplace no)
+			(effects
+				(font
+					(size 1.27 1.27)
+				)
+			)
+		)
+		(property "Digikey URL" "https://www.digikey.com/en/products/detail/texas-instruments/TPS259830LNRGER/22106807"
+			(at 57.15 53.34 0)
+			(hide yes)
+			(show_name no)
+			(do_not_autoplace no)
+			(effects
+				(font
+					(size 1.27 1.27)
+				)
+			)
+		)
+		(property "Manufacturer" "Texas Instruments"
+			(at 57.15 53.34 0)
+			(hide yes)
+			(show_name no)
+			(do_not_autoplace no)
+			(effects
+				(font
+					(size 1.27 1.27)
+				)
+			)
+		)
+		(property "Manufacturer Part Number" "TPS259830LNRGER"
+			(at 57.15 53.34 0)
+			(hide yes)

Commit message: all components sourced
Parts:
- C38, C39, C41, C42, C44, C45: footprint (none) -> Capacitor_SMD:C_0603_1608Metric_Pad1.08x0.95mm_HandSolder; Digikey Part Number (none) -> 311-1085-1-ND; Digikey URL (none) -> https://www.digikey.com/en/products/detail/yageo/CC0603KRX7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; Manufacturer (none) -> YAGEO; Manufacturer Part Number (none) -> CC0603KRX7R9BB103
- C40, C43, C46: footprint (none) -> Capacitor_SMD:C_0603_1608Metric_Pad1.08x0.95mm_HandSolder; Digikey Part Number (none) -> 311-1423-1-ND; Digikey URL (none) -> https://www.digikey.com/en/products/detail/yageo/CC0603JRNP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; Manufacturer (none) -> YAGEO; Manufacturer Part Number (none) -> CC0603JRNPO9BN102
- R14, R16, R18: footprint (none) -> Resistor_SMD:R_0603_1608Metric_Pad0.98x0.95mm_HandSolder; Digikey Part Number (none) -> 311-113HRCT-ND; Digikey URL (none) -> https://www.digikey.com/en/products/detail/yageo/RC0603FR-0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; Manufacturer (none) -> YAGEO; Manufacturer Part Number (none) -> RC0603FR-07113RL
- R15, R17, R19: footprint (none) -> Resistor_SMD:R_0603_1608Metric_Pad0.98x0.95mm_HandSolder; Digikey Part Number (none) -> 311-1.05KHRCT-ND; Digikey URL (none) -> https://www.digikey.com/en/products/detail/yageo/RC0603FR-0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; Manufacturer (none) -> YAGEO; Manufacturer Part Number (none) -> RC0603FR-071K05L
