File: fuse-board/efuses.kicad_sch (KiCad schematic)
At the start: 38 parts, among them U4 PTPS259830LNRGER, U5 PTPS259830LNRGER, U6 PTPS259830LNRGER, U7 PTPS259830LNRGER, U8 PTPS259830LNRGER, U9 PTPS259830LNRGER

Commit message: update tmux1308
Parts:
- added C53, C56, C57, C58: 1nF, Capacitor_SMD:C_0603_1608Metric_Pad1.08x0.95mm_HandSolder, symbol Device:C
Connections:
- net GND: now also C53.2, C56.2, C57.1, C58.1
- net at U4.15 (DVDT/_BGATE): now also C57.2
- net at U4.7 (ITIMER): now also C56.1
- net at R6.2: no longer U6.8 (ILIM)
- net at U6.15 (DVDT/_BGATE): now also C58.2
- net at U6.7 (ITIMER): now also C53.1
- no-connect marks 16 -> 12
Other:
- note added: "U4 PEB / U6 Telemetry / U7 TBB (7A to emulate a 5A blade): R_ILIM = 210 Ω → I_LIM = 1460/210 + 0.11 = 7.0 A R_IMON = 1.91 kΩ → V_IMON @ 7 A = 7 × 1.91k × 243 µA/A ≈ 3.25 V C_ITIMER = 1 nF → t_ITIMER = 0.47 ms C_dVdt = 1 nF → SR ≈ 4.6 V/ms (turn-on ~2.6 ms @ 12 V) U5 Shutdown / U8 Inverter / U9 VCU (13A to emulate a 10A blade): R_ILIM = 113 Ω → I_LIM = 1460/113 + 0.11 = 13.0 A R_IMON = 1.05 kΩ → V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"
- note removed: "U4 PEB / U6 Telemetry / U7 TBB (7A to emulate a 5A blade): R_ILIM = 210 Ω → I_LIM = 1460/210 + 0.11 = 7.0 A R_IMON = 1.91 kΩ → V_IMON @ 7 A = 7 × 1.91k × 243 µA/A ≈ 3.25 V C_ITIMER / C_dVdt = open (max slew) U5 Shutdown / U8 Inverter / U9 VCU (13A to emulate a 10A blade): R_ILIM = 113 Ω → I_LIM = 1460/113 + 0.11 = 13.0 A R_IMON = 1.05 kΩ → V_IMON @ 13 A = 13 × 1.05k × 243 µA/A ≈ 3.32 V C_ITIMER =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"
- moved on the sheet: C24, C25, C29, C30, C31, R2, R3, R6, R7, R8, R9, U7

Commit message: switch efuse config and symbol
passives still need to be sourced
Parts:
- removed C24, C25, C26, C27, C28, C29, C30, C31, C32, C33, C34, C35, C36, C37, C53, C56: 1nF, Capacitor_SMD:C_0603_1608Metric_Pad1.08x0.95mm_HandSolder, symbol Device:C
- removed R11, R13: 1.05k, Resistor_SMD:R_0603_1608Metric_Pad0.98x0.95mm_HandSolder, symbol Device:R
- removed R12: 113, Resistor_SMD:R_0603_1608Metric_Pad0.98x0.95mm_HandSolder, symbol Device:R
- removed U4, U5, U6, U7, U8, U9: PTPS259830LNRGER, formula_slug_footprint_library:VQFN24_RGE_TEX, symbol formula_slug_symbol_library:PTPS259830LNRGER
- added C20, C21, C22: 1uF, Capacitor_SMD:C_0603_1608Metric_Pad1.08x0.95mm_HandSolder, symbol Device:C
- added C59: 1nF, Capacitor_SMD:C_0603_1608Metric_Pad1.08x0.95mm_HandSolder, symbol Device:C
- added C60, C63, C65, C68, C71, C74, C77, C80, C83: 3.3nF, Capacitor_SMD:C_0603_1608Metric_Pad1.08x0.95mm_HandSolder, symbol Device:C
- added C61, C62, C64, C66, C67, C69, C70, C72, C73, C75, C76, C78, C79, C81, C82, C84: 15nF, Capacitor_SMD:C_0603_1608Metric_Pad1.08x0.95mm_HandSolder, symbol Device:C
- added R31, R34, R36, R37, R38, R39: 113, Resistor_SMD:R_0603_1608Metric_Pad0.98x0.95mm_HandSolder, symbol Device:R
- added R32, R33, R35: 210, Resistor_SMD:R_0603_1608Metric_Pad0.98x0.95mm_HandSolder, symbol Device:R
- added U10, U11, U12, U4, U5, U6, U7, U8, U9: TPS259830ONRGER, formula_slug_footprint_library:TPS259830ONRGER, symbol formula_slug_symbol_library:TPS259830ONRGER
- C57, C58: value 1nF -> 15nF; Digikey Part Number 311-1423-1-ND -> (none); Digikey URL https://www.digikey.com/en/products/detail/yageo/CC0603JRNP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 -> (none); Manufacturer YAGEO -> (none); Manufacturer Part Number CC0603JRNPO9BN102 -> (none)
- R10: value 113 -> 1.02k; Digikey Part Number 311-113HRCT-ND -> (none); Digikey URL https://www.digikey.com/en/products/detail/yageo/RC0603FR-0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 -> (none); Manufacturer YAGEO -> (none); Manufacturer Part Number RC0603FR-07113RL -> (none)
- R3, R8: value 210 -> 1.02k; Digikey Part Number 311-210HRCT-ND -> (none); Digikey URL https://www.digikey.com/en/products/detail/yageo/RC0603FR-0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 -> (none); Manufacturer YAGEO -> (none); Manufacturer Part Number RC0603FR-07210RL -> (none)
- R4: value 113 -> 1.91k; Digikey Part Number 311-113HRCT-ND -> 13-AC0603FR-071K91LCT-ND; Digikey URL https://www.digikey.com/en/products/detail/yageo/RC0603FR-0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 -> https://www.digikey.com/en/products/detail/yageo/AC0603FR-0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; Manufacturer Part Number RC0603FR-07113RL -> AC0603FR-071K91L
- R5: value 1.05k -> 1.02k; Digikey Part Number 311-1.05KHRCT-ND -> (none); Digikey URL https://www.digikey.com/en/products/detail/yageo/RC0603FR-0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 -> (none); Manufacturer YAGEO -> (none); Manufacturer Part Number RC0603FR-071K05L -> (none)
- R6: value 210 -> 1.91k; Digikey Part Number 311-210HRCT-ND -> 13-AC0603FR-071K91LCT-ND; Digikey URL https://www.digikey.com/en/products/detail/yageo/RC0603FR-0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 -> https://www.digikey.com/en/products/detail/yageo/AC0603FR-0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; Manufacturer Part Number RC0603FR-07210RL -> AC0603FR-071K91L
- R7, R9: value 1.91k -> 1.02k; Digikey Part Number 13-AC0603FR-071K91LCT-ND -> (none); Digikey URL https://www.digikey.com/en/products/detail/yageo/AC0603FR-0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 -> (none); Manufacturer YAGEO -> (none); Manufacturer Part Number AC0603FR-071K91L -> (none)
Connections:
- net 12V_IN: now also C14.2, C15.2, C16.2, C17.2, C18.2, C19.2, C20.2, C21.2, C22.2, U10.[1,2,3,16,25] (IN), U11.[1,2,3,16,25] (IN), U12.[1,2,3,16,25] (IN), U4.[1,2,3,16,25] (IN), U5.[1,2,3,16,25] (IN), U6.[1,2,3,16,25] (IN), U7.[1,2,3,16,25] (IN), U8.[1,2,3,16,25] (IN), U9.[1,2,3,16,25] (IN); no longer C14.1, C15.1, C16.1, C17.1, C18.1, C19.1
- net GND: now also C14.1, C15.1, C16.1, C17.1, C18.1, C19.1, C57.2, C58.2, R10.2, R2.2, R3.2, R4.2, R5.2, R6.2, R7.2, R8.2, R9.2, C20.1, C21.1, C22.1, C60.2, C61.2, C62.2, C63.2, C64.2, C65.2, C66.2, C67.2, C68.2, C69.2, C70.2, C71.2, C72.2, C73.2, C74.2, C75.2, C76.2, C77.2, C78.2, C79.2, C80.2, C81.2, C82.2, C83.2, C84.2, R31.1, R32.1, R33.1, R34.1, R35.1, R36.1, R37.1, R38.1, R39.1, U10.10 (RETRY_DLY), U10.12 (OVLO), U10.[4,5,14,26] (GND), U11.10 (RETRY_DLY), U11.12 (OVLO), U11.[4,5,14,26] (GND), U12.10 (RETRY_DLY), U12.12 (OVLO), U12.[4,5,14,26] (GND), U4.10 (RETRY_DLY), U4.12 (OVLO), U4.[4,5,14,26] (GND), U5.10 (RETRY_DLY), U5.12 (OVLO), U5.[4,5,14,26] (GND), U6.10 (RETRY_DLY), U6.12 (OVLO), U6.[4,5,14,26] (GND), U7.10 (RETRY_DLY), U7.12 (OVLO), U7.[4,5,14,26] (GND), U8.10 (RETRY_DLY), U8.12 (OVLO), U8.[4,5,14,26] (GND), U9.10 (RETRY_DLY), U9.12 (OVLO), U9.[4,5,14,26] (GND); no longer C14.2, C15.2, C16.2, C17.2, C18.2, C19.2, C57.1, C58.1, R10.1, R2.1, R3.1, R4.1, R5.1, R6.1, R7.1, R8.1, R9.1
- net Inver_EN: now also U8.6 (EN/UVLO)
- net Inver_IMON: now also R5.1, C69.1, U8.9 (IMON)
- net Inver_OUT: now also U8.[17,18,19,20,21,22,23,24] (OUT)
- net PEB_EN: now also U4.6 (EN/UVLO)
- net PEB_IMON: now also R2.1, C61.1, U4.9 (IMON); no longer R2.2
- net PEB_OUT: now also U4.[17,18,19,20,21,22,23,24] (OUT)
- net Shutdn_EN: now also U5.6 (EN/UVLO)
- net Shutdn_IMON: now also R3.1, C64.1, U5.9 (IMON); no longer R5.2
- net Shutdn_OUT: now also U5.[17,18,19,20,21,22,23,24] (OUT)
- net TBB_EN: now also U7.6 (EN/UVLO)
- net TBB_IMON: now also R6.1, C72.1, U7.9 (IMON); no longer R9.2
- net TBB_OUT: now also U7.[17,18,19,20,21,22,23,24] (OUT)
- net Telem_EN: now also U6.6 (EN/UVLO)
- net Telem_IMON: now also R4.1, C66.1, U6.9 (IMON); no longer R7.2
- net Telem_OUT: now also U6.[17,18,19,20,21,22,23,24] (OUT)
- net VCU_EN: now also U9.6 (EN/UVLO)
- net VCU_IMON: now also R7.1, C75.1, U9.9 (IMON)
- net VCU_OUT: now also U9.[17,18,19,20,21,22,23,24] (OUT)
- new net: C60.1, U4.15 (DVDT)
- new net: C57.1, U4.7 (ITIMER)
- new net: R32.2, U4.8 (ILIM)
- new net: R38.2, U11.8 (ILIM)
- new net: C63.1, U5.15 (DVDT)
- new net: C62.1, U5.7 (ITIMER)
- new net: R31.2, U5.8 (ILIM)
- new net: R33.2, U6.8 (ILIM)
- new net: C74.1, U9.15 (DVDT)
- new net: C73.1, U9.7 (ITIMER)
- new net: R36.2, U9.8 (ILIM)
- new net: C71.1, U7.15 (DVDT)
- new net: R37.2, U10.8 (ILIM)
- new net: C70.1, U7.7 (ITIMER)
- new net: R35.2, U7.8 (ILIM)
- new net: C65.1, U6.15 (DVDT)
- new net: C80.1, U11.15 (DVDT)
- new net: C79.1, U11.7 (ITIMER)
- new net: C83.1, U12.15 (DVDT)
- new net: C68.1, U8.15 (DVDT)
- new net: C67.1, U8.7 (ITIMER)
- new net: R34.2, U8.8 (ILIM)
- new net: C58.1, U6.7 (ITIMER)
- new net: C82.1, U12.7 (ITIMER)
- new net: R39.2, U12.8 (ILIM)
- new net: C77.1, U10.15 (DVDT)
- new net: C76.1, U10.7 (ITIMER)
- new net FANA_EN: U10.6 (EN/UVLO)
- new net FANA_IMON: C78.1, R8.1, U10.9 (IMON)
- new net FANA_OUT: U10.[17,18,19,20,21,22,23,24] (OUT)
- new net FANB_EN: U11.6 (EN/UVLO)
- new net FANB_IMON: C81.1, R9.1, U11.9 (IMON)
- new net FANB_OUT: U11.[17,18,19,20,21,22,23,24] (OUT)
- new net FANC_EN: U12.6 (EN/UVLO)
- new net FANC_IMON: C84.1, R10.1, U12.9 (IMON)
- new net FANC_OUT: U12.[17,18,19,20,21,22,23,24] (OUT)
- no-connect marks 12 -> 18
Other:
- note added: "PEB (U4), Telemetry (U6), TBB (U7): Blade Current ATM: 5A eFuse Current Limit Set: 7A (7.0624A) R_ILIM: 210 Ohm R_IMON: 1.91 kOhm C_ITIMER: 15nF C_dVdt: 3.3nF V_IMON_MAX = 3.28V (@ 7.0624A) SR_ON = 1.15 V/ms @ 12V (Table 6.7) t_D,ON = 3.83 ms @ 12V (Table 6.7) t_ITIMER = 7ms Shutdown (U5), Inverter (U8), VCU (U9): Blade Current ATM: 10A eFuse Current Limit Set: 13A (13.0304A) R_ILIM: 113 Ohm R_IM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"
- note removed: "U4 PEB / U6 Telemetry / U7 TBB (7A to emulate a 5A blade): R_ILIM = 210 Ω → I_LIM = 1460/210 + 0.11 = 7.0 A R_IMON = 1.91 kΩ → V_IMON @ 7 A = 7 × 1.91k × 243 µA/A ≈ 3.25 V C_ITIMER = 1 nF → t_ITIMER = 0.47 ms C_dVdt = 1 nF → SR ≈ 4.6 V/ms (turn-on ~2.6 ms @ 12 V) U5 Shutdown / U8 Inverter / U9 VCU (13A to emulate a 10A blade): R_ILIM = 113 Ω → I_LIM = 1460/113 + 0.11 = 13.0 A R_IMON = 1.05 kΩ → V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"
- moved on the sheet: C14, C57, R2

Commit message: add connectors and source components
Parts:
- removed C59: 1nF, Capacitor_SMD:C_0603_1608Metric_Pad1.08x0.95mm_HandSolder, symbol Device:C
- C57, C58, C61, C62, C64, C66, C67, C69, C70, C72, C73, C75, C76, C78, C79, C81, C82, C84: Digikey Part Number (none) -> 311-1430-1-ND; Digikey URL (none) -> https://www.digikey.com/en/products/detail/yageo/CC0603KRX7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; Manufacturer (none) -> YAGEO; Manufacturer Part Number (none) -> CC0603KRX7R9BB153
- C60, C63, C65, C68, C71, C74, C77, C80, C83: Digikey Part Number (none) -> 311-1082-1-ND; Digikey URL (none) -> https://www.digikey.com/en/products/detail/yageo/CC0603KRX7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; Manufacturer (none) -> YAGEO; Manufacturer Part Number (none) -> CC0603KRX7R9BB332
- R10, R3, R5, R7, R8, R9: Digikey Part Number (none) -> 13-AC0603FR-071K02LCT-ND; Digikey URL (none) -> https://www.digikey.com/en/products/detail/yageo/AC0603FR-0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; Manufacturer (none) -> YAGEO; Manufacturer Part Number (none) -> AC0603FR-071K02L
- U10, U11, U12, U4, U5, U6, U7, U8, U9: Digikey Part Number (none) -> 296-TPS259830ONRGERCT-ND; Digikey URL (none) -> https://www.digikey.com/en/products/detail/texas-instrument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; Manufacturer (none) -> Texas Instruments; Manufacturer Part Number (none) -> TPS259830ONRGER

Commit message: fix RC filters
Parts:
- removed C61, C64: 15nF, Capacitor_SMD:C_0603_1608Metric_Pad1.08x0.95mm_HandSolder, symbol Device:C
- added C85, C86, C87: 15nF, Capacitor_SMD:C_0603_1608Metric_Pad1.08x0.95mm_HandSolder, symbol Device:C
- added R11, R12, R13, R14, R15, R16, R17, R18, R19: 1.91k, Resistor_SMD:R_0603_1608Metric_Pad0.98x0.95mm_HandSolder, symbol Device:R
Connections:
- net FANA_IMON: now also R17.2; no longer R8.1, U10.9 (IMON)
- net FANB_IMON: now also R18.2; no longer R9.1, U11.9 (IMON)
- net FANC_IMON: now also R19.2; no longer R10.1, U12.9 (IMON)
- net GND: now also C85.2, C86.2, C87.2
- net Inver_IMON: now also C87.1, R15.2; no longer C69.1, R5.1, U8.9 (IMON)
- net PEB_IMON: now also C85.1, R12.2; no longer R2.1, U4.9 (IMON)
- net Shutdn_IMON: now also C72.1, R14.2; no longer R3.1, U5.9 (IMON)
- net TBB_IMON: now also C86.1, R13.2; no longer C72.1, R6.1, U7.9 (IMON)
- net Telem_IMON: now also R11.2; no longer R4.1, U6.9 (IMON)
- net VCU_IMON: now also R16.2; no longer R7.1, U9.9 (IMON)
- new net: C69.1, R15.1, R5.1, U8.9 (IMON)
- new net: R12.1, R2.1, U4.9 (IMON)
- new net: R11.1, R4.1, U6.9 (IMON)
- new net: R14.1, R3.1, U5.9 (IMON)
- new net: R16.1, R7.1, U9.9 (IMON)
- new net: R13.1, R6.1, U7.9 (IMON)
- new net: R18.1, R9.1, U11.9 (IMON)
- new net: R17.1, R8.1, U10.9 (IMON)
- new net: R10.1, R19.1, U12.9 (IMON)
Other:
- moved on the sheet: C66

Commit message: Update efuses.kicad_sch
Parts:
- removed C69: 15nF, Capacitor_SMD:C_0603_1608Metric_Pad1.08x0.95mm_HandSolder, symbol Device:C
Changed lines of the file:
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@@
 	)
 	(junction
-		(at 130.81 101.6)
-		(diameter 0)
-		(color 0 0 0 0)
-	)
-	(junction
 		(at 92.71 66.04)
 		(diameter 0)
@@
 	)
 	(junction
-		(at 140.97 109.22)
-		(diameter 0)
-		(color 0 0 0 0)
-	)
-	(junction
 		(at 92.71 53.34)
 		(diameter 0)
@@
 	(wire
 		(pts
-			(xy 140.97 109.22) (xy 140.97 116.84)
+			(xy 140.97 97.79) (xy 140.97 116.84)
 		)
 		(stroke
@@
 	(wire
 		(pts
-			(xy 130.81 101.6) (xy 133.35 101.6)
-		)
-		(stroke
-			(width 0)
-			(type default)
-		)
-	)
-	(wire
-		(pts
 			(xy 63.5 74.93) (xy 67.31 74.93)
 		)
@@
 	(wire
 		(pts
-			(xy 133.35 101.6) (xy 133.35 109.22)
-		)
-		(stroke
-			(width 0)
-			(type default)
-		)
-	)
-	(wire
-		(pts
 			(xy 73.66 116.84) (xy 63.5 116.84)
 		)
@@
 	(wire
 		(pts
-			(xy 140.97 97.79) (xy 140.97 109.22)
-		)
-		(stroke
-			(width 0)
-			(type default)
-		)
-	)
-	(wire
-		(pts
 			(xy 254 140.97) (xy 256.54 140.97)
 		)
@@
 					(unit 1)
 				)
-			)
-		)
-	)
-	(symbol
-		(lib_id "Device:C")
-		(at 137.16 109.22 90)
-		(unit 1)
-		(body_style 1)
-		(exclude_from_sim no)
-		(in_bom yes)
-		(on_board yes)
-		(in_pos_files yes)
-		(dnp no)
-		(property "Reference" "C69"
-			(at 139.573 104.775 90)
-			(show_name no)
-			(do_not_autoplace no)
-			(effects
-				(font
-					(size 1.27 1.27)
-				)
-				(justify left)
-			)
-		)
-		(property "Value" "15nF"
-			(at 139.573 102.235 90)
-			(show_name no)
-			(do_not_autoplace no)
-			(effects
-				(font
-					(size 1.27 1.27)
-				)
-				(justify left)
-			)
-		)
-		(property "Footprint" "Capacitor_SMD:C_0603_1608Metric_Pad1.08x0.95mm_HandSolder"
-			(at 140.97 108.2548 0)
-			(hide yes)
-			(show_name no)
-			(do_not_autoplace no)
-			(effects
-				(font
-					(size 1.27 1.27)
-				)
-			)
-		)
-		(property "Datasheet" "https://yageogroup.com/content/datasheet/asset/file/UPY-GPHC_X7R_6_3V-TO-250V"
-			(at 137.16 109.22 0)
-			(hide yes)
-			(show_name no)
-			(do_not_autoplace no)
-			(effects
-				(font
-					(size 1.27 1.27)
-				)
-			)
-		)
-		(property "Description" "Unpolarized capacitor"
-			(at 137.16 109.22 0)
-			(hide yes)
-			(show_name no)
-			(do_not_autoplace no)
-			(effects
-				(font
-					(size 1.27 1.27)
-				)
-			)
-		)
-		(property "Digikey Part Number" "311-1430-1-ND"
-			(at 137.16 109.22 0)
-			(hide yes)
-			(show_name no)
-			(do_not_autoplace no)
-			(effects
-				(font
-					(size 1.27 1.27)
-				)
-			)
-		)
-		(property "Digikey URL" "https://www.digikey.com/en/products/detail/yageo/CC0603KRX7R9BB153/2833595?s=N4IgjCBcoEwAwBYCcVQAcAuUQFUB2AlhgPIBmAsgKYCGAzgK4BOlIANCPdmgGJsgC2BPNjABWOBL79qADxHjJAX0XsYUANogAwlrgA2OAGYA0gCUAGgHZTSAEK2QAXUVA"
-			(at 137.16 109.22 0)
-			(hide yes)
-			(show_name no)
-			(do_not_autoplace no)
-			(effects
-				(font
-					(size 1.27 1.27)
-				)
-			)
-		)
-		(property "Manufacturer" "YAGEO"
-			(at 137.16 109.22 0)
-			(hide yes)
-			(show_name no)
-			(do_not_autoplace no)
-			(effects
-				(font
-					(size 1.27 1.27)
-				)
-			)
-		)
-		(property "Manufacturer Part Number" "CC0603KRX7R9BB153"
-			(at 137.16 109.22 0)
-			(hide yes)
-			(show_name no)
-			(do_not_autoplace no)
-			(effects
-				(font
-					(size 1.27 1.27)
-				)
-			)
-		)
-		(pin "2"
-		)
-		(pin "1"
-		)
-		(instances
-			(project "fuse-board"
-				(path "/e994741c-7c7d-4124-9d00-43b883baa61d/d86ad6f9-6ecb-4228-85b7-377c89926190"
-					(reference "C69")
-					(unit 1)
-				)

Commit message: update to have >10kohm series r
reccomended by TI in datasheet
Parts:
- removed C66, C72: 15nF, Capacitor_SMD:C_0603_1608Metric_Pad1.08x0.95mm_HandSolder, symbol Device:C
- removed R11, R12, R13, R14, R15, R16, R17, R18, R19: 1.91k, Resistor_SMD:R_0603_1608Metric_Pad0.98x0.95mm_HandSolder, symbol Device:R
- added C88, C89: 3.3nF, Capacitor_SMD:C_0603_1608Metric_Pad1.08x0.95mm_HandSolder, symbol Device:C
- added R40, R41, R42, R43, R44, R45, R46, R47, R48: 10k, Resistor_SMD:R_0603_1608Metric_Pad0.98x0.95mm_HandSolder, symbol Device:R
- C75, C78, C81, C84, C85, C86, C87: value 15nF -> 3.3nF; Digikey Part Number 311-1430-1-ND -> 311-1082-1-ND; Digikey URL https://www.digikey.com/en/products/detail/yageo/CC0603KRX7R9BB153/2833595?s=N4IgjCBcoEwAwBYCcVQAcAuUQFUB2AlhgPIBmAsgKYCGAzgK4BOlIANCPdmgGJsgC2BPNjABWOBL79qADxHjJAX0XsYUANogAwlrgA2OAGYA0gCUAGgHZTSAEK2QAXUVA -> https://www.digikey.com/en/products/detail/yageo/CC0603KRX7R9BB332/302816?s=N4IgjCBcoEwAwBYCcVQAcAuUQFUB2AlhgPIBmAsgKYCGAzgK4BOlIANCPdmgGJsgC2BPNgDMIuHD79qAD1HjJAX0XsYUANogAwlrgA2OCIDSAJQAaAdhNIAQjZABdRUA; Manufacturer Part Number CC0603KRX7R9BB153 -> CC0603KRX7R9BB332
Connections:
- net FANA_IMON: now also C87.1, R46.1; no longer C78.1
- net FANB_IMON: now also C88.1, R47.1; no longer C81.1
- net FANC_IMON: now also C89.1, R48.1; no longer C84.1
- net GND: now also C88.2, C89.2
- net Inver_IMON: now also C85.1, R44.1; no longer C87.1
- net PEB_IMON: now also C75.1, R40.1; no longer C85.1
- net Shutdn_IMON: now also C86.1, R45.1
- net TBB_IMON: now also C81.1, R42.1; no longer C86.1
- net Telem_IMON: now also C78.1, R41.1
- net VCU_IMON: now also C84.1, R43.1; no longer C75.1
- net at R5.1, U8.9 (IMON): now also R44.2
- net at R2.1, U4.9 (IMON): now also R40.2
- net at R4.1, U6.9 (IMON): now also R41.2
- net at R3.1, U5.9 (IMON): now also R45.2
- net at R7.1, U9.9 (IMON): now also R43.2
- net at R6.1, U7.9 (IMON): now also R42.2
- net at R9.1, U11.9 (IMON): now also R47.2
- net at R8.1, U10.9 (IMON): now also R46.2
- net at R10.1, U12.9 (IMON): now also R48.2

Commit message: OVLO/UVLO Lockout + DNP ITIMER
Parts:
- removed C14: 1uF, Capacitor_SMD:C_0603_1608Metric_Pad1.08x0.95mm_HandSolder, symbol Device:C
- added C24: 1uF, Capacitor_SMD:C_0603_1608Metric_Pad1.08x0.95mm_HandSolder, symbol Device:C
- added R11, R14, R17, R20, R50, R53, R56, R59, R62: 9k, symbol Device:R
- added R12, R15, R18, R21, R51, R54, R57, R60, R63: 29k, symbol Device:R
- added R13, R16, R19, R49, R52, R55, R58, R61, R64: 48.38k, symbol Device:R
- C57, C58, C62, C67, C70, C73, C76, C79, C82: now not fitted
Connections:
- net 12V_IN: now also C15.1, C16.1, C17.1, C18.1, C19.1, C20.1, C21.1, C22.1, C24.1; no longer C15.2, C16.2, C17.2, C18.2, C19.2, C20.2, C21.2, C22.2
- net FANA_EN: now also R56.2, R57.1
- net FANB_EN: now also R59.2, R60.1
- net FANC_EN: now also R62.2, R63.1
- net GND: now also R13.2, R16.2, R19.2, R49.2, R52.2, R55.2, R58.2, R61.2, R64.2; no longer C15.1, C16.1, C17.1, C18.1, C19.1, C20.1, C21.1, C22.1, U10.12 (OVLO), U11.12 (OVLO), U12.12 (OVLO), U4.12 (OVLO), U5.12 (OVLO), U6.12 (OVLO), U7.12 (OVLO), U8.12 (OVLO), U9.12 (OVLO)
- net Inver_EN: now also R50.2, R51.1
- net PEB_EN: now also R11.2, R12.1
- net Shutdn_EN: now also R14.2, R15.1
- net TBB_EN: now also R20.2, R21.1
- net Telem_EN: now also R17.2, R18.1
- net VCU_EN: now also R53.2, R54.1
- new net: C18.2, R20.1
- new net: R12.2, R13.1, U4.12 (OVLO)
- new net: R15.2, R16.1, U5.12 (OVLO)
- new net: R54.2, R55.1, U9.12 (OVLO)
- new net: C19.2, R53.1
- new net: C20.2, R56.1
- new net: R60.2, R61.1, U11.12 (OVLO)
- new net: C15.2, R11.1
- new net: R21.2, R49.1, U7.12 (OVLO)
- new net: R51.2, R52.1, U8.12 (OVLO)
- new net: C21.2, R59.1
- new net: C16.2, R14.1
- new net: R18.2, R19.1, U6.12 (OVLO)
- new net: R63.2, R64.1, U12.12 (OVLO)
- new net: C17.2, R50.1
- new net: C22.2, R62.1
- new net: C24.2, R17.1
- new net: R57.2, R58.1, U10.12 (OVLO)
Other:
- note added: "Do Not Populate Capacitors: Leave NC (NOT grounded), and only add cap if we need to set ITIMER higher"
- moved on the sheet: C15

Commit message: fix decoupling cap gnd
Connections:
- net GND: now also C15.2, C16.2, C17.2, C18.2, C19.2, C20.2, C21.2, C22.2, C24.2, R11.1, R14.1, R17.1, R20.1, R50.1, R53.1, R56.1, R59.1, R62.1
