File: fuse-board/mcu.kicad_sch (KiCad schematic)
At the start: 65 parts, among them IC1 TMUX1308QPWRQ1, J1 FTSH-107-01-F-DV-K-P-TR, J10 Conn_01x03, J11 Conn_01x03, J12 Conn_01x03, J13 Conn_01x03, J14 Conn_01x03, J6 Conn_01x03, J7 Conn_01x03, J8 Conn_01x03, J9 Conn_01x03, SW1 Y97KT23B5NAFP, U1 STM32G491KCUx, U13 74AHCT1G125, Y1 ECS-240-8-37B-CKY-TR

Commit message: mcu -> g441, remove jumpers
Parts:
- removed J10, J11, J12, J13, J14, J6, J7, J8, J9: Conn_01x03, Connector_PinHeader_2.54mm:PinHeader_1x03_P2.54mm_Vertical, symbol Connector_Generic:Conn_01x03
- removed U1: STM32G491KCUx, Package_DFN_QFN:QFN-32-1EP_5x5mm_P0.5mm_EP3.45x3.45mm, symbol MCU_ST_STM32G4:STM32G491KCUx
- added U1: STM32G441KBTx, Package_QFP:LQFP-32_7x7mm_P0.8mm, symbol MCU_ST_STM32G4:STM32G441KBTx
- C1, C2: Digi PN (none) -> 311-3874-1-ND; Digi URL (none) -> https://www.digikey.com/en/products/detail/yageo/CC0603DRNP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; Digikey Part Number 311-3874-1-ND -> (none); Digikey URL https://www.digikey.com/en/products/detail/yageo/CC0603DRNP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 -> (none); MFG (none) -> Yageo; MFG PN (none) -> CC0603DRNPO9BN6R8; Manufacturer YAGEO -> (none); Manufacturer Part Number CC0603DRNPO9BN6R8 -> (none)
- C3, C5, C6, C8: Digi PN (none) -> 311-1344-1-ND; Digi URL (none) -> https://www.digikey.com/en/products/detail/yageo/CC0603KRX7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; Digikey Part Number 311-1344-1-ND -> (none); Digikey URL https://www.digikey.com/en/products/detail/yageo/CC0603KRX7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 -> (none); MFG (none) -> Yageo; MFG PN (none) -> CC0603KRX7R9BB104; Manufacturer YAGEO -> (none); Manufacturer Part Number CC0603KRX7R9BB104 -> (none)
- C4: Digi PN (none) -> 1276-CL10A106KO8NQNCCT-ND; Digi URL (none) -> https://www.digikey.com/en/products/detail/samsung-electro-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; Digikey Part Number 1276-CL10A106KO8NQNCCT-ND -> (none); Digikey URL https://www.digikey.com/en/products/detail/samsung-electro-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 -> (none); MFG (none) -> Samsung Electro-Mechanics; MFG PN (none) -> CL10A106KO8NQNC; Manufacturer Samsung Electro-Mechanics -> (none); Manufacturer Part Number CL10A106KO8NQNC -> (none)
- C7: Digi PN (none) -> 1276-CL10B105KB9VPJCCT-ND; Digi URL (none) -> https://www.digikey.com/en/products/detail/samsung-electro-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; Digikey Part Number 1276-CL10B105KB9VPJCCT-ND -> (none); Digikey URL https://www.digikey.com/en/products/detail/samsung-electro-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 -> (none); MFG (none) -> Samsung Electro-Mechanics; MFG PN (none) -> CL10B105KB9VPJC; Manufacturer Samsung Electro-Mechanics -> (none); Manufacturer Part Number CL10B105KB9VPJC -> (none)
- FB1: Digi PN (none) -> 4816-FCM1608KF-601T03CT-ND; Digi URL (none) -> https://www.digikey.com/en/products/detail/tai-tech-advance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; Digikey Part Number 4816-FCM1608KF-601T03CT-ND -> (none); Digikey URL https://www.digikey.com/en/products/detail/tai-tech-advance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 -> (none); MFG (none) -> TAI-TECH Advanced Electronics Co., Ltd.; MFG PN (none) -> FCM 1608KF-601T03; Manufacturer TAI-TECH Advanced Electronics Co., Ltd. -> (none); Manufacturer Part Number FCM 1608KF-601T03 -> (none)
- J1: Digi PN (none) -> SAM13170CT-ND; Digi URL (none) -> https://www.digikey.com/en/products/detail/samtec-inc/FTSH-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; Digikey Part Number SAM13170CT-ND -> (none); Digikey URL https://www.digikey.com/en/products/detail/samtec-inc/FTSH-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 -> (none); MFG (none) -> Samtec Inc.; MFG PN (none) -> FTSH-107-01-F-DV-K-P-TR; Manufacturer Samtec Inc. -> (none); Manufacturer Part Number FTSH-107-01-F-DV-K-P-TR -> (none)
- R1: value 10K -> 10k; Digi PN (none) -> 311-10KLDCT-ND; Digi URL (none) -> https://www.digikey.com/en/products/detail/yageo/AC0603FR-0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; Digikey Part Number 311-10KLDCT-ND -> (none); Digikey URL https://www.digikey.com/en/products/detail/yageo/AC0603FR-0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 -> (none); MFG (none) -> Yageo; MFG PN (none) -> AC0603FR-0710KL; Manufacturer YAGEO -> (none); Manufacturer Part Number AC0603FR-0710KL -> (none)
- SW1: Digi PN (none) -> 108-Y97KT23B5NAFPCT-ND; Digi URL (none) -> https://www.digikey.com/en/products/detail/c-k/y97kt23b5naf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; Digikey Part Number 108-Y97KT23B5NAFPCT-ND -> (none); Digikey URL https://www.digikey.com/en/products/detail/c-k/y97kt23b5naf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 -> (none); MFG (none) -> C&K; MFG PN (none) -> Y97KT23B5NAFP; Manufacturer C&K -> (none); Manufacturer Part Number Y97KT23B5NAFPY97KT23B5NAFP -> (none)
- Y1: Digi PN (none) -> XC3063CT-ND; Digi URL (none) -> https://www.digikey.com/en/products/detail/ecs-inc/ECS-240-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; Digikey Part Number XC3063CT-ND -> (none); Digikey URL https://www.digikey.com/en/products/detail/ecs-inc/ECS-240-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 -> (none); MFG (none) -> ECS; MFG PN (none) -> ECS-240-8-37B-CKY-TR; Manufacturer ECS -> (none); Manufacturer Part Number ECS-240-8-37B-CKY-TR -> (none)
Connections:
- net FANA_EN is gone; now on net MCU_FANA_EN: R29.2
- net FANB_EN is gone; now on net MCU_FANB_EN: R28.2
- net FANC_EN is gone; now on net MCU_FANC_EN: R30.2
- net Inver_EN is gone; now on net MCU_Inver_EN: R25.2
- net PEB_EN is gone; now on net MCU_PEB_EN: R22.2
- net Shutdn_EN is gone; now on net MCU_Shutdn_EN: R26.2
- net TBB_EN is gone; now on net MCU_TBB_EN: R23.2
- net Telem_EN is gone; now on net MCU_Telem_EN: R24.2
- net VCU_EN is gone; now on net MCU_VCU_EN: R27.2
- net +3V3: now also U1.1 (VDD), U1.17 (VDD)
- net +3V3_A: now also U1.15 (VDDA)
- net ADC_MUXED_IMON: now also U1.5 (PA0)
- net ADC_Shutdn_IMON: now also U1.6 (PA1)
- net BOOT0: now also U1.31 (PB8)
- net CANRX: now also U1.21 (PA11)
- net CANTX: now also U1.22 (PA12)
- net GND: now also U1.14 (VSSA), U1.16 (VSS), U1.32 (VSS)
- net LED_SIGNAL: now also U1.28 (PB5)
- net MCU_FANA_EN: now also U1.25 (PA15)
- net MCU_FANB_EN: now also U1.13 (PB0)
- net MCU_FANC_EN: now also U1.27 (PB4)
- net MCU_Inver_EN: now also U1.29 (PB6)
- net MCU_PEB_EN: now also U1.12 (PA7)
- net MCU_Shutdn_EN: now also U1.20 (PA10)
- net MCU_TBB_EN: now also U1.18 (PA8)
- net MCU_Telem_EN: now also U1.19 (PA9)
- net MCU_VCU_EN: now also U1.30 (PB7)
- net MUX_SEL0: now also U1.9 (PA4)
- net MUX_SEL1: now also U1.10 (PA5)
- net MUX_SEL2: now also U1.11 (PA6)
- net NRST: now also U1.4 (PG10)
- net OSC_IN: now also U1.2 (PF0)
- net OSC_OUT: now also U1.3 (PF1)
- net STLINK_SWCLK: now also U1.24 (PA14)
- net STLINK_SWDIO: now also U1.23 (PA13)
- net STLINK_SWO: now also U1.26 (PB3)
- net VCP_UART_RX: now also U1.8 (PA3)
- net VCP_UART_TX: now also U1.7 (PA2)
Other:
- note added: "Current sensing mux and voltage clamps"
- note added: "Enables and pull-ups"
- note added: "STM32G441KBTx MCU"
- note removed: "Jumpers and pull-ups"
- note removed: "Mux and filters"
- note removed: "STM32G491KCU6 MCU"
- moved on the sheet: C53, C56, C57, C58, C59, C60, C61, C62, C63, C64, C65, C66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

Commit message: Document eFuse enable behavior and update LED data resistor
Parts:
- R31: value 33 -> 330R
Other:
- note added: "EN GPIOs open-drain; 10k pullups default eFuses ON at MCU boot."

Commit message: get rid of LEDs and add LED_SIGNAL
Parts:
- removed C53, C56, C57, C58, C59, C60, C61, C62, C63, C64: 100nF, Capacitor_SMD:C_0603_1608Metric_Pad1.08x0.95mm_HandSolder, symbol Device:C
- removed C65, C66: 47uF, Capacitor_SMD:C_0805_2012Metric_Pad1.18x1.45mm_HandSolder, symbol Device:C
- removed D10, D11, D12, D13, D5, D6, D7, D8, D9: Inolux_IN-PI554FCH, LED_SMD:LED_Inolux_IN-PI554FCH_PLCC4_5.0x5.0mm_P3.2mm, symbol LED:Inolux_IN-PI554FCH
- removed R31: 330R, Resistor_SMD:R_1206_3216Metric_Pad1.30x1.75mm_HandSolder, symbol Device:R
- removed U13: 74AHCT1G125, Package_TO_SOT_SMD:SOT-23-5_HandSoldering, symbol 74xGxx:74AHCT1G125
Connections:
- no-connect marks 5 -> 4

Commit message: update tmux1308
Parts:
- removed IC1: TMUX1308QPWRQ1, formula_slug_footprint_library:SOP65P640X120-16N, symbol formula_slug_symbol_library:TMUX1308QPWRQ1
- added U13: TMUX1308QPWRQ1, formula_slug_footprint_library:SOP65P640X120-16N, symbol formula_slug_symbol_library:TMUX1308QPWRQ1
Connections:
- net +3V3: now also U13.16 (VDD)
- net FANA_IMON: now also U13.5 (S5)
- net FANB_IMON: now also U13.2 (S6)
- net FANC_IMON: now also U13.4 (S7)
- net GND: now also U13.6 (~{EN}), U13.8 (GND)
- net Inver_IMON: now also U13.12 (S3)
- net MUX_IMON_OUT: now also U13.3 (D)
- net MUX_SEL0: now also U13.11 (A0)
- net MUX_SEL1: now also U13.10 (A1)
- net MUX_SEL2: now also U13.9 (A2)
- net PEB_IMON: now also U13.13 (S0)
- net TBB_IMON: now also U13.14 (S1)
- net Telem_IMON: now also U13.15 (S2)
- net VCU_IMON: now also U13.1 (S4)
Other:
- moved on the sheet: C50, C51, C52, D14, D15, D16, D17, R20, R21

Commit message: more changes task 8 almost done waiting for calcs
Other:
- note added: "PCB: Place C50 (100 nF) immediately next to U13 VDD and GND pins."
Changed lines of the file:
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@@
+		)
+	)
+	(text "PCB: Place C50 (100 nF) \nimmediately next to U13 \nVDD and GND pins."
+		(exclude_from_sim no)
+		(at 38.862 148.844 0)
+		(effects
+			(font
+				(size 1.27 1.27)
+			)
 		)
 	)

Commit message: add connectors and source components
Parts:
- C1, C2: Digikey Part Number (none) -> 311-3874-1-ND; Digikey URL (none) -> https://www.digikey.com/en/products/detail/yageo/CC0603DRNP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; Manufacturer (none) -> YAGEO; Manufacturer Part Number (none) -> CC0603DRNPO9BN6R8
- C3, C5, C6, C8: Digikey Part Number (none) -> 311-1344-1-ND; Digikey URL (none) -> https://www.digikey.com/en/products/detail/yageo/CC0603KRX7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; Manufacturer (none) -> YAGEO; Manufacturer Part Number (none) -> CC0603KRX7R9BB104
- C4: Digikey Part Number (none) -> 1276-CL10A106KO8NQNCCT-ND; Digikey URL (none) -> https://www.digikey.com/en/products/detail/samsung-electro-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; Manufacturer (none) -> Samsung Electro-Mechanics; Manufacturer Part Number (none) -> CL10A106KO8NQNC
- C7: Digikey Part Number (none) -> 1276-1860-1-ND; Digikey URL (none) -> https://www.digikey.com/en/products/detail/samsung-electro-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; Manufacturer (none) -> Samsung Electro-Mechanics; Manufacturer Part Number (none) -> CL10A105KB8NNNC
- FB1: Digikey Part Number (none) -> 4816-FCM1608KF-601T03CT-ND; Digikey URL (none) -> https://www.digikey.com/en/products/detail/tai-tech-advance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; Manufacturer (none) -> TAI-TECH Advanced Electronics Co., Ltd.; Manufacturer Part Number (none) -> FCM 1608KF-601T03
- J1: Digikey Part Number (none) -> SAM13170CT-ND; Digikey URL (none) -> https://www.digikey.com/en/products/detail/samtec-inc/FTSH-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; Manufacturer (none) -> Samtec Inc.; Manufacturer Part Number (none) -> FTSH-107-01-F-DV-K-P-TR
- R1: Digikey Part Number (none) -> 311-10KLDCT-ND; Digikey URL (none) -> https://www.digikey.com/en/products/detail/yageo/AC0603FR-0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; Manufacturer (none) -> YAGEO; Manufacturer Part Number (none) -> AC0603FR-0710KL
- R22, R23, R24, R25, R26, R27, R28, R29, R30: value 10K -> 10k
- SW1: Digikey Part Number (none) -> 108-PTS647SK38SMTR2LFSCT-ND; Digikey URL (none) -> https://www.digikey.com/en/products/detail/c-k/PTS647SK38SM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; Manufacturer (none) -> C&K; Manufacturer Part Number (none) -> PTS647SK38SMTR2 LFS
- U1: Digikey Part Number (none) -> 497-STM32G441KBT6-ND; Digikey URL (none) -> https://www.digikey.com/en/products/detail/stmicroelectroni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; Manufacturer (none) -> STMicroelectronics; Manufacturer Part Number (none) -> STM32G441KBT6
- U13: Digikey Part Number (none) -> 296-TMUX1308QPWRQ1CT-ND; Digikey URL (none) -> https://www.digikey.com/en/products/detail/texas-instrument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; Manufacturer (none) -> Texas Instruments; Manufacturer Part Number (none) -> TMUX1308QPWRQ1
- Y1: Digikey Part Number (none) -> XC3063CT-ND; Digikey URL (none) -> https://www.digikey.com/en/products/detail/ecs-inc/ECS-240-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; Manufacturer (none) -> ECS Inc.; Manufacturer Part Number (none) -> ECS-240-8-37B-CKY-TR

Commit message: OVLO/UVLO Lockout + DNP ITIMER
Parts:
- removed C51, C52: 100pF, Capacitor_SMD:C_0603_1608Metric_Pad1.08x0.95mm_HandSolder, symbol Device:C
- removed R20, R21: 1k, Resistor_SMD:R_0603_1608Metric_Pad0.98x0.95mm_HandSolder, symbol Device:R
Connections:
- net MUX_IMON_OUT is gone; now on net ADC_MUXED_IMON: U13.3 (D)

Commit message: combine pins, 9 adc pins, notes
Parts:
- removed C50: 100nF, Capacitor_SMD:C_0603_1608Metric_Pad1.08x0.95mm_HandSolder, symbol Device:C
- removed D14, D15, D16, D17: SS34, Diode_SMD:D_SMB-SMC_Universal_Handsoldering, symbol Device:D_Schottky
- removed R24, R28, R30: 10k, Resistor_SMD:R_0603_1608Metric_Pad0.98x0.95mm_HandSolder, symbol Device:R
- removed U13: TMUX1308QPWRQ1, formula_slug_footprint_library:SOP65P640X120-16N, symbol formula_slug_symbol_library:TMUX1308QPWRQ1
Connections:
- net ADC_MUXED_IMON is gone; now on net TBB_IMON: U1.5 (PA0)
- net ADC_Shutdn_IMON is gone; now on net Telem_IMON: U1.6 (PA1)
- net MCU_FANB_EN is gone; now on net FANC_IMON: U1.13 (PB0)
- net MCU_FANC_EN is gone; now on net VCP_UART_RX: U1.27 (PB4)
- net MUX_SEL0 is gone; now on net FANA_IMON: U1.9 (PA4)
- net MUX_SEL1 is gone; now on net FANB_IMON: U1.10 (PA5)
- net Inver_IMON: now also U1.7 (PA2)
- net MCU_PEB_EN: now also U1.30 (PB7); no longer U1.12 (PA7)
- net PEB_IMON: now also U1.12 (PA7)
- net VCP_UART_RX: no longer U1.8 (PA3)
- net VCP_UART_TX: now also U1.26 (PB3); no longer U1.7 (PA2)
- net VCU_IMON: now also U1.8 (PA3)
- net MCU_FANA_EN renamed MCU_FAN_EN
- net MCU_Telem_EN renamed MCU_VCU_Telem_EN
- net MCU_VCU_Telem_EN: now also R27.2
- removed net MCU_VCU_EN: R27.2, U1.30 (PB7)
- net MUX_SEL2 renamed Shutdn_IMON
- net STLINK_SWO: no longer names the net of J1.8 (Pin_8)
- net STLINK_SWO: no longer U1.26 (PB3)
- no-connect marks 4 -> 5
Other:
- note removed: "Current sensing mux and voltage clamps"
- note removed: "PCB: Place C50 (100 nF) immediately next to U13 VDD and GND pins."
- moved on the sheet: R22, R23, R25, R26, R27, R29
