File: fs5-telemetry-peripheral-board.kicad_sch (KiCad schematic)
At the start: 0 parts

Commit message: Started work on wheel speed circuitry
Parts:
- added C1: 10pF, symbol Device:C_Small
- added C2: 22nF, symbol Device:C_Small
- added C3: 100nF, symbol Device:C_Small
- added J1: ATS668LSM, symbol Symbols:ATS668LSM
- added R1, R4: 1K, symbol Device:R_US
- added R2: 10K, symbol Device:R_US
- added R3: 22K, symbol Device:R_US
Connections:
- new net: C1.1, R1.2
- new net: R2.2, R3.1
- new net +5V: R1.1, R2.1
- new net GND: C1.2, C2.2, C3.2, R3.2, R4.2
Other:
- note added: "Wheel Speed Sensor Connector"
