File: fs5-telemetry-peripheral-board.kicad_sch (KiCad schematic)
At the start: 9 parts, among them J1 ATS668LSM, U2 LM2907M/NOPB

Commit message: finished wheel speed sensor part
Parts:
- removed U2: LM2907M/NOPB, symbol Symbols:LM2907M_NOPB
- added C4, C5: 100nF, symbol Device:C_Small
- added R5: 10K, symbol Device:R_US
- added R6: 100k, symbol Device:R_US
- added U1: LM2907M/NOPB, symbol Symbols:LM2907M_NOPB
Connections:
- net +5V: now also C4.1, U1.8 (COL), U1.9 (V+)
- net GND: now also C4.2, C5.2, R5.2, U1.12 (GND)
- net at C2.1: now also U1.2 (CP)
- net at C3.1, R4.1: now also U1.3 (CP), U1.4 (IN+)
- net at C1.1, R1.2: now also U1.1 (TACH+)
- net at R2.2, R3.1: now also U1.11 (TACH-)
- new net: R5.1, R6.1, U1.10 (IN-), U1.5 (EMIT)
- new net: C5.1, R6.2

Commit message: Added schematic for sensors, CAN transceiver, voltage regulator and instrumentation amplifier
Parts:
- added C10, C7, C8, C9: 100nF, symbol Device:C_Small
- added C6: 330nF, symbol Device:C_Small
- added J2: Potentiometer, symbol Connector:Conn_01x03_Pin
- added J3: Conn_01x10_Pin, symbol Connector:Conn_01x10_Pin
- added J4: Strain Gauge, symbol Connector:Conn_01x02_Pin
- added J5: 1x8 Tire Surface Temperature Sensor, symbol Connector_Generic_MountingPin:Conn_01x04_MountingPin
- added J6: Tire Temperature Sensor, symbol Connector_Generic_MountingPin:Conn_01x04_MountingPin
- added J7: 1x1 Tire Air Temperature Sensor, symbol Connector_Generic_MountingPin:Conn_01x04_MountingPin
- added J8: Conn_01x09_Pin, symbol Connector:Conn_01x09_Pin
- added J9: Conn_01x04_MountingPin, symbol Connector_Generic_MountingPin:Conn_01x04_MountingPin
- added R10: Extra, symbol Device:R_Small_US
- added R11: 60.4R, symbol Device:R_Small_US
- added R12, R9: 4.7k, symbol Device:R_Small_US
- added R7: 120R, symbol Device:R_US
- added R8: 120R, symbol Device:R_Small_US
- added RV1: 200R, symbol Device:R_Potentiometer
- added U2: LM7805CV, symbol Symbols:LM7805CV
- added U3: INA125U, symbol Symbols:INA125U
- added U4: ISO1050DUB, Package_SO:SOP-8_6.62x9.15mm_P2.54mm, symbol Interface_CAN_LIN:ISO1050DUB
Connections:
- net +5V: now also C10.1, C7.1, C8.1, C9.1, J2.1 (Pin_1), J3.8 (Pin_8), J4.2 (Pin_2), J5.2 (Pin_2), J6.1 (Pin_1), J7.2 (Pin_2), R12.2, R7.1, R9.2, U2.3 (VO), U3.1 (V+), U3.2 (SLEEP), U4.1 (VCC1), U4.8 (VCC2)
- net GND: now also C10.2, C6.2, C7.2, C8.2, C9.2, J2.3 (Pin_3), J3.9 (Pin_9), J5.1 (Pin_1), J6.4 (Pin_4), J7.1 (Pin_1), J9.4 (Pin_4), R8.2, RV1.3 (1), U2.2 (GND), U3.12 (VREFCOM), U3.3 (V-), U4.4 (GND1), U4.5 (GND2)
- net PC3: now reaches C5.1, R6.2
- net PC3: now also J3.5 (Pin_5)
- new net: R10.1, R11.1, U3.8 (RG)
- new net: R10.2, R11.2, U3.9 (RG)
- new net: U3.4 (VREFOUT), U3.5 (IAREF)
- new net +12V: C6.1, J9.1 (Pin_1), U2.1 (VI)
- new net CAN1_RX: U4.2 (RXD)
- new net CAN1_TX: U4.3 (TXD)
- new net CANH: J6.3 (Pin_3), J9.3 (Pin_3), U4.7 (CANH)
- new net CANL: J6.2 (Pin_2), J9.2 (Pin_2), U4.6 (CANL)
- new net PA1: J3.6 (Pin_6)
- new net PA2: J3.7 (Pin_7)
- new net PA6: J2.2 (Pin_2)
- new net PA7: U3.10 (VO), U3.11 (SENSE)
- new net PB0: J3.1 (Pin_1), J5.4 (Pin_4), J7.4 (Pin_4), R12.1
- new net PB1: J5.3 (Pin_3), J7.3 (Pin_3), J8.1 (Pin_1), R9.1
- new net PB2: J8.2 (Pin_2)
- new net PB3: J8.3 (Pin_3)
- new net PB4: J8.4 (Pin_4)
- new net PB5: J8.5 (Pin_5)
- new net PB6: J8.6 (Pin_6)
- new net PB7: J8.7 (Pin_7)
- new net PB8: J8.8 (Pin_8)
- new net PB9: J8.9 (Pin_9)
- new net PC0: J3.2 (Pin_2)
- new net PC1: J3.3 (Pin_3)
- new net PC2: J3.4 (Pin_4)
- new net UPDI: J3.10 (Pin_10)
- new net Vin+: J4.1 (Pin_1), R8.1, U3.6 (VIN+)
- new net Vin-: R7.2, RV1.1 (3), RV1.2, U3.7 (VIN-)
- new net VrefBG: U3.13 (VREFBG)
Other:
- note added: "CAN Transceiver"
- note added: "Connectors"
- note added: "Sensors"
- note added: "Wheelstone Bridge"

Commit message: added
Parts:
- added C11: 100nF, symbol Device:C
- added C12, C13: 6.8pF, symbol Device:C
- added C14: 10uF, symbol Device:C_Small
- added C15, C16, C18: 100nF, symbol Device:C_Small
- added C17: 1uF, symbol Device:C_Small
- added FB1: FCM1608KF-601T03, symbol Device:FerriteBead
- added J10: FTSH-107-01-F-DV-K-P-TR, symbol Connector_Generic:Conn_02x07_Odd_Even
- added R13: 10k, symbol Device:R
- added SW1: Y97KT23B5NAFP, symbol Switch:SW_Push
- added U5: STM32G441KBTx, Package_QFP:LQFP-32_7x7mm_P0.8mm, symbol MCU_ST_STM32G4:STM32G441KBTx
- added Y1: 24MHz, symbol Device:Crystal_GND24_Small
Connections:
- net GND: now also C11.1, C12.1, C13.1, C14.2, C15.2, C16.2, C17.2, C18.2, J10.11 (Pin_11), J10.12 (Pin_12), J10.5 (Pin_5), J10.7 (Pin_7), R13.2, SW1.1, U5.14 (VSSA), U5.16 (VSS), U5.32 (VSS), Y1.2 (G), Y1.4 (G)
- new net: C11.2, SW1.2, U5.4 (PG10)
- new net +3V3: C14.1, C15.1, C16.1, C17.1, C18.1, FB1.1, FB1.2, J10.3 (Pin_3), U5.1 (VDD), U5.15 (VDDA), U5.17 (VDD)
- new net B00T0: R13.1, U5.31 (PB8)
- new net OSC_In: C12.2, U5.2 (PF0), Y1.3
- new net OSC_Out: C13.2, U5.3 (PF1), Y1.1
- new net STLINK_SWCLK: J10.6 (Pin_6), U5.24 (PA14)
- new net STLINK_SWDIO: J10.4 (Pin_4), U5.23 (PA13)
- new net STLINK_SWO: J10.8 (Pin_8), U5.26 (PB3)
- new net VCP_UART_RX: U5.8 (PA3)
- new net VCP_UART_TX: U5.7 (PA2)
- new net VCT_UART_RX: J10.13 (Pin_13)
- new net VCT_UART_TX: J10.14 (Pin_14)
Other:
- note added: "ST-Link Programming/Debug Connector"
- note added: "in-progress"
