File: llc-prototype-2/SR_Rect_Stage.sch.kicad_sch (KiCad schematic)
At the start: 12 parts, among them U2 UCC24624DR

Commit message: Rev 1.2
added output caps, resonant caps, feedback compensation, fast turn off for primary fets
Other:
- moved on the sheet: C8, C9, U2
