File: telemetry-logging-board/rf.kicad_sch (KiCad schematic)
At the start: 37 parts, among them J6 LF, J7 HF, U5 LR2021IMLTRT, Y2 21MHz

Commit message: mostly CAN work
Parts:
- removed C12: C_Small, symbol Device:C_Small
- removed Y2: 21MHz, symbol Device:Crystal
- added C20, C21: 2.2uF, symbol Device:C_Small
- added C22: 100nF, symbol Device:C_Small
- added C23: 4.7uF, symbol Device:C_Small
- added C24: 1nF, symbol Device:C_Small
- added C25, C26: 1uF, symbol Device:C_Small
- added D1, D2: RClamp2271ZC, symbol Device:D_TVS
- added FB1, FB2, FB3: FerriteBead_Small, symbol Device:FerriteBead_Small
- added L16: 2.2uH, symbol Device:L
- added R13, R14: 470R, symbol Device:R_Small
- added R15: 120k, symbol Device:R_Small
- added TH1: ERT-JZER104F, symbol Device:Thermistor_NTC
- added Y2: 32MHz, symbol Device:Crystal_GND23
- C10: value C_Small -> 3.9pF
- C11, C9: value C_Small -> 1.8pF
- C13, C5: value C_Small -> 18pF
- C14: value C_Small -> 6.8pF
- C15: value C_Small -> 2pF
- C16, C19: value C_Small -> 1.2pF
- C17: value C_Small -> 1.1pF
- C18: value C_Small -> 2.7pF
- C4: value C_Small -> 2.2pF
- C6: value C_Small -> 47pF
- C7: value C_Small -> 22pF
- C8: value C_Small -> 7.5pF
- J6, J7: footprint (none) -> Connector_Coaxial:SMA_Amphenol_132203-12_Horizontal
- L10: value L -> 2.4nH
- L11: value L -> 1.1nH
- L12: value L -> 1.6nH
- L13: value L -> 1.5nH
- L14, L9: value L -> 22nH
- L15: value L -> 18nH
- L4: value L -> 24nH
- L5: value L -> 4.7nH
- L6: value L -> 12nH
- L7: value L -> 3.9nH
- L8: value L -> 7.5nH
- R12: value 0R -> 470R
Connections:
- net GND: now also C20.2, C21.2, C22.2, C23.2, C24.2, C25.2, C26.2, D1.1 (A1), D2.1 (A1), TH1.2, Y2.2 (G), Y2.3 (G)
- net at C11.1, C5.1, J6.1 (In)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: now also D1.2 (A2)
- net at C15.1, J7.1 (In), L11.1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: now also D2.2 (A2)
- net at U5.1 (VR_PA): now also C24.1
- net at U5.10 (DIO8): now also R13.2
- net at U5.11 (DIO7): now also R12.2
- net at U5.12 (VDCC1): now also C26.1, FB3.2
- net at U5.13 (VPAX1): now also C20.1, FB1.2
- net at U5.14 (LXB): now also L16.2
- net at U5.16 (LXA): now also L16.1
- net at U5.17 (VBAT): now also C22.1, C23.1, FB2.2
- net VPAX: now reaches U5.2 (VPAX2)
- net VPAX: now also C21.1, FB1.1
- net RF_MISO: now reaches U5.21 (MISO)
- net RF_MISO: no longer R12.2
- net at U5.25 (BUSY): now also R14.1
- net VDCC: now reaches U5.26 (VDCC2)
- net VDCC: now also C25.1, FB3.1
- net at U5.3 (NTC): now also R15.1, TH1.1
- net at U5.4 (XTA): now also Y2.1
- net at U5.5 (XTB): now also Y2.4
- net VNTC: now reaches U5.6 (VTCXO/VNTC)
- net VNTC: now also R15.2
- net RF_DIO11: now reaches U5.7 (DIO11)
- net RF_DIO7: now reaches R12.1
- net RF_~{RST}: now reaches R2.1
- net RF_~{RST}: now also R14.2
- net RF_MOSI: now reaches R11.1
- net RF_~{SS}: now reaches R3.1
- net RF_SCK: now reaches R10.1
- new net RF_DIO8: R13.1
- new net VBAT: FB2.1
- no-connect marks 0 -> 4
Other:
- company: (none) -> Formula Slug
- title: (none) -> Telemetry Logging Board
- moved on the sheet: C13, C17, C19, C4, C5, C6, C9, L10, L15, L4, L6, R10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
