File: telemetry-logging-board/telemetry-logging-board.kicad_sch (KiCad schematic)
At the start: 0 parts

Commit message: mostly CAN work
Parts:
- added J12: Wifi, Connector_Coaxial:SMA_Amphenol_132203-12_Horizontal, symbol Connector:Conn_Coaxial
- added J13: ESP, Connector_Coaxial:U.FL_Hirose_U.FL-R-SMT-1_Vertical, symbol Connector:Conn_Coaxial
- added J5: USB_C_Receptacle_USB2.0_16P, Connector_USB:USB_C_Receptacle_G-Switch_GT-USB-7051x, symbol Connector:USB_C_Receptacle_USB2.0_16P
- added J8: Micro_SD_Card, Connector_Card:microSD_HC_Wuerth_693072010801, symbol Connector:Micro_SD_Card
- added R4, R5: 5.1k, symbol Device:R_Small
- added U1: ESP32-S3-MINI-1U, RF_Module:ESP32-S2-MINI-1U, symbol RF_Module:ESP32-S3-MINI-1U
- added U6: USBLC6-2SC6, Package_TO_SOT_SMD:SOT-23-6, symbol Power_Protection:USBLC6-2SC6
Connections:
- new net: J12.1 (In), J13.1 (In)
- new net: J12.2 (Ext), J13.2 (Ext)
- new net: J5.A5 (CC1), R5.2
- new net: U1.23 (USB_D-), U6.1 (I/O1)
- new net: U1.24 (USB_D+), U6.3 (I/O2)
- new net: J5.B5 (CC2), R4.2
- new net: J5.A7 (D-), J5.B7 (D-), U6.4 (I/O2)
- new net: J5.A6 (D+), J5.B6 (D+), U6.6 (I/O1)
- new net +3.3V: J8.4 (VDD), U1.3 (3V3), U1.45 (EN)
- new net GND: J5.A1 (GND), J5.A12 (GND), J5.B1 (GND), J5.B12 (GND), J8.6 (VSS), R4.1, R5.1, U1.1 (GND), U1.2 (GND), U1.42 (GND), U1.43 (GND), U1.46 (GND), U1.47 (GND), U1.48 (GND), U1.49 (GND), U1.50 (GND), U1.51 (GND), U1.52 (GND), U1.53 (GND), U1.54 (GND), U1.55 (GND), U1.56 (GND), U1.57 (GND), U1.58 (GND), U1.59 (GND), U1.60 (GND), U1.61 (GND), U1.62 (GND), U1.63 (GND), U1.64 (GND), U1.65 (GND), U6.2 (GND)
- new net GNDPWR: J5.SH (SHIELD), J8.SH (SHIELD)
- new net SPI2_CS_RF: U1.34 (IO38)
- new net SPI2_CS_SD: J8.2 (DAT3/CD)
- new net SPI2_MISO: J8.7 (DAT0), U1.33 (IO37)
- new net SPI2_MOSI: J8.3 (CMD), U1.31 (IO35)
- new net SPI2_SCK: J8.5 (CLK), U1.32 (IO36)
- new net VBUS: J5.A4 (VBUS), J5.A9 (VBUS), J5.B4 (VBUS), J5.B9 (VBUS), U6.5 (VBUS)
- no-connect marks 0 -> 2
Other:
- removed sheet MCU
- sheet CAN Busses ports: added CS_A, CS_B, CS_C, MISO, MOSI, SCK; removed none
- sheet LR Radio ports: added RF_DIO11, RF_DIO7, RF_DIO8, RF_MISO, RF_MOSI, RF_SCK, RF_~{RST}, RF_~{SS}; removed none
- note added: "Strap"
- company: (none) -> Formula Slug
- title: (none) -> Telemetry Logging Board

Commit message: eth chip
Changed lines of the file:
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@@
+		)
+	)
+	(label "CAN_CS_C"
+		(at 107.95 147.32 0)
+		(effects
+			(font
+				(size 1.27 1.27)
+			)
+			(justify left bottom)
 		)
 	)
@@
 			)
 			(justify right bottom)
+		)
+	)
+	(label "CAN_CS_B"
+		(at 107.95 144.78 0)
+		(effects
+			(font
+				(size 1.27 1.27)
+			)
+			(justify left bottom)
+		)
+	)
+	(label "SPI3_SCK"
+		(at 107.95 137.16 0)
+		(effects
+			(font
+				(size 1.27 1.27)
+			)
+			(justify left bottom)
 		)
 	)
@@
 			)
 			(justify right bottom)
+		)
+	)
+	(label "SPI3_MOSI"
+		(at 107.95 134.62 0)
+		(effects
+			(font
+				(size 1.27 1.27)
+			)
+			(justify left bottom)
 		)
 	)
@@
 		)
 	)
+	(label "CAN_CS_A"
+		(at 107.95 142.24 0)
+		(effects
+			(font
+				(size 1.27 1.27)
+			)
+			(justify left bottom)
+		)
+	)
 	(label "SPI2_MOSI"
 		(at 86.36 113.03 180)
@@
 		)
 	)
+	(label "SPI3_MISO"
+		(at 107.95 139.7 0)
+		(effects
+			(font
+				(size 1.27 1.27)
+			)
+			(justify left bottom)
+		)
+	)

Commit message: ethernet hardware side
Connections:
- net SPI2_MISO: no longer J8.7 (DAT0)
- net SPI2_MOSI: no longer J8.3 (CMD)
- net SPI2_SCK: no longer J8.5 (CLK)
- net SD_DAT2: now reaches J8.1 (DAT2)
- net SD_DAT1: now reaches J8.8 (DAT1)
- net SPI2_CS_SD renamed SD_DAT3
- new net SD_CLK: J8.5 (CLK)
- new net SD_CMD: J8.3 (CMD)
- new net SD_DAT0: J8.7 (DAT0)
- no-connect marks 2 -> 0
Changed lines of the file:
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@@
 		(color 0 0 0 0)
 	)
-	(no_connect
-		(at 73.66 100.33)
-	)
-	(no_connect
-		(at 73.66 118.11)
-	)
 	(wire
 		(pts
@@
 	(wire
 		(pts
+			(xy 73.66 118.11) (xy 86.36 118.11)
+		)
+		(stroke
+			(width 0)
+			(type default)
+		)
+	)
+	(wire
+		(pts
 			(xy 196.85 123.19) (xy 196.85 124.46)
 		)
@@
 	(wire
 		(pts
+			(xy 78.74 144.78) (xy 91.44 144.78)
+		)
+		(stroke
+			(width 0)
+			(type default)
+		)
+	)
+	(wire
+		(pts
 			(xy 228.6 100.33) (xy 228.6 97.79)
 		)
@@
 	(wire
 		(pts
+			(xy 78.74 147.32) (xy 91.44 147.32)
+		)
+		(stroke
+			(width 0)
+			(type default)
+		)
+	)
+	(wire
+		(pts
 			(xy 212.09 100.33) (xy 212.09 97.79)
 		)
@@
 	(wire
 		(pts
+			(xy 78.74 160.02) (xy 91.44 160.02)
+		)
+		(stroke
+			(width 0)
+			(type default)
+		)
+	)
+	(wire
+		(pts
+			(xy 78.74 149.86) (xy 91.44 149.86)
+		)
+		(stroke
+			(width 0)
+			(type default)
+		)
+	)
+	(wire
+		(pts
 			(xy 187.96 130.81) (xy 187.96 133.35)
+		)
+		(stroke
+			(width 0)
+			(type default)
+		)
+	)
+	(wire
+		(pts
+			(xy 73.66 100.33) (xy 86.36 100.33)
 		)
 		(stroke
@@
 		)
 	)
+	(label "SD_DAT0"
+		(at 107.95 161.29 0)
+		(effects
+			(font
+				(size 1.27 1.27)
+			)
+			(justify left bottom)
+		)
+	)
+	(label "RF_IO7"
+		(at 91.44 144.78 180)
+		(effects
+			(font
+				(size 1.27 1.27)
+			)
+			(justify right bottom)
+		)
+	)
 	(label "SPI2_CS_RF"
 		(at 91.44 162.56 180)
@@
 		)
 	)
+	(label "RF_IO8"
+		(at 91.44 147.32 180)
+		(effects
+			(font
+				(size 1.27 1.27)
+			)
+			(justify right bottom)
+		)
+	)
+	(label "RF_IO7"
+		(at 107.95 176.53 0)
+		(effects
+			(font
+				(size 1.27 1.27)
+			)
+			(justify left bottom)
+		)
+	)
 	(label "CAN_CS_B"
 		(at 107.95 144.78 0)
@@
 		)
 	)
-	(label "SPI2_CS_SD"
-		(at 173.99 146.05 180)
-		(effects
-			(font
-				(size 1.27 1.27)
-			)
-			(justify right bottom)
+	(label "RF_RST"
+		(at 91.44 160.02 180)
+		(effects
+			(font
+				(size 1.27 1.27)
+			)
+			(justify right bottom)
+		)
+	)
+	(label "SD_DAT2"
+		(at 86.36 118.11 180)
+		(effects
+			(font
+				(size 1.27 1.27)
+			)
+			(justify right bottom)
+		)
+	)
+	(label "SD_CLK"
+		(at 107.95 158.75 0)
+		(effects
+			(font
+				(size 1.27 1.27)
+			)
+			(justify left bottom)
+		)
+	)
+	(label "SD_CMD"
+		(at 107.95 156.21 0)
+		(effects
+			(font
+				(size 1.27 1.27)
+			)
+			(justify left bottom)
 		)
 	)
@@
 		)
 	)
-	(label "SPI2_MISO"
+	(label "SD_DAT1"
+		(at 107.95 163.83 0)
+		(effects
+			(font
+				(size 1.27 1.27)
+			)
+			(justify left bottom)
+		)
+	)
+	(label "SD_DAT0"
 		(at 86.36 102.87 180)
 		(effects
@@
 		)
 	)
-	(label "SPI2_CS_SD"
+	(label "SD_DAT3"
 		(at 86.36 115.57 180)
 		(effects
@@
 			)
 			(justify right bottom)
+		)
+	)
+	(label "RF_IO11"
+		(at 107.95 171.45 0)
+		(effects
+			(font
+				(size 1.27 1.27)
+			)
+			(justify left bottom)
+		)
+	)
+	(label "RF_IO8"
+		(at 107.95 173.99 0)
+		(effects
+			(font
+				(size 1.27 1.27)
+			)
+			(justify left bottom)
+		)
+	)
+	(label "SD_DAT2"
+		(at 107.95 151.13 0)
+		(effects
+			(font
+				(size 1.27 1.27)
+			)
+			(justify left bottom)
+		)
+	)
+	(label "SD_DAT3"
+		(at 107.95 153.67 0)
+		(effects
+			(font
+				(size 1.27 1.27)
+			)
+			(justify left bottom)
 		)
 	)
@@
 		)
 	)
-	(label "SPI2_MOSI"
+	(label "SD_DAT1"
+		(at 86.36 100.33 180)
+		(effects
+			(font
+				(size 1.27 1.27)
+			)
+			(justify right bottom)
+		)
+	)
+	(label "RF_IO11"
+		(at 91.44 149.86 180)
+		(effects
+			(font
+				(size 1.27 1.27)
+			)
+			(justify right bottom)
+		)
+	)
+	(label "SD_CMD"
 		(at 86.36 113.03 180)
 		(effects
@@
 		)
 	)
-	(label "SPI2_SCK"
+	(label "SD_CLK"
 		(at 86.36 107.95 180)
 		(effects
@@
 		)
 	)
+	(label "RF_RST"
+		(at 107.95 168.91 0)
+		(effects
+			(font
+				(size 1.27 1.27)
+			)
+			(justify left bottom)
+		)
+	)
