File: telemetry-logging-board/telemetry-logging-board.kicad_sch (KiCad schematic)
At the start: 8 parts, among them J12 Wifi, J13 ESP, J5 USB_C_Receptacle_USB2.0_16P, J8 Micro_SD_Card, U1 ESP32-S3-MINI-1U, U6 USBLC6-2SC6

Commit message: use every pin
Parts:
- added JP10, JP8, JP9: SD_SPI, symbol Jumper:SolderJumper_2_Open
- added R108, R109: 10k, symbol Device:R
- added SW1: FLASH, symbol Switch:SW_SPST
- added TP3: GP44, symbol Connector:TestPoint
- added TP5: TX, symbol Connector:TestPoint
- added TP6: RX, symbol Connector:TestPoint
Connections:
- net +3V3: now also R108.1
- net CAN_CS_A: now also U1.35 (IO39)
- net CAN_CS_B: now also U1.36 (IO40)
- net CAN_CS_C: now also U1.37 (IO41)
- net CAN_INT_A: now also U1.27 (IO47)
- net CAN_INT_B: now also U1.38 (IO42)
- net CAN_INT_C: now also U1.29 (IO34)
- net GND: now also R109.2, SW1.2 (B)
- net RF_IO11: now also U1.28 (IO33)
- net RF_IO7: now also U1.30 (IO48)
- net RF_IO8: now also U1.34 (IO38)
- net SD_CLK: now also U1.11 (IO7), JP9.2 (B)
- net SD_CMD: now also U1.10 (IO6), JP8.2 (B)
- net SD_DAT0: now also U1.19 (IO15), JP10.2 (B)
- net SD_DAT1: now also U1.25 (IO21)
- net SD_DAT2: now also U1.7 (IO3)
- net SD_DAT3: now also U1.14 (IO10)
- net SPI2_CS_RF: now also U1.13 (IO9); no longer U1.34 (IO38)
- net SPI2_MISO: now also U1.17 (IO13), JP10.1 (A); no longer U1.33 (IO37)
- net SPI2_MOSI: now also U1.15 (IO11), JP8.1 (A); no longer U1.31 (IO35)
- net SPI2_SCK: now also U1.16 (IO12), JP9.1 (A); no longer U1.32 (IO36)
- net SPI3_MISO: now also U1.33 (IO37)
- net SPI3_MOSI: now also U1.31 (IO35)
- net SPI3_SCK: now also U1.32 (IO36)
- net ETH_~{CS}: now reaches U1.12 (IO8)
- net SW_UART_RX: now reaches U1.18 (IO14)
- net SW_UART_TX: now reaches U1.20 (IO16)
- net ETH_~{INT}: now reaches U1.21 (IO17)
- net ETH_~{RST}: now reaches U1.22 (IO18)
- net RF_~{RST}: now reaches U1.26 (IO26)
- net at U1.39 (TXD0): now also TP5.1
- net at U1.4 (IO0): now also R108.2, SW1.1 (A)
- net at U1.40 (RXD0): now also TP6.1
- net CHRG: now reaches U1.41 (IO45)
- net at U1.44 (IO46): now also R109.1, TP3.1
- net ETH_EN: now reaches U1.5 (IO1)
- net PERIPH_EN: now reaches U1.6 (IO2)
- net CAN_A_EN: now reaches U1.8 (IO4)
- net BATT_SENS: now reaches U1.9 (IO5)
Other:
- sheet Ethernet ports: added MISO, MOSI, SCLK, SW_RST, SW_UART_RX, SW_UART_TX, ~{CS}_ETH, ~{INT}, ~{RST}; removed none
- sheet Power Supply ports: added BAT_SENS, CAN_A_EN, CHRG, ETH_EN, PERIPH_EN; removed none
- note added: "Jump ESP32 WiFi from U.fl to SMA"
- note added: "Must be low for USB-Serial-JTAG/UART boot"
- note added: "SD_CS"
- note added: "Strap Fully ovveridable by efuse"
- note removed: "Strap"
- moved on the sheet: J12, J13, J5, J8, R4, R5, U1, U6

Commit message: replace LR2021 with seeed wio LR2021, rework psu
Parts:
- added JP11: SD_SPI, symbol Jumper:SolderJumper_2_Open
Connections:
- net CHRG: now also JP11.1 (A)
- net CAN_A_EN: no longer names the net of U1.8 (IO4)
- new net Power Supply/CHRG: JP11.2 (B)
Other:
- sheet LR Radio: file rf.kicad_sch -> rf_mod.kicad_sch
- sheet Power Supply ports: added none; removed CAN_A_EN
- moved on the sheet: R109, TP3
Changed lines of the file:
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@@
 	(text "Must be low for USB-Serial-JTAG/UART boot"
 		(exclude_from_sim no)
-		(at 219.456 147.32 0)
+		(at 225.806 147.32 0)
 		(effects
 			(font
@@
 	(text "Strap Fully ovveridable by efuse"
 		(exclude_from_sim no)
-		(at 213.106 144.526 0)
+		(at 219.456 144.526 0)
 		(effects
 			(font
@@
 	)
 	(junction
-		(at 195.58 147.32)
+		(at 201.93 147.32)
 		(diameter 0)
 		(color 0 0 0 0)
@@
 	(wire
 		(pts
-			(xy 80.01 35.56) (xy 92.71 35.56)
+			(xy 80.01 35.56) (xy 91.44 35.56)
 		)
 		(stroke
@@
 	(wire
 		(pts
-			(xy 199.39 138.43) (xy 195.58 138.43)
-		)
-		(stroke
-			(width 0)
-			(type default)
-		)
-	)
-	(wire
-		(pts
 			(xy 189.23 101.6) (xy 180.34 101.6)
 		)
@@
 	(wire
 		(pts
-			(xy 80.01 43.18) (xy 92.71 43.18)
+			(xy 80.01 40.64) (xy 92.71 40.64)
 		)
 		(stroke
@@
 	(wire
 		(pts
-			(xy 195.58 138.43) (xy 195.58 147.32)
+			(xy 201.93 143.51) (xy 201.93 147.32)
 		)
 		(stroke
@@
 	(wire
 		(pts
-			(xy 180.34 147.32) (xy 195.58 147.32)
+			(xy 180.34 147.32) (xy 201.93 147.32)
 		)
 		(stroke
@@
 	(wire
 		(pts
-			(xy 215.9 114.3) (xy 223.52 114.3)
+			(xy 101.6 35.56) (xy 106.68 35.56)
 		)
 		(stroke
@@
 	(wire
 		(pts
-			(xy 137.16 111.76) (xy 149.86 111.76)
+			(xy 215.9 114.3) (xy 223.52 114.3)
 		)
 		(stroke
@@
 	(wire
 		(pts
-			(xy 215.9 40.64) (xy 227.33 40.64)
+			(xy 137.16 111.76) (xy 149.86 111.76)
 		)
 		(stroke
@@
 	(wire
 		(pts
-			(xy 137.16 109.22) (xy 149.86 109.22)
+			(xy 215.9 40.64) (xy 227.33 40.64)
 		)
 		(stroke
@@
 	(wire
 		(pts
-			(xy 82.55 120.65) (xy 82.55 105.41)
+			(xy 137.16 109.22) (xy 149.86 109.22)
 		)
 		(stroke
@@
 	(wire
 		(pts
-			(xy 78.74 154.94) (xy 91.44 154.94)
+			(xy 82.55 120.65) (xy 82.55 105.41)
 		)
 		(stroke
@@
 	(wire
 		(pts
-			(xy 66.04 113.03) (xy 87.63 113.03)
+			(xy 78.74 154.94) (xy 91.44 154.94)
 		)
 		(stroke
@@
 	(wire
 		(pts
-			(xy 137.16 114.3) (xy 149.86 114.3)
+			(xy 66.04 113.03) (xy 87.63 113.03)
 		)
 		(stroke
@@
 	(wire
 		(pts
-			(xy 80.01 40.64) (xy 92.71 40.64)
+			(xy 137.16 114.3) (xy 149.86 114.3)
 		)
 		(stroke
@@
 	(wire
 		(pts
-			(xy 80.01 45.72) (xy 92.71 45.72)
+			(xy 80.01 43.18) (xy 92.71 43.18)
 		)
 		(stroke
@@
 		)
 	)
-	(label "CAN_A_EN"
-		(at 137.16 116.84 0)
-		(effects
-			(font
-				(size 1.27 1.27)
-			)
-			(justify left bottom)
-		)
-	)
 	(label "CAN_INT_B"
 		(at 193.04 142.24 180)
@@
 		)
 	)
-	(label "CAN_A_EN"
-		(at 92.71 40.64 180)
-		(effects
-			(font
-				(size 1.27 1.27)
-			)
-			(justify right bottom)
-		)
-	)
 	(label "SD_CMD"
 		(at 78.74 113.03 180)
@@
 	)
 	(label "CHRG"
-		(at 92.71 35.56 180)
+		(at 106.68 35.56 180)
 		(effects
 			(font
@@
 	)
 	(label "ETH_EN"
-		(at 92.71 45.72 180)
+		(at 92.71 43.18 180)
 		(effects
 			(font
@@
 	)
 	(label "PERIPH_EN"
-		(at 92.71 43.18 180)
+		(at 92.71 40.64 180)
 		(effects
 			(font
@@
 	(symbol
 		(lib_id "power:GND")
-		(at 195.58 154.94 0)
+		(at 201.93 154.94 0)
 		(unit 1)
 		(body_style 1)
@@
 		(dnp no)
 		(property "Reference" "#PWR0127"
-			(at 195.58 161.29 0)
+			(at 201.93 161.29 0)
 			(hide yes)
 			(show_name no)
@@
 		)
 		(property "Value" "GND"
-			(at 195.58 158.75 0)
+			(at 201.93 158.75 0)
 			(show_name no)
 			(do_not_autoplace no)
@@
 		)
 		(property "Footprint" ""
-			(at 195.58 154.94 0)
+			(at 201.93 154.94 0)
 			(hide yes)
 			(show_name no)
@@
 		)
 		(property "Datasheet" ""
-			(at 195.58 154.94 0)
+			(at 201.93 154.94 0)
 			(hide yes)
 			(show_name no)
@@
 		)
 		(property "Description" "Power symbol creates a global label with name \"GND\" , ground"
-			(at 195.58 154.94 0)
+			(at 201.93 154.94 0)
 			(hide yes)
 			(show_name no)
@@
 	)
 	(symbol
+		(lib_id "Jumper:SolderJumper_2_Open")
+		(at 96.52 35.56 180)
+		(unit 1)
+		(body_style 1)
+		(exclude_from_sim no)
+		(in_bom no)
+		(on_board yes)
+		(in_pos_files yes)
+		(dnp no)
+		(property "Reference" "JP11"
+			(at 92.964 34.036 0)
+			(show_name no)
+			(do_not_autoplace no)
+			(effects
+				(font
+					(size 1.27 1.27)
+				)
+			)
+		)
+		(property "Value" "SD_SPI"
+			(at 96.52 33.02 0)
+			(hide yes)
+			(show_name no)
+			(do_not_autoplace no)
+			(effects
+				(font
+					(size 1.27 1.27)
+				)
+			)
+		)
+		(property "Footprint" ""
+			(at 96.52 35.56 0)
+			(hide yes)
+			(show_name no)
+			(do_not_autoplace no)
+			(effects
+				(font
+					(size 1.27 1.27)
+				)
+			)
+		)
+		(property "Datasheet" ""
+			(at 96.52 27.94 0)
+			(hide yes)
+			(show_name no)
+			(do_not_autoplace no)
+			(effects
+				(font
+					(size 1.27 1.27)
+				)
+			)
+		)
+		(property "Description" "Solder Jumper, 2-pole, open"
+			(at 96.52 30.48 0)
+			(hide yes)
+			(show_name no)
+			(do_not_autoplace no)
+			(effects
+				(font
+					(size 1.27 1.27)
+				)
+			)
+		)
+		(pin "2"
+		)
+		(pin "1"
+		)
+		(instances
+			(project "telemetry-logging-board"
+				(path "/77f08122-c609-410b-9d24-33eebdb4af2b"
+					(reference "JP11")
+					(unit 1)
+				)
+			)
+		)
+	)
+	(symbol
 		(lib_id "Device:R")
 		(at 124.46 102.87 0)
@@
 	(symbol
 		(lib_id "Connector:TestPoint")
-		(at 199.39 138.43 270)
+		(at 201.93 143.51 0)
 		(unit 1)
 		(body_style 1)
@@
 		(fields_autoplaced yes)
 		(property "Reference" "TP3"
-			(at 204.47 137.1599 90)
+			(at 204.47 138.9379 0)
 			(show_name no)
 			(do_not_autoplace no)
@@
 		)
 		(property "Value" "GP44"
-			(at 204.47 139.6999 90)
+			(at 204.47 141.4779 0)
 			(show_name no)
 			(do_not_autoplace no)
@@
 		)
 		(property "Footprint" ""
-			(at 199.39 143.51 0)
+			(at 207.01 143.51 0)
 			(hide yes)
 			(show_name no)
@@
 		)
 		(property "Datasheet" ""
-			(at 199.39 143.51 0)
+			(at 207.01 143.51 0)
 			(hide yes)
 			(show_name no)
@@
 		)
 		(property "Description" "test point"
-			(at 199.39 138.43 0)
+			(at 201.93 143.51 0)
 			(hide yes)
 			(show_name no)
@@
 	(symbol
 		(lib_id "Device:R")
-		(at 195.58 151.13 0)
+		(at 201.93 151.13 0)
 		(unit 1)
 		(body_style 1)
@@
 		(fields_autoplaced yes)
 		(property "Reference" "R109"
-			(at 198.12 149.8599 0)
+			(at 204.47 149.8599 0)
 			(show_name no)
 			(do_not_autoplace no)
@@
 		)
 		(property "Value" "10k"
-			(at 198.12 152.3999 0)
+			(at 204.47 152.3999 0)
 			(show_name no)
 			(do_not_autoplace no)
@@
 		)
 		(property "Footprint" ""
-			(at 193.802 151.13 90)
+			(at 200.152 151.13 90)
 			(hide yes)
 			(show_name no)
@@
 		)
 		(property "Datasheet" ""
-			(at 195.58 151.13 0)
+			(at 201.93 151.13 0)
 			(hide yes)
 			(show_name no)
@@
 		)
 		(property "Description" "Resistor"
-			(at 195.58 151.13 0)
+			(at 201.93 151.13 0)
 			(hide yes)
 			(show_name no)
@@
 			)
 		)
-		(pin "CAN_A_EN" input
-			(at 80.01 40.64 0)
-			(effects
-				(font
-					(size 1.27 1.27)
-				)
-				(justify right)
-			)
-		)
 		(pin "CHRG" output
 			(at 80.01 35.56 0)
@@
 		)
 		(pin "ETH_EN" input
-			(at 80.01 45.72 0)
+			(at 80.01 43.18 0)
 			(effects
 				(font
@@
 		)
 		(pin "PERIPH_EN" input
-			(at 80.01 43.18 0)
+			(at 80.01 40.64 0)
 			(effects
 				(font
@@
 			)
 		)
-		(property "Sheetfile" "rf.kicad_sch"
+		(property "Sheetfile" "rf_mod.kicad_sch"
 			(at 24.13 182.1946 0)
 			(show_name no)

Commit message: idek
Parts:
- JP1: renamed from JP10; footprint (none) -> Jumper:SolderJumper-2_P1.3mm_Open_RoundedPad1.0x1.5mm
- JP2: renamed from JP9; footprint (none) -> Jumper:SolderJumper-2_P1.3mm_Open_RoundedPad1.0x1.5mm
- JP3: renamed from JP8; footprint (none) -> Jumper:SolderJumper-2_P1.3mm_Open_RoundedPad1.0x1.5mm
- JP4: renamed from JP11; footprint (none) -> Jumper:SolderJumper-2_P1.3mm_Open_RoundedPad1.0x1.5mm
- R1: renamed from R108; footprint (none) -> Resistor_SMD:R_0603_1608Metric
- R2: renamed from R109; footprint (none) -> Resistor_SMD:R_0603_1608Metric
- R3: renamed from R4; footprint (none) -> Resistor_SMD:R_0603_1608Metric
- R4: renamed from R5; footprint (none) -> Resistor_SMD:R_0603_1608Metric
- SW1: footprint (none) -> Button_Switch_SMD:SW_Push_1P1T-SH_NO_CK_KMR2xxG
- TP1: renamed from TP5; footprint (none) -> TestPoint:TestPoint_Pad_2.0x2.0mm
- TP2: renamed from TP6; footprint (none) -> TestPoint:TestPoint_Pad_2.0x2.0mm
- TP3: footprint (none) -> TestPoint:TestPoint_Pad_2.0x2.0mm
- renumbered J8 to J1, J13 to J2, J12 to J3, J5 to J4, U6 to U2
