File: telemetry-logging-board/can-if-trx.kicad_sch (KiCad schematic)
At the start: 7 parts, among them U2 MCP2518FD-xQBB, U3 ISO1044BD, Y1 ECS-200-12-33Q-JES-TR

Commit message: mostly CAN work
Parts:
- added D4: NUP2105L, Package_TO_SOT_SMD:SOT-23, symbol Power_Protection:NUP2105L
- added GD2: GDT_2Pin, symbol Device:GDT_2Pin
- added R29, R30, R31, R32, R33, R35, R36: 0R, symbol Device:R_Small
- added R34, R37, R38: 1M, symbol Device:R_Small
- added R40: 60R, Resistor_SMD:R_0805_2012Metric, symbol Device:R
- added R41, R42: 1k, Resistor_SMD:R_0805_2012Metric, symbol Device:R
- added SW3: TERM, symbol Switch:SW_DPST
- added U11: CRE1S0505SC, Converter_DCDC:Converter_DCDC_Murata_CRE1xxxxxxSC_THT, symbol Converter_DCDC_Isolated:CRE1S0505SC
- R39: renamed from R1; value 120R -> 60R
- renumbered C1 to C12, C2 to C36, C3 to C39, U3 to U12, U2 to U7, Y1 to Y3
Connections:
- net CAN_H: now also D4.2 (K), R41.1
- net CAN_L: now also D4.1 (K), R40.2, R42.2; no longer R39.2
- net GND: now also GD2.3, R34.1, R36.1, U11.1 (-VIN); no longer C39.1, U12.7 (GND2)
- net at C12.1, U7.5 (OSC2), Y3.1: now also R29.2
- net at U7.1 (TXCAN): now also R31.2, R32.2; no longer U12.2 (TXD)
- net at U12.3 (RXD): now also R30.1, R32.1; no longer U7.2 (RXCAN)
- net CLKOUT: now reaches U7.3 (CLKO/SOF)
- net 5v renamed ISO_5V
- net ISO_5V: now also R35.2, U11.4 (+VOUT)
- new net: R39.2, SW3.3
- new net: R34.2, R37.1
- new net: R40.1, SW3.1
- new net: R31.1, R33.1, U12.2 (TXD)
- new net: R30.2, R33.2, U7.2 (RXCAN)
- new net: R37.2, R38.1
- new net CLKIN: R29.1
- new net ISO_0V: C39.1, D4.3 (A), GD2.1, R36.2, R38.2, R41.2, R42.1, SW3.2, SW3.4, U11.3 (-VOUT), U12.7 (GND2)
- new net VDD_CAN: R35.1, U11.2 (+VIN)
Other:
- note added: "Arrests strong common mode events"
- note added: "Crystal and oscillators can be de-populated if CLKIN is available"
- note added: "Populate Left for ISO1044. Populate Right for ADM3050"
- note added: "Prevents slow common mode accumulation"
- note added: "Resistors depopulated for isolation must be large footprint! Per IEC 60664-1 Table F.2: 2.5kv : 1.5mm 4kv : 3.0mm 6kv : 5.5mm R1206 : 1.8mm gap"
- company: (none) -> Formula Slug
- title: (none) -> Telemetry Logging Board: CAN Interface
- moved on the sheet: C12, C36, C39, R39, U12, U7, Y3

Commit message: ethernet hardware side
Connections:
- net GPIO1 renamed ~{INT-1}(RX)
- net ~{INT-I} renamed ~{INT-0}(TX)
- net ~{INT-O} renamed ~{INT}
Changed lines of the file:
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@@
 		)
 	)
-	(hierarchical_label "~{INT-I}"
-		(shape bidirectional)
+	(hierarchical_label "~{INT-0}(TX)"
+		(shape output)
 		(at 114.3 111.76 0)
 		(effects
@@
 		)
 	)
-	(hierarchical_label "~{INT-O}"
-		(shape bidirectional)
+	(hierarchical_label "~{INT}"
+		(shape output)
 		(at 114.3 109.22 0)
 		(effects
@@
 		)
 	)
-	(hierarchical_label "GPIO1"
-		(shape bidirectional)
+	(hierarchical_label "~{INT-1}(RX)"
+		(shape output)
 		(at 114.3 114.3 0)
 		(effects

Commit message: update title block
Other:
- title: Telemetry Logging Board: CAN Interface -> Telemetry Logging Board
Changed lines of the file:
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@@
 	(paper "A4")
 	(title_block
-		(title "Telemetry Logging Board: CAN Interface")
+		(title "Telemetry Logging Board")
 		(date "2026-07-30")
 		(rev "R2.0")
