File: telemetry-logging-board/eth.kicad_sch (KiCad schematic)
At the start: 5 parts, among them J1 RJ45_Bel_SI-60062-F, J2 RJ45_Bel_SI-60062-F, J3 RJ45_Bel_SI-60062-F, J4 RJ45_Bel_SI-60062-F, U4 LAN9370T-I/KCX

Commit message: mostly CAN work
Other:
- company: (none) -> Formula Slug
- title: (none) -> Telemetry Logging Board
Changed lines of the file:
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@@
 	(generator_version "10.0")
 	(paper "A4")
+	(title_block
+		(title "Telemetry Logging Board")
+		(date "2026-07-30")
+		(rev "R2.0")
+		(company "Formula Slug")
+		(comment 1 "Designed by Luca Younes")
+	)
 	(symbol
 		(lib_id "Connector:RJ45_Bel_SI-60062-F")

Commit message: eth chip
Parts:
- removed J4: RJ45_Bel_SI-60062-F, Connector_RJ:RJ45_Pulse_JK00177NL_Horizontal, symbol Connector:RJ45_Bel_SI-60062-F
- added U9: W5500, Package_QFP:LQFP-48_7x7mm_P0.5mm, symbol Interface_Ethernet:W5500
Connections:
- new net: U9.11 (AVDD), U9.15 (AVDD), U9.17 (AVDD), U9.21 (AVDD), U9.4 (AVDD), U9.8 (AVDD)
- new net: U9.14 (AGND), U9.16 (AGND), U9.19 (AGND), U9.3 (AGND), U9.48 (AGND), U9.9 (AGND)
Other:
- moved on the sheet: J1, J2, J3, U4
Changed lines of the file:
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@@
 	(generator "eeschema")
 	(generator_version "10.0")
-	(paper "A4")
+	(paper "A3")
 	(title_block
 		(title "Telemetry Logging Board")
@@
 	(symbol
 		(lib_id "Connector:RJ45_Bel_SI-60062-F")
-		(at 248.92 53.34 0)
+		(at 349.25 104.14 0)
 		(unit 1)
 		(body_style 1)
@@
 		(fields_autoplaced yes)
 		(property "Reference" "J1"
-			(at 250.19 39.37 0)
+			(at 350.52 90.17 0)
 			(show_name no)
 			(do_not_autoplace no)
@@
 		)
 		(property "Value" "RJ45_Bel_SI-60062-F"
-			(at 250.19 41.91 0)
+			(at 350.52 92.71 0)
 			(show_name no)
 			(do_not_autoplace no)
@@
 		)
 		(property "Footprint" "Connector_RJ:RJ45_Pulse_JK00177NL_Horizontal"
-			(at 248.92 40.64 0)
+			(at 349.25 91.44 0)
 			(hide yes)
 			(show_name no)
@@
 		)
 		(property "Datasheet" "https://belfuse.com/resources/drawings/magneticsolutions/dr-mag-si-60062-f.pdf"
-			(at 248.92 38.1 0)
+			(at 349.25 88.9 0)
 			(hide yes)
 			(show_name no)
@@
 		)
 		(property "Description" "1 Port RJ45 Magjack Connector Through Hole 10/100 Base-T, AutoMDIX"
-			(at 248.92 53.34 0)
+			(at 349.25 104.14 0)
 			(hide yes)
 			(show_name no)
@@
 	)
 	(symbol
-		(lib_id "Connector:RJ45_Bel_SI-60062-F")
-		(at 248.92 132.08 0)
+		(lib_id "Interface_Ethernet:W5500")
+		(at 196.85 219.71 0)
 		(unit 1)
 		(body_style 1)
@@
 		(dnp no)
 		(fields_autoplaced yes)
-		(property "Reference" "J4"
-			(at 250.19 118.11 0)
-			(show_name no)
-			(do_not_autoplace no)
-			(effects
-				(font
-					(size 1.27 1.27)
-				)
-			)
-		)
-		(property "Value" "RJ45_Bel_SI-60062-F"
-			(at 250.19 120.65 0)
-			(show_name no)
-			(do_not_autoplace no)
-			(effects
-				(font
-					(size 1.27 1.27)
-				)
-			)
-		)
-		(property "Footprint" "Connector_RJ:RJ45_Pulse_JK00177NL_Horizontal"
-			(at 248.92 119.38 0)
-			(hide yes)
-			(show_name no)
-			(do_not_autoplace no)
-			(effects
-				(font
-					(size 1.27 1.27)
-				)
-			)
-		)
-		(property "Datasheet" "https://belfuse.com/resources/drawings/magneticsolutions/dr-mag-si-60062-f.pdf"
-			(at 248.92 116.84 0)
-			(hide yes)
-			(show_name no)
-			(do_not_autoplace no)
-			(effects
-				(font
-					(size 1.27 1.27)
-				)
-			)
-		)
-		(property "Description" "1 Port RJ45 Magjack Connector Through Hole 10/100 Base-T, AutoMDIX"
-			(at 248.92 132.08 0)
-			(hide yes)
-			(show_name no)
-			(do_not_autoplace no)
-			(effects
-				(font
-					(size 1.27 1.27)
-				)
-			)
-		)
-		(pin "L3"
+		(property "Reference" "U9"
+			(at 201.5333 186.69 0)
+			(show_name no)
+			(do_not_autoplace no)
+			(effects
+				(font
+					(size 1.27 1.27)
+				)
+				(justify left)
+			)
+		)
+		(property "Value" "W5500"
+			(at 201.5333 189.23 0)
+			(show_name no)
+			(do_not_autoplace no)
+			(effects
+				(font
+					(size 1.27 1.27)
+				)
+				(justify left)
+			)
+		)
+		(property "Footprint" "Package_QFP:LQFP-48_7x7mm_P0.5mm"
+			(at 196.85 177.8 0)
+			(hide yes)
+			(show_name no)
+			(do_not_autoplace no)
+			(effects
+				(font
+					(size 1.27 1.27)
+				)
+			)
+		)
+		(property "Datasheet" "http://wizwiki.net/wiki/lib/exe/fetch.php/products:w5500:w5500_ds_v109e.pdf"
+			(at 196.85 194.31 0)
+			(hide yes)
+			(show_name no)
+			(do_not_autoplace no)
+			(effects
+				(font
+					(size 1.27 1.27)
+				)
+			)
+		)
+		(property "Description" "10/100Mb SPI Ethernet controller with TCP/IP stack, LQFP-48"
+			(at 196.85 219.71 0)
+			(hide yes)
+			(show_name no)
+			(do_not_autoplace no)
+			(effects
+				(font
+					(size 1.27 1.27)
+				)
+			)
+		)
+		(pin "25"
+		)
+		(pin "22"
+		)
+		(pin "37"
+		)
+		(pin "27"
+		)
+		(pin "30"
+		)
+		(pin "13"
+		)
+		(pin "10"
+		)
+		(pin "2"
+		)
+		(pin "26"
+		)
+		(pin "21"
+		)
+		(pin "43"
+		)
+		(pin "3"
+		)
+		(pin "15"
+		)
+		(pin "40"
+		)
+		(pin "42"
 		)
 		(pin "7"
 		)
-		(pin "L4"
+		(pin "35"
+		)
+		(pin "39"
+		)
+		(pin "47"
+		)
+		(pin "1"
+		)
+		(pin "32"
+		)
+		(pin "38"
+		)
+		(pin "28"
+		)
+		(pin "14"
+		)
+		(pin "36"
+		)
+		(pin "33"
+		)
+		(pin "11"
+		)
+		(pin "41"
+		)
+		(pin "29"
+		)
+		(pin "12"
+		)
+		(pin "19"
+		)
+		(pin "20"
+		)
+		(pin "46"
+		)
+		(pin "18"
+		)
+		(pin "34"
+		)
+		(pin "23"
+		)
+		(pin "44"
+		)
+		(pin "24"
+		)
+		(pin "45"
+		)
+		(pin "16"
+		)
+		(pin "48"
+		)
+		(pin "31"
+		)
+		(pin "17"
+		)
+		(pin "6"
+		)
+		(pin "5"
+		)
+		(pin "4"
 		)
 		(pin "8"
 		)
-		(pin "L1"
-		)
-		(pin "6"
-		)
-		(pin "SH"
-		)
-		(pin "1"
-		)
-		(pin "L2"
-		)
-		(pin "4"
-		)
-		(pin "5"
-		)
-		(pin "3"
-		)
-		(pin "2"
+		(pin "9"
 		)
 		(instances
 			(project "telemetry-logging-board"
 				(path "/77f08122-c609-410b-9d24-33eebdb4af2b/7979997a-7ce3-4ea9-80ba-9abc2907bb28"
-					(reference "J4")
+					(reference "U9")
 					(unit 1)
 				)
@@
 	(symbol
 		(lib_id "allwinner-sip-lib:LAN9370T-I_KCX")
-		(at 73.66 50.8 0)
+		(at 210.82 172.72 180)
 		(unit 1)
 		(body_style 1)
@@
 		(fields_autoplaced yes)
 		(property "Reference" "U4"
-			(at 129.54 40.64 0)
+			(at 154.94 81.28 0)
 			(show_name no)
 			(do_not_autoplace no)
@@
 		)
 		(property "Value" "LAN9370T-I/KCX"
-			(at 129.54 43.18 0)
+			(at 154.94 83.82 0)
 			(show_name no)
 			(do_not_autoplace no)
@@
 		)
 		(property "Footprint" "QFN_LAN9370T-I/KCX_MCH"
-			(at 73.66 50.8 0)
+			(at 210.82 172.72 0)
 			(hide yes)
 			(show_name no)
@@
 		)
 		(property "Datasheet" "LAN9370T-I/KCX"
-			(at 73.66 50.8 0)
+			(at 210.82 172.72 0)
 			(hide yes)
 			(show_name no)
@@
 		)
 		(property "Description" ""
-			(at 73.66 50.8 0)
+			(at 210.82 172.72 0)
 			(hide yes)
 			(show_name no)
@@
 	(symbol
 		(lib_id "Connector:RJ45_Bel_SI-60062-F")
-		(at 248.92 78.74 0)
+		(at 349.25 129.54 0)
 		(unit 1)
 		(body_style 1)
@@
 		(fields_autoplaced yes)
 		(property "Reference" "J2"
-			(at 250.19 64.77 0)
+			(at 350.52 115.57 0)
 			(show_name no)
 			(do_not_autoplace no)
@@
 		)
 		(property "Value" "RJ45_Bel_SI-60062-F"
-			(at 250.19 67.31 0)
+			(at 350.52 118.11 0)
 			(show_name no)
 			(do_not_autoplace no)
@@
 		)
 		(property "Footprint" "Connector_RJ:RJ45_Pulse_JK00177NL_Horizontal"
-			(at 248.92 66.04 0)
+			(at 349.25 116.84 0)
 			(hide yes)
 			(show_name no)
@@
 		)
 		(property "Datasheet" "https://belfuse.com/resources/drawings/magneticsolutions/dr-mag-si-60062-f.pdf"
-			(at 248.92 63.5 0)
+			(at 349.25 114.3 0)
 			(hide yes)
 			(show_name no)
@@
 		)
 		(property "Description" "1 Port RJ45 Magjack Connector Through Hole 10/100 Base-T, AutoMDIX"
-			(at 248.92 78.74 0)
+			(at 349.25 129.54 0)
 			(hide yes)
 			(show_name no)
@@
 	(symbol
 		(lib_id "Connector:RJ45_Bel_SI-60062-F")
-		(at 248.92 105.41 0)
+		(at 349.25 156.21 0)
 		(unit 1)
 		(body_style 1)
@@
 		(fields_autoplaced yes)
 		(property "Reference" "J3"
-			(at 250.19 91.44 0)
+			(at 350.52 142.24 0)
 			(show_name no)
 			(do_not_autoplace no)
@@
 		)
 		(property "Value" "RJ45_Bel_SI-60062-F"
-			(at 250.19 93.98 0)
+			(at 350.52 144.78 0)
 			(show_name no)
 			(do_not_autoplace no)
@@
 		)
 		(property "Footprint" "Connector_RJ:RJ45_Pulse_JK00177NL_Horizontal"
-			(at 248.92 92.71 0)
+			(at 349.25 143.51 0)
 			(hide yes)
 			(show_name no)
@@
 		)
 		(property "Datasheet" "https://belfuse.com/resources/drawings/magneticsolutions/dr-mag-si-60062-f.pdf"
-			(at 248.92 90.17 0)
+			(at 349.25 140.97 0)
 			(hide yes)
 			(show_name no)
@@
 		)
 		(property "Description" "1 Port RJ45 Magjack Connector Through Hole 10/100 Base-T, AutoMDIX"
-			(at 248.92 105.41 0)
-			(hide yes)
-			(show_name no)
+			(at 349.25 156.21 0)
+			(hide yes)
+			(show_name no)

Commit message: ethernet hardware side
Parts:
- removed J1, J2, J3: RJ45_Bel_SI-60062-F, Connector_RJ:RJ45_Pulse_JK00177NL_Horizontal, symbol Connector:RJ45_Bel_SI-60062-F
- removed U4: LAN9370T-I/KCX, QFN_LAN9370T-I/KCX_MCH, symbol allwinner-sip-lib:LAN9370T-I_KCX
- added C30, C31: 18pF, symbol Device:C_Small
- added C34: 10nF, symbol Device:C_Small
- added C35: 4.7uF, symbol Device:C_Small
- added C40, C53, C55, C56: 33nF, symbol Device:C_Small
- added C41, C54, C57, C58: DNP, symbol Device:C_Small
- added C51: 100nF, symbol Device:C_Small
- added C52: 1nF, symbol Device:C_Small
- added D3: LED_ABGR, symbol Device:LED_ABGR
- added D6: LED, symbol Device:LED
- added J1: RJ45, Connector_RJ:RJ45_OST_PJ012-8P8CX_Vertical, symbol Connector:RJ45
- added L1: HH-1M1608-121JT, symbol Device:L_Small
- added R22, R57, R58: DNP, symbol Device:R_Small
- added R59: 12k4 1%, symbol Device:R_Small
- added R60: 10k, symbol Device:R_Small
- added R75, R76, R77, R78: 75R, symbol Device:R_Small
- added R8: 1M, symbol Device:R_Small
- added TP1: VBG, symbol Connector:TestPoint
- added TP2: 1v2, symbol Connector:TestPoint
- added TR5: PT61020EL, Transformer_SMD:Transformer_Ethernet_Bourns_PT61020EL, symbol Transformer:PT61020EL
- added U4: (no value), formula_slug_footprint_library:128-TQFP-ECAP, symbol formula_slug_symbol_library:LAN96455F-I/8MW
- added Y5: 25MHz, symbol Device:Crystal
Connections:
- net INT_RXP: now reaches U9.1 (TXN)
- net INT_RXP: now also U9.6 (RXP), C41.2, C55.2
- net at U9.10 (EXRES1): now also R59.1
- net ETH_AVDD: now reaches U9.11 (AVDD), U9.15 (AVDD), U9.17 (AVDD), U9.21 (AVDD), U9.4 (AVDD), U9.8 (AVDD)
- net ETH_AVDD: now also L1.2
- net GND: now reaches U9.14 (AGND), U9.16 (AGND), U9.19 (AGND), U9.3 (AGND), U9.48 (AGND), U9.9 (AGND)
- net GND: now also U9.29 (GND), C30.2, C31.2, C34.2, C35.2, C51.2, C52.2, R22.2, R57.2, R58.2, R59.2
- net at U9.18 (VBG): now also TP1.1
- net INT_TXP: now reaches U9.2 (TXP)
- net INT_TXP: now also U9.5 (RXN), C40.2, C57.2
- net at U9.20 (TOCAP): now also C35.1
- net at U9.22 (1V2O): now also C34.1, TP2.1
- net at U9.24 (SPDLED): now also D3.4 (RK)
- net at U9.25 (LINKLED): now also D6.1 (K)
- net at U9.26 (DUPLED): now also D3.3 (GK)
- net at U9.27 (ACTLED): now also D3.2 (BK)
- net +3.3V: now reaches U9.28 (VDD)
- net +3.3V: now also D3.1 (A), D6.2 (A), L1.1, R60.1
- net at U9.30 (XI/CLKIN): now also C30.1, R8.1, Y5.1
- net at U9.31 (XO): now also C31.1, R8.2, Y5.2
- net ~{CS}_ETH: now reaches U9.32 (~{SCS})
- net SCLK: now reaches U9.33 (SCLK)
- net MISO: now reaches U9.34 (MISO)
- net MOSI: now reaches U9.35 (MOSI)
- net ~{INT}: now reaches U9.36 (~{INT})
- net ~{INT}: now also R60.2
- net ~{RST}: now reaches U9.37 (~{RST})
- net at U9.43 (PMODE2): now also R22.1
- net at U9.44 (PMODE1): now also R57.1
- net at U9.45 (PMODE0): now also R58.1
- new net: C53.1, C54.1, U4.22 (P4_AN)
- new net: C40.1, C41.1, U4.21 (P4_AP)
- new net: C55.1, C57.1, U4.23 (P4_BP)
- new net: C56.1, C58.1, U4.24 (P4_BN)
- new net: C52.1, R75.2, R76.2, R77.2, R78.2
- new net: R75.1, TR5.15 (MCT4)
- new net: R76.1, TR5.18 (MCT3)
- new net: C51.1, TR5.1 (TCT1), TR5.10 (TCT4), TR5.4 (TCT2), TR5.7 (TCT3)
- new net: TR5.11 (TD4+), U4.19 (P3_DP)
- new net: TR5.12 (TD4-), U4.20 (P3_DN)
- new net: TR5.2 (TD1+), U4.11 (P3_AP)
- new net: R77.1, TR5.21 (MCT2)
- new net: R78.1, TR5.24 (MCT1)
- new net: TR5.3 (TD1-), U4.12 (P3_AN)
- new net: TR5.5 (TD2+), U4.13 (P3_BP)
- new net: TR5.6 (TD2-), U4.14 (P3_BN)
- new net: TR5.8 (TD3+), U4.17 (P3_CP)
- new net: TR5.9 (TD3-), U4.18 (P3_CN)
- new net AUX_TRAN: J1.2, TR5.22 (MX1-)
- new net AUX_TRAP: J1.1, TR5.23 (MX1+)
- new net AUX_TRBN: J1.4, TR5.19 (MX2-)
- new net AUX_TRBP: J1.3, TR5.20 (MX2+)
- new net AUX_TRCN: J1.7, TR5.16 (MX3-)
- new net AUX_TRCP: J1.8, TR5.17 (MX3+)
- new net AUX_TRDN: J1.6, TR5.13 (MX4-)
- new net AUX_TRDP: J1.5, TR5.14 (MX4+)
- new net INT_RXN: C54.2, C56.2
- new net INT_TXN: C53.2, C58.2
- new net M12X_TR/AN: U4.103 (P0_AN)
- new net M12X_TR/AP: U4.102 (P0_AP)
- new net M12X_TR/BN: U4.106 (P0_BN)
- new net M12X_TR/BP: U4.105 (P0_BP)
- new net M12X_TR/CN: U4.109 (P0_CN)
- new net M12X_TR/CP: U4.108 (P0_CP)
- new net M12X_TR/DN: U4.111 (P0_DN)
- new net M12X_TR/DP: U4.110 (P0_DP)
- new net M12X_TR1/AN: U4.113 (P1_AN)
- new net M12X_TR1/AP: U4.112 (P1_AP)
- new net M12X_TR1/BN: U4.115 (P1_BN)
- new net M12X_TR1/BP: U4.114 (P1_BP)
- new net M12X_TR1/CN: U4.118 (P1_CN)
- new net M12X_TR1/CP: U4.117 (P1_CP)
- new net M12X_TR1/DN: U4.121 (P1_DN)
- new net M12X_TR1/DP: U4.120 (P1_DP)
- new net M12X_TR2/AN: U4.2 (P2_AN)
- new net M12X_TR2/AP: U4.1 (P2_AP)
- new net M12X_TR2/BN: U4.5 (P2_BN)
- new net M12X_TR2/BP: U4.4 (P2_BP)
- new net M12X_TR2/CN: U4.8 (P2_CN)
- new net M12X_TR2/CP: U4.7 (P2_CP)
- new net M12X_TR2/DN: U4.10 (P2_DN)
- new net M12X_TR2/DP: U4.9 (P2_DP)
- no-connect marks 0 -> 10
Other:
- added sheet M12X_TR (m12x_tr.kicad_sch)
- added sheet M12X_TR1 (m12x_tr.kicad_sch)
- added sheet M12X_TR2 (m12x_tr.kicad_sch)
- note added: "Debug/PC port, under weather cover"
- note added: "Device Port"
- note added: "Ethernet Switch"
- note added: "PMODE[0-2] Pulled up internally to set auto negotiate mode"
- moved on the sheet: U9

Commit message: update title block
Changed lines of the file:
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@@
 	(hierarchical_label "~{CS}_SW"
 		(shape input)
-		(at 114.9866 178.2994 180)
+		(at 119.38 153.67 180)
 		(effects
 			(font

Commit message: finish ethernet, power supply arch, some other things
Parts:
- added C63, C64: 12pF, symbol Device:C_Small
- added C65: 100nF, symbol Device:C_Small
- added D13, D14, D15, D16: LED, symbol Device:LED
- added R100, R97, R98, R99: R_Small, symbol Device:R_Small
- added R103: 200R, symbol Device:R_Small
- added R104: 6.04k, symbol Device:R_Small
- added R16, R20, R21, R35, R36, R49, R50, R61, R62, R79, R80, R81, R82, R83, R89, R9, R90, R91: 10k, symbol formula_slug_symbol_library:R_small_selectable
- added R84, R85, R86, R87, R88: 10k, symbol Device:R_Small
- added Y6: 25Mhz, symbol Device:Crystal
Connections:
- net +3.3V is gone; now on net VDD: D3.1 (A), D6.2 (A), L1.1, R60.1, U9.28 (VDD)
- net GND: now also U4.PAD (GND), C63.2, C64.2, R103.1, R104.2, R16.3, R20.3, R21.1, R35.1, R36.1, R49.1, R50.1, R61.3, R62.3, R79.3, R80.1, R81.3, R82.1, R83.1, R89.1, R9.1, R90.3, R91.3
- net ETH_1.15: now reaches U4.104 (VDD_AL)
- net ETH_1.15: now also U4.119 (VDD_AL), U4.15 (VDD_AL), U4.28 (VDD_AL), U4.3 (VDD_AL)
- net VDD: now reaches U4.107 (VDD_AH)
- net VDD: now also U4.116 (VDD_AH), U4.128 (VDD_AH), U4.16 (VDD_AH), U4.25 (VDD_AH), U4.32 (VDD_IO_E), U4.39 (VDD_IO_E), U4.44 (VDD_AHS), U4.52 (VDD_AHS), U4.58 (VDD_IO_D), U4.6 (VDD_AH), U4.69 (VDD_IO_C), U4.77 (VDD_IO_C), U4.84 (VDD_IO_B), U4.92 (VDD_IO_B), U4.96 (VDD_IO_A), R100.1, R16.1, R20.1, R21.3, R35.3, R36.3, R49.3, R50.3, R61.1, R62.1, R79.1, R80.3, R81.1, R82.3, R83.3, R84.1, R85.1, R86.1, R87.1, R88.1, R89.3, R9.3, R90.1, R91.1, R97.1, R98.1, R99.1
- net VDDA: now reaches U4.122 (VDD)
- net VDDA: now also U4.126 (VDD_PLL), U4.37 (VDD), U4.47 (VDD_ALS0), U4.54 (VDD_ALS1), U4.59 (VDD), U4.73 (VDD), U4.88 (VDD), C65.1
- net at U4.123 (X_O): now also C63.1, Y6.1
- net at U4.124 (X_I): now also C64.1, Y6.2
- net at U4.125 (RTN_PLL): now also C65.2
- net at U4.127 (I_SET): now also R104.1
- net at U4.51 (RESREF): now also R103.2
- net SW_RST: now reaches U4.101 (~{RST})
- net SW_RST: now also R91.2
- net PHY0_LED1: now reaches U4.31 (GPIO43)
- net PHY0_LED0: now reaches U4.33 (GPIO42)
- net SW_XMII_MODE0: now reaches U4.34 (GPIO41_XMII_MODE0)
- net SW_XMII_MODE0: now also R50.2
- net SW_SD_MODE0: now reaches U4.35 (GPIO40_SD_MODE1)
- net SW_SD_MODE0: now also R88.2
- net SW_SD_MODE1: now reaches U4.36 (GPIO40_SD_MODE0)
- net SW_SD_MODE1: now also R87.2
- net SW_XMII_MODE1: now reaches U4.38 (GPIO38_XMII_MODE1)
- net SW_XMII_MODE1: now also R83.2
- net SW_GPIO_MODE1: now reaches U4.40 (GPIO37_GPIO_MODE1)
- net SW_GPIO_MODE1: now also D14.1 (K), R89.2
- net SW_GPIO_MODE0: now reaches U4.41 (GPIO36_GPIO_MODE0)
- net SW_GPIO_MODE0: now also D13.1 (K), R90.2
- net SW_LOOP_EN: now reaches U4.42 (GPIO35_LOOP_EN)
- net SW_LOOP_EN: now also D16.1 (K), R61.2
- net SW_JTAG_EN: now reaches U4.43 (GPIO34_JTAG_ENB)
- net SW_JTAG_EN: now also D15.1 (K), R36.2
- net SW_EEPROM_SIZE: now reaches U4.60 (GPIO_33_EEPROM_SIZE)
- net SW_EEPROM_SIZE: now also R84.2
- net SW_UART_TX: now reaches U4.62 (GPIO_31)
- net SW_UART_RX: now reaches U4.63 (GPIO_30)
- net SW_MGMT_MODE1: now reaches U4.65 (GPIO_28_MGMT_MODE1)
- net SW_MGMT_MODE1: now also R21.2
- net SW_MGMT_MODE0: now reaches U4.66 (GPIO_27_MGMT_MODE0)
- net SW_MGMT_MODE0: now also R35.2
- net SW_BOOT_MODE2: now reaches U4.67 (GPIO_26_BOOT_MODE2)
- net SW_BOOT_MODE2: now also R9.2
- net SW_BOOT_MODE1: now reaches U4.68 (GPIO_25_BOOT_MODE1)
- net SW_BOOT_MODE1: now also R16.2
- net SW_BOOT_MODE0: now reaches U4.70 (GPIO_24_BOOT_MODE0)
- net SW_BOOT_MODE0: now also R20.2
- net SW_SerDes_125M_CLK_EN: now reaches U4.71 (GPIO_23_SD_125M)
- net SW_SerDes_125M_CLK_EN: now also R49.2
- net SW_SGPIO_EN: now reaches U4.72 (GPIO_22_SGPIO_EN)
- net SW_SGPIO_EN: now also R86.2
- net SW_SFP_NEG: now reaches U4.81 (GPIO_15_SEP_EN)
- net SW_SFP_NEG: now also R85.2
- net SW_GBE_PHY_EN: now reaches U4.82 (GPIO_14_CUPHY_MODE)
- net SW_LED_MODE: now reaches U4.83 (GPIO_13_LED_MODE)
- net SW_LED_MODE: now also R81.2
- net SW_ENGY_EF_EN: now reaches U4.85 (GPIO_12_EEE_EN)
- net SW_ENGY_EF_EN: now also R80.2
- net SW_FLW_CTRL_EN: now reaches U4.86 (GPIO_11_ELOW_EN)
- net SW_FLW_CTRL_EN: now also R79.2
- net SW_GBE_PHY_~{EN}: now reaches U4.87 (GPIO_10_E2E_CLOCK_EN)
- net SW_GBE_PHY_~{EN}: now also R82.2
- new net: D15.2 (A), R99.2
- new net: D13.2 (A), R97.2
- new net: D14.2 (A), R98.2
- new net: D16.2 (A), R100.2
- new net SW_E2E_CLK_EN: R62.2
- no-connect marks 10 -> 37
Other:
- sheet M12X_TR ports: added LED0, LED1, VDD_LED; removed none
- sheet M12X_TR1 ports: added LED0, LED1, VDD_LED; removed none
- sheet M12X_TR2 ports: added LED0, LED1, VDD_LED; removed none
- note added: "Allow GBE in auto-negotiation"
- note added: "Boot Mode 3 (ROM Boot)"
- note added: "Disable Energy Effecient Eth Mode"
- note added: "Disable JTAG"
- note added: "Enable End To End Clock"
- note added: "Enable Flow Control"
- note added: "Enable Loop Detection"
- note added: "Enable More Verbose "Tri-Color" Mode"
- note added: "Irrelevant/Unused"
- note added: "Management Mode 0 (UART CLI)"
- note added: "PHY1_LED0"
- note added: "PHY1_LED1"
- note added: "PHY2_LED1"
- note added: "PHY2_LED2"
- note added: "PHY3_LED1"
- note added: "PHY3_LED2"
- note added: "PHY4_LED1"
- note added: "PHY4_LED2"
- note added: "Set GPIO Mode B"
- note added: "Use CuPHY4, RMII in GPIO MODE B"
- note added: "We aint Using SerDes, No ref CLK input"
- moved on the sheet: C30, C31, C34, C35, C40, C41, C51, C52, C53, C54, C55, C56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

Commit message: use every pin
Other:
- moved on the sheet: R36, R89, R90
