File: telemetry-logging-board/eth.kicad_sch (KiCad schematic)
At the start: 71 parts, among them J1 RJ45, U9 W5500, Y5 25MHz, Y6 25Mhz

Commit message: idek
Parts:
- removed D3: LED_ABGR, symbol Device:LED_ABGR
- removed Y5: 25MHz, symbol Device:Crystal
- removed Y6: 25Mhz, symbol Device:Crystal
- added D18, D19, D20: LED, Diode_SMD:D_0603_1608Metric, symbol Device:LED
- added R90, R91, R92: R_Small, Resistor_SMD:R_0603_1608Metric, symbol Device:R_Small
- added Y1, Y2: 25MHz, Crystal:Crystal_SMD_3225-4Pin_3.2x2.5mm, symbol Device:Crystal_GND24
- C19: renamed from C63; footprint (none) -> Capacitor_SMD:C_0603_1608Metric
- C20: renamed from C64; footprint (none) -> Capacitor_SMD:C_0603_1608Metric
- C21: renamed from C30; footprint (none) -> Capacitor_SMD:C_0603_1608Metric
- C22: renamed from C65; footprint (none) -> Capacitor_SMD:C_0603_1608Metric
- C23: renamed from C31; footprint (none) -> Capacitor_SMD:C_0603_1608Metric
- C24: renamed from C34; footprint (none) -> Capacitor_SMD:C_0603_1608Metric
- C25: renamed from C35; footprint (none) -> Capacitor_SMD:C_0603_1608Metric
- C26: renamed from C40; footprint (none) -> Capacitor_SMD:C_0603_1608Metric
- C27: renamed from C53; footprint (none) -> Capacitor_SMD:C_0603_1608Metric
- C28: renamed from C55; footprint (none) -> Capacitor_SMD:C_0603_1608Metric
- C29: renamed from C56; footprint (none) -> Capacitor_SMD:C_0603_1608Metric
- C30: renamed from C41; footprint (none) -> Capacitor_SMD:C_0603_1608Metric
- C31: renamed from C54; footprint (none) -> Capacitor_SMD:C_0603_1608Metric
- C32: renamed from C57; footprint (none) -> Capacitor_SMD:C_0603_1608Metric
- C33: renamed from C58; footprint (none) -> Capacitor_SMD:C_0603_1608Metric
- C34: renamed from C51; footprint (none) -> Capacitor_SMD:C_0603_1608Metric
- C35: renamed from C52; footprint (none) -> Capacitor_SMD:C_0603_1608Metric
- D3: renamed from D6; footprint (none) -> Diode_SMD:D_0603_1608Metric
- D5: renamed from D15; footprint (none) -> Diode_SMD:D_0603_1608Metric
- D6: renamed from D16; footprint (none) -> Diode_SMD:D_0603_1608Metric
- D7: renamed from D13; footprint (none) -> Diode_SMD:D_0603_1608Metric
- D8: renamed from D14; footprint (none) -> Diode_SMD:D_0603_1608Metric
- L4: renamed from L1; footprint (none) -> Inductor_SMD:L_0603_1608Metric
- R15: renamed from R9; footprint (none) -> formula_slug_footprint_library:R_0603_Selectable
- R16: footprint (none) -> formula_slug_footprint_library:R_0603_Selectable
- R17: renamed from R20; footprint (none) -> formula_slug_footprint_library:R_0603_Selectable
- R18: renamed from R104; footprint (none) -> Resistor_SMD:R_0603_1608Metric
- R19: renamed from R22; footprint (none) -> Resistor_SMD:R_0603_1608Metric
- R20: renamed from R57; footprint (none) -> Resistor_SMD:R_0603_1608Metric
- R21: renamed from R58; footprint (none) -> Resistor_SMD:R_0603_1608Metric
- R22: renamed from R21; footprint (none) -> formula_slug_footprint_library:R_0603_Selectable
- R23: renamed from R35; footprint (none) -> formula_slug_footprint_library:R_0603_Selectable
- R24: renamed from R60; footprint (none) -> Resistor_SMD:R_0603_1608Metric
- R25: renamed from R103; footprint (none) -> Resistor_SMD:R_0603_1608Metric
- R26: renamed from R8; footprint (none) -> Resistor_SMD:R_0603_1608Metric
- R27: renamed from R49; footprint (none) -> formula_slug_footprint_library:R_0603_Selectable
- R28: renamed from R36; footprint (none) -> formula_slug_footprint_library:R_0603_Selectable
- R29: renamed from R89; footprint (none) -> formula_slug_footprint_library:R_0603_Selectable
- R30: renamed from R90; footprint (none) -> formula_slug_footprint_library:R_0603_Selectable
- R31: renamed from R59; footprint (none) -> Resistor_SMD:R_0603_1608Metric
- R32: renamed from R88; footprint (none) -> Resistor_SMD:R_0603_1608Metric
- R33: renamed from R87; footprint (none) -> Resistor_SMD:R_0603_1608Metric
- R34: renamed from R86; footprint (none) -> Resistor_SMD:R_0603_1608Metric
- R35: renamed from R84; footprint (none) -> Resistor_SMD:R_0603_1608Metric
- R36: renamed from R85; footprint (none) -> Resistor_SMD:R_0603_1608Metric
- R37: renamed from R82; footprint (none) -> formula_slug_footprint_library:R_0603_Selectable
- R38: renamed from R81; footprint (none) -> formula_slug_footprint_library:R_0603_Selectable
- R39: renamed from R80; footprint (none) -> formula_slug_footprint_library:R_0603_Selectable
- R40: renamed from R79; footprint (none) -> formula_slug_footprint_library:R_0603_Selectable
- R41: renamed from R62; footprint (none) -> formula_slug_footprint_library:R_0603_Selectable
- R42: renamed from R61; footprint (none) -> formula_slug_footprint_library:R_0603_Selectable
- R43: renamed from R50; footprint (none) -> formula_slug_footprint_library:R_0603_Selectable
- R44: renamed from R83; footprint (none) -> formula_slug_footprint_library:R_0603_Selectable
- R45: renamed from R99; footprint (none) -> Resistor_SMD:R_0603_1608Metric
- R46: renamed from R100; footprint (none) -> Resistor_SMD:R_0603_1608Metric
- R47: renamed from R91; footprint (none) -> formula_slug_footprint_library:R_0603_Selectable
- R48: renamed from R97; footprint (none) -> Resistor_SMD:R_0603_1608Metric
- R49: renamed from R75; footprint (none) -> Resistor_SMD:R_0603_1608Metric
- R50: renamed from R98; footprint (none) -> Resistor_SMD:R_0603_1608Metric
- R51: renamed from R76; footprint (none) -> Resistor_SMD:R_0603_1608Metric
- R52: renamed from R77; footprint (none) -> Resistor_SMD:R_0603_1608Metric
- R53: renamed from R78; footprint (none) -> Resistor_SMD:R_0603_1608Metric
- TP6: renamed from TP1; footprint (none) -> TestPoint:TestPoint_Pad_2.0x2.0mm
- TP7: renamed from TP2; footprint (none) -> TestPoint:TestPoint_Pad_2.0x2.0mm
- renumbered J1 to J10, TR5 to TR1, U4 to U10, U9 to U11
Connections:
- net GND: now also Y1.2 (G), Y1.4 (G), Y2.2 (G), Y2.4 (G)
- net VDD: now also D18.2 (A), D19.2 (A), D20.2 (A)
- net at C23.1, R26.2, U11.31 (XO): now also Y2.3
- net at C21.1, R26.1, U11.30 (XI/CLKIN): now also Y2.1
- net at U11.24 (SPDLED): now also R90.2
- net at U11.26 (DUPLED): now also R91.2
- net at U11.27 (ACTLED): now also R92.2
- net at C19.1, U10.123 (X_O): now also Y1.1
- net at C20.1, U10.124 (X_I): now also Y1.3
- new net: D18.1 (K), R90.1
- new net: D20.1 (K), R92.1
- new net: D19.1 (K), R91.1
Other:
- moved on the sheet: C21, C23
