File: telemetry-logging-board/rf_mod.kicad_sch (KiCad schematic)
At the start: 3 parts, among them J17 HF, J18 LF, U5 Value

Commit message: idek
Parts:
- renumbered J18 to J5, J17 to J6, U5 to U9
Changed lines of the file:
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@@
 		(dnp no)
 		(fields_autoplaced yes)
-		(property "Reference" "U5"
+		(property "Reference" "U9"
 			(at 139.7 76.2 0)
 			(show_name no)
@@
 			(project "telemetry-logging-board"
 				(path "/77f08122-c609-410b-9d24-33eebdb4af2b/98a8033c-6556-440f-bb5e-fa89586975aa"
-					(reference "U5")
+					(reference "U9")
 					(unit 1)
 				)
@@
 		(dnp no)
 		(fields_autoplaced yes)
-		(property "Reference" "#PWR03"
+		(property "Reference" "#PWR041"
 			(at 139.7 121.92 0)
 			(hide yes)
@@
 			(project "telemetry-logging-board"
 				(path "/77f08122-c609-410b-9d24-33eebdb4af2b/98a8033c-6556-440f-bb5e-fa89586975aa"
-					(reference "#PWR03")
+					(reference "#PWR041")
 					(unit 1)
 				)
@@
 		(dnp no)
 		(fields_autoplaced yes)
-		(property "Reference" "J17"
+		(property "Reference" "J6"
 			(at 162.56 105.7031 0)
 			(show_name no)
@@
 			(project "telemetry-logging-board"
 				(path "/77f08122-c609-410b-9d24-33eebdb4af2b/98a8033c-6556-440f-bb5e-fa89586975aa"
-					(reference "J17")
+					(reference "J6")
 					(unit 1)
 				)
@@
 		(in_pos_files yes)
 		(dnp no)
-		(property "Reference" "J18"
+		(property "Reference" "J5"
 			(at 116.84 105.7031 0)
 			(show_name no)
@@
 			(project "telemetry-logging-board"
 				(path "/77f08122-c609-410b-9d24-33eebdb4af2b/98a8033c-6556-440f-bb5e-fa89586975aa"
-					(reference "J18")
+					(reference "J5")
 					(unit 1)
 				)
@@
 		(dnp no)
 		(fields_autoplaced yes)
-		(property "Reference" "#PWR04"
+		(property "Reference" "#PWR040"
 			(at 125.73 86.36 0)
 			(hide yes)
@@
 			(project "telemetry-logging-board"
 				(path "/77f08122-c609-410b-9d24-33eebdb4af2b/98a8033c-6556-440f-bb5e-fa89586975aa"
-					(reference "#PWR04")
+					(reference "#PWR040")
 					(unit 1)
 				)
