File: telemetry-logging-board/m12x_tr.kicad_sch (KiCad schematic)
At the start: 12 parts, among them J14 M12-X

Commit message: idek
Parts:
- C48: renamed from C43; footprint (none) -> Capacitor_SMD:C_0603_1608Metric
- C49: renamed from C44; footprint (none) -> Capacitor_SMD:C_0603_1608Metric
- D12: renamed from D7; footprint (none) -> Diode_SMD:D_0603_1608Metric
- D13: renamed from D10; footprint (none) -> Diode_SMD:D_0603_1608Metric
- J11: renamed from J14; footprint (none) -> Jumper:SolderJumper-2_P1.3mm_Open_RoundedPad1.0x1.5mm
- R72: renamed from R93; footprint (none) -> Resistor_SMD:R_0603_1608Metric
- R73: renamed from R94; footprint (none) -> Resistor_SMD:R_0603_1608Metric
- R74: renamed from R63; footprint (none) -> Resistor_SMD:R_0603_1608Metric
- R75: renamed from R64; footprint (none) -> Resistor_SMD:R_0603_1608Metric
- R76: renamed from R65; footprint (none) -> Resistor_SMD:R_0603_1608Metric
- R77: renamed from R66; footprint (none) -> Resistor_SMD:R_0603_1608Metric

Commit message: remove incorrect footprint assignments
Parts:
- J11: footprint Jumper:SolderJumper-2_P1.3mm_Open_RoundedPad1.0x1.5mm -> (none)
Changed lines of the file:
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@@
 			)
 		)
-		(property "Footprint" "Jumper:SolderJumper-2_P1.3mm_Open_RoundedPad1.0x1.5mm"
+		(property "Footprint" ""
 			(at 194.31 91.44 0)
 			(hide yes)
