File: telemetry-logging-board/can.kicad_sch (KiCad schematic)
At the start: 3 parts, among them J10 CAN_B, J11 CAN_C, J9 CAN_A

Commit message: replace LR2021 with seeed wio LR2021, rework psu
Parts:
- added JP1, JP19, JP2, JP20: CAN_INTER_ISO, symbol Jumper:SolderJumper_2_Open
Connections:
- net CAN-IF/ISO_0V: now also JP19.2 (B)
- net CAN-IF/ISO_5V: now also JP1.2 (B)
- net CAN-IF1/ISO_0V: now also JP19.1 (A), JP20.2 (B)
- net CAN-IF1/ISO_5V: now also JP1.1 (A), JP2.2 (B)
- net CAN-IF2/ISO_0V: now also JP20.1 (A)
- net CAN-IF2/ISO_5V: now also JP2.1 (A)

Commit message: idek
Parts:
- added J14: M8-6P, symbol Connector_Generic:Conn_01x06
- JP5: renamed from JP1; footprint (none) -> Jumper:SolderJumper-2_P1.3mm_Open_RoundedPad1.0x1.5mm
- JP6: renamed from JP2; footprint (none) -> Jumper:SolderJumper-2_P1.3mm_Open_RoundedPad1.0x1.5mm
- JP7: renamed from JP19; footprint (none) -> Jumper:SolderJumper-2_P1.3mm_Open_RoundedPad1.0x1.5mm
- JP8: renamed from JP20; footprint (none) -> Jumper:SolderJumper-2_P1.3mm_Open_RoundedPad1.0x1.5mm
- renumbered J9 to J7, J10 to J8, J11 to J9
Other:
- note added: "Male, Right Angle"
- note added: "https://www.aliexpress.us/item/3256806106157547.html"
Changed lines of the file:
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@@
+		)
+	)
+	(text "Male, Right Angle"
+		(exclude_from_sim no)
+		(at 243.586 66.802 0)
+		(effects
+			(font
+				(size 1.27 1.27)
+			)
+		)
+	)
+	(text "https://www.aliexpress.us/item/3256806106157547.html"
+		(exclude_from_sim no)
+		(at 244.602 62.738 0)
+		(effects
+			(font
+				(size 1.27 1.27)
+			)
 		)
 	)
@@
 		(dnp no)
 		(fields_autoplaced yes)
-		(property "Reference" "#PWR061"
+		(property "Reference" "#PWR044"
 			(at 97.79 125.73 0)
 			(hide yes)
@@
 			(project "telemetry-logging-board"
 				(path "/77f08122-c609-410b-9d24-33eebdb4af2b/7f3d1692-3ca8-4973-8724-6cc30343bbd5"
-					(reference "#PWR061")
+					(reference "#PWR044")
 					(unit 1)
 				)
@@
 		(dnp no)
 		(fields_autoplaced yes)
-		(property "Reference" "#PWR0134"
+		(property "Reference" "#PWR047"
 			(at 104.14 123.19 0)
 			(hide yes)
@@
 			(project "telemetry-logging-board"
 				(path "/77f08122-c609-410b-9d24-33eebdb4af2b/7f3d1692-3ca8-4973-8724-6cc30343bbd5"
-					(reference "#PWR0134")
+					(reference "#PWR047")
 					(unit 1)
 				)
@@
 		(dnp no)
 		(fields_autoplaced yes)
-		(property "Reference" "JP19"
+		(property "Reference" "JP7"
 			(at 203.2 93.9799 90)
 			(show_name no)
@@
 			)
 		)
-		(property "Footprint" ""
+		(property "Footprint" "Jumper:SolderJumper-2_P1.3mm_Open_RoundedPad1.0x1.5mm"
 			(at 200.66 95.25 0)
 			(hide yes)
@@
 			(project "telemetry-logging-board"
 				(path "/77f08122-c609-410b-9d24-33eebdb4af2b/7f3d1692-3ca8-4973-8724-6cc30343bbd5"
-					(reference "JP19")
+					(reference "JP7")
 					(unit 1)
 				)
@@
 		(dnp no)
 		(fields_autoplaced yes)
-		(property "Reference" "J10"
+		(property "Reference" "J8"
 			(at 167.64 91.4399 0)
 			(show_name no)
@@
 			(project "telemetry-logging-board"
 				(path "/77f08122-c609-410b-9d24-33eebdb4af2b/7f3d1692-3ca8-4973-8724-6cc30343bbd5"
-					(reference "J10")
+					(reference "J8")
 					(unit 1)
 				)
@@
 		(dnp no)
 		(fields_autoplaced yes)
-		(property "Reference" "#PWR059"
+		(property "Reference" "#PWR042"
 			(at 97.79 46.99 0)
 			(hide yes)
@@
 			(project "telemetry-logging-board"
 				(path "/77f08122-c609-410b-9d24-33eebdb4af2b/7f3d1692-3ca8-4973-8724-6cc30343bbd5"
-					(reference "#PWR059")
+					(reference "#PWR042")
 					(unit 1)
 				)
@@
 		(dnp no)
 		(fields_autoplaced yes)
-		(property "Reference" "JP1"
+		(property "Reference" "JP5"
 			(at 184.15 72.3899 90)
 			(show_name no)
@@
 			)
 		)
-		(property "Footprint" ""
+		(property "Footprint" "Jumper:SolderJumper-2_P1.3mm_Open_RoundedPad1.0x1.5mm"
 			(at 181.61 73.66 0)
 			(hide yes)
@@
 			(project "telemetry-logging-board"
 				(path "/77f08122-c609-410b-9d24-33eebdb4af2b/7f3d1692-3ca8-4973-8724-6cc30343bbd5"
-					(reference "JP1")
+					(reference "JP5")
 					(unit 1)
 				)
@@
 		(dnp no)
 		(fields_autoplaced yes)
-		(property "Reference" "JP20"
+		(property "Reference" "JP8"
 			(at 203.2 133.3499 90)
 			(show_name no)
@@
 			)
 		)
-		(property "Footprint" ""
+		(property "Footprint" "Jumper:SolderJumper-2_P1.3mm_Open_RoundedPad1.0x1.5mm"
 			(at 200.66 134.62 0)
 			(hide yes)
@@
 			(project "telemetry-logging-board"
 				(path "/77f08122-c609-410b-9d24-33eebdb4af2b/7f3d1692-3ca8-4973-8724-6cc30343bbd5"
-					(reference "JP20")
+					(reference "JP8")
 					(unit 1)
 				)
@@
 		(dnp no)
 		(fields_autoplaced yes)
-		(property "Reference" "#PWR063"
+		(property "Reference" "#PWR045"
 			(at 104.14 44.45 0)
 			(hide yes)
@@
 			(project "telemetry-logging-board"
 				(path "/77f08122-c609-410b-9d24-33eebdb4af2b/7f3d1692-3ca8-4973-8724-6cc30343bbd5"
-					(reference "#PWR063")
+					(reference "#PWR045")
 					(unit 1)
 				)
@@
 		(dnp no)
 		(fields_autoplaced yes)
-		(property "Reference" "#PWR062"
+		(property "Reference" "#PWR046"
 			(at 104.14 83.82 0)
 			(hide yes)
@@
 			(project "telemetry-logging-board"
 				(path "/77f08122-c609-410b-9d24-33eebdb4af2b/7f3d1692-3ca8-4973-8724-6cc30343bbd5"
-					(reference "#PWR062")
+					(reference "#PWR046")
 					(unit 1)
 				)
@@
 		(dnp no)
 		(fields_autoplaced yes)
-		(property "Reference" "J9"
+		(property "Reference" "J7"
 			(at 167.64 52.0699 0)
 			(show_name no)
@@
 			(project "telemetry-logging-board"
 				(path "/77f08122-c609-410b-9d24-33eebdb4af2b/7f3d1692-3ca8-4973-8724-6cc30343bbd5"
-					(reference "J9")
+					(reference "J7")
+					(unit 1)
+				)
+			)
+		)
+	)
+	(symbol
+		(lib_id "Connector_Generic:Conn_01x06")
+		(at 245.11 78.74 0)
+		(unit 1)
+		(body_style 1)
+		(exclude_from_sim no)
+		(in_bom yes)
+		(on_board yes)
+		(in_pos_files yes)
+		(dnp no)
+		(fields_autoplaced yes)
+		(property "Reference" "J14"
+			(at 247.65 78.7399 0)
+			(show_name no)
+			(do_not_autoplace no)
+			(effects
+				(font
+					(size 1.27 1.27)
+				)
+				(justify left)
+			)
+		)
+		(property "Value" "M8-6P"
+			(at 247.65 81.2799 0)
+			(show_name no)
+			(do_not_autoplace no)
+			(effects
+				(font
+					(size 1.27 1.27)
+				)
+				(justify left)
+			)
+		)
+		(property "Footprint" ""
+			(at 245.11 78.74 0)
+			(hide yes)
+			(show_name no)
+			(do_not_autoplace no)
+			(effects
+				(font
+					(size 1.27 1.27)
+				)
+			)
+		)
+		(property "Datasheet" ""
+			(at 245.11 78.74 0)
+			(hide yes)
+			(show_name no)
+			(do_not_autoplace no)
+			(effects
+				(font
+					(size 1.27 1.27)
+				)
+			)
+		)
+		(property "Description" "Generic connector, single row, 01x06, script generated (kicad-library-utils/schlib/autogen/connector/)"
+			(at 245.11 78.74 0)
+			(hide yes)
+			(show_name no)
+			(do_not_autoplace no)
+			(effects
+				(font
+					(size 1.27 1.27)
+				)
+			)
+		)
+		(pin "5"
+		)
+		(pin "2"
+		)
+		(pin "6"
+		)
+		(pin "1"
+		)
+		(pin "3"
+		)
+		(pin "4"
+		)
+		(instances
+			(project "telemetry-logging-board"
+				(path "/77f08122-c609-410b-9d24-33eebdb4af2b/7f3d1692-3ca8-4973-8724-6cc30343bbd5"
+					(reference "J14")
 					(unit 1)
 				)
@@
 		(dnp no)
 		(fields_autoplaced yes)
-		(property "Reference" "J11"
+		(property "Reference" "J9"
 			(at 167.64 130.8099 0)
 			(show_name no)
@@
 			(project "telemetry-logging-board"
 				(path "/77f08122-c609-410b-9d24-33eebdb4af2b/7f3d1692-3ca8-4973-8724-6cc30343bbd5"
-					(reference "J11")
+					(reference "J9")
 					(unit 1)
 				)
@@
 		(dnp no)
 		(fields_autoplaced yes)
-		(property "Reference" "JP2"
+		(property "Reference" "JP6"
 			(at 184.15 111.7599 90)
 			(show_name no)
@@
 			)
 		)
-		(property "Footprint" ""
+		(property "Footprint" "Jumper:SolderJumper-2_P1.3mm_Open_RoundedPad1.0x1.5mm"
 			(at 181.61 113.03 0)
 			(hide yes)
@@
 			(project "telemetry-logging-board"
 				(path "/77f08122-c609-410b-9d24-33eebdb4af2b/7f3d1692-3ca8-4973-8724-6cc30343bbd5"
-					(reference "JP2")
+					(reference "JP6")
 					(unit 1)
 				)
@@
 		(dnp no)
 		(fields_autoplaced yes)
-		(property "Reference" "#PWR060"
+		(property "Reference" "#PWR043"
 			(at 97.79 86.36 0)
 			(hide yes)
@@
 			(project "telemetry-logging-board"
 				(path "/77f08122-c609-410b-9d24-33eebdb4af2b/7f3d1692-3ca8-4973-8724-6cc30343bbd5"
-					(reference "#PWR060")
+					(reference "#PWR043")
 					(unit 1)
 				)

Commit message: add can connector
Parts:
- removed J14: M8-6P, symbol Connector_Generic:Conn_01x06
- added J14: M12, symbol Connector:Conn_01x08_Pin
- added JP27, JP28, JP29, JP30, JP31, JP32: CAN_A_HV_ISO, symbol Jumper:SolderJumper_2_Bridged
Connections:
- net CAN-IF/CAN_H: now also JP28.1 (A)
- net CAN-IF/CAN_L: now also JP27.1 (A)
- net CAN-IF1/CAN_H: now also JP30.1 (A)
- net CAN-IF1/CAN_L: now also JP29.1 (A)
- net CAN-IF2/CAN_H: now also JP32.1 (A)
- net CAN-IF2/CAN_L: now also JP31.1 (A)
- new net: J14.3 (Pin_3), JP27.2 (B)
- new net: J14.7 (Pin_7), JP31.2 (B)
- new net: J14.4 (Pin_4), JP28.2 (B)
- new net: J14.5 (Pin_5), JP29.2 (B)
- new net: J14.6 (Pin_6), JP30.2 (B)
- new net: J14.8 (Pin_8), JP32.2 (B)
- new net +12V: J14.1 (Pin_1)
- new net GND: J14.2 (Pin_2)
Other:
- note removed: "Male, Right Angle"
- note removed: "https://www.aliexpress.us/item/3256806106157547.html"
- moved on the sheet: JP7, JP8
