File: telemetry-logging-board/psu.kicad_sch (KiCad schematic)
At the start: 30 parts, among them U10 AP61300Z6, U8 AP61300Z6, U9 AP61300Z6

Commit message: mostly CAN work
Parts:
- removed C30, C31, C34, C35: 22uF, symbol Device:C_Polarized
- removed C40, C43: 1uF, symbol Device:C_Small
- removed C41, C44: 100nF, symbol Device:C_Small
- removed L1, L3: 1uH, symbol Device:L
- removed R4, R8: 200k, symbol Device:R_Small
- removed R5: 100k, symbol Device:R_Small
- removed R9: 400k, symbol Device:R_Small
- removed TP2: 0v9, symbol Connector:TestPoint
- removed TP3: 1v8, symbol Connector:TestPoint
- removed U10, U9: AP61300Z6, Package_TO_SOT_SMD:SOT-563, symbol Regulator_Switching:AP61300Z6
Other:
- note added: "3.3v Regulator"
- note removed: "SIP Power Supplies"
- company: (none) -> Formula Slug
- title: (none) -> Telemetry Logging Board
- moved on the sheet: C27, C28, C29, C32, C33, C37, C38, L2, R6, R7, TP4, U8

Commit message: finish ethernet, power supply arch, some other things
Parts:
- added C59, C60: 22uF, symbol Device:C_Polarized
- added C61: 1uF, symbol Device:C_Small
- added C62: 100nF, symbol Device:C_Small
- added L3: 1uH, symbol Device:L
- added R101: 200k, symbol Device:R_Small
- added R102: 220k, symbol Device:R_Small
- added U10, U16, U17: TPS22919DCK, Package_TO_SOT_SMD:SOT-363_SC-70-6, symbol Power_Management:TPS22919DCK
- added U18: AP61300Z6, Package_TO_SOT_SMD:SOT-563, symbol Regulator_Switching:AP61300Z6
Connections:
- net +3V3: now also U16.1 (IN), U17.1 (IN)
- net +5V: now also U10.1 (IN)
- net GND: now also C32.2, C33.2, C37.1, C38.1, R7.1, U8.2 (GND), C59.2, C60.2, C61.1, C62.1, R102.1, U10.2 (GND), U16.2 (GND), U17.2 (GND), U18.2 (GND)
- new net: R101.1, R102.2, U18.1 (FB)
- new net: L3.1, U18.4 (SW)
- new net +3.3V: U16.5 (QOD), U16.6 (OUT)
- new net VCC: U10.5 (QOD), U10.6 (OUT)
- new net VDD: C59.1, U17.5 (QOD), U17.6 (OUT), U18.3 (VIN), U18.5 (EN)
- new net VDDA: C60.1, C61.2, C62.2, L3.2, R101.2, U18.6 (OUT)
Other:
- note added: "+3.3V"
- note added: "+3V3"
- note added: "+5V"
- note added: "+BATT"
- note added: "+BATT : Battery positive terminal, after protections +5V : Boosted Battery output supply, always on when battery is alive +3V3 : Battery backed supply, always on when battery is alive VDD : Ethernet Subsystem Switched Power Supply derrived from +3V3 +3.3V : Switched peripheral power supply for radio, CAN. derrived from +3V3 VCC : CAN TRX Supply, switched from +5V VDDA : Switched ethernet subsyste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"
- note added: "1.15V REG"
- note added: "3.3 V REG"
- note added: "5V boost"
- note added: "CAN TRX BUS Side"
- note added: "CAN TRX MCU Side"
- note added: "ETH"
- note added: "Ethernet Switch 1.15v"
- note added: "MCU"
- note added: "MCU SW"
- note added: "Protections"
- note added: "Radio"
- note added: "VCC"
- note added: "VDD"
- note added: "VDDA"
- note removed: "3.3v Regulator"
- moved on the sheet: C27, C28, C29, C32, C33, C37, C38, L2, R6, R7, TP4, U8

Commit message: use every pin
Connections:
- net ETH_EN: now reaches U17.3 (ON)
- net CAN_A_EN: now reaches U10.3 (ON)
- net PERIPH_EN: now reaches U16.3 (ON)
Other:
- moved on the sheet: U10, U16, U17

Commit message: replace LR2021 with seeed wio LR2021, rework psu
Parts:
- removed U10: TPS22919DCK, Package_TO_SOT_SMD:SOT-363_SC-70-6, symbol Power_Management:TPS22919DCK
- added BT1: LiPo, symbol Device:Battery_Cell
- added C66, C68: 4.7uF, symbol Device:C_Polarized
- added C67, C69: 100nF, symbol Device:C_Small
- added C70: 10uF, symbol Device:C_Small
- added D17: LED, symbol Device:LED
- added L17: 2.2uH, symbol Device:L_Small
- added R105: 10k, symbol Device:R_Small
- added R106, R107: 500k, symbol Device:R_Small
- added R110: 100R, symbol Device:R_Small
- added U19: BQ24072RGT, Package_DFN_QFN:VQFN-16-1EP_3x3mm_P0.5mm_EP1.6x1.6mm, symbol Battery_Management:BQ24072RGT
- added U20: TPS63002, Package_SON:Texas_DRC0010J_ThermalVias, symbol Regulator_Switching:TPS63002
Connections:
- net +3V3: now also D17.2 (A), R105.1
- net BAT_SENS: now also C67.2, R106.2, R107.1
- net CHRG: now also R105.2, U19.9 (~{CHG})
- net GND: now also BT1.2 (-), C66.2, C67.1, C68.2, C69.1, C70.1, R107.2, U19.14 (TMR), U19.17 (VSS), U19.4 (~{CE}), U19.6 (EN1), U19.8 (VSS), U20.11 (PGND), U20.3 (PGND), U20.9 (GND)
- new net: C68.1, C70.2, R110.1, U19.10 (OUT), U19.11 (OUT), U19.5 (EN2), U20.5 (VIN)
- new net: C69.2, R110.2, U20.6 (EN), U20.7 (PS/SYNC), U20.8 (VINA)
- new net: L17.2, U20.2 (L2)
- new net: L17.1, U20.4 (L1)
- new net: BT1.1 (+), C66.1, R106.1, U19.2 (BAT), U19.3 (BAT)
- new net: D17.1 (K), U19.7 (~{PGOOD})
Other:
- note added: "+BATT : Battery positive terminal, after protections +3V3 : Battery backed supply, always on when battery is alive VDD : Ethernet Subsystem Switched Power Supply derrived from +3V3 +3.3V : Switched peripheral power supply for radio, CAN. derrived from +3V3 VDDA : Switched ethernet subsystem supply, derrived from +3V3"
- note added: "3 Years to Disch"
- note added: "3.3V boost"
- note added: "CAN TRX"
- note removed: "+5V"
- note removed: "+BATT : Battery positive terminal, after protections +5V : Boosted Battery output supply, always on when battery is alive +3V3 : Battery backed supply, always on when battery is alive VDD : Ethernet Subsystem Switched Power Supply derrived from +3V3 +3.3V : Switched peripheral power supply for radio, CAN. derrived from +3V3 VCC : CAN TRX Supply, switched from +5V VDDA : Switched ethernet subsyste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"
- note removed: "3.3 V REG"
- note removed: "5V boost"
- note removed: "CAN TRX BUS Side"
- note removed: "CAN TRX MCU Side"
- note removed: "VCC"
- moved on the sheet: C59, C60, C61, C62, L3, R101, R102, U16, U17, U18

Commit message: idek
Parts:
- removed C27: 10uF, symbol Device:C_Small
- removed C28, C37: 1uF, symbol Device:C_Small
- removed C29, C38: 100nF, symbol Device:C_Small
- removed C32, C33: 22uF, symbol Device:C_Polarized
- removed L2: 1uH, symbol Device:L
- removed R6: 200k, symbol Device:R_Small
- removed R7: 44.2k, symbol Device:R_Small
- removed TP4: 3v3, symbol Connector:TestPoint
- removed U20: TPS63002, Package_SON:Texas_DRC0010J_ThermalVias, symbol Regulator_Switching:TPS63002
- removed U8: AP61300Z6, Package_TO_SOT_SMD:SOT-563, symbol Regulator_Switching:AP61300Z6
- added C18, C6: 1uF, Capacitor_SMD:C_0603_1608Metric, symbol Device:C_Small
- added D1: D_Small, Diode_SMD:D_0603_1608Metric, symbol Device:D_Small
- added R10: 1.13k, Resistor_SMD:R_0603_1608Metric, symbol Device:R_Small
- added R9: 1.18k, Resistor_SMD:R_0603_1608Metric, symbol Device:R_Small
- added TP5: 3v3, TestPoint:TestPoint_Pad_2.0x2.0mm, symbol Connector:TestPoint
- added U4: TPS63001, Package_SON:Texas_DRC0010J_ThermalVias, symbol Regulator_Switching:TPS63001
- BT1: footprint (none) -> Connector_JST:JST_PH_B2B-PH-K_1x02_P2.00mm_Vertical
- C11: renamed from C61; footprint (none) -> Capacitor_SMD:C_0603_1608Metric
- C12: renamed from C62; footprint (none) -> Capacitor_SMD:C_0603_1608Metric
- C13: renamed from C68; footprint (none) -> Capacitor_SMD:C_0603_1608Metric
- C14: renamed from C66; footprint (none) -> Capacitor_SMD:C_0603_1608Metric
- C15: renamed from C70; footprint (none) -> Capacitor_SMD:C_0603_1608Metric
- C16: renamed from C67; footprint (none) -> Capacitor_SMD:C_0603_1608Metric
- C17: renamed from C69; footprint (none) -> Capacitor_SMD:C_0603_1608Metric
- C5: renamed from C59; footprint (none) -> Capacitor_SMD:C_0603_1608Metric
- C9: renamed from C60; footprint (none) -> Capacitor_SMD:C_0603_1608Metric
- D2: renamed from D17; footprint (none) -> Diode_SMD:D_0603_1608Metric
- L2: renamed from L3; footprint (none) -> Inductor_SMD:L_Coilcraft_LPS4018
- L3: renamed from L17; footprint (none) -> Inductor_SMD:L_Coilcraft_LPS4018
- R11: renamed from R105; footprint (none) -> Resistor_SMD:R_0603_1608Metric
- R12: renamed from R106; footprint (none) -> Resistor_SMD:R_0603_1608Metric
- R13: renamed from R107; footprint (none) -> Resistor_SMD:R_0603_1608Metric
- R14: renamed from R110; footprint (none) -> Resistor_SMD:R_0603_1608Metric
- R7: renamed from R101; footprint (none) -> Resistor_SMD:R_0603_1608Metric
- R8: renamed from R102; footprint (none) -> Resistor_SMD:R_0603_1608Metric
- renumbered U16 to U3, U18 to U5, U17 to U6, U19 to U7
Connections:
- net +3V3: now also C18.2, TP5.1, U4.1 (VOUT), U4.10 (FB)
- net GND: now also U7.15 (TD), C18.1, C6.1, R10.1, R9.1, U4.11 (PGND), U4.3 (PGND), U4.9 (GND)
- net UNREG_SAFE: now reaches C13.1, C15.2, R14.1, U7.10 (OUT), U7.11 (OUT), U7.5 (EN2)
- net UNREG_SAFE: now also U4.5 (VIN)
- net at C17.2, R14.2: now also U4.6 (EN), U4.7 (PS/SYNC), U4.8 (VINA)
- net at L3.2: now also U4.2 (L2)
- net at L3.1: now also U4.4 (L1)
- net BATT: now reaches BT1.1 (+), C14.1, R12.1, U7.2 (BAT), U7.3 (BAT)
- net at U7.12 (ILIM): now also R9.2
- net at U7.13 (IN): now also C6.2, D1.1 (K)
- net at U7.16 (ISET): now also R10.2
- new net VBUS: D1.2 (A)
Other:
- note added: "TBD 5v input block"
- note removed: "General +3v3"
- moved on the sheet: BT1, C13, C14, C15, C16, C17, D2, L3, R11, R12, R13, R14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

Commit message: add can connector
Changed lines of the file:
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@@
 		)
 	)
+	(wire
+		(pts
+			(xy 19.05 128.27) (xy 19.05 124.46)
+		)
+		(stroke
+			(width 0)
+			(type default)
+		)
+	)
 	(polyline
 		(pts
@@
 	)
 	(symbol
+		(lib_id "power:+12V")
+		(at 19.05 124.46 0)
+		(unit 1)
+		(body_style 1)
+		(exclude_from_sim no)
+		(in_bom yes)
+		(on_board yes)
+		(in_pos_files yes)
+		(dnp no)
+		(fields_autoplaced yes)
+		(property "Reference" "#PWR028"
+			(at 19.05 128.27 0)
+			(hide yes)
+			(show_name no)
+			(do_not_autoplace no)
+			(effects
+				(font
+					(size 1.27 1.27)
+				)
+			)
+		)
+		(property "Value" "+12V"
+			(at 19.05 119.38 0)
+			(show_name no)
+			(do_not_autoplace no)
+			(effects
+				(font
+					(size 1.27 1.27)
+				)
+			)
+		)
+		(property "Footprint" ""
+			(at 19.05 124.46 0)
+			(hide yes)
+			(show_name no)
+			(do_not_autoplace no)
+			(effects
+				(font
+					(size 1.27 1.27)
+				)
+			)
+		)
+		(property "Datasheet" ""
+			(at 19.05 124.46 0)
+			(hide yes)
+			(show_name no)
+			(do_not_autoplace no)
+			(effects
+				(font
+					(size 1.27 1.27)
+				)
+			)
+		)
+		(property "Description" "Power symbol creates a global label with name \"+12V\""
+			(at 19.05 124.46 0)
+			(hide yes)
+			(show_name no)
+			(do_not_autoplace no)
+			(effects
+				(font
+					(size 1.27 1.27)
+				)
+			)
+		)
+		(pin "1"
+		)
+		(instances
+			(project "telemetry-logging-board"
+				(path "/77f08122-c609-410b-9d24-33eebdb4af2b/4a560299-de31-4079-a217-7e1626a60243"
+					(reference "#PWR028")
+					(unit 1)
+				)
+			)
+		)
+	)
+	(symbol
 		(lib_id "Device:C_Polarized")
 		(at 147.32 116.84 0)
@@
 					(unit 1)
 				)
+			)
+		)
+	)
+	(symbol
+		(lib_id "power:GND")
+		(at 19.05 132.08 0)
+		(unit 1)
+		(body_style 1)
+		(exclude_from_sim no)
+		(in_bom yes)
+		(on_board yes)
+		(in_pos_files yes)
+		(dnp no)
+		(fields_autoplaced yes)
+		(property "Reference" "#PWR021"
+			(at 19.05 138.43 0)
+			(hide yes)
+			(show_name no)
+			(do_not_autoplace no)
+			(effects
+				(font
+					(size 1.27 1.27)
+				)
+			)
+		)
+		(property "Value" "GND"
+			(at 19.05 137.16 0)
+			(show_name no)
+			(do_not_autoplace no)
+			(effects
+				(font
+					(size 1.27 1.27)
+				)
+			)
+		)
+		(property "Footprint" ""
+			(at 19.05 132.08 0)
+			(hide yes)
+			(show_name no)
+			(do_not_autoplace no)
+			(effects
+				(font
+					(size 1.27 1.27)
+				)
+			)
+		)
+		(property "Datasheet" ""
+			(at 19.05 132.08 0)
+			(hide yes)
+			(show_name no)
+			(do_not_autoplace no)
+			(effects
+				(font
+					(size 1.27 1.27)
+				)
+			)
+		)
+		(property "Description" "Power symbol creates a global label with name \"GND\" , ground"
+			(at 19.05 132.08 0)
+			(hide yes)
+			(show_name no)
+			(do_not_autoplace no)
+			(effects
+				(font
+					(size 1.27 1.27)
+				)
+			)
+		)
+		(pin "1"
+		)
+		(instances
+			(project "telemetry-logging-board"
+				(path "/77f08122-c609-410b-9d24-33eebdb4af2b/4a560299-de31-4079-a217-7e1626a60243"
+					(reference "#PWR021")
+					(unit 1)
+				)
