File: tractive-system-status-indicator/tractive-system-status-indicator.kicad_pcb (KiCad board)
At the start: 2 copper layers, 50.6 x 16.1 mm, 0 parts

Commit message: schematic
Put footprints in and stuff, will start layout soon
Parts:
- added D1: LED, LED_SMD:LED_0805_2012Metric_Pad1.15x1.40mm_HandSolder, F.Cu at (126.0, 73.2)
- added D10: LED, LED_SMD:LED_0805_2012Metric_Pad1.15x1.40mm_HandSolder, F.Cu at (153.9, 84.3)
- added D11: LED, LED_SMD:LED_0805_2012Metric_Pad1.15x1.40mm_HandSolder, F.Cu at (161.0, 84.3)
- added D12: LED, LED_SMD:LED_0805_2012Metric_Pad1.15x1.40mm_HandSolder, F.Cu at (167.6, 84.3)
- added D13: LED, LED_SMD:LED_0603_1608Metric_Pad1.05x0.95mm_HandSolder, F.Cu at (140.7, 130.3)
- added D14: LED, LED_SMD:LED_0603_1608Metric_Pad1.05x0.95mm_HandSolder, F.Cu at (140.7, 132.9)
- added D15: LED, LED_SMD:LED_0603_1608Metric_Pad1.05x0.95mm_HandSolder, F.Cu at (140.7, 135.5)
- added D16: LED, LED_SMD:LED_0603_1608Metric_Pad1.05x0.95mm_HandSolder, F.Cu at (140.7, 138.1)
- added D17: LED, LED_SMD:LED_0603_1608Metric_Pad1.05x0.95mm_HandSolder, F.Cu at (140.7, 140.7)
- added D18: LED, LED_SMD:LED_0603_1608Metric_Pad1.05x0.95mm_HandSolder, F.Cu at (145.1, 130.3)
- added D19: LED, LED_SMD:LED_0603_1608Metric_Pad1.05x0.95mm_HandSolder, F.Cu at (145.1, 132.9)
- added D2: LED, LED_SMD:LED_0805_2012Metric_Pad1.15x1.40mm_HandSolder, F.Cu at (132.1, 73.2)
- added D20: LED, LED_SMD:LED_0603_1608Metric_Pad1.05x0.95mm_HandSolder, F.Cu at (145.1, 135.5)
- added D21: LED, LED_SMD:LED_0603_1608Metric_Pad1.05x0.95mm_HandSolder, F.Cu at (145.1, 138.1)
- added D22: LED, LED_SMD:LED_0603_1608Metric_Pad1.05x0.95mm_HandSolder, F.Cu at (145.1, 140.7)
- added D23: LED, LED_SMD:LED_0603_1608Metric_Pad1.05x0.95mm_HandSolder, F.Cu at (149.5, 130.3)
- added D24: LED, LED_SMD:LED_0603_1608Metric_Pad1.05x0.95mm_HandSolder, F.Cu at (149.5, 132.9)
- added D25: LED, LED_SMD:LED_0603_1608Metric_Pad1.05x0.95mm_HandSolder, F.Cu at (149.5, 135.5)
- added D26: LED, LED_SMD:LED_0603_1608Metric_Pad1.05x0.95mm_HandSolder, F.Cu at (149.5, 138.1)
- added D27: LED, LED_SMD:LED_0603_1608Metric_Pad1.05x0.95mm_HandSolder, F.Cu at (149.5, 140.7)
- added D3: LED, LED_SMD:LED_0805_2012Metric_Pad1.15x1.40mm_HandSolder, F.Cu at (138.7, 73.2)
- added D4: LED, LED_SMD:LED_0805_2012Metric_Pad1.15x1.40mm_HandSolder, F.Cu at (126.0, 84.3)
- added D5: LED, LED_SMD:LED_0805_2012Metric_Pad1.15x1.40mm_HandSolder, F.Cu at (132.1, 84.3)
- added D6: LED, LED_SMD:LED_0805_2012Metric_Pad1.15x1.40mm_HandSolder, F.Cu at (138.7, 84.3)
- added D7: LED, LED_SMD:LED_0805_2012Metric_Pad1.15x1.40mm_HandSolder, F.Cu at (153.9, 73.2)
- added D8: LED, LED_SMD:LED_0805_2012Metric_Pad1.15x1.40mm_HandSolder, F.Cu at (161.0, 73.2)
- added D9: LED, LED_SMD:LED_0805_2012Metric_Pad1.15x1.40mm_HandSolder, F.Cu at (167.6, 73.2)
- added G***: LOGO, formula_slug_footprint_library:FORMULA SLUG, F.Cu at (149.4, 73.7)
- added J1: Conn_01x06, Connector_Molex:Molex_Micro-Fit_3.0_43650-0610_1x06-1MP_P3.00mm_Horizontal, F.Cu at (145.3, 106.7)
- added R1: 220, Resistor_SMD:R_0603_1608Metric_Pad0.98x0.95mm_HandSolder, F.Cu at (136.3, 130.3)
- added R2: 220, Resistor_SMD:R_0603_1608Metric_Pad0.98x0.95mm_HandSolder, F.Cu at (136.3, 132.8)
- added R3: 360, Resistor_SMD:R_0603_1608Metric_Pad0.98x0.95mm_HandSolder, F.Cu at (136.3, 135.3)
- added R4: 360, Resistor_SMD:R_0603_1608Metric_Pad0.98x0.95mm_HandSolder, F.Cu at (136.3, 137.8)
- added R5: 200, Resistor_SMD:R_0603_1608Metric_Pad0.98x0.95mm_HandSolder, F.Cu at (136.3, 140.3)
- added R6: 200, Resistor_SMD:R_0603_1608Metric_Pad0.98x0.95mm_HandSolder, F.Cu at (136.3, 142.8)
- added R7: 200, Resistor_SMD:R_0603_1608Metric_Pad0.98x0.95mm_HandSolder, F.Cu at (136.3, 145.4)
- added R8: 200, Resistor_SMD:R_0603_1608Metric_Pad0.98x0.95mm_HandSolder, F.Cu at (136.3, 147.9)
- added R9: 200, Resistor_SMD:R_0603_1608Metric_Pad0.98x0.95mm_HandSolder, F.Cu at (136.3, 150.4)
Other:
- board size 50.6 x 16.1 mm -> 125.2 x 46.9 mm

Commit message: layout
oved to new template, also did layout. Satisfies area requirements
Parts:
- removed G***: LOGO, formula_slug_footprint_library:FORMULA SLUG
- removed J1: Conn_01x06, Connector_Molex:Molex_Micro-Fit_3.0_43650-0610_1x06-1MP_P3.00mm_Horizontal
- moved D27 73.0 mm to (198.3, 86.4)
- moved R9 68.2 mm to (184.9, 102.6)
- moved R3 63.3 mm to (157.5, 75.7), turned to 90 degrees
- moved D25 61.7 mm to (198.1, 97.5), turned to 180 degrees
- moved R4 60.5 mm to (157.5, 81.2), turned to -90 degrees
- moved D15 57.8 mm to (110.2, 86.4), turned to 180 degrees
- moved R8 57.5 mm to (171.7, 102.6)
- moved D26 56.1 mm to (198.1, 110.2)
- moved R1 56.0 mm to (121.9, 76.2), turned to 90 degrees
- moved D22 55.4 mm to (179.2, 97.0), turned to 180 degrees
- moved D24 55.3 mm to (179.3, 86.4)
- moved D21 53.9 mm to (160.0, 86.4)
- moved R2 53.0 mm to (121.9, 81.8), turned to -90 degrees
- moved R7 47.5 mm to (157.0, 102.6)
- moved D18 45.4 mm to (134.0, 86.4)
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Connections:
- net /RTD_LED_Anode renamed /RTM_In
- net /RTD_LED_Cathode renamed /RTM_Out
- D11 pad 1: /TSSI_RED_Cathode -> Net-(D11-K)
- D11 pad 2: Net-(D11-A) -> Net-(D10-K)
- D12 pad 2: Net-(D10-K) -> Net-(D11-K)
- D8 pad 1: Net-(D10-A) -> Net-(D8-K)
- D8 pad 2: Net-(D8-A) -> Net-(D7-K)
- D9 pad 1: Net-(D11-A) -> /TSSI_RED_Cathode
- D9 pad 2: Net-(D7-K) -> Net-(D8-K)
- R4 pad 2: Net-(D8-A) -> Net-(D10-A)
Routing:
- net /RTM_In: track 0.00 -> 112.2 mm
- net /RTM_Out: track 0.00 -> 90.7 mm
- net Net-(D20-K): track 0.00 -> 25.6 mm
- net Net-(D17-K): track 0.00 -> 25.5 mm
- net Net-(D14-K): track 0.00 -> 25.5 mm
- net Net-(D26-K): track 0.00 -> 24.7 mm
- net Net-(D23-K): track 0.00 -> 24.6 mm
- net Net-(D19-K): track 0.00 -> 13.9 mm
- net Net-(D25-A): track 0.00 -> 13.5 mm
- net Net-(D16-K): track 0.00 -> 13.4 mm
- net Net-(D22-K): track 0.00 -> 13.3 mm
- net Net-(D13-K): track 0.00 -> 12.9 mm
- net Net-(D13-A): track 0.00 -> 12.8 mm
- net Net-(D25-K): track 0.00 -> 12.7 mm
- net Net-(D16-A): track 0.00 -> 8.96 mm
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Other:
- board size 125.2 x 46.9 mm -> 137.5 x 46.9 mm

Commit message: Updated template, resourced LED's,  placed components
Parts:
- removed D15, D21, D22, D23, D24: LED, LED_SMD:LED_0603_1608Metric_Pad1.05x0.95mm_HandSolder
- added D28: LED, LED_SMD:LED_Avago_PLCC4_3.2x2.8mm_CW, F.Cu at (163.1, 105.7)
- added D29: LED, LED_SMD:LED_Avago_PLCC4_3.2x2.8mm_CW, F.Cu at (163.1, 113.8)
- added D30: LED, LED_SMD:LED_Avago_PLCC4_3.2x2.8mm_CW, F.Cu at (149.4, 109.2)
- added D31: LED, LED_SMD:LED_Avago_PLCC4_3.2x2.8mm_CW, F.Cu at (135.1, 116.3)
- added D32: LED, LED_SMD:LED_Avago_PLCC4_3.2x2.8mm_CW, F.Cu at (129.0, 113.8)
- added D33: LED, LED_SMD:LED_Avago_PLCC4_3.2x2.8mm_CW, F.Cu at (142.2, 116.3)
- added D34: LED, LED_SMD:LED_Avago_PLCC4_3.2x2.8mm_CW, F.Cu at (149.4, 116.3)
- added D35: LED, LED_SMD:LED_Avago_PLCC4_3.2x2.8mm_CW, F.Cu at (157.0, 116.3)
- added D36: LED, LED_SMD:LED_Avago_PLCC4_3.2x2.8mm_CW, F.Cu at (157.0, 109.2)
- added D37: LED, LED_SMD:LED_Avago_PLCC4_3.2x2.8mm_CW, F.Cu at (125.5, 87.4)
- added D38: LED, LED_SMD:LED_Avago_PLCC4_3.2x2.8mm_CW, F.Cu at (132.6, 87.4)
- added D39: LED, LED_SMD:LED_Everlight-SMD3528_3.5x2.8mm_67-21ST, F.Cu at (158.5, 94.5)
- added D40: LED, LED_SMD:LED_Everlight-SMD3528_3.5x2.8mm_67-21ST, F.Cu at (165.6, 94.5)
- added D41: LED, LED_SMD:LED_Everlight-SMD3528_3.5x2.8mm_67-21ST, F.Cu at (151.4, 94.5)
- added D42: LED, LED_SMD:LED_Avago_PLCC4_3.2x2.8mm_CW, F.Cu at (135.1, 102.1)
- added D43: LED, LED_SMD:LED_Avago_PLCC4_3.2x2.8mm_CW, F.Cu at (142.7, 102.1)
- added D44: LED, LED_SMD:LED_Avago_PLCC4_3.2x2.8mm_CW, F.Cu at (149.9, 102.1)
- added D45: LED, LED_SMD:LED_Avago_PLCC4_3.2x2.8mm_CW, F.Cu at (157.0, 102.1)
- added J1: Conn_01x06, Connector_Molex:Molex_Micro-Fit_3.0_43650-0610_1x06-1MP_P3.00mm_Horizontal, F.Cu at (113.0, 153.4)
- added R10: 220, Resistor_SMD:R_0603_1608Metric_Pad0.98x0.95mm_HandSolder, F.Cu at (132.1, 139.2)
- added R11: 220, Resistor_SMD:R_0603_1608Metric_Pad0.98x0.95mm_HandSolder, F.Cu at (132.0, 141.4)
- D1, D10, D2, D3, D4, D5, D6, D7, D8, D9: footprint LED_SMD:LED_0805_2012Metric_Pad1.15x1.40mm_HandSolder -> LED_SMD:LED_Avago_PLCC4_3.2x2.8mm_CW
- D11, D12: footprint LED_SMD:LED_0805_2012Metric_Pad1.15x1.40mm_HandSolder -> LED_SMD:LED_Everlight-SMD3528_3.5x2.8mm_67-21ST
- D13, D14, D16, D17, D18, D19, D20: footprint LED_SMD:LED_0603_1608Metric_Pad1.05x0.95mm_HandSolder -> LED_SMD:LED_Everlight-SMD3528_3.5x2.8mm_67-21ST
- D25, D26, D27: footprint LED_SMD:LED_0603_1608Metric_Pad1.05x0.95mm_HandSolder -> LED_SMD:LED_Avago_PLCC4_3.2x2.8mm_CW
- R3, R4: value 360 -> 220
- R5, R6, R7, R8, R9: value 200 -> 220
- moved D25 69.6 mm to (129.0, 105.7)
- moved D14 69.1 mm to (172.7, 80.3)
- moved R3 67.6 mm to (127.7, 136.3), turned to 0 degrees
- moved D9 66.8 mm to (118.4, 94.5), turned to 0 degrees
- moved R4 64.9 mm to (127.7, 138.8), turned to 0 degrees
- moved D13 63.3 mm to (172.7, 87.4)
- moved D26 63.0 mm to (135.1, 109.2)
- moved R9 62.7 mm to (132.0, 136.3)
- moved D27 60.5 mm to (142.2, 109.2)
- moved R1 55.4 mm to (127.7, 131.3), turned to 0 degrees
- moved R2 52.4 mm to (127.7, 133.8), turned to 0 degrees
- moved D8 50.7 mm to (125.5, 94.5), turned to 0 degrees
- moved R8 50.5 mm to (132.0, 133.8)
- moved D10 44.8 mm to (118.4, 87.4), turned to 0 degrees
- moved R6 43.3 mm to (127.7, 143.9)
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Connections:
- D11 pad 2: Net-(D10-K) -> Net-(D11-A)
- D12 pad 1: /TSSI_RED_Cathode -> Net-(D12-K)
- D13 pad 2: Net-(D13-A) -> Net-(D12-K)
- D14 pad 1: Net-(D14-K) -> /TSSI_RED_Cathode
- D18 pad 1: /RTM_Out -> Net-(D18-K)
- D19 pad 1: Net-(D19-K) -> /TSSI_RED_Cathode
- D19 pad 2: Net-(D19-A) -> Net-(D18-K)
- D20 pad 2: Net-(D19-K) -> Net-(D20-A)
- D27 pad 1: /RTM_Out -> Net-(D27-K)
- D9 pad 1: /TSSI_RED_Cathode -> /TSSI_GREEN_Cathode
- R3 pad 1: /TSSI_RED_Anode -> /TSSI_GREEN_Anode
- R4 pad 1: /TSSI_RED_Anode -> /TSSI_GREEN_Anode
- R5 pad 1: /RTM_In -> /TSSI_RED_Anode
- R5 pad 2: Net-(D13-A) -> Net-(D11-A)
- R6 pad 1: /RTM_In -> /TSSI_RED_Anode
- R7 pad 2: Net-(D19-A) -> Net-(D42-A)
- R8 pad 2: Net-(D22-A) -> Net-(D25-A)
- R9 pad 2: Net-(D25-A) -> Net-(D29-A)
Routing:
- net /RTM_In: track 112.2 -> 0.00 mm
- net /RTM_Out: track 90.7 -> 0.00 mm
- net Net-(D20-K): track 25.6 -> 0.00 mm
- net Net-(D17-K): track 25.5 -> 0.00 mm
- net Net-(D14-K): track 25.5 -> 0.00 mm
- net Net-(D26-K): track 24.7 -> 0.00 mm
- net Net-(D23-K): track 24.6 -> 0.00 mm
- net Net-(D19-K): track 13.9 -> 0.00 mm
- net Net-(D25-A): track 13.5 -> 0.00 mm
- net Net-(D16-K): track 13.4 -> 0.00 mm
- net Net-(D22-K): track 13.3 -> 0.00 mm
- net Net-(D13-K): track 12.9 -> 0.00 mm
- net Net-(D13-A): track 12.8 -> 0.00 mm
- net Net-(D25-K): track 12.7 -> 0.00 mm
- net Net-(D16-A): track 8.96 -> 0.00 mm
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
Commit message: Schematic
Found resistor values (used 70-80% of max current draw for LED's)
Parts:
- moved R5 65.7 mm to (169.2, 90.4)
- moved R6 60.0 mm to (154.9, 90.4), turned to 180 degrees
- moved R11 59.1 mm to (162.1, 90.4), turned to 180 degrees
- moved R2 51.7 mm to (136.1, 82.8)
- moved R4 49.3 mm to (121.9, 89.9), turned to 180 degrees
- moved R1 48.8 mm to (121.9, 82.8), turned to 180 degrees
- moved R3 46.4 mm to (129.0, 89.9)
- moved R7 6.66 mm to (126.0, 134.1)
- moved D10 1.02 mm to (118.4, 86.4)
- moved D11 1.02 mm to (172.7, 93.5), turned to 180 degrees
- moved D12 1.02 mm to (165.6, 86.4)
- moved D13 1.02 mm to (172.7, 86.4), turned to 180 degrees
- moved D16 1.02 mm to (151.4, 86.4)
- moved D20 1.02 mm to (158.5, 86.4)
- moved D37 1.02 mm to (125.5, 86.4), turned to 180 degrees
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Routing:
- net /TSSI_GREEN_Cathode: track 0.00 -> 48.9 mm
- net /TSSI_GREEN_Anode: track 0.00 -> 37.7 mm
- net /TSSI_RED_Cathode: track 0.00 -> 32.5 mm
- net /TSSI_RED_Anode: track 0.00 -> 22.2 mm
- net Net-(D40-K): track 0.00 -> 16.9 mm
- net Net-(D11-K): track 0.00 -> 11.3 mm
- net Net-(D37-K): track 0.00 -> 9.31 mm
- net Net-(D12-K): track 0.00 -> 9.29 mm
- net Net-(D5-K): track 0.00 -> 8.93 mm
- net Net-(D10-K): track 0.00 -> 8.80 mm
- net Net-(D20-K): track 0.00 -> 7.33 mm
- net Net-(D16-K): track 0.00 -> 7.33 mm
- net Net-(D13-K): track 0.00 -> 7.33 mm
- net Net-(D7-A): track 0.00 -> 6.22 mm
- net Net-(D10-A): track 0.00 -> 6.12 mm
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
Commit message: Layout
Parts:
- removed J1: Conn_01x06, Connector_Molex:Molex_Micro-Fit_3.0_43650-0610_1x06-1MP_P3.00mm_Horizontal
- moved R9 44.8 mm to (168.6, 110.5), turned to 180 degrees
- moved R7 36.7 mm to (139.2, 99.8), turned to 180 degrees
- moved R10 26.0 mm to (138.7, 114.0)
- moved R8 25.4 mm to (123.4, 110.0)
- moved D25 0.24 mm to (129.0, 106.4)
- moved D27 0.24 mm to (142.2, 110.0), turned to 180 degrees
- moved D28 0.24 mm to (163.0, 106.4)
- moved D29 0.24 mm to (163.0, 114.5)
- moved D30 0.24 mm to (149.3, 110.0)
- moved D32 0.24 mm to (129.0, 114.5)
- moved D36 0.24 mm to (156.9, 110.0)
- moved D43 0.24 mm to (142.7, 102.9)
- moved D44 0.24 mm to (149.8, 102.9)
- moved D45 0.24 mm to (156.9, 102.9)
- moved D26 0.24 mm to (135.1, 110.0)
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Routing:
- net /RTM_In: track 0.00 -> 117.9 mm
- net /RTM_Out: track 0.00 -> 93.2 mm
- net Net-(D27-K): track 0.00 -> 29.9 mm
- net Net-(D30-K): track 0.00 -> 16.4 mm
- net Net-(D35-K): track 0.00 -> 15.5 mm
- net Net-(D29-K): track 0.00 -> 12.6 mm
- net Net-(D26-K): track 0.00 -> 10.1 mm
- net Net-(D42-A): track 0.00 -> 7.56 mm
- net Net-(D25-K): track 0.00 -> 6.95 mm
- net Net-(D33-A): track 0.00 -> 5.62 mm
- net Net-(D25-A): track 0.00 -> 4.95 mm
- net Net-(D29-A): track 0.00 -> 4.63 mm
- net Net-(D34-K): track 0.00 -> 4.62 mm
- net Net-(D42-K): track 0.00 -> 4.62 mm
- net Net-(D31-K): track 0.00 -> 4.15 mm
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
Commit message: Documentation,  symbol fields, connector changes
Parts:
- added J1: Conn_01x06, formula_slug_footprint_library:1054301106, B.Cu at (182.4, 107.2)
- R1, R2, R3, R4: value 220 -> 60
- R10, R7, R8, R9: value 220 -> 100
- R11, R5, R6: value 220 -> 80
- moved D35 0.48 mm to (156.5, 117.1)
- moved D36 0.48 mm to (156.5, 110.0)
- moved D44 0.48 mm to (149.4, 102.9)
- moved D45 0.48 mm to (156.5, 102.9)
- moved D43 0.48 mm to (142.2, 102.9)
- moved D42 0.05 mm to (135.2, 102.9)
Routing:
- net /TSSI_GREEN_Anode: track 37.7 -> 130.8 mm, vias 0 -> 1
- net /TSSI_GREEN_Cathode: track 48.9 -> 126.2 mm, vias 0 -> 1
- net /TSSI_RED_Anode: track 22.2 -> 60.9 mm, vias 0 -> 1
- net /TSSI_RED_Cathode: track 32.5 -> 59.8 mm, vias 0 -> 1
- net /RTM_In: track 117.9 -> 137.8 mm, vias 0 -> 1
- net /RTM_Out: track 93.2 -> 103.4 mm, vias 0 -> 1

Commit message: Added filled zones to layout
- Rewired using the filled zones
- Flipped resistors to back
Parts:
- R1, R10, R11, R2, R3, R4, R5, R6, R7, R8, R9: moved to B.Cu
- moved J1 11.1 mm to (190.5, 99.6)
- turned R1 to 0 degrees
- turned R10 to 180 degrees
- turned R11 to 0 degrees
- turned R2 to 180 degrees
- turned R3 to 180 degrees
- turned R4 to 0 degrees
- turned R5 to 180 degrees
- turned R6 to 0 degrees
- turned R7 to 0 degrees
- turned R8 to 180 degrees
- turned R9 to 0 degrees
Routing:
- net /RTM_In: track 137.8 -> 28.4 mm, vias 1 -> 0
- net /RTM_Out: track 103.4 -> 27.8 mm
- net /TSSI_GREEN_Cathode: track 126.2 -> 75.1 mm
- net /TSSI_RED_Cathode: track 59.8 -> 25.1 mm
- net /TSSI_GREEN_Anode: track 130.8 -> 96.5 mm, vias 1 -> 0
- net /TSSI_RED_Anode: track 60.9 -> 36.3 mm, vias 1 -> 0
- net Net-(D29-A): track 4.63 -> 12.8 mm, vias 0 -> 1
- net Net-(D35-K): track 15.5 -> 22.2 mm
- net Net-(D27-K): track 30.1 -> 24.4 mm
- net Net-(D25-A): track 4.95 -> 10.7 mm, vias 0 -> 1
- net Net-(D33-A): track 5.62 -> 8.16 mm, vias 0 -> 1
- net Net-(D1-A): track 5.31 -> 7.13 mm, vias 0 -> 1
- net Net-(D10-A): track 6.12 -> 7.71 mm, vias 0 -> 1
- net Net-(D30-K): track 16.4 -> 17.8 mm
- net Net-(D11-A): track 3.81 -> 5.01 mm, vias 0 -> 1
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- added copper zone on B.Cu, net /RTM_In
- added copper zone on F.Cu, net /RTM_Out
- added copper zone on B.Cu, net /TSSI_GREEN_Anode
- added copper zone on F.Cu, net /TSSI_GREEN_Cathode
- added copper zone on B.Cu, net /TSSI_RED_Anode
- added copper zone on F.Cu, net /TSSI_RED_Cathode

Commit message: added 3d models
Parts:
- D11, D12, D13, D14, D16, D17, D18, D19, D20, D39, D40, D41: footprint LED_SMD:LED_Everlight-SMD3528_3.5x2.8mm_67-21ST -> LED_SMD:LED_Avago_PLCC4_3.2x2.8mm_CW
- moved R7 9.47 mm to (130.0, 102.4)
Routing:
- net Net-(D42-A): track 8.01 -> 3.60 mm
- net Net-(D16-A): track 5.58 -> 8.36 mm
- net Net-(D13-K): track 7.33 -> 10.0 mm
- net Net-(D12-K): track 10.2 -> 7.94 mm
- net Net-(D20-A): track 5.85 -> 8.09 mm
- net Net-(D11-A): track 5.01 -> 7.04 mm
- net Net-(D20-K): track 7.33 -> 9.08 mm
- net Net-(D16-K): track 7.33 -> 5.61 mm
- net Net-(D40-K): track 16.4 -> 15.1 mm
- net /TSSI_RED_Cathode: track 25.1 -> 26.3 mm
- net Net-(D39-K): track 4.96 -> 4.11 mm
- net Net-(D18-K): track 4.96 -> 4.11 mm
- net Net-(D17-K): track 4.96 -> 4.11 mm
- net Net-(D11-K): track 11.7 -> 11.1 mm
- net Net-(D5-K): track 8.67 -> 8.11 mm
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