File: tractive-system-status-indicator/tractive-system-status-indicator.kicad_sch (KiCad schematic)
At the start: 25 parts, among them J1 Conn_01x06

Commit message: schematic
Put footprints in and stuff, will start layout soon
Parts:
- added D19, D20, D21, D22, D23, D24, D25, D26, D27: LED, LED_SMD:LED_0603_1608Metric_Pad1.05x0.95mm_HandSolder, symbol Device:LED
- added R7, R8, R9: 200, Resistor_SMD:R_0603_1608Metric_Pad0.98x0.95mm_HandSolder, symbol Device:R
- D1, D10, D11, D12, D2, D3, D4, D5, D6, D7, D8, D9: footprint (none) -> LED_SMD:LED_0805_2012Metric_Pad1.15x1.40mm_HandSolder; Digi URL (none) -> https://www.digikey.com/en/products/detail/xinglight/XL-TD2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
- D13, D14, D15, D16, D17, D18: footprint (none) -> LED_SMD:LED_0603_1608Metric_Pad1.05x0.95mm_HandSolder; Digi URL (none) -> https://www.digikey.com/en/products/detail/ams-osram-usa-in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
- J1: footprint (none) -> Connector_Molex:Molex_Micro-Fit_3.0_43650-0610_1x06-1MP_P3.00mm_Horizontal; Digi URL (none) -> https://www.digikey.com/en/products/detail/molex/0436500612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
- R1, R2: value R -> 220; footprint (none) -> Resistor_SMD:R_0603_1608Metric_Pad0.98x0.95mm_HandSolder
- R3, R4: value R -> 360; footprint (none) -> Resistor_SMD:R_0603_1608Metric_Pad0.98x0.95mm_HandSolder
- R5, R6: value R -> 200; footprint (none) -> Resistor_SMD:R_0603_1608Metric_Pad0.98x0.95mm_HandSolder
Connections:
- net RTD_LED_Anode: now also R7.1, R8.1, R9.1
- net RTD_LED_Cathode: now also D15.1 (K), D21.1 (K), D24.1 (K), D27.1 (K); no longer D17.1 (K)
- net at D14.2 (A): now also D13.1 (K); no longer R6.2
- net at D17.2 (A): now also D16.1 (K); no longer D15.1 (K)
- net at D14.1 (K): now also D15.2 (A); no longer D16.2 (A)
- net at D18.2 (A): now also D17.1 (K); no longer D16.1 (K)
- new net: D26.1 (K), D27.2 (A)
- new net: D25.1 (K), D26.2 (A)
- new net: D23.1 (K), D24.2 (A)
- new net: D22.1 (K), D23.2 (A)
- new net: D20.1 (K), D21.2 (A)
- new net: D19.1 (K), D20.2 (A)
- new net: D19.2 (A), R7.2
- new net: D25.2 (A), R9.2
- new net: D16.2 (A), R6.2
- new net: D22.2 (A), R8.2
Other:
- company: (none) -> Formula Slug
- title: (none) -> TSSI Board
- moved on the sheet: D1, D10, D11, D12, D13, D2, D3, D4, D5, D6, D7, D8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

Commit message: layout
oved to new template, also did layout. Satisfies area requirements
Connections:
- net TSSI_RED_Cathode: now also D9.1 (K); no longer D11.1 (K)
- net at R4.2: now also D10.2 (A); no longer D8.2 (A)
- net at D8.1 (K): now also D9.2 (A); no longer D10.2 (A)
- net at D11.2 (A): now also D10.1 (K); no longer D9.1 (K)
- net at D7.1 (K): now also D8.2 (A); no longer D9.2 (A)
- net at D12.2 (A): now also D11.1 (K); no longer D10.1 (K)
- net RTD_LED_Anode renamed RTM_In
- net RTD_LED_Cathode renamed RTM_Out
Other:
- note added: "VCU / PEB"
- note removed: "VCU"
- title: TSSI Board -> ${BOARD_TITLE}

Commit message: Updated template, resourced LED's,  placed components
Parts:
- removed D15, D21, D22, D23, D24: LED, LED_SMD:LED_0603_1608Metric_Pad1.05x0.95mm_HandSolder, symbol Device:LED
- added D28, D29, D30, D31, D32, D33, D34, D35, D36, D37, D38, D42, D43, D44, D45: LED, LED_SMD:LED_Avago_PLCC4_3.2x2.8mm_CW, symbol Device:LED
- added D39, D40, D41: LED, LED_SMD:LED_Everlight-SMD3528_3.5x2.8mm_67-21ST, symbol Device:LED
- added R10, R11: 220, Resistor_SMD:R_0603_1608Metric_Pad0.98x0.95mm_HandSolder, symbol Device:R
- D1, D10, D2, D3, D4, D5, D6, D7, D8, D9: footprint LED_SMD:LED_0805_2012Metric_Pad1.15x1.40mm_HandSolder -> LED_SMD:LED_Avago_PLCC4_3.2x2.8mm_CW; Digi URL https://www.digikey.com/en/products/detail/xinglight/XL-TD2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 -> (none)
- D11, D12: footprint LED_SMD:LED_0805_2012Metric_Pad1.15x1.40mm_HandSolder -> LED_SMD:LED_Everlight-SMD3528_3.5x2.8mm_67-21ST; Digi URL https://www.digikey.com/en/products/detail/xinglight/XL-TD2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 -> (none)
- D13, D14, D16, D17, D18, D19, D20: footprint LED_SMD:LED_0603_1608Metric_Pad1.05x0.95mm_HandSolder -> LED_SMD:LED_Everlight-SMD3528_3.5x2.8mm_67-21ST; Digi URL https://www.digikey.com/en/products/detail/ams-osram-usa-in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 -> (none)
- D25, D26, D27: footprint LED_SMD:LED_0603_1608Metric_Pad1.05x0.95mm_HandSolder -> LED_SMD:LED_Avago_PLCC4_3.2x2.8mm_CW; Digi URL https://www.digikey.com/en/products/detail/ams-osram-usa-in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 -> (none)
- R3, R4: value 360 -> 220
- R5, R6, R7, R8, R9: value 200 -> 220
Connections:
- net RTM_In: now also R10.1; no longer R5.1, R6.1
- net RTM_Out: now also D28.1 (K), D32.1 (K), D36.1 (K), D45.1 (K); no longer D18.1 (K), D27.1 (K)
- net TSSI_GREEN_Anode: now also R3.1, R4.1
- net TSSI_GREEN_Cathode: now also D9.1 (K), D38.1 (K)
- net TSSI_RED_Anode: now also R5.1, R6.1, R11.1; no longer R3.1, R4.1
- net TSSI_RED_Cathode: now also D14.1 (K), D19.1 (K), D41.1 (K); no longer D12.1 (K), D9.1 (K)
- net at D11.2 (A): now also R5.2; no longer D10.1 (K)
- net at D13.2 (A): now also D12.1 (K); no longer R5.2
- net at D20.2 (A): now also R11.2; no longer D19.1 (K)
- net at R7.2: now also D42.2 (A); no longer D19.2 (A)
- net at R8.2: now also D25.2 (A)
- net at R9.2: now also D29.2 (A); no longer D25.2 (A)
- net at D20.1 (K): now also D39.2 (A)
- new net: D40.1 (K), D41.2 (A)
- new net: D33.2 (A), R10.2
- new net: D30.1 (K), D31.2 (A)
- new net: D29.1 (K), D30.2 (A)
- new net: D34.1 (K), D35.2 (A)
- new net: D33.1 (K), D34.2 (A)
- new net: D39.1 (K), D40.2 (A)
- new net: D37.1 (K), D38.2 (A)
- new net: D10.1 (K), D37.2 (A)
- new net: D35.1 (K), D36.2 (A)
- new net: D18.1 (K), D19.2 (A)
- new net: D42.1 (K), D43.2 (A)
- new net: D44.1 (K), D45.2 (A)
- new net: D43.1 (K), D44.2 (A)
- new net: D27.1 (K), D28.2 (A)
- new net: D31.1 (K), D32.2 (A)

Commit message: Schematic
Found resistor values (used 70-80% of max current draw for LED's)
Parts:
- R1, R2, R3, R4: value 220 -> 60
- R10, R7, R8, R9: value 220 -> 100
- R11, R5, R6: value 220 -> 80
Other:
- moved on the sheet: D1, D10, D11, D16, D2, D20, D25, D29, D3, D33, D37, D38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

Commit message: Documentation,  symbol fields, connector changes
Parts:
- D1, D10, D2, D3, D37, D38, D4, D5, D6, D7, D8, D9: Digi URL (none) -> https://www.digikey.com/en/products/detail/w%C3%BCrth-elekt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
- D11, D12, D13, D16, D17, D18, D19, D20, D39, D40, D41: Digi URL (none) -> https://www.digikey.com/en/products/detail/quelighting-corp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
- D14: Digi URL (none) -> https://www.digikey.com/en/products/detail/quelighting-corp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; MFG (none) -> (none)
- D25, D26, D27, D28, D29, D30, D31, D32, D33, D34, D35, D36, D42, D43, D44, D45: Digi URL (none) -> https://www.digikey.com/en/products/detail/ams-osram-ag/LA-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
- J1: footprint Connector_Molex:Molex_Micro-Fit_3.0_43650-0610_1x06-1MP_P3.00mm_Horizontal -> formula_slug_footprint_library:1054301106
Other:
- added sheet rules (rules.kicad_sch)
- added sheet rules2 (rules2.kicad_sch)
- note added: "For amber LED resistors: 2.15V * 4 = 8.6V 12V - 8.6V = 3.4V Also has a max current draw of 50 mA. 3.4V/0.034 amps = 100 ohms I used 0.034 amps instead of 0.04 to get a standard resistor value"
- note added: "For red LED resistors: 2.2V * 4 = 8.8V 12V - 8.8V = 3.2V Also has a max current draw of 50 mA. 3.2V / 0.04 amps = 80 ohms"
- note added: "Green LED resistor value calculations: LED forward voltage = 3.2V 3.2 * 3 = 9.6V (3 in series) Using Ohm's law, 12-9.6V = 2.4V The LED's max current draw is 50 mA. Using 80% (for longevity): 2.4V / 0.04 amps = 60 ohms"

Commit message: added 3d models
Parts:
- D11, D12, D13, D14, D16, D17, D18, D19, D20, D39, D40, D41: footprint LED_SMD:LED_Everlight-SMD3528_3.5x2.8mm_67-21ST -> LED_SMD:LED_Avago_PLCC4_3.2x2.8mm_CW
Changed lines of the file:
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@@
 			)
 		)
-		(property "Footprint" "LED_SMD:LED_Everlight-SMD3528_3.5x2.8mm_67-21ST"
+		(property "Footprint" "LED_SMD:LED_Avago_PLCC4_3.2x2.8mm_CW"
 			(at 133.35 109.22 0)
 			(hide yes)
@@
 			)
 		)
-		(property "Footprint" "LED_SMD:LED_Everlight-SMD3528_3.5x2.8mm_67-21ST"
+		(property "Footprint" "LED_SMD:LED_Avago_PLCC4_3.2x2.8mm_CW"
 			(at 96.52 95.25 0)
 			(hide yes)
@@
 			)
 		)
-		(property "Footprint" "LED_SMD:LED_Everlight-SMD3528_3.5x2.8mm_67-21ST"
+		(property "Footprint" "LED_SMD:LED_Avago_PLCC4_3.2x2.8mm_CW"
 			(at 120.65 109.22 0)
 			(hide yes)
@@
 			)
 		)
-		(property "Footprint" "LED_SMD:LED_Everlight-SMD3528_3.5x2.8mm_67-21ST"
+		(property "Footprint" "LED_SMD:LED_Avago_PLCC4_3.2x2.8mm_CW"
 			(at 107.95 95.25 0)
 			(hide yes)
@@
 			)
 		)
-		(property "Footprint" "LED_SMD:LED_Everlight-SMD3528_3.5x2.8mm_67-21ST"
+		(property "Footprint" "LED_SMD:LED_Avago_PLCC4_3.2x2.8mm_CW"
 			(at 107.95 81.28 0)
 			(hide yes)
@@
 			)
 		)
-		(property "Footprint" "LED_SMD:LED_Everlight-SMD3528_3.5x2.8mm_67-21ST"
+		(property "Footprint" "LED_SMD:LED_Avago_PLCC4_3.2x2.8mm_CW"
 			(at 133.35 95.25 0)
 			(hide yes)
@@
 			)
 		)
-		(property "Footprint" "LED_SMD:LED_Everlight-SMD3528_3.5x2.8mm_67-21ST"
+		(property "Footprint" "LED_SMD:LED_Avago_PLCC4_3.2x2.8mm_CW"
 			(at 133.35 81.28 0)
 			(hide yes)
@@
 			)
 		)
-		(property "Footprint" "LED_SMD:LED_Everlight-SMD3528_3.5x2.8mm_67-21ST"
+		(property "Footprint" "LED_SMD:LED_Avago_PLCC4_3.2x2.8mm_CW"
 			(at 96.52 81.28 0)
 			(hide yes)
@@
 			)
 		)
-		(property "Footprint" "LED_SMD:LED_Everlight-SMD3528_3.5x2.8mm_67-21ST"
+		(property "Footprint" "LED_SMD:LED_Avago_PLCC4_3.2x2.8mm_CW"
 			(at 120.65 81.28 0)
 			(hide yes)
@@
 			)
 		)
-		(property "Footprint" "LED_SMD:LED_Everlight-SMD3528_3.5x2.8mm_67-21ST"
+		(property "Footprint" "LED_SMD:LED_Avago_PLCC4_3.2x2.8mm_CW"
 			(at 120.65 95.25 0)
 			(hide yes)
@@
 			)
 		)
-		(property "Footprint" "LED_SMD:LED_Everlight-SMD3528_3.5x2.8mm_67-21ST"
+		(property "Footprint" "LED_SMD:LED_Avago_PLCC4_3.2x2.8mm_CW"
 			(at 107.95 109.22 0)
 			(hide yes)
@@
 			)
 		)
-		(property "Footprint" "LED_SMD:LED_Everlight-SMD3528_3.5x2.8mm_67-21ST"
+		(property "Footprint" "LED_SMD:LED_Avago_PLCC4_3.2x2.8mm_CW"
 			(at 96.52 109.22 0)
 			(hide yes)

Commit message: Changed shape
Parts:
- removed D10, D14, D19, D20, D37, D38, D39, D40, D41, D7, D8, D9: LED, LED_SMD:LED_Avago_PLCC4_3.2x2.8mm_CW, symbol Device:LED
- removed R11: 80, Resistor_SMD:R_0603_1608Metric_Pad0.98x0.95mm_HandSolder, symbol Device:R
- removed R3, R4: 60, Resistor_SMD:R_0603_1608Metric_Pad0.98x0.95mm_HandSolder, symbol Device:R
- R5, R6: value 80 -> 150
- renumbered D16 to D14, D17 to D15, D18 to D16
Connections:
- net TSSI_RED_Cathode: now also D13.1 (K), D16.1 (K)
Other:
- note added: "For amber LED resistors: 2.15V * 4 = 8.6V 12V - 8.6V = 3.4V Also has a max current draw of 50 mA. 3.4V/0.034 amps = 100 ohms"
- note added: "For red LED resistors: 2.2V * 3 = 6.6 12V - 6.6V = 5.4V Also has a max current draw of 50 mA. 5.4V / 0.036 amps = 150 ohms"
- note added: "Green LED resistor value calculations: LED forward voltage = 3.2V 3.2 * 3 = 9.6V (3 in series) Using Ohm's law, 12-9.6V = 2.4V The LED's max current draw is 50 mA. 2.4V / 0.04 amps = 60 ohms"
- note removed: "For amber LED resistors: 2.15V * 4 = 8.6V 12V - 8.6V = 3.4V Also has a max current draw of 50 mA. 3.4V/0.034 amps = 100 ohms I used 0.034 amps instead of 0.04 to get a standard resistor value"
- note removed: "For red LED resistors: 2.2V * 4 = 8.8V 12V - 8.8V = 3.2V Also has a max current draw of 50 mA. 3.2V / 0.04 amps = 80 ohms"
- note removed: "Green LED resistor value calculations: LED forward voltage = 3.2V 3.2 * 3 = 9.6V (3 in series) Using Ohm's law, 12-9.6V = 2.4V The LED's max current draw is 50 mA. Using 80% (for longevity): 2.4V / 0.04 amps = 60 ohms"
- moved on the sheet: D11, D12, D13, D14, D15, D16, D25, D26, D27, D28, D29, D30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

Commit message: readded 3d models
Parts:
- D1, D11, D12, D13, D14, D15, D16, D2, D25, D26, D27, D28, D29, D3, D30, D31, D32, D33, D34, D35, D36, D4, D42, D43, D44, D45, D5, D6: footprint LED_SMD:LED_Avago_PLCC4_3.2x2.8mm_CW -> LED_SMD:LED_Avago_PLCC4_3.2x2.8mm_CW_3DMODEL
Changed lines of the file:
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@@
 			)
 		)
-		(property "Footprint" "LED_SMD:LED_Avago_PLCC4_3.2x2.8mm_CW"
+		(property "Footprint" "LED_SMD:LED_Avago_PLCC4_3.2x2.8mm_CW_3DMODEL"
 			(at 113.03 40.64 0)
 			(hide yes)
@@
 			)
 		)
-		(property "Footprint" "LED_SMD:LED_Avago_PLCC4_3.2x2.8mm_CW"
+		(property "Footprint" "LED_SMD:LED_Avago_PLCC4_3.2x2.8mm_CW_3DMODEL"
 			(at 96.52 71.12 0)
 			(hide yes)
@@
 			)
 		)
-		(property "Footprint" "LED_SMD:LED_Avago_PLCC4_3.2x2.8mm_CW"
+		(property "Footprint" "LED_SMD:LED_Avago_PLCC4_3.2x2.8mm_CW_3DMODEL"
 			(at 107.95 116.84 0)
 			(hide yes)
@@
 			)
 		)
-		(property "Footprint" "LED_SMD:LED_Avago_PLCC4_3.2x2.8mm_CW"
+		(property "Footprint" "LED_SMD:LED_Avago_PLCC4_3.2x2.8mm_CW_3DMODEL"
 			(at 107.95 129.54 0)
 			(hide yes)
@@
 			)
 		)
-		(property "Footprint" "LED_SMD:LED_Avago_PLCC4_3.2x2.8mm_CW"
+		(property "Footprint" "LED_SMD:LED_Avago_PLCC4_3.2x2.8mm_CW_3DMODEL"
 			(at 97.79 40.64 0)
 			(hide yes)
@@
 			)
 		)
-		(property "Footprint" "LED_SMD:LED_Avago_PLCC4_3.2x2.8mm_CW"
+		(property "Footprint" "LED_SMD:LED_Avago_PLCC4_3.2x2.8mm_CW_3DMODEL"
 			(at 130.81 27.94 0)
 			(hide yes)
@@
 			)
 		)
-		(property "Footprint" "LED_SMD:LED_Avago_PLCC4_3.2x2.8mm_CW"
+		(property "Footprint" "LED_SMD:LED_Avago_PLCC4_3.2x2.8mm_CW_3DMODEL"
 			(at 107.95 71.12 0)
 			(hide yes)
@@
 			)
 		)
-		(property "Footprint" "LED_SMD:LED_Avago_PLCC4_3.2x2.8mm_CW"
+		(property "Footprint" "LED_SMD:LED_Avago_PLCC4_3.2x2.8mm_CW_3DMODEL"
 			(at 107.95 57.15 0)
 			(hide yes)
@@
 			)
 		)
-		(property "Footprint" "LED_SMD:LED_Avago_PLCC4_3.2x2.8mm_CW"
+		(property "Footprint" "LED_SMD:LED_Avago_PLCC4_3.2x2.8mm_CW_3DMODEL"
 			(at 120.65 129.54 0)
 			(hide yes)
@@
 			)
 		)
-		(property "Footprint" "LED_SMD:LED_Avago_PLCC4_3.2x2.8mm_CW"
+		(property "Footprint" "LED_SMD:LED_Avago_PLCC4_3.2x2.8mm_CW_3DMODEL"
 			(at 96.52 91.44 0)
 			(hide yes)
@@
 			)
 		)
-		(property "Footprint" "LED_SMD:LED_Avago_PLCC4_3.2x2.8mm_CW"
+		(property "Footprint" "LED_SMD:LED_Avago_PLCC4_3.2x2.8mm_CW_3DMODEL"
 			(at 113.03 27.94 0)
 			(hide yes)
@@
 			)
 		)
-		(property "Footprint" "LED_SMD:LED_Avago_PLCC4_3.2x2.8mm_CW"
+		(property "Footprint" "LED_SMD:LED_Avago_PLCC4_3.2x2.8mm_CW_3DMODEL"
 			(at 107.95 104.14 0)
 			(hide yes)
@@
 			)
 		)
-		(property "Footprint" "LED_SMD:LED_Avago_PLCC4_3.2x2.8mm_CW"
+		(property "Footprint" "LED_SMD:LED_Avago_PLCC4_3.2x2.8mm_CW_3DMODEL"
 			(at 96.52 104.14 0)
 			(hide yes)
@@
 			)
 		)
-		(property "Footprint" "LED_SMD:LED_Avago_PLCC4_3.2x2.8mm_CW"
+		(property "Footprint" "LED_SMD:LED_Avago_PLCC4_3.2x2.8mm_CW_3DMODEL"
 			(at 96.52 129.54 0)
 			(hide yes)
@@
 			)
 		)
-		(property "Footprint" "LED_SMD:LED_Avago_PLCC4_3.2x2.8mm_CW"
+		(property "Footprint" "LED_SMD:LED_Avago_PLCC4_3.2x2.8mm_CW_3DMODEL"
 			(at 120.65 91.44 0)
 			(hide yes)
@@
 			)
 		)
-		(property "Footprint" "LED_SMD:LED_Avago_PLCC4_3.2x2.8mm_CW"
+		(property "Footprint" "LED_SMD:LED_Avago_PLCC4_3.2x2.8mm_CW_3DMODEL"
 			(at 96.52 57.15 0)
 			(hide yes)
@@
 			)
 		)
-		(property "Footprint" "LED_SMD:LED_Avago_PLCC4_3.2x2.8mm_CW"
+		(property "Footprint" "LED_SMD:LED_Avago_PLCC4_3.2x2.8mm_CW_3DMODEL"
 			(at 134.62 104.14 0)
 			(hide yes)
@@
 			)
 		)
-		(property "Footprint" "LED_SMD:LED_Avago_PLCC4_3.2x2.8mm_CW"
+		(property "Footprint" "LED_SMD:LED_Avago_PLCC4_3.2x2.8mm_CW_3DMODEL"
 			(at 129.54 40.64 0)
 			(hide yes)
@@
 			)
 		)
-		(property "Footprint" "LED_SMD:LED_Avago_PLCC4_3.2x2.8mm_CW"
+		(property "Footprint" "LED_SMD:LED_Avago_PLCC4_3.2x2.8mm_CW_3DMODEL"
 			(at 134.62 129.54 0)
 			(hide yes)
@@
 			)
 		)
-		(property "Footprint" "LED_SMD:LED_Avago_PLCC4_3.2x2.8mm_CW"
+		(property "Footprint" "LED_SMD:LED_Avago_PLCC4_3.2x2.8mm_CW_3DMODEL"
 			(at 120.65 57.15 0)
 			(hide yes)
@@
 			)
 		)
-		(property "Footprint" "LED_SMD:LED_Avago_PLCC4_3.2x2.8mm_CW"
+		(property "Footprint" "LED_SMD:LED_Avago_PLCC4_3.2x2.8mm_CW_3DMODEL"
 			(at 120.65 116.84 0)
 			(hide yes)
@@
 			)
 		)
-		(property "Footprint" "LED_SMD:LED_Avago_PLCC4_3.2x2.8mm_CW"
+		(property "Footprint" "LED_SMD:LED_Avago_PLCC4_3.2x2.8mm_CW_3DMODEL"
 			(at 134.62 116.84 0)
 			(hide yes)
@@
 			)
 		)
-		(property "Footprint" "LED_SMD:LED_Avago_PLCC4_3.2x2.8mm_CW"
+		(property "Footprint" "LED_SMD:LED_Avago_PLCC4_3.2x2.8mm_CW_3DMODEL"
 			(at 120.65 71.12 0)
 			(hide yes)
@@
 			)
 		)
-		(property "Footprint" "LED_SMD:LED_Avago_PLCC4_3.2x2.8mm_CW"
+		(property "Footprint" "LED_SMD:LED_Avago_PLCC4_3.2x2.8mm_CW_3DMODEL"
 			(at 134.62 91.44 0)
 			(hide yes)
@@
 			)
 		)
-		(property "Footprint" "LED_SMD:LED_Avago_PLCC4_3.2x2.8mm_CW"
+		(property "Footprint" "LED_SMD:LED_Avago_PLCC4_3.2x2.8mm_CW_3DMODEL"
 			(at 96.52 116.84 0)
 			(hide yes)
@@
 			)
 		)
-		(property "Footprint" "LED_SMD:LED_Avago_PLCC4_3.2x2.8mm_CW"
+		(property "Footprint" "LED_SMD:LED_Avago_PLCC4_3.2x2.8mm_CW_3DMODEL"
 			(at 97.79 27.94 0)
 			(hide yes)
@@
 			)
 		)
+		(property "Digikey Part Number" ""
+			(at 97.79 27.94 0)
+			(hide yes)
+			(show_name no)
+			(do_not_autoplace no)
+			(effects
+				(font
+					(size 1.27 1.27)
+				)
+			)
+		)
+		(property "Digikey URL" ""
+			(at 97.79 27.94 0)
+			(hide yes)
+			(show_name no)
+			(do_not_autoplace no)
+			(effects
+				(font
+					(size 1.27 1.27)
+				)
+			)
+		)
+		(property "Manufacturer" ""
+			(at 97.79 27.94 0)
+			(hide yes)
+			(show_name no)
+			(do_not_autoplace no)
+			(effects
+				(font
+					(size 1.27 1.27)
+				)
+			)
+		)
+		(property "Manufacturer Part Number" ""
+			(at 97.79 27.94 0)
+			(hide yes)
+			(show_name no)
+			(do_not_autoplace no)
+			(effects
+				(font
+					(size 1.27 1.27)
+				)
+			)
+		)
 		(pin "2"
 		)
@@
 			)
 		)
-		(property "Footprint" "LED_SMD:LED_Avago_PLCC4_3.2x2.8mm_CW"
+		(property "Footprint" "LED_SMD:LED_Avago_PLCC4_3.2x2.8mm_CW_3DMODEL"
 			(at 120.65 104.14 0)
 			(hide yes)
@@
 			)
 		)
-		(property "Footprint" "LED_SMD:LED_Avago_PLCC4_3.2x2.8mm_CW"
+		(property "Footprint" "LED_SMD:LED_Avago_PLCC4_3.2x2.8mm_CW_3DMODEL"
 			(at 107.95 91.44 0)
 			(hide yes)
