File: tractive-system-status-indicator/rules.kicad_sch (KiCad schematic)
At the start: 0 parts

Commit message: fields
Other:
- note added: "EV.6.1.5 A: Minimum height and width is satisfied (see PCB editor) - Green & Red: 19.304x10.414mm - Amber: 39.116x17.272 mm C: Distance - Green to Red: 7.712 mm - Green & Red to Amber: 7.874 mm D: Center - All LED's smallest illuminated dimension is 2.40mm in diameter - All LED distance is 7.112mm E: Visibility - Each LED's brightness is sufficient to visible in direct sunlight - Green: 5000 mcd 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"
- note removed: "EV.6.1.5 A: Minimum height and width is satisfied (see PCB editor) - Green & Red: 26.416x17.272 mm - Amber: 39.116x17.272 mm C: Distance - Green to Red: 6.604mm - Green & Red to Amber: 6.35mm D: Center - All LED's smallest illuminated dimension is 2.40mm in diameter - All LED distance is 7.112mm E: Visibility - Each LED's brightness is sufficient to visible in direct sunlight - Green: 5000 mcd - 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"
Changed lines of the file:
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@@
 	(generator_version "10.0")
 	(paper "A4")
-	(text "EV.6.1.5\nA: Minimum height and width is satisfied (see PCB editor)\n	- Green & Red: 26.416x17.272 mm\n	- Amber: 39.116x17.272 mm\nC: Distance\n	- Green to Red: 6.604mm\n	- Green & Red to Amber: 6.35mm\nD: Center \n	- All LED's smallest illuminated dimension is 2.40mm in diameter\n	- All LED distance is 7.112mm\nE: Visibility\n	- Each LED's brightness is sufficient to visible in direct sunlight\n	- Green: 5000 mcd\n	- Red: 2750 mcd\n	- Amber: 3370 mcd\n	- The brightness differes, but it doesn't matter because only LED will be on at a time."
+	(text "EV.6.1.5\nA: Minimum height and width is satisfied (see PCB editor)\n	- Green & Red: 19.304x10.414mm\n	- Amber: 39.116x17.272 mm\nC: Distance\n	- Green to Red: 7.712 mm\n	- Green & Red to Amber: 7.874 mm\nD: Center \n	- All LED's smallest illuminated dimension is 2.40mm in diameter\n	- All LED distance is 7.112mm\nE: Visibility\n	- Each LED's brightness is sufficient to visible in direct sunlight\n	- Green: 5000 mcd\n	- Red: 2750 mcd\n	- Amber: 4450 mcd\n	- The brightness differes, but it doesn't matter because only LED will be on at a time."
 		(exclude_from_sim no)
 		(at 21.59 133.604 0)
