File: telemetry-logging-board/_restore_backup_2026-09-03T20-03-23-319/can-if-trx.kicad_sch (KiCad schematic)
At the start: 23 parts, among them SW3 TERM, U11 CRE1S0505SC, U12 ISO1044BD, U7 MCP2518FD-xQBB, Y3 ECS-200-12-33Q-JES-TR

Commit message: finish ethernet, power supply arch, some other things
Parts:
- removed JP1, JP4: ISO, symbol Jumper:SolderJumper_2_Open
- added GD2: GDT_2Pin, symbol Device:GDT_2Pin
- added R35, R36: 0R, symbol Device:R_Small
Connections:
- net GND: now also GD2.3, R36.1
- net ISO_0V: now also GD2.1, R36.2
- net ISO_5V: now also R35.2
- net VDD_CAN: now also R35.1
Other:
- note added: "Arrests strong common mode events"
- note added: "Resistors depopulated for isolation must be large footprint! Per IEC 60664-1 Table F.2: 2.5kv : 1.5mm 4kv : 3.0mm 6kv : 5.5mm R1206 : 1.8mm gap"
