File: telemetry-logging-board/_restore_backup_2026-09-03T20-03-23-319/m12x_tr.kicad_sch (KiCad schematic)
At the start: 12 parts, among them J14 M12-X

Commit message: finish ethernet, power supply arch, some other things
Parts:
- removed D10, D7: LED, symbol Device:LED
- removed R93, R94: R_Small, symbol Device:R_Small
