File: telemetry-logging-board/_restore_backup_2026-09-03T20-03-23-319/telemetry-logging-board.kicad_sch (KiCad schematic)
At the start: 8 parts, among them J12 Wifi, J13 ESP, J5 USB_C_Receptacle_USB2.0_16P, J8 Micro_SD_Card, U1 ESP32-S3-MINI-1U, U6 USBLC6-2SC6

Commit message: finish ethernet, power supply arch, some other things
Connections:
- net +3V3 renamed +3.3V
Other:
- sheet CAN Busses ports: added none; removed INT_A, INT_B, INT_C
