File: vehicle-control-unit/IMU.kicad_sch (KiCad schematic)
At the start: 11 parts, among them U28 BME688, U29 BNO086

Commit message: vcu changes progess
-new mcu added and pairing progess
-grounding clips added
-changed schematic symbols to fs_components library
Parts:
- U28: footprint FS_4_Global_Footprint_Library:BME_688_Bosch_LGA-8_3x3mm_P0.8mm_ClockwisePinNumbering -> formula_slug_footprint_library:BME_688_Bosch_LGA-8_3x3mm_P0.8mm_ClockwisePinNumbering
- U29: footprint FS_4_Global_Footprint_Library:BNO086_LGA-28_5.2x3.8mm_P0.5mm -> formula_slug_footprint_library:BNO086_LGA-28_5.2x3.8mm_P0.5mm
Changed lines of the file:
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@@
 			)
 		)
-		(property "Footprint" "FS_4_Global_Footprint_Library:BNO086_LGA-28_5.2x3.8mm_P0.5mm"
+		(property "Footprint" "formula_slug_footprint_library:BNO086_LGA-28_5.2x3.8mm_P0.5mm"
 			(at 189.23 104.14 0)
 			(hide yes)
@@
 		)
 		(property "Sim.Device" ""
+			(at 214.63 119.38 0)
+			(hide yes)
+			(show_name no)
+			(do_not_autoplace no)
+			(effects
+				(font
+					(size 1.27 1.27)
+				)
+			)
+		)
+		(property "Digikey Part Number" ""
+			(at 214.63 119.38 0)
+			(hide yes)
+			(show_name no)
+			(do_not_autoplace no)
+			(effects
+				(font
+					(size 1.27 1.27)
+				)
+			)
+		)
+		(property "Digikey URL" ""
+			(at 214.63 119.38 0)
+			(hide yes)
+			(show_name no)
+			(do_not_autoplace no)
+			(effects
+				(font
+					(size 1.27 1.27)
+				)
+			)
+		)
+		(property "Manufacturer Part Number" ""
 			(at 214.63 119.38 0)
 			(hide yes)
@@
 			)
 		)
-		(property "Footprint" "FS_4_Global_Footprint_Library:BME_688_Bosch_LGA-8_3x3mm_P0.8mm_ClockwisePinNumbering"
+		(property "Footprint" "formula_slug_footprint_library:BME_688_Bosch_LGA-8_3x3mm_P0.8mm_ClockwisePinNumbering"
 			(at 205.74 177.8 0)
 			(hide yes)
@@
 			(at 205.74 177.8 0)
 			(hide yes)
+			(show_name no)
+			(do_not_autoplace no)
+			(effects
+				(font
+					(size 1.27 1.27)
+				)
+			)
+		)
+		(property "Digikey Part Number" ""
+			(at 205.74 177.8 0)
+			(hide yes)
+			(show_name no)
+			(do_not_autoplace no)
+			(effects
+				(font
+					(size 1.27 1.27)
+				)
+			)
+		)
+		(property "Digikey URL" ""
+			(at 205.74 177.8 0)
+			(hide yes)
+			(show_name no)
+			(do_not_autoplace no)
+			(effects
+				(font
+					(size 1.27 1.27)
+				)
+			)
+		)
+		(property "Manufacturer Part Number" ""
+			(at 205.74 177.8 0)
+			(hide yes)
