File: vehicle-control-unit/vehicle-control-unit.kicad_sch (KiCad schematic)
At the start: 0 parts

Commit message: Copied VCU and added TSSI changes
Parts:
- added C1: 10uF 0805, Capacitor_SMD:C_0805_2012Metric_Pad1.18x1.45mm_HandSolder, symbol Device:C
- added C2, C4: 1uF, Capacitor_SMD:C_0603_1608Metric_Pad1.08x0.95mm_HandSolder, symbol Device:C
- added C3: 0.1uF, Capacitor_SMD:C_0603_1608Metric_Pad1.08x0.95mm_HandSolder, symbol Device:C
- added C5: 47uF, Capacitor_SMD:C_0805_2012Metric_Pad1.18x1.45mm_HandSolder, symbol Device:C
- added H1, H2, H3, H4: MountingHole_Pad, MountingHole:MountingHole_3.2mm_M3_Pad, symbol Mechanical:MountingHole_Pad
- added J1: ATS13-34PB2-BM01, FS_4_Global_Footprint_Library:ATS13-34PB2-BM01, symbol Connector_Generic:Conn_01x34
- added J2: SS-60400-023, FS_4_Global_Footprint_Library:SS-60400-023, symbol Connector_Generic_Shielded:Conn_01x08_Shielded
- added J3: ATS13-34PA2-BM01, FS_4_Global_Footprint_Library:ATS13-34PA2-BM01, symbol Connector_Generic:Conn_01x34
- added L1: 4.7uH, Inductor_SMD:L_Bourns_SRP5030T, symbol Device:L
- added U1: AP63205WU, Package_TO_SOT_SMD:TSOT-23-6, symbol Regulator_Switching:AP63205WU
- added U2: MIC5504-3.3YM5, Package_TO_SOT_SMD:SOT-23-5, symbol Regulator_Linear:MIC5504-3.3YM5
Connections:
- new net: C3.2, L1.1, U1.5 (SW)
- new net: C3.1, U1.6 (BST)
- new net +12V: C1.2, J1.24 (Pin_24), J1.25 (Pin_25), J1.9 (Pin_9), J2.7 (Pin_7), U1.2 (EN), U1.3 (IN)
- new net +3V3: C4.2, U2.5 (VOUT)
- new net +5V: C2.2, C5.2, J3.10 (Pin_10), J3.11 (Pin_11), J3.12 (Pin_12), J3.13 (Pin_13), J3.27 (Pin_27), L1.2, U1.1 (FB), U2.1 (VIN), U2.3 (EN)
- new net APPS_1_Raw: J3.1 (Pin_1)
- new net APPS_2_Raw: J3.2 (Pin_2)
- new net BMS_LED_Anode: J3.14 (Pin_14)
- new net BMS_LED_Cathode: J3.5 (Pin_5)
- new net BOTS_Neg: J3.31 (Pin_31)
- new net BOTS_Pos: J3.29 (Pin_29)
- new net BPPS_1_Raw: J3.3 (Pin_3)
- new net BSPD_LED_Anode: J3.16 (Pin_16)
- new net BSPD_LED_Cathode: J3.7 (Pin_7)
- new net BSPD_Shutdown_Out: J1.19 (Pin_19)
- new net Brake_LED_Anode: J1.20 (Pin_20)
- new net Brake_LED_Cathode: J1.12 (Pin_12)
- new net CAN_Data_H: J1.18 (Pin_18), J2.2 (Pin_2)
- new net CAN_Data_L: J1.26 (Pin_26), J2.1 (Pin_1)
- new net CAN_Powertrain_H: J1.1 (Pin_1)
- new net CAN_Powertrain_L: J1.10 (Pin_10)
- new net Current_Analog_Raw: J1.7 (Pin_7)
- new net Current_Vref_Raw: J1.8 (Pin_8)
- new net Dash_Lap: J2.4 (Pin_4)
- new net Dash_Launch: J2.3 (Pin_3)
- new net Driverless_Signal: J1.14 (Pin_14)
- new net E_Stop_Neg: J3.22 (Pin_22)
- new net E_Stop_Pos: J3.30 (Pin_30)
- new net Front_Brake_Raw: J1.16 (Pin_16)
- new net GND: C1.1, C2.1, C4.1, C5.1, H1.1, H2.1, H3.1, H4.1, J1.17 (Pin_17), J1.33 (Pin_33), J1.34 (Pin_34), J2.8 (Pin_8), J2.SH (Shield), J3.18 (Pin_18), J3.19 (Pin_19), J3.20 (Pin_20), J3.21 (Pin_21), J3.28 (Pin_28), U1.4 (GND), U2.2 (GND)
- new net IMD_LED_Anode: J3.15 (Pin_15)
- new net IMD_LED_Cathode: J3.6 (Pin_6)
- new net Inertia_Neg: J3.24 (Pin_24)
- new net Inertia_Pos: J3.23 (Pin_23)
- new net MCU/SPS_1_Raw: J3.26 (Pin_26)
- new net MCU/Solenoid_Neg: J3.33 (Pin_33)
- new net RTD_Button_Neg: J3.8 (Pin_8)
- new net RTD_Button_Pos: J3.25 (Pin_25)
- new net RTD_Buzzer_Neg: J1.13 (Pin_13)
- new net RTD_Buzzer_Pos: J1.21 (Pin_21)
- new net RTD_LED_Anode: J3.17 (Pin_17)
- new net RTD_LED_Cathode: J3.9 (Pin_9)
- new net Rear_Brake_Raw: J1.15 (Pin_15)
- new net Reset_Button: J1.11 (Pin_11)
- new net Shutdown_In: J1.4 (Pin_4)
- new net Solenoid_12V: J3.34 (Pin_34)
- new net Status_Indicator_Strip: J3.4 (Pin_4)
- new net TSSI_GREEN_Anode: J1.32 (Pin_32)
- new net TSSI_GREEN_Cathode: J1.23 (Pin_23)
- new net TSSI_RED_Anode: J1.31 (Pin_31)
- new net TSSI_RED_Cathode: J1.22 (Pin_22)
- new net UART5_RX: J1.5 (Pin_5)
- new net UART5_TX: J1.6 (Pin_6)
- new net nBMS_Fault: J1.3 (Pin_3)
- new net nIMD_Fault: J1.2 (Pin_2)
- no-connect marks 0 -> 7
Other:
- added sheet MCU (MCU.kicad_sch)
- added sheet Shutdown_VCU (Shutdown_VCU.kicad_sch)
- note added: "APPS_1_5V"
- note added: "APPS_1_GND"
- note added: "APPS_2_5V"
- note added: "APPS_2_GND"
- note added: "BPPS_1_5V"
- note added: "BPPS_1_GND"
- note added: "Brake_Front_12V"
- note added: "Brake_Rear_12V"
- note added: "Brake_Rear_GND"
- note added: "Dash Board"
- note added: "Everything Else"
- note added: "External IMU UART"
- note added: "Front_Brake_GND"
- note added: "Power Supply"
- note added: "SIS_Bin/GND"
- note added: "SPS_1_5V"
- note added: "SPS_1_GND"
- note added: "Status_Indicator_Strip_5V"
- note added: "Steering Wheel PCB"
- note added: "Steering_Wheel_Power"

Commit message: progress on new mcu, ground clip added
Parts:
- added J6: 5019, CONN1_5019_KEY, symbol formula_slug_symbol_library:5019
Connections:
- net GND: now also J6.1
Changed lines of the file:
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@@
+	)
+	(symbol
+		(lib_id "formula_slug_symbol_library:5019")
+		(at 140.97 26.67 0)
+		(unit 1)
+		(body_style 1)
+		(exclude_from_sim no)
+		(in_bom yes)
+		(on_board yes)
+		(in_pos_files yes)
+		(dnp no)
+		(fields_autoplaced yes)
+		(property "Reference" "J6"
+			(at 154.94 25.3999 0)
+			(show_name no)
+			(do_not_autoplace no)
+			(effects
+				(font
+					(size 1.524 1.524)
+				)
+				(justify left)
+			)
+		)
+		(property "Value" "5019"
+			(at 154.94 27.9399 0)
+			(show_name no)
+			(do_not_autoplace no)
+			(effects
+				(font
+					(size 1.524 1.524)
+				)
+				(justify left)
+			)
+		)
+		(property "Footprint" "CONN1_5019_KEY"
+			(at 140.97 26.67 0)
+			(hide yes)
+			(show_name no)
+			(do_not_autoplace no)
+			(effects
+				(font
+					(size 1.27 1.27)
+					(italic yes)
+				)
+			)
+		)
+		(property "Datasheet" "5019"
+			(at 140.97 26.67 0)
+			(hide yes)
+			(show_name no)
+			(do_not_autoplace no)
+			(effects
+				(font
+					(size 1.27 1.27)
+					(italic yes)
+				)
+			)
+		)
+		(property "Description" ""
+			(at 140.97 26.67 0)
+			(hide yes)
+			(show_name no)
+			(do_not_autoplace no)
+			(effects
+				(font
+					(size 1.27 1.27)
+				)
+			)
+		)
+		(pin "1"
+		)
+		(instances
+			(project "vehicle-control-unit"
+				(path "/e994741c-7c7d-4124-9d00-43b883baa61d"
+					(reference "J6")
+					(unit 1)
+				)
+			)
+		)
 	)
 	(symbol
@@
 					(unit 1)
 				)
+			)
+		)
+	)
+	(symbol
+		(lib_id "power:GND")
+		(at 140.97 26.67 0)
+		(unit 1)
+		(body_style 1)
+		(exclude_from_sim no)
+		(in_bom yes)
+		(on_board yes)
+		(in_pos_files yes)
+		(dnp no)
+		(fields_autoplaced yes)
+		(property "Reference" "#PWR0216"
+			(at 140.97 33.02 0)
+			(hide yes)
+			(show_name no)
+			(do_not_autoplace no)
+			(effects
+				(font
+					(size 1.27 1.27)
+				)
+			)
+		)
+		(property "Value" "GND"
+			(at 140.97 31.75 0)
+			(show_name no)
+			(do_not_autoplace no)
+			(effects
+				(font
+					(size 1.27 1.27)
+				)
+			)
+		)
+		(property "Footprint" ""
+			(at 140.97 26.67 0)
+			(hide yes)
+			(show_name no)
+			(do_not_autoplace no)
+			(effects
+				(font
+					(size 1.27 1.27)
+				)
+			)
+		)
+		(property "Datasheet" ""
+			(at 140.97 26.67 0)
+			(hide yes)
+			(show_name no)
+			(do_not_autoplace no)
+			(effects
+				(font
+					(size 1.27 1.27)
+				)
+			)
+		)
+		(property "Description" "Power symbol creates a global label with name \"GND\" , ground"
+			(at 140.97 26.67 0)
+			(hide yes)
+			(show_name no)
+			(do_not_autoplace no)
+			(effects
+				(font
+					(size 1.27 1.27)
+				)
+			)
+		)
+		(pin "1"
+		)
+		(instances
+			(project "vehicle-control-unit"
+				(path "/e994741c-7c7d-4124-9d00-43b883baa61d"
+					(reference "#PWR0216")
+					(unit 1)
+				)

Commit message: Schematic changes
-STM32G473 mcu added
-sampling of shutdown nets
-test points to important nets
-debug led
Parts:
- J1: footprint FS_4_Global_Footprint_Library:ATS13-34PB2-BM01 -> formula_slug_footprint_library:ATS13-34PB2-BM01
- J3: footprint FS_4_Global_Footprint_Library:ATS13-34PA2-BM01 -> formula_slug_footprint_library:ATS13-34PB2-BM01
Changed lines of the file:
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@@
 			)
 		)
-		(property "Footprint" "FS_4_Global_Footprint_Library:ATS13-34PA2-BM01"
+		(property "Footprint" "formula_slug_footprint_library:ATS13-34PB2-BM01"
 			(at 345.44 133.35 0)
 			(hide yes)
@@
 		)
 		(property "Sim.Device" ""
+			(at 345.44 135.89 0)
+			(hide yes)
+			(show_name no)
+			(do_not_autoplace no)
+			(effects
+				(font
+					(size 1.27 1.27)
+				)
+			)
+		)
+		(property "Digikey Part Number" ""
+			(at 345.44 135.89 0)
+			(hide yes)
+			(show_name no)
+			(do_not_autoplace no)
+			(effects
+				(font
+					(size 1.27 1.27)
+				)
+			)
+		)
+		(property "Digikey URL" ""
+			(at 345.44 135.89 0)
+			(hide yes)
+			(show_name no)
+			(do_not_autoplace no)
+			(effects
+				(font
+					(size 1.27 1.27)
+				)
+			)
+		)
+		(property "Manufacturer Part Number" ""
 			(at 345.44 135.89 0)
 			(hide yes)
@@
 			)
 		)
-		(property "Footprint" "FS_4_Global_Footprint_Library:ATS13-34PB2-BM01"
+		(property "Footprint" "formula_slug_footprint_library:ATS13-34PB2-BM01"
 			(at 38.1 97.79 0)
 			(hide yes)
@@
 			(at 38.1 97.79 0)
 			(hide yes)
+			(show_name no)
+			(do_not_autoplace no)
+			(effects
+				(font
+					(size 1.27 1.27)
+				)
+			)
+		)
+		(property "Digikey Part Number" ""
+			(at 38.1 97.79 0)
+			(hide yes)
+			(show_name no)
+			(do_not_autoplace no)
+			(effects
+				(font
+					(size 1.27 1.27)
+				)
+			)
+		)
+		(property "Digikey URL" ""
+			(at 38.1 97.79 0)
+			(hide yes)
+			(show_name no)
+			(do_not_autoplace no)
+			(effects
+				(font
+					(size 1.27 1.27)
+				)
+			)
+		)
+		(property "Manufacturer Part Number" ""
+			(at 38.1 97.79 0)
+			(hide yes)
