File: vehicle-control-unit/Shutdown_LEDS.kicad_sch (KiCad schematic)
At the start: 72 parts, among them Q1 AO3400A, Q2 AO3400A, Q3 AO3400A, Q4 AO3400A, Q5 AO3400A, U10 SN74HCS08DR, U13 SN74HC14DR, U15 SN74HC14DR, U16 LM555CMX

Commit message: Schematic changes
-STM32G473 mcu added
-sampling of shutdown nets
-test points to important nets
-debug led
Parts:
- added TP10: Hard_Braking_High_Current, TestPoint:TestPoint_Pad_D1.0mm, symbol Connector:TestPoint
- added TP20: BSDP_Fault, TestPoint:TestPoint_Pad_D1.0mm, symbol Connector:TestPoint
Connections:
- net BSDP_Fault: now also TP20.1
- net Hard_Braking_High_Current: now also TP10.1

Commit message: added lamp check and removed imu pins
Parts:
- added C37: 100uF, Capacitor_SMD:C_0603_1608Metric_Pad1.08x0.95mm_HandSolder, symbol Device:C
- added Q11, Q6: AO3400A, Package_TO_SOT_SMD:SOT-23, symbol Transistor_FET:AO3400A
- added R71: 36k, Resistor_SMD:R_0603_1608Metric_Pad0.98x0.95mm_HandSolder, symbol Device:R
- added unit 1 of U13
Connections:
- net +5V: now also R71.1
- net GND: now also C37.1, Q11.2 (S), Q6.2 (S)
- net TSSI_GREEN_Cathode: now also Q6.3 (D)
- net TSSI_RED_Cathode: now also Q11.3 (D)
- new net: C37.2, R71.2, U13.1
- new net Lamp_Check: Q11.1 (G), Q6.1 (G), U13.2
Other:
- moved on the sheet: D14, D15, D16, D17
