File: vehicle-control-unit/Shutdown_VCU.kicad_sch (KiCad schematic)
At the start: 54 parts, among them K2 G6SK-2G, K3 G6DN-1A, SW1 61-6441.4047, SW2 A165E-S, SW3 Typ- 505, U10 SN74HCS08DR, U11 MCP6004, U12 SN74HCS32DR, U13 SN74HC14DR, U14 SZNUD3124DMT1G, U3 HASS-300S, U4 X05PSA02000P18, U5 X05PSA02000P18, U6 MCP6004, U7 MCP6004, U8 MCP6004, U9 SN74HCS32DR

Commit message: added pot to BSPD current threshold
Parts:
- added R93, R94: 10k, Resistor_SMD:R_0603_1608Metric_Pad0.98x0.95mm_HandSolder, symbol Device:R
- added RV4: 3296W_20K, Potentiometer_THT:Potentiometer_Bourns_3296W_Vertical, symbol Device:R_Potentiometer
Connections:
- net High_Current_Threshold: now also R93.1, R94.1, RV4.2; no longer R13.1, R14.2
- new net: R13.1, R93.2, RV4.1
- new net: R14.2, R94.2, RV4.3
Other:
- moved on the sheet: R1, R13, R14, R2, R3, R8, U6A, U6B

Commit message: added lamp check and removed imu pins
Parts:
- removed unit 1 of U13
Connections:
- no-connect marks 16 -> 14
Changed lines of the file:
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@@
 	)
 	(no_connect
-		(at 345.44 121.92)
-	)
-	(no_connect
 		(at 308.61 124.46)
 	)
 	(no_connect
-		(at 330.2 121.92)
-	)
-	(no_connect
 		(at 364.49 121.92)
 	)
@@
 				)
 			)
-		)
-	)
-	(symbol
-		(lib_id "74xx:74HC14")
-		(at 337.82 121.92 0)
-		(unit 1)
-		(body_style 1)
-		(exclude_from_sim no)
-		(in_bom yes)
-		(on_board yes)
-		(in_pos_files yes)
-		(dnp no)
-		(fields_autoplaced yes)
-		(property "Reference" "U13"
-			(at 337.82 113.03 0)
-			(show_name no)
-			(do_not_autoplace no)
-			(effects
-				(font
-					(size 1.27 1.27)
-				)
-			)
-		)
-		(property "Value" "SN74HC14DR"
-			(at 337.82 115.57 0)
-			(show_name no)
-			(do_not_autoplace no)
-			(effects
-				(font
-					(size 1.27 1.27)
-				)
-			)
-		)
-		(property "Footprint" "Package_SO:SOIC-14_3.9x8.7mm_P1.27mm"
-			(at 337.82 121.92 0)
-			(hide yes)
-			(show_name no)
-			(do_not_autoplace no)
-			(effects
-				(font
-					(size 1.27 1.27)
-				)
-			)
-		)
-		(property "Datasheet" "https://www.ti.com/lit/ds/symlink/sn74hc14.pdf"
-			(at 337.82 121.92 0)
-			(hide yes)
-			(show_name no)
-			(do_not_autoplace no)
-			(effects
-				(font
-					(size 1.27 1.27)
-				)
-			)
-		)
-		(property "Description" "Hex inverter schmitt trigger"
-			(at 337.82 121.92 0)
-			(hide yes)
-			(show_name no)
-			(do_not_autoplace no)
-			(effects
-				(font
-					(size 1.27 1.27)
-				)
-			)
-		)
-		(property "Digi PN" "296-1194-1-ND"
-			(at 337.82 121.92 0)
-			(hide yes)
-			(show_name no)
-			(do_not_autoplace no)
-			(effects
-				(font
-					(size 1.27 1.27)
-				)
-			)
-		)
-		(property "Digi URL" "https://www.digikey.com/en/products/detail/texas-instruments/SN74HC14DR/276837"
-			(at 337.82 121.92 0)
-			(hide yes)
-			(show_name no)
-			(do_not_autoplace no)
-			(effects
-				(font
-					(size 1.27 1.27)
-				)
-			)
-		)
-		(property "MFG" "TI"
-			(at 337.82 121.92 0)
-			(hide yes)
-			(show_name no)
-			(do_not_autoplace no)
-			(effects
-				(font
-					(size 1.27 1.27)
-				)
-			)
-		)
-		(property "MFG PN" "SN74HC14DR"
-			(at 337.82 121.92 0)
-			(hide yes)
-			(show_name no)
-			(do_not_autoplace no)
-			(effects
-				(font
-					(size 1.27 1.27)
-				)
-			)
-		)
-		(property "MANUFACTURER" ""
-			(at 337.82 121.92 0)
-			(hide yes)
-			(show_name no)
-			(do_not_autoplace no)
-			(effects
-				(font
-					(size 1.27 1.27)
-				)
-			)
-		)
-		(property "Sim.Type" ""
-			(at 337.82 121.92 0)
-			(hide yes)
-			(show_name no)
-			(do_not_autoplace no)
-			(effects
-				(font
-					(size 1.27 1.27)
-				)
-			)
-		)
-		(property "Digikey Link" ""
-			(at 337.82 121.92 0)
-			(hide yes)
-			(show_name no)
-			(do_not_autoplace no)
-			(effects
-				(font
-					(size 1.27 1.27)
-				)
-			)
-		)
-		(property "MFP PN" ""
-			(at 337.82 121.92 0)
-			(hide yes)
-			(show_name no)
-			(do_not_autoplace no)
-			(effects
-				(font
-					(size 1.27 1.27)
-				)
-			)
-		)
-		(property "Manufacturer" ""
-			(at 337.82 121.92 0)
-			(hide yes)
-			(show_name no)
-			(do_not_autoplace no)
-			(effects
-				(font
-					(size 1.27 1.27)
-				)
-			)
-		)
-		(property "Part Name" ""
-			(at 337.82 121.92 0)
-			(hide yes)
-			(show_name no)
-			(do_not_autoplace no)
-			(effects
-				(font
-					(size 1.27 1.27)
-				)
-			)
-		)
-		(property "Sim.Device" ""
-			(at 337.82 121.92 0)
-			(hide yes)
-			(show_name no)
-			(do_not_autoplace no)
-			(effects
-				(font
-					(size 1.27 1.27)
-				)
-			)
-		)
-		(pin "5"
-		)
-		(pin "1"
-		)
-		(pin "11"
-		)
-		(pin "10"
-		)
-		(pin "8"
-		)
-		(pin "13"
-		)
-		(pin "12"
-		)
-		(pin "14"
-		)
-		(pin "7"
-		)
-		(pin "3"
-		)
-		(pin "4"
-		)
-		(pin "2"
-		)
-		(pin "9"
-		)
-		(pin "6"
-		)
-		(instances
-			(project "vehicle-control-unit"
-				(path "/e994741c-7c7d-4124-9d00-43b883baa61d/ea6a280a-2379-492f-a1be-47be4daa3461"
-					(reference "U13")
-					(unit 1)
-				)
-			)
