File: temp-sense_bms-board/BMS.kicad_sch (KiCad schematic)
At the start: 40 parts, among them J1 84952-5, J2 84952-5, J3 1053131202, J4 512810598, J5 1053131202, J6 1053131202, J7 1053131202, Q1 NSV1C201MZ4, SW1 SW_DIP_x04, U17 LTC6810IG-2-TRPBF

Commit message: first layout
Placed all temp & humidity sensors. Placed all bms components. Unsure if LV/HV isolation is proper, so will review in future. Will also review traces cuz they're lowk hella jank.
Parts:
- J1, J2: footprint FS_4_Global_Footprint_Library:849525 -> Connector_FFC-FPC:TE_84952-5_1x05-1MP_P1.0mm_Horizontal
- L1: footprint FS_4_Global_Footprint_Library:HM2113ZNLT -> FS_4_Global_Footprint_Libary:HM2113ZNLT
- SW1: footprint FS_4_Global_Footprint_Library:SW_A6H-4101_OMR -> FS_4_Global_Footprint_Libary:SW_A6H-4101_OMR

Commit message: Added water drop sensors
Added pads for sensors and added PCF8574T I/O expander IC
Parts:
- J1: footprint Connector_FFC-FPC:TE_84952-5_1x05-1MP_P1.0mm_Horizontal -> FS_4_Global_Footprint_Library:849525
- J3, J5, J6, J7: footprint FS_4_Global_Footprint_Library:Nano-Fit_1054301102 -> FS_4_Global_Footprint_Libary:CONN_SD-105430-001_02_MOL
- renumbered U17 to U29
Changed lines of the file:
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@@
 		(dnp no)
 		(fields_autoplaced yes)
-		(property "Reference" "U17"
+		(property "Reference" "U29"
 			(at 166.37 66.04 0)
 			(show_name no)
@@
 			(project "temp-sense_bms-board"
 				(path "/2578a7cf-fb3a-4f93-9944-b46c757ff050/9f846a03-efdf-4167-b509-f0c25752b18e"
-					(reference "U17")
+					(reference "U29")
 					(unit 1)
 				)
@@
 			)
 		)
-		(property "Footprint" "FS_4_Global_Footprint_Library:Nano-Fit_1054301102"
+		(property "Footprint" "FS_4_Global_Footprint_Libary:CONN_SD-105430-001_02_MOL"
 			(at 318.77 102.87 0)
 			(hide yes)
@@
 			)
 		)
-		(property "Footprint" "Connector_FFC-FPC:TE_84952-5_1x05-1MP_P1.0mm_Horizontal"
+		(property "Footprint" "FS_4_Global_Footprint_Library:849525"
 			(at 45.72 74.93 0)
 			(hide yes)
@@
 			)
 		)
-		(property "Footprint" "FS_4_Global_Footprint_Library:Nano-Fit_1054301102"
+		(property "Footprint" "FS_4_Global_Footprint_Libary:CONN_SD-105430-001_02_MOL"
 			(at 318.77 95.25 0)
 			(hide yes)
@@
 			)
 		)
-		(property "Footprint" "FS_4_Global_Footprint_Library:Nano-Fit_1054301102"
+		(property "Footprint" "FS_4_Global_Footprint_Libary:CONN_SD-105430-001_02_MOL"
 			(at 273.05 144.78 0)
 			(hide yes)
@@
 			)
 		)
-		(property "Footprint" "FS_4_Global_Footprint_Library:Nano-Fit_1054301102"
+		(property "Footprint" "FS_4_Global_Footprint_Libary:CONN_SD-105430-001_02_MOL"
 			(at 295.91 147.32 0)
 			(hide yes)

Commit message: connector replacement
replaced balance board connectors with mezzanine connector
Parts:
- removed J4: 512810598, FS_4_Global_Footprint_Library:512810598, symbol Connector_Generic:Conn_01x05
- removed R13: 5k, Resistor_SMD:R_0805_2012Metric_Pad1.20x1.40mm_HandSolder, symbol Device:R
Connections:
- net ALERT renamed WATER_SENSE
- no-connect marks 7 -> 4
