File: temp-sense_bms-board/temp-sense_bms-board.kicad_pcb (KiCad board)
At the start: 2 copper layers, 154 parts, among them J1 84952-5, J2 84952-5, J3 1053131202, J4 512810598, J5 1053131202, J6 1053131202, J7 1053131202, Q1 NSV1C201MZ4, Q2 AO3400A, Q3 AO3400A, Q4 AO3400A, Q5 AO3400A, Q6 AO3400A, Q7 AO3400A, SW1 SW_DIP_x04, U1 TMP1075D, U10 TMP1075D, U11 TMP1075D, U12 TMP1075D, U13 TMP1075D, U14 TMP1075D, U15 TMP1075D, U16 TMP1075D, U17 TMP1075D, U18 TMP1075D, U19 TMP1075D, U2 TMP1075D, U20 TMP1075D, U21 TMP1075D, U22 TMP1075D, U23 TMP1075D, U24 TMP1075D, U25 HDC1010YPAR, U26 HDC1010YPAR, U27 HDC1010YPAR, U28 HDC1010YPAR, U29 LTC6810IG-2-TRPBF, U3 TMP1075D, U30 PCF8574T, U4 TMP1075D, U5 TMP1075D, U6 TMP1075D, U7 TMP1075D, U8 TMP1075D, U9 TMP1075D

Commit message: connector replacement
replaced balance board connectors with mezzanine connector
Parts:
- removed J4: 512810598, FS_4_Global_Footprint_Libary:512810598
- removed R13: 5k, Resistor_SMD:R_0805_2012Metric_Pad1.20x1.40mm_HandSolder
Connections:
- U1 pad 3: ALERT -> unconnected-(U1-ALERT-Pad3)
- U10 pad 3: ALERT -> unconnected-(U10-ALERT-Pad3)
- U11 pad 3: ALERT -> unconnected-(U11-ALERT-Pad3)
- U12 pad 3: ALERT -> unconnected-(U12-ALERT-Pad3)
- U13 pad 3: ALERT -> unconnected-(U13-ALERT-Pad3)
- U14 pad 3: ALERT -> unconnected-(U14-ALERT-Pad3)
- U15 pad 3: ALERT -> unconnected-(U15-ALERT-Pad3)
- U16 pad 3: ALERT -> unconnected-(U16-ALERT-Pad3)
- U17 pad 3: ALERT -> unconnected-(U17-ALERT-Pad3)
- U18 pad 3: ALERT -> unconnected-(U18-ALERT-Pad3)
- U19 pad 3: ALERT -> unconnected-(U19-ALERT-Pad3)
- U2 pad 3: ALERT -> unconnected-(U2-ALERT-Pad3)
- U20 pad 3: ALERT -> unconnected-(U20-ALERT-Pad3)
- U21 pad 3: ALERT -> unconnected-(U21-ALERT-Pad3)
- U22 pad 3: ALERT -> unconnected-(U22-ALERT-Pad3)
- U23 pad 3: ALERT -> unconnected-(U23-ALERT-Pad3)
- U24 pad 3: ALERT -> unconnected-(U24-ALERT-Pad3)
- U3 pad 3: ALERT -> unconnected-(U3-ALERT-Pad3)
- U4 pad 3: ALERT -> unconnected-(U4-ALERT-Pad3)
- U5 pad 3: ALERT -> unconnected-(U5-ALERT-Pad3)
- U6 pad 3: ALERT -> unconnected-(U6-ALERT-Pad3)
- U7 pad 3: ALERT -> unconnected-(U7-ALERT-Pad3)
- U8 pad 3: ALERT -> unconnected-(U8-ALERT-Pad3)
- U9 pad 3: ALERT -> unconnected-(U9-ALERT-Pad3)
Routing:
- net ALERT: track 1052.5 -> 0.77 mm, vias 11 -> 0
- net Net-(J3-Pin_1): track 32.2 -> 0.02 mm
- net DQ: track 28.8 -> 0.03 mm
- net unconnected-(U21-ALERT-Pad3): track 0.00 -> 0.87 mm
- net unconnected-(U1-ALERT-Pad3): track 0.00 -> 0.66 mm
- net unconnected-(U2-ALERT-Pad3): track 0.00 -> 0.49 mm, vias 0 -> 1
