File: temp-sense_bms-board/temp-sense_bms-board.kicad_sch (KiCad schematic)
At the start: 0 parts

Commit message: first work
Parts:
- added C1: 10nf, Capacitor_SMD:C_0603_1608Metric_Pad1.08x0.95mm_HandSolder, symbol Device:C
- added C10, C11, C12, C2, C3, C4, C5, C6, C7, C8, C9: .01uF, Capacitor_SMD:C_0603_1608Metric_Pad1.08x0.95mm_HandSolder, symbol Device:C
- added U1, U2, U6, U7: HDC1010YPAR, symbol 2026-08-22_00-16-12:HDC1010YPAR
- added U10, U11, U12, U13, U14, U15, U16, U3, U4, U5, U8, U9: TMP1075D, Package_SO:SO-8_3.9x4.9mm_P1.27mm, symbol Sensor_Temperature:TMP1075D
Connections:
- new net ALERT: U10.3 (ALERT), U11.3 (ALERT), U12.3 (ALERT), U13.3 (ALERT), U14.3 (ALERT), U15.3 (ALERT), U16.3 (ALERT), U3.3 (ALERT), U4.3 (ALERT), U5.3 (ALERT), U8.3 (ALERT), U9.3 (ALERT)
- new net I2C_SCL: U1.A1 (SCL), U10.2 (SCL), U10.6 (A1), U11.2 (SCL), U12.2 (SCL), U13.2 (SCL), U14.2 (SCL), U15.2 (SCL), U16.2 (SCL), U2.A1 (SCL), U3.2 (SCL), U4.2 (SCL), U5.2 (SCL), U6.A1 (SCL), U7.A1 (SCL), U8.2 (SCL), U9.2 (SCL)
- new net I2C_SDA: U1.A2 (SDA), U10.1 (SDA), U11.1 (SDA), U12.1 (SDA), U13.1 (SDA), U13.7 (A0), U14.1 (SDA), U15.1 (SDA), U15.7 (A0), U16.1 (SDA), U16.7 (A0), U2.A2 (SDA), U3.1 (SDA), U4.1 (SDA), U5.1 (SDA), U6.A2 (SDA), U7.A2 (SDA), U8.1 (SDA), U9.1 (SDA)
- new net V-: C1.2, C10.2, C11.2, C12.2, C2.2, C3.2, C4.2, C5.2, C6.2, C7.2, C8.2, C9.2, U1.B2 (GND), U1.C1 (ADR0), U1.D1 (ADR1), U10.4 (GND), U10.5 (A2), U10.7 (A0), U11.4 (GND), U11.5 (A2), U11.7 (A0), U12.4 (GND), U12.7 (A0), U13.4 (GND), U13.6 (A1), U14.4 (GND), U14.6 (A1), U14.7 (A0), U15.4 (GND), U15.6 (A1), U16.4 (GND), U2.B2 (GND), U2.C1 (ADR0), U3.4 (GND), U3.5 (A2), U3.6 (A1), U3.7 (A0), U4.4 (GND), U4.5 (A2), U4.6 (A1), U5.4 (GND), U5.5 (A2), U6.B2 (GND), U6.D1 (ADR1), U7.B2 (GND), U8.4 (GND), U9.4 (GND), U9.5 (A2), U9.6 (A1)
- new net VREG: C1.1, C10.1, C11.1, C12.1, C2.1, C3.1, C4.1, C5.1, C6.1, C7.1, C8.1, C9.1, U1.B1 (VDD), U10.8 (V+), U11.6 (A1), U11.8 (V+), U12.5 (A2), U12.6 (A1), U12.8 (V+), U13.5 (A2), U13.8 (V+), U14.5 (A2), U14.8 (V+), U15.5 (A2), U15.8 (V+), U16.5 (A2), U16.6 (A1), U16.8 (V+), U2.B1 (VDD), U2.D1 (ADR1), U3.8 (V+), U4.7 (A0), U4.8 (V+), U5.6 (A1), U5.7 (A0), U5.8 (V+), U6.B1 (VDD), U6.C1 (ADR0), U7.B1 (VDD), U7.C1 (ADR0), U7.D1 (ADR1), U8.5 (A2), U8.6 (A1), U8.7 (A0), U8.8 (V+), U9.7 (A0), U9.8 (V+)
- no-connect marks 0 -> 4
Other:
- added sheet BMS (BMS.kicad_sch)

Commit message: first layout
Placed all temp & humidity sensors. Placed all bms components. Unsure if LV/HV isolation is proper, so will review in future. Will also review traces cuz they're lowk hella jank.
Parts:
- added C27, C28, C29, C30: 100nf, Capacitor_SMD:C_0603_1608Metric_Pad1.08x0.95mm_HandSolder, symbol Device:C
- C10, C11, C12, C2, C3, C4, C5, C6, C7, C8, C9: value .01uF -> 10nf
- U1, U2, U6, U7: footprint (none) -> Sensors:HDC1010_YPA
Connections:
- net V-: now also C27.2, C28.2, C29.2, C30.2
- net VREG: now also C27.1, C28.1, C29.1, C30.1

Commit message: Added water drop sensors
Added pads for sensors and added PCF8574T I/O expander IC
Parts:
- added C31, C32, C33, C34, C35, C36, C37, C38, C39, C40, C41, C42: 10nf, Capacitor_SMD:C_0603_1608Metric_Pad1.08x0.95mm_HandSolder, symbol Device:C
- added C43: 100nf, Capacitor_SMD:C_0603_1608Metric_Pad1.08x0.95mm_HandSolder, symbol Device:C
- added R43, R44, R45, R46: 100k, Resistor_SMD:R_0603_1608Metric_Pad0.98x0.95mm_HandSolder, symbol Device:R
- added U13, U14, U15, U16, U17, U18, U19, U20, U21, U22, U23, U24: TMP1075D, Package_SO:SO-8_3.9x4.9mm_P1.27mm, symbol Sensor_Temperature:TMP1075D
- added U30: PCF8574T, Package_SO:SOIC-16W_7.5x10.3mm_P1.27mm, symbol Interface_Expansion:PCF8574T
- added W1, W2, W3, W4: Conn_01x02_Pin, FS_4_Global_Footprint_Libary:Water_Droplet_Comb_Sensor, symbol Connector:Conn_01x02_Pin
- renumbered U3 to U1, U14 to U10, U15 to U11, U16 to U12, U4 to U2, U1 to U25, U2 to U26, U6 to U27, U7 to U28, U5 to U3, U8 to U4, U9 to U5, U10 to U6, U11 to U7, U12 to U8, U13 to U9
Connections:
- net ALERT: now also U13.3 (ALERT), U14.3 (ALERT), U15.3 (ALERT), U16.3 (ALERT), U17.3 (ALERT), U18.3 (ALERT), U19.3 (ALERT), U20.3 (ALERT), U21.3 (ALERT), U22.3 (ALERT), U23.3 (ALERT), U24.3 (ALERT)
- net I2C_SCL: now also U10.7 (A0), U12.7 (A0), U13.2 (SCL), U14.2 (SCL), U14.7 (A0), U15.2 (SCL), U16.2 (SCL), U16.7 (A0), U17.2 (SCL), U18.2 (SCL), U19.2 (SCL), U19.6 (A1), U20.2 (SCL), U20.6 (A1), U21.2 (SCL), U22.2 (SCL), U23.2 (SCL), U23.7 (A0), U24.2 (SCL), U24.6 (A1), U30.14 (SCL); no longer U6.6 (A1)
- net I2C_SDA: now also U13.1 (SDA), U13.7 (A0), U14.1 (SDA), U15.1 (SDA), U15.7 (A0), U16.1 (SDA), U17.1 (SDA), U17.6 (A1), U18.1 (SDA), U18.6 (A1), U19.1 (SDA), U20.1 (SDA), U21.1 (SDA), U21.6 (A1), U22.1 (SDA), U22.6 (A1), U23.1 (SDA), U24.1 (SDA), U30.15 (SDA); no longer U12.7 (A0)
- net V-: now also U10.5 (A2), U12.5 (A2), U3.7 (A0), U4.5 (A2), U5.7 (A0), U6.6 (A1), U9.5 (A2), C31.2, C32.2, C33.2, C34.2, C35.2, C36.2, C37.2, C38.2, C39.2, C40.2, C41.2, C42.2, C43.2, U13.4 (GND), U13.6 (A1), U14.4 (GND), U14.6 (A1), U15.4 (GND), U16.4 (GND), U17.4 (GND), U17.5 (A2), U17.7 (A0), U18.4 (GND), U18.5 (A2), U19.4 (GND), U19.5 (A2), U19.7 (A0), U20.4 (GND), U20.5 (A2), U21.4 (GND), U21.7 (A0), U22.4 (GND), U23.4 (GND), U23.6 (A1), U24.4 (GND), U30.1 (A0), U30.2 (A1), U30.3 (A2), U30.8 (GND), W1.2 (Pin_2), W2.2 (Pin_2), W3.2 (Pin_2), W4.2 (Pin_2); no longer U10.7 (A0), U5.5 (A2), U6.5 (A2), U6.7 (A0), U7.5 (A2), U8.7 (A0)
- net VREG: now also U5.5 (A2), U6.5 (A2), U6.7 (A0), U7.5 (A2), U8.7 (A0), C31.1, C32.1, C33.1, C34.1, C35.1, C36.1, C37.1, C38.1, C39.1, C40.1, C41.1, C42.1, C43.1, R43.1, R44.1, R45.1, R46.1, U13.5 (A2), U13.8 (V+), U14.5 (A2), U14.8 (V+), U15.5 (A2), U15.6 (A1), U15.8 (V+), U16.5 (A2), U16.6 (A1), U16.8 (V+), U17.8 (V+), U18.7 (A0), U18.8 (V+), U19.8 (V+), U20.7 (A0), U20.8 (V+), U21.5 (A2), U21.8 (V+), U22.5 (A2), U22.7 (A0), U22.8 (V+), U23.5 (A2), U23.8 (V+), U24.5 (A2), U24.7 (A0), U24.8 (V+), U30.16 (VDD); no longer U10.5 (A2), U12.5 (A2), U3.7 (A0), U4.5 (A2), U5.7 (A0), U9.5 (A2)
- new net Sense_W1: R43.2, U30.4 (P0), W1.1 (Pin_1)
- new net Sense_W2: R44.2, U30.5 (P1), W2.1 (Pin_1)
- new net Sense_W3: R45.2, U30.6 (P2), W3.1 (Pin_1)
- new net Sense_W4: R46.2, U30.7 (P3), W4.1 (Pin_1)
- no-connect marks 4 -> 9
Other:
- moved on the sheet: C10, C11, C12, C27, C28, C29, C30, C4, C5, C6, C7, C8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

Commit message: connector replacement
replaced balance board connectors with mezzanine connector
Parts:
- removed C43: 100nf, Capacitor_SMD:C_0603_1608Metric_Pad1.08x0.95mm_HandSolder, symbol Device:C
- removed U30: PCF8574T, Package_SO:SOIC-16W_7.5x10.3mm_P1.27mm, symbol Interface_Expansion:PCF8574T
- added R13: 100k, Resistor_SMD:R_0805_2012Metric_Pad1.20x1.40mm_HandSolder, symbol Device:R
- added U31: DS18B20Z+, Package_SO:SO-8_3.9x4.9mm_P1.27mm, symbol 2026-01-10_01-54-57:DS18B20Z+
- R43: value 100k -> 200k; footprint Resistor_SMD:R_0603_1608Metric_Pad0.98x0.95mm_HandSolder -> Resistor_SMD:R_0805_2012Metric_Pad1.20x1.40mm_HandSolder
- R44: value 100k -> 400k; footprint Resistor_SMD:R_0603_1608Metric_Pad0.98x0.95mm_HandSolder -> Resistor_SMD:R_0805_2012Metric_Pad1.20x1.40mm_HandSolder
- R45: value 100k -> 800k; footprint Resistor_SMD:R_0603_1608Metric_Pad0.98x0.95mm_HandSolder -> Resistor_SMD:R_0805_2012Metric_Pad1.20x1.40mm_HandSolder
- R46: footprint Resistor_SMD:R_0603_1608Metric_Pad0.98x0.95mm_HandSolder -> Resistor_SMD:R_0805_2012Metric_Pad1.20x1.40mm_HandSolder
Connections:
- net Sense_W1: now also R13.2; no longer R43.2
- net Sense_W2: now also R43.2; no longer R44.2
- net Sense_W3: now also R44.2; no longer R45.2
- net Sense_W4: now also R45.2; no longer R46.2
- net VREG: no longer R43.1, R44.1, R45.1
- removed net ALERT: U1.3 (ALERT), U10.3 (ALERT), U11.3 (ALERT), U12.3 (ALERT), U13.3 (ALERT), U14.3 (ALERT), U15.3 (ALERT), U16.3 (ALERT), U17.3 (ALERT), U18.3 (ALERT), U19.3 (ALERT), U2.3 (ALERT), U20.3 (ALERT), U21.3 (ALERT), U22.3 (ALERT), U23.3 (ALERT), U24.3 (ALERT), U3.3 (ALERT), U4.3 (ALERT), U5.3 (ALERT), U6.3 (ALERT), U7.3 (ALERT), U8.3 (ALERT), U9.3 (ALERT)
- new net DQ: U31.4 (DQ)
- new net WATER_SENSE: R13.1, R43.1, R44.1, R45.1, R46.2
- no-connect marks 9 -> 28
Other:
- moved on the sheet: W1, W2, W3, W4
