File: tractive-battery-board/HVIL.kicad_sch (KiCad schematic)
At the start: 10 parts, among them J13 TS, J14 HVIL+/HVIL-, U17 MCP6004

Commit message: HVIL Isolation
Parts:
- removed unit 5 of U17
- added U?: MCP6004, symbol Amplifier_Operational:MCP6004
- added U?: (no value), Package_TO_SOT_SMD:SOT-23-6_Handsoldering, symbol formula_slug_symbol_library:AP3032KTR-G1
- added U?: PC817, Package_DIP:DIP-4_W7.62mm, symbol Isolator:PC817
Connections:
- net HVIL_P: now also U?.1; no longer J14.1 (Pin_1)
- net TS_N: now also U?.11 (V-), U?.2, U?.2 (GND); no longer J14.2 (Pin_2)
- net TS_P: now also U?.1 (SW), U?.4 (V+)
- new net GND Isolated: J14.2 (Pin_2), U?.3, U?.5 (OV)
- new net HV Isolated: U?.4, U?.6 (VIN)
- new net HVIL Signal: J14.1 (Pin_1)
- no-connect marks 3 -> 5

Commit message: Fixed MCU PINs
Parts:
- added R?: 1.7k, symbol Device:R_Small_US
Connections:
- net GND Isolated: no longer U?.3
- net HVIL Signal: now also U?.3
- net HVIL_P: now also R?.1; no longer U?.1
- net HV Isolated renamed +5V
- new net: R?.2, U?.1
Other:
- moved on the sheet: U?

Commit message: Removed Isolation from HVIL
Parts:
- removed R?: 1.7k, symbol Device:R_Small_US
- removed U?: (no value), Package_TO_SOT_SMD:SOT-23-6_Handsoldering, symbol formula_slug_symbol_library:AP3032KTR-G1
- removed U?: PC817, Package_DIP:DIP-4_W7.62mm, symbol Isolator:PC817
Connections:
- net GND Isolated is gone; now on net TS_N: J14.2 (Pin_2)
- net HVIL Signal is gone; now on net HVIL_P: J14.1 (Pin_1)
- net TS_P: no longer U?.4 (V+)
- net at C41.2, PS1.6 (+VOUT), R50.1: now also U?.4 (V+)
- no-connect marks 5 -> 3
Other:
- moved on the sheet: U?E
