File: tractive-battery-board/tractive-battery-board.kicad_sch (KiCad schematic)
At the start: 0 parts

Commit message: FS4 TBB schematic moved to FS5
Parts:
- added C1, C2: 6.8pF, Capacitor_SMD:C_0603_1608Metric_Pad1.08x0.95mm_HandSolder, symbol Device:C
- added C10, C11, C13, C14, C15, C16, C17, C18, C19, C20, C25, C26, C3, C6, C7, C8, C9: 100nF, Capacitor_SMD:C_0603_1608Metric_Pad1.08x0.95mm_HandSolder, symbol Device:C
- added C12, C22, C24: 1uF, Capacitor_SMD:C_0603_1608Metric_Pad1.08x0.95mm_HandSolder, symbol Device:C
- added C21: 15nF, Capacitor_SMD:C_0603_1608Metric_Pad1.08x0.95mm_HandSolder, symbol Device:C
- added C23, C5: 10uF, Resistor_SMD:R_0805_2012Metric_Pad1.20x1.40mm_HandSolder, symbol Device:C
- added C27: 47uF, Capacitor_SMD:C_0805_2012Metric_Pad1.18x1.45mm_HandSolder, symbol Device:C
- added C4: 4.7uF, Capacitor_SMD:C_0805_2012Metric_Pad1.18x1.45mm_HandSolder, symbol Device:C
- added D1, D2, D3, D4, D5, D6: PLZ3V3B-G3/H, Diode_SMD:D_SMF, symbol Device:D_Zener
- added FB1: FCM 1608KF-601T03, Inductor_SMD:L_0603_1608Metric_Pad1.05x0.95mm_HandSolder, symbol Device:FerriteBead
- added H1, H2: MountingHole_Pad, MountingHole:MountingHole_3.2mm_M3_Pad, symbol Mechanical:MountingHole_Pad
- added J1: FTSH-107-01-F-DV-K-P-TR, Connector_PinHeader_1.27mm:PinHeader_2x07_P1.27mm_Vertical_SMD, symbol Connector_Generic:Conn_02x07_Odd_Even
- added J2: IMD_Connector, FS_4_Global_Footprint_Library:1054311103 - 3-Pin Molex Nano-fit, symbol Connector_Generic:Conn_01x03
- added J3: Busbar_Temp_Sense, FS_4_Global_Footprint_Library:1054311202 - 2-Pin Molex Nano-fit, symbol Connector_Generic:Conn_01x02
- added J4: Cooling_TS, FS_4_Global_Footprint_Library:1054311202 - 2-Pin Molex Nano-fit, symbol Connector_Generic:Conn_01x02
- added J5: E-Meter, FS_4_Global_Footprint_Library:1054311202 - 2-Pin Molex Nano-fit, symbol Connector_Generic:Conn_01x02
- added J6: BMS_TS, FS_4_Global_Footprint_Library:1054311202 - 2-Pin Molex Nano-fit, symbol Connector_Generic:Conn_01x02
- added J7: Conn_02x13_Counter_Clockwise, FS_4_Global_Footprint_Library:ATS15-26PA-BM01, symbol Connector_Generic:Conn_02x13_Counter_Clockwise
- added JP1: Jumper_2_Open, Connector_PinHeader_2.54mm:PinHeader_2x01_P2.54mm_Vertical, symbol Jumper:Jumper_2_Open
- added L1: 4.7uH, Inductor_SMD:L_Bourns_SRP5030T, symbol Device:L
- added Q1: AO3400A, Package_TO_SOT_SMD:SOT-23, symbol Transistor_FET:AO3400A
- added Q2: AO3401A, Package_TO_SOT_SMD:SOT-23, symbol Transistor_FET:AO3401A
- added R1, R2, R24, R25, R28: 10k, Resistor_SMD:R_0603_1608Metric_Pad0.98x0.95mm_HandSolder, symbol Device:R
- added R10, R12, R5, R7: 20k, Resistor_SMD:R_0603_1608Metric_Pad0.98x0.95mm_HandSolder, symbol Device:R
- added R11, R13, R6, R8: 6.8k, Resistor_SMD:R_0603_1608Metric_Pad0.98x0.95mm_HandSolder, symbol Device:R
- added R14, R15, R16, R17, R18, R29: 15k, Resistor_SMD:R_0603_1608Metric_Pad0.98x0.95mm_HandSolder, symbol Device:R
- added R19: 1.3k, Resistor_SMD:R_2010_5025Metric_Pad1.40x2.65mm_HandSolder, symbol Device:R
- added R20: 330, Resistor_SMD:R_1206_3216Metric_Pad1.30x1.75mm_HandSolder, symbol Device:R
- added R21: 560, Resistor_SMD:R_1206_3216Metric_Pad1.30x1.75mm_HandSolder, symbol Device:R
- added R22, R23, R9: 100k, Resistor_SMD:R_0603_1608Metric_Pad0.98x0.95mm_HandSolder, symbol Device:R
- added R26: 4.7k, Resistor_SMD:R_0603_1608Metric_Pad0.98x0.95mm_HandSolder, symbol Device:R
- added R27: 5.1k, Resistor_SMD:R_0603_1608Metric_Pad0.98x0.95mm_HandSolder, symbol Device:R
- added R3, R4: 120, Resistor_SMD:R_0603_1608Metric_Pad0.98x0.95mm_HandSolder, symbol Device:R
- added SW1: Y97KT23B5NAFP, Button_Switch_SMD:SW_SPST_PTS647_Sx38, symbol Switch:SW_Push
- added SW2: SW_Push, Resistor_SMD:R_0603_1608Metric_Pad0.98x0.95mm_HandSolder, symbol Switch:SW_Push
- added TP1: MISO_TP, TestPoint:TestPoint_Pad_D1.0mm, symbol Connector:TestPoint
- added TP16: PC13_TP, TestPoint:TestPoint_Pad_D1.0mm, symbol Connector:TestPoint
- added TP17: PC14_TP, TestPoint:TestPoint_Pad_D1.0mm, symbol Connector:TestPoint
- added TP18: PC15_TP, TestPoint:TestPoint_Pad_D1.0mm, symbol Connector:TestPoint
- added TP19: PC7_TP, TestPoint:TestPoint_Pad_D1.0mm, symbol Connector:TestPoint
- added TP2: MOSI_TP, TestPoint:TestPoint_Pad_D1.0mm, symbol Connector:TestPoint
- added TP20: PC8_TP, TestPoint:TestPoint_Pad_D1.0mm, symbol Connector:TestPoint
- added TP3: SCK_TP, TestPoint:TestPoint_Pad_D1.0mm, symbol Connector:TestPoint
- added TP4: CK_TP, TestPoint:TestPoint_Pad_D1.0mm, symbol Connector:TestPoint
- added U1: STLINK-V3MODS, FS_4_Global_Footprint_Library:MODULE_STLINK-V3MODS, symbol FS_4_Global_Symbol_Library:STLINK-V3MODS
- added U2: STM32F446RETx, Package_QFP:LQFP-64_10x10mm_P0.5mm, symbol MCU_ST_STM32F4:STM32F446RETx
- added U3, U4: ISO1044BD, FS_4_Global_Footprint_Library:SOIC-8_ISO1044BD, symbol Interface_CAN_LIN:ISO1044BD
- added U5: DS18B20Z+, Package_SO:SOIC-8_3.9x4.9mm_P1.27mm, symbol Sensor_Temperature:DS18B20Z
- added U6: MIC5504-3.3YM5, Package_TO_SOT_SMD:SOT-23-5, symbol Regulator_Linear:MIC5504-3.3YM5
- added U7: AP63205WU, Package_TO_SOT_SMD:TSOT-23-6, symbol Regulator_Switching:AP63205WU
- added Y1: ECS-240-8-37B-CKY-TR, Crystal:Crystal_SMD_2016-4Pin_2.0x1.6mm, symbol Device:Crystal_GND24
Connections:
- new net: Q1.1 (G), R24.1
- new net: J4.1 (Pin_1), J5.1 (Pin_1), J6.1 (Pin_1), JP1.1 (A)
- new net: TP16.1, U2.2 (PC13)
- new net: TP17.1, U2.3 (PC14)
- new net: C4.2, U2.30 (VCAP_1)
- new net: TP20.1, U2.37 (PC6)
- new net: TP19.1, U2.38 (PC7)
- new net: TP18.1, U2.4 (PC15)
- new net: R27.2, R28.2, R29.1
- new net: R20.2, R21.1, R22.1
- new net: R16.1, R7.1, R8.2
- new net: R15.1, R5.1, R6.2
- new net: R10.1, R11.2, R17.1
- new net: R12.1, R13.2, R18.1
- new net: C25.1, L1.1, U7.5 (SW)
- new net: C25.2, U7.6 (BST)
- new net +12V: C23.2, J2.2 (Pin_2), J7.1 (Pin_1), R5.2, U7.2 (EN), U7.3 (IN)
- new net +3V3: C10.1, C11.1, C24.2, C5.2, C6.1, C7.1, C8.1, C9.1, FB1.1, J1.3 (Pin_3), Q2.3 (D), R26.1, U1.30 (T_VCC), U2.1 (VBAT), U2.19 (VDD), U2.32 (VDD), U2.48 (VDD), U2.64 (VDD), U3.1 (VCC1), U4.1 (VCC1), U6.5 (VOUT)
- new net +3V3_A: C12.1, C13.1, FB1.2, U2.13 (VDDA)
- new net +5V: C14.1, C15.1, C22.2, C27.2, J7.26 (Pin_26), L1.2, R25.1, SW2.1, U1.22 (5V_OPT), U3.8 (VCC2), U4.8 (VCC2), U6.1 (VIN), U6.3 (EN), U7.1 (FB)
- new net BOOT0: R1.1, U2.60 (BOOT0)
- new net BOOT1: R2.1, U2.28 (PB2)
- new net CAN_2_RD: U2.33 (PB12), U3.3 (RXD)
- new net CAN_2_TD: U2.34 (PB13), U3.2 (TXD)
- new net CAN_H_1: J7.3 (Pin_3), J7.5 (Pin_5), U4.6 (CANH)
- new net CAN_H_2: J7.14 (Pin_14), J7.17 (Pin_17), U3.6 (CANH)
- new net CAN_L_1: J7.4 (Pin_4), R4.2, U4.5 (CANL)
- new net CAN_L_2: J7.15 (Pin_15), R3.2, U3.5 (CANL)
- new net CAN_L_RES_1: J7.6 (Pin_6), R4.1
- new net CAN_L_RES_2: J7.16 (Pin_16), R3.1
- new net CAN_POWERTRAIN_RD: U2.44 (PA11), U4.3 (RXD)
- new net CAN_POWERTRAIN_TD: U2.45 (PA12), U4.2 (TXD)
- new net Charge_State: J7.24 (Pin_24), R14.1, R9.1
- new net Charge_State_Filtered: C16.1, D3.1 (K), R14.2, U2.10 (PC2)
- new net Fan_PWM: J7.7 (Pin_7), U2.39 (PC8)
- new net GLV_Voltage: C17.1, D1.1 (K), R15.2, U2.23 (PA7)
- new net GND: C1.2, C10.2, C11.2, C12.2, C13.2, C14.2, C15.2, C16.2, C17.2, C18.2, C19.2, C2.2, C20.2, C21.2, C22.1, C23.1, C24.1, C26.2, C27.1, C3.1, C4.1, C5.1, C6.2, C7.2, C8.2, C9.2, D1.2 (A), D2.2 (A), D3.2 (A), D4.2 (A), D5.2 (A), D6.2 (A), H1.1, H2.1, J1.11 (Pin_11), J1.5 (Pin_5), J1.7 (Pin_7), J2.3 (Pin_3), J3.2 (Pin_2), J4.2 (Pin_2), J5.2 (Pin_2), J6.2 (Pin_2), J7.2 (Pin_2), Q1.2 (S), R1.2, R11.1, R13.1, R2.2, R21.2, R23.1, R28.1, R6.1, R8.1, R9.2, SW1.1, U1.24 (GND), U1.26 (GND2), U1.27 (GND3), U1.29 (GND4), U1.5 (GNDDETECT), U1.8 (GND_2), U2.12 (VSSA), U2.18 (VSS), U2.31 (VSS), U2.47 (VSS), U2.63 (VSS), U3.4 (GND1), U3.7 (GND2), U4.4 (GND1), U4.7 (GND2), U5.3 (V_{DD}), U5.5 (GND), U6.2 (GND), U7.4 (GND), Y1.2, Y1.4
- new net IMD_FAULT_12V: J2.1 (Pin_1), R19.1
- new net IMD_Fault_3V3: C21.1, D6.1 (K), R22.2, U2.24 (PC4)
- new net IRs_Final: J7.20 (Pin_20), R7.2
- new net NRST: C3.2, J1.12 (Pin_12), SW1.2, U1.31 (T_NRST), U2.7 (NRST)
- new net OSC_IN: C1.1, U2.5 (PH0), Y1.3
- new net OSC_OUT: C2.1, U2.6 (PH1), Y1.1
- new net SH_RESET-: J7.25 (Pin_25), R27.1, SW2.2
- new net SH_RESET_3V3: C26.1, R29.2, U2.16 (PA2)
- new net SPI_BMS_CS: TP4.1, U2.20 (PA4)
- new net SPI_MISO: TP1.1, U2.56 (PB4)
- new net SPI_MOSI: TP2.1, U2.57 (PB5)
- new net SPI_SCK: TP3.1, U2.21 (PA5)
- new net STLINK_SWCLK: J1.6 (Pin_6), U1.13 (T_JCLK/T_SWCLK), U2.49 (PA14)
- new net STLINK_SWDIO: J1.4 (Pin_4), U1.4 (T_JTMS/T_SWDIO), U2.46 (PA13)
- new net STLINK_SWO: J1.8 (Pin_8), U1.6 (T_JTDO/T_SWO), U2.55 (PB3)
- new net Shutdown + IMD Delay/BMS_FAULT_5V: Q1.3 (D), R25.2
- new net Shutdown_In: J7.23 (Pin_23), R10.2
- new net Shutdown_In_3V3_Filtered: C19.1, D4.1 (K), R17.2, U2.14 (PA0)
- new net Shutdown_Measure: C18.1, D2.1 (K), R16.2, U2.22 (PA6)
- new net Shutdown_Out: J7.22 (Pin_22), R12.2
- new net Shutdown_Out_3V3_Filtered: C20.1, D5.1 (K), R18.2, U2.15 (PA1)
- new net TS1W: J3.1 (Pin_1), JP1.2 (B), Q2.2 (S), R26.2, U2.35 (PB14), U5.4 (DQ)
- new net TS1W_PU_Control: Q2.1 (G), U2.36 (PB15)
- new net TS_READY: J7.19 (Pin_19), U2.40 (PC9)
- new net VCP_UART_RX: J1.13 (Pin_13), U1.15 (T_VCP_RX), U2.43 (PA10)
- new net VCP_UART_TX: J1.14 (Pin_14), U1.12 (T_VCP_TX), U2.42 (PA9)
- new net V_Curr_Out: J7.8 (Pin_8)
- new net V_Curr_Ref: J7.9 (Pin_9)
- new net V_Out_Negative: J7.10 (Pin_10), U2.9 (PC1)
- new net V_Out_Positive: J7.11 (Pin_11), U2.8 (PC0)
- new net nBMS_FAULT_VCU: J7.12 (Pin_12)
- new net nBMS_Fault_3V3: R23.2, R24.2, U2.25 (PC5)
- new net nIMD_FAULT_5V: R19.2, R20.1
- new net nIMD_FAULT_VCU: J7.13 (Pin_13)
- new net nPreCharge_Control: U2.26 (PB0)
- no-connect marks 0 -> 38
Other:
- added sheet Current Sensors + Filtering (Current_Sensors.kicad_sch)
- added sheet HVIL (HVIL.kicad_sch)
- added sheet IsoSPI (TB_IsoSPI.kicad_sch)
- added sheet Precharge Circuit (TB_Precharge.kicad_sch)
- added sheet Shutdown + IMD Delay (Shutdown Logic.kicad_sch)
- note added: "24MHz"
- note added: "Auxillary Connectors"
- note added: "CAN Transciever"
- note added: "Current Sensor + Filtering"
- note added: "Decoupling 100nF capacitors need to be placed as close to respective Vdd/Vss as possible. Note that VSS contains all VSS mcu pins for each VDD/VSS pair."
- note added: "E-Meters"
- note added: "HV Voltage Indicator"
- note added: "IsoSPI"
- note added: "MCU Protections"
- note added: "NOTE: CAN Bridge left disconnected for now, but if we can figure out the protocol on the usb side to access it, we can connect it"
- note added: "Power Block"
- note added: "Precharge Circuit"
- note added: "SH_RESET+"
- note added: "SH_Reset"
- note added: "ST-Link Programming/Debugging Connector"
- note added: "STLINKV3-MODS Programmer"
- note added: "STM32F446RETx MCU"
- note added: "Shutdown + IMD Delay"
- note added: "TB Board Mount E-Meter"
- note added: "include diagraam for IRs"
- note added: "source digikey part"
- note added: "~100Hz RC Filter"

Commit message: Nano-Fit for IMD CAN
Purpose is to
Parts:
- added J?: IMD_CAN, symbol Connector_Generic:Conn_02x02_Counter_Clockwise
Connections:
- net CAN_H_2: now also J?.4 (Pin_4)
- net CAN_L_2: now also J?.3 (Pin_3)
- net at J7.18 (Pin_18): now also J?.1 (Pin_1)
- net at J7.21 (Pin_21): now also J?.2 (Pin_2)
- no-connect marks 38 -> 36
Changed lines of the file:
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@@
 	)
 	(junction
+		(at 327.66 191.77)
+		(diameter 0)
+		(color 0 0 0 0)
+	)
+	(junction
 		(at 396.24 59.69)
 		(diameter 0)
@@
 	)
 	(junction
+		(at 330.2 189.23)
+		(diameter 0)
+		(color 0 0 0 0)
+	)
+	(junction
 		(at 170.815 69.215)
 		(diameter 0)
@@
 	)
 	(no_connect
-		(at 334.01 173.99)
-	)
-	(no_connect
 		(at 97.79 68.58)
 	)
@@
 	)
 	(no_connect
-		(at 334.01 181.61)
-	)
-	(no_connect
 		(at 97.79 66.04)
 	)
@@
 	(wire
 		(pts
+			(xy 320.04 199.39) (xy 327.66 199.39)
+		)
+		(stroke
+			(width 0)
+			(type default)
+		)
+	)
+	(wire
+		(pts
+			(xy 320.04 201.93) (xy 330.2 201.93)
+		)
+		(stroke
+			(width 0)
+			(type default)
+		)
+	)
+	(wire
+		(pts
 			(xy 102.87 140.97) (xy 102.87 144.78)
 		)
@@
 	(wire
 		(pts
+			(xy 330.2 201.93) (xy 330.2 189.23)
+		)
+		(stroke
+			(width 0)
+			(type default)
+		)
+	)
+	(wire
+		(pts
 			(xy 189.23 134.62) (xy 190.5 134.62)
 		)
@@
 	(wire
 		(pts
-			(xy 326.39 191.77) (xy 334.01 191.77)
+			(xy 326.39 191.77) (xy 327.66 191.77)
 		)
 		(stroke
@@
 	(wire
 		(pts
+			(xy 307.34 199.39) (xy 307.34 181.61)
+		)
+		(stroke
+			(width 0)
+			(type default)
+		)
+	)
+	(wire
+		(pts
 			(xy 92.71 129.54) (xy 102.87 129.54)
 		)
@@
 	(wire
 		(pts
+			(xy 303.53 201.93) (xy 303.53 173.99)
+		)
+		(stroke
+			(width 0)
+			(type default)
+		)
+	)
+	(wire
+		(pts
+			(xy 330.2 189.23) (xy 334.01 189.23)
+		)
+		(stroke
+			(width 0)
+			(type default)
+		)
+	)
+	(wire
+		(pts
 			(xy 297.18 116.84) (xy 297.18 119.38)
 		)
@@
 	(wire
 		(pts
+			(xy 307.34 201.93) (xy 303.53 201.93)
+		)
+		(stroke
+			(width 0)
+			(type default)
+		)
+	)
+	(wire
+		(pts
 			(xy 125.095 69.215) (xy 137.795 69.215)
 		)
@@
 	(wire
 		(pts
+			(xy 327.66 191.77) (xy 334.01 191.77)
+		)
+		(stroke
+			(width 0)
+			(type default)
+		)
+	)
+	(wire
+		(pts
 			(xy 118.11 160.02) (xy 144.78 160.02)
 		)
@@
 	(wire
 		(pts
+			(xy 327.66 199.39) (xy 327.66 191.77)
+		)
+		(stroke
+			(width 0)
+			(type default)
+		)
+	)
+	(wire
+		(pts
 			(xy 97.79 140.97) (xy 100.33 140.97)
 		)
@@
 	(wire
 		(pts
+			(xy 307.34 181.61) (xy 334.01 181.61)
+		)
+		(stroke
+			(width 0)
+			(type default)
+		)
+	)
+	(wire
+		(pts
 			(xy 354.33 41.91) (xy 354.33 43.18)
 		)
@@
 	(wire
 		(pts
-			(xy 326.39 189.23) (xy 334.01 189.23)
+			(xy 326.39 189.23) (xy 330.2 189.23)
+		)
+		(stroke
+			(width 0)
+			(type default)
+		)
+	)
+	(wire
+		(pts
+			(xy 303.53 173.99) (xy 334.01 173.99)
 		)
 		(stroke
@@
 					(unit 1)
 				)
+			)
+		)
+	)
+	(symbol
+		(lib_id "Connector_Generic:Conn_02x02_Counter_Clockwise")
+		(at 312.42 199.39 0)
+		(unit 1)
+		(body_style 1)
+		(exclude_from_sim no)
+		(in_bom yes)
+		(on_board yes)
+		(in_pos_files yes)
+		(dnp no)
+		(fields_autoplaced yes)
+		(property "Reference" "J?"
+			(at 313.69 193.04 0)
+			(show_name no)
+			(do_not_autoplace no)
+			(effects
+				(font
+					(size 1.27 1.27)
+				)
+			)
+		)
+		(property "Value" "IMD_CAN"
+			(at 313.69 195.58 0)
+			(show_name no)
+			(do_not_autoplace no)
+			(effects
+				(font
+					(size 1.27 1.27)
+				)
+			)
+		)
+		(property "Footprint" ""
+			(at 312.42 199.39 0)
+			(hide yes)
+			(show_name no)
+			(do_not_autoplace no)
+			(effects
+				(font
+					(size 1.27 1.27)
+				)
+			)
+		)
+		(property "Datasheet" ""
+			(at 312.42 199.39 0)
+			(hide yes)
+			(show_name no)
+			(do_not_autoplace no)
+			(effects
+				(font
+					(size 1.27 1.27)
+				)
+			)
+		)
+		(property "Description" "Generic connector, double row, 02x02, counter clockwise pin numbering scheme (similar to DIP package numbering), script generated (kicad-library-utils/schlib/autogen/connector/)"
+			(at 312.42 199.39 0)
+			(hide yes)
+			(show_name no)
+			(do_not_autoplace no)
+			(effects
+				(font
+					(size 1.27 1.27)
+				)
+			)
+		)
+		(pin "2"
+		)
+		(pin "3"
+		)
+		(pin "1"
+		)
+		(pin "4"
+		)
+		(instances
+			(project "tractive-battery-board"
+				(path "/e994741c-7c7d-4124-9d00-43b883baa61d"
+					(reference "J?")
+					(unit 1)
+				)

Commit message: HVIL Isolation
Parts:
- U2: value STM32F446RETx -> STM32G473RBT6
Changed lines of the file:
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@@
 			)
 		)
-		(property "Value" "STM32F446RETx"
+		(property "Value" "STM32G473RBT6"
 			(at 73.406 142.24 0)
 			(show_name no)
@@
 			)
 		)
-		(property "Datasheet" "https://www.st.com/resource/en/datasheet/stm32f446re.pdf"
+		(property "Datasheet" "https://www.st.com/resource/en/datasheet/stm32g473cb.pdf"
 			(at 95.25 193.04 0)
 			(hide yes)
@@
 			(at 95.25 193.04 0)
 			(hide yes)
+			(show_name no)
+			(do_not_autoplace no)
+			(effects
+				(font
+					(size 1.27 1.27)
+				)
+			)
+		)
+		(property "Digikey Part Number" ""
+			(at 95.25 193.04 0)
+			(hide yes)
+			(show_name no)
+			(do_not_autoplace no)
+			(effects
+				(font
+					(size 1.27 1.27)
+				)
+			)
+		)
+		(property "Digikey URL" ""
+			(at 95.25 193.04 0)
+			(hide yes)

Commit message: MCU Update
Parts:
- U2: symbol MCU_ST_STM32F4:STM32F446RETx -> MCU_ST_STM32G4:STM32G473RBTx
Connections:
- net +3V3: now also U2.16 (VDD); no longer U2.19 (VDD)
- net +3V3_A: now also U2.29 (VDDA); no longer U2.13 (VDDA)
- net BOOT0: now also U2.7 (PG10); no longer U2.60 (BOOT0)
- net BOOT1: now also U2.26 (PB2); no longer U2.28 (PB2)
- net CAN_POWERTRAIN_RD: now also U2.45 (PA11); no longer U2.44 (PA11)
- net CAN_POWERTRAIN_TD: now also U2.46 (PA12); no longer U2.45 (PA12)
- net Fan_PWM: now also U2.40 (PC8); no longer U2.39 (PC8)
- net GLV_Voltage: now also U2.21 (PA7); no longer U2.23 (PA7)
- net GND: now also U2.15 (VSS), U2.27 (VSSA); no longer U2.12 (VSSA), U2.18 (VSS)
- net IMD_Fault_3V3: now also U2.22 (PC4); no longer U2.24 (PC4)
- net NRST: now also U2.28 (VREF+); no longer U2.7 (NRST)
- net SH_RESET_3V3: now also U2.14 (PA2); no longer U2.16 (PA2)
- net SPI_BMS_CS: now also U2.18 (PA4); no longer U2.20 (PA4)
- net SPI_MISO: now also U2.57 (PB4); no longer U2.56 (PB4)
- net SPI_MOSI: now also U2.58 (PB5); no longer U2.57 (PB5)
- net SPI_SCK: now also U2.19 (PA5); no longer U2.21 (PA5)
- net STLINK_SWCLK: now also U2.50 (PA14); no longer U2.49 (PA14)
- net STLINK_SWDIO: now also U2.49 (PA13); no longer U2.46 (PA13)
- net STLINK_SWO: now also U2.56 (PB3); no longer U2.55 (PB3)
- net Shutdown_In_3V3_Filtered: now also U2.12 (PA0); no longer U2.14 (PA0)
- net Shutdown_Measure: now also U2.20 (PA6); no longer U2.22 (PA6)
- net Shutdown_Out_3V3_Filtered: now also U2.13 (PA1); no longer U2.15 (PA1)
- net TS_READY: now also U2.41 (PC9); no longer U2.40 (PC9)
- net VCP_UART_RX: now also U2.44 (PA10); no longer U2.43 (PA10)
- net VCP_UART_TX: now also U2.43 (PA9); no longer U2.42 (PA9)
- net nBMS_Fault_3V3: now also U2.23 (PC5); no longer U2.25 (PC5)
- net nPreCharge_Control: now also U2.24 (PB0); no longer U2.26 (PB0)
- net at U2.30 (PB10): no longer C4.2
- net at U2.37 (PB15): no longer TP20.1
- net at U2.38 (PC6): now also TP20.1; no longer TP19.1
- new net: TP19.1, U2.39 (PC7)
- no-connect marks 36 -> 37
Other:
- moved on the sheet: U2

Commit message: Fixed GND C4 4.7uF pin
Connections:
- net at U2.30 (PB10): now also C4.2
- no-connect marks 37 -> 36
Other:
- moved on the sheet: C4
Changed lines of the file:
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@@
 	)
 	(no_connect
-		(at 113.03 220.98)
-	)
-	(no_connect
 		(at 97.79 78.74)
 	)
@@
 	(wire
 		(pts
+			(xy 140.97 238.76) (xy 127 238.76)
+		)
+		(stroke
+			(width 0)
+			(type default)
+		)
+	)
+	(wire
+		(pts
 			(xy 328.93 217.17) (xy 331.47 217.17)
 		)
@@
 	(wire
 		(pts
+			(xy 140.97 220.98) (xy 140.97 238.76)
+		)
+		(stroke
+			(width 0)
+			(type default)
+		)
+	)
+	(wire
+		(pts
 			(xy 189.23 110.49) (xy 189.23 106.68)
 		)
@@
 	(wire
 		(pts
+			(xy 113.03 220.98) (xy 140.97 220.98)
+		)
+		(stroke
+			(width 0)
+			(type default)
+		)
+	)
+	(wire
+		(pts
 			(xy 77.47 102.87) (xy 76.2 102.87)
 		)
@@
 	(symbol
 		(lib_id "Device:C")
-		(at 71.12 218.44 90)
+		(at 123.19 238.76 90)
 		(mirror x)
 		(unit 1)
@@
 		(dnp no)
 		(property "Reference" "C4"
-			(at 72.39 221.742 90)
+			(at 124.46 242.062 90)
 			(show_name no)
 			(do_not_autoplace no)
@@
 		)
 		(property "Value" "4.7uF"
-			(at 73.406 223.52 90)
+			(at 125.476 243.84 90)
 			(show_name no)
 			(do_not_autoplace no)
@@
 		)
 		(property "Footprint" "Capacitor_SMD:C_0805_2012Metric_Pad1.18x1.45mm_HandSolder"
-			(at 74.93 219.4052 0)
+			(at 127 239.7252 0)
 			(hide yes)
 			(show_name no)
@@
 		)
 		(property "Datasheet" "https://mm.digikey.com/Volume0/opasdata/d220001/medias/docus/41/CL21A475KAQNNNE_Spec.pdf"
-			(at 71.12 218.44 0)
+			(at 123.19 238.76 0)
 			(hide yes)
 			(show_name no)
@@
 		)
 		(property "Description" "Unpolarized capacitor"
-			(at 71.12 218.44 0)
+			(at 123.19 238.76 0)
 			(hide yes)
 			(show_name no)
@@
 		)
 		(property "Digi PN" "1276-1244-1-ND"
-			(at 71.12 218.44 0)
+			(at 123.19 238.76 0)
 			(hide yes)
 			(show_name no)
@@
 		)
 		(property "MFG" "Samsung Electro-Mechanics"
-			(at 71.12 218.44 0)
+			(at 123.19 238.76 0)
 			(hide yes)
 			(show_name no)
@@
 		)
 		(property "MFG PN" "CL21A475KAQNNNE"
-			(at 71.12 218.44 0)
+			(at 123.19 238.76 0)
 			(hide yes)
 			(show_name no)
@@
 		)
 		(property "Digi URL" "https://www.digikey.com/en/products/detail/samsung-electro-mechanics/CL21A475KAQNNNE/3886902"
-			(at 71.12 218.44 90)
+			(at 123.19 238.76 90)
 			(hide yes)
 			(show_name no)
@@
 		)
 		(property "Digikey Link" ""
-			(at 71.12 218.44 90)
+			(at 123.19 238.76 90)
 			(hide yes)
 			(show_name no)
@@
 		)
 		(property "MAXIMUM_PACKAGE_HEIGHT" ""
-			(at 71.12 218.44 90)
+			(at 123.19 238.76 90)
 			(hide yes)
 			(show_name no)
@@
 		)
 		(property "MFP PN" ""
-			(at 71.12 218.44 90)
+			(at 123.19 238.76 90)
 			(hide yes)
 			(show_name no)
@@
 		)
 		(property "Manufacturer" ""
-			(at 71.12 218.44 90)
+			(at 123.19 238.76 90)
 			(hide yes)
 			(show_name no)
@@
 		)
 		(property "Manufacturer Part Number" ""
-			(at 71.12 218.44 90)
+			(at 123.19 238.76 90)
 			(hide yes)
 			(show_name no)
@@
 		)
 		(property "PN" ""
-			(at 71.12 218.44 90)
+			(at 123.19 238.76 90)
 			(hide yes)
 			(show_name no)
@@
 		)
 		(property "Part Name" ""
-			(at 71.12 218.44 90)
+			(at 123.19 238.76 90)
 			(hide yes)
 			(show_name no)
@@
 		)
 		(property "Sim.Device" ""
-			(at 71.12 218.44 90)
+			(at 123.19 238.76 90)
 			(hide yes)
 			(show_name no)
@@
 		)
 		(property "Sim.Pins" ""
-			(at 71.12 218.44 90)
+			(at 123.19 238.76 90)
 			(hide yes)
 			(show_name no)
@@
 		)
 		(property "Sim.Type" ""
-			(at 71.12 218.44 90)
+			(at 123.19 238.76 90)
 			(hide yes)
 			(show_name no)
@@
 	(symbol
 		(lib_id "power:GND")
-		(at 67.31 218.44 0)
+		(at 119.38 238.76 0)
 		(unit 1)
 		(body_style 1)
@@
 		(dnp no)
 		(property "Reference" "#PWR012"
-			(at 67.31 224.79 0)
+			(at 119.38 245.11 0)
 			(hide yes)
 			(show_name no)
@@
 		)
 		(property "Value" "GND"
-			(at 63.5 220.218 0)
+			(at 115.57 240.538 0)
 			(show_name no)
 			(do_not_autoplace no)
@@
 		)
 		(property "Footprint" ""
-			(at 67.31 218.44 0)
+			(at 119.38 238.76 0)
 			(hide yes)
 			(show_name no)
@@
 		)
 		(property "Datasheet" ""
-			(at 67.31 218.44 0)
+			(at 119.38 238.76 0)
 			(hide yes)
 			(show_name no)
@@
 		)
 		(property "Description" "Power symbol creates a global label with name \"GND\" , ground"
-			(at 67.31 218.44 0)
+			(at 119.38 238.76 0)
 			(hide yes)
 			(show_name no)

Commit message: Fixed MCU PINs
Connections:
- net BOOT0: now also U2.2 (PC13); no longer U2.7 (PG10)
- net BOOT1: now also U2.37 (PB15); no longer U2.26 (PB2)
- net CAN_2_RD: now also U2.34 (PB12); no longer U2.33 (PB11)
- net CAN_2_TD: now also U2.35 (PB13); no longer U2.34 (PB12)
- net CAN_POWERTRAIN_RD: now also U2.61 (PB8); no longer U2.45 (PA11)
- net CAN_POWERTRAIN_TD: now also U2.62 (PB9); no longer U2.46 (PA12)
- net Charge_State_Filtered: now also U2.26 (PB2); no longer U2.10 (PC2)
- net Fan_PWM: now also U2.38 (PC6); no longer U2.40 (PC8)
- net GLV_Voltage: now also U2.36 (PB14); no longer U2.21 (PA7)
- net GND: no longer U2.15 (VSS), U2.31 (VSS), U2.47 (VSS), U2.63 (VSS)
- net IMD_Fault_3V3: now also U2.39 (PC7); no longer U2.22 (PC4)
- net NRST: now also U2.7 (PG10); no longer U2.28 (VREF+)
- net SH_RESET_3V3: now also U2.58 (PB5); no longer U2.14 (PA2)
- net SPI_BMS_CS: now also U2.57 (PB4); no longer U2.18 (PA4)
- net SPI_MISO: now also U2.20 (PA6); no longer U2.57 (PB4)
- net SPI_MOSI: now also U2.21 (PA7); no longer U2.58 (PB5)
- net SPI_SCK: now also U2.52 (PC10); no longer U2.19 (PA5)
- net Shutdown_In_3V3_Filtered: now also U2.24 (PB0); no longer U2.12 (PA0)
- net Shutdown_Measure: now also U2.33 (PB11); no longer U2.20 (PA6)
- net Shutdown_Out_3V3_Filtered: now also U2.25 (PB1); no longer U2.13 (PA1)
- net TS1W: now also U2.19 (PA5); no longer U2.35 (PB13)
- net TS1W_PU_Control: now also U2.18 (PA4); no longer U2.36 (PB14)
- net TS_READY: now also U2.9 (PC1); no longer U2.41 (PC9)
- net VCP_UART_RX: now also U2.17 (PA3); no longer U2.44 (PA10)
- net VCP_UART_TX: now also U2.14 (PA2); no longer U2.43 (PA9)
- net V_Out_Negative: no longer U2.9 (PC1)
- net V_Out_Positive: now also U2.23 (PC5); no longer U2.8 (PC0)
- net nBMS_Fault_3V3: now also U2.10 (PC2); no longer U2.23 (PC5)
- net nPreCharge_Control: now also U2.42 (PA8); no longer U2.24 (PB0)
- net at TP16.1: now also U2.8 (PC0); no longer U2.2 (PC13)
- net at U2.3 (PC14): no longer TP17.1
- net at C4.2: now also U2.15 (VSS), U2.31 (VSS), U2.47 (VSS), U2.63 (VSS); no longer U2.30 (PB10)
- net at TP20.1: now also U2.12 (PA0); no longer U2.38 (PC6)
- net at TP19.1: now also U2.13 (PA1); no longer U2.39 (PC7)
- net at U2.4 (PC15): no longer TP18.1
- new net: TP17.1, U2.40 (PC8)
- new net: TP18.1, U2.41 (PC9)
- no-connect marks 36 -> 37
Other:
- moved on the sheet: C3, C4, R1, R2, SW1, TP1, TP16, TP17, TP18, TP19, TP2, TP20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

Commit message: Removed Isolation from HVIL
Changed lines of the file:
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@@
-	)
-	(junction
-		(at 68.58 220.98)
-		(diameter 0)
-		(color 0 0 0 0)
 	)
 	(junction
@@
 		)
 		(stroke
-			(width 0)
-			(type default)
-		)
-	)
-	(wire
-		(pts
-			(xy 67.31 220.98) (xy 68.58 220.98)
-		)
-		(stroke

Commit message: IMD reset fix
Other:
- title: ${BOARD_TITLE} -> Tractive Battery Board
Changed lines of the file:
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@@
 	(paper "B")
 	(title_block
-		(title "${BOARD_TITLE}")
+		(title "Tractive Battery Board")
 		(date "${CURRENT_DATE}")
 		(rev "${REVISION}")
 		(company "Formula Slug")
-		(comment 1 "${NAMES}")
+		(comment 1 "Kaylee Kramer")
 		(comment 2 "${COMMENT1}")
 		(comment 3 "${COMMENT2}")
@@
 		)
 		(pin "56"
+			(alternate "SYS_JTDO-SWO")
 		)
 		(pin "57"
+			(alternate "SPI1_MISO")
 		)
 		(pin "33"
@@
 		)
 		(pin "62"
+			(alternate "FDCAN1_TX")
 		)
 		(pin "58"
@@
 		)
 		(pin "35"
+			(alternate "FDCAN2_TX")
 		)
 		(pin "27"
 		)
 		(pin "61"
+			(alternate "FDCAN1_RX")
 		)
 		(pin "34"
+			(alternate "FDCAN2_RX")
 		)
 		(pin "40"
@@
 		)
 		(pin "6"
+			(alternate "RCC_OSC_OUT")
 		)
 		(pin "5"
+			(alternate "RCC_OSC_IN")
 		)
 		(pin "11"
@@
 		)
 		(pin "21"
+			(alternate "SPI1_MOSI")
 		)
 		(pin "22"
@@
 		)
 		(pin "49"
+			(alternate "SYS_JTMS-SWDIO")
 		)
 		(pin "50"
+			(alternate "SYS_JTCK-SWCLK")
 		)
 		(pin "36"
 		)
 		(pin "52"
+			(alternate "SPI3_SCK")
 		)
 		(pin "51"
 		)
 		(pin "14"
+			(alternate "USART2_TX")
 		)
 		(pin "64"
@@
 		)
 		(pin "17"
+			(alternate "USART2_RX")
 		)
 		(pin "15"
 		)
 		(pin "20"
+			(alternate "SPI1_MISO")
 		)
 		(pin "13"
