File: llc-prototype/GateDriver.kicad_sch (KiCad schematic)
At the start: 12 parts, among them U1 UCC256612DDBR

Commit message: updated symbols from fs4 to fs5
Parts:
- U1: symbol FS_4_Global_Symbol_Library:UCC256612DDBR -> formula_slug_symbol_library:UCC256612DDBR
Changed lines of the file:
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@@
 	)
 	(symbol
-		(lib_id "FS_4_Global_Symbol_Library:UCC256612DDBR")
-		(at 134.62 110.49 0)
+		(lib_id "formula_slug_symbol_library:UCC256612DDBR")
+		(at 134.62 109.22 0)
 		(unit 1)
 		(body_style 1)
@@
 		(dnp no)
 		(property "Reference" "U1"
-			(at 138.176 95.504 0)
+			(at 138.176 94.234 0)
 			(show_name no)
 			(do_not_autoplace no)
@@
 		)
 		(property "Value" "UCC256612DDBR"
-			(at 138.176 98.044 0)
+			(at 138.176 96.774 0)
 			(show_name no)
 			(do_not_autoplace no)
@@
 		)
 		(property "Footprint" "Package_SO:SOIC-16_3.9x9.9mm_P1.27mm"
-			(at 134.62 110.49 0)
+			(at 135.128 78.74 0)
 			(hide yes)
 			(show_name no)
@@
 		)
 		(property "Datasheet" "https://www.ti.com/lit/ds/symlink/ucc25661.pdf?ts=1754894386115&ref_url=https%253A%252F%252Fwww.ti.com%252Fproduct%252FUCC25661%252Fpart-details%252FUCC256610DDBR"
-			(at 134.62 110.49 0)
+			(at 134.874 74.422 0)
 			(hide yes)
 			(show_name no)
@@
 		)
 		(property "Description" "LLC Controller/Half-Bridge Gate Driver"
-			(at 134.62 110.49 0)
+			(at 114.046 87.884 0)
 			(hide yes)
 			(show_name no)
+			(do_not_autoplace no)
+			(effects
+				(font
+					(size 1.27 1.27)
+				)
+			)
+		)
+		(property "Digikey Part Number" ""
+			(at 134.62 109.22 0)
+			(hide yes)
+			(show_name no)
+			(do_not_autoplace no)
+			(effects
+				(font
+					(size 1.27 1.27)
+				)
+			)
+		)
+		(property "Digikey URL" ""
+			(at 134.62 109.22 0)
+			(hide yes)
+			(show_name no)
+			(do_not_autoplace no)
+			(effects
+				(font
+					(size 1.27 1.27)
+				)
+			)
+		)
+		(property "Manufacturer" ""
+			(at 134.62 109.22 0)
+			(hide yes)
+			(show_name no)
+			(do_not_autoplace no)
+			(effects
+				(font
+					(size 1.27 1.27)
+				)
+			)
+		)
+		(property "Manufacturer Part Number" ""
+			(at 134.62 109.22 0)
+			(hide yes)
+			(show_name no)

Commit message: fixed HV gnds
Changed lines of the file:
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@@
 	(text "LL Pin HFBurstEntry at ~160W i.e ~23% of max load"
 		(exclude_from_sim no)
-		(at 79.756 87.376 0)
+		(at 75.184 75.692 0)
 		(effects
 			(font
@@
 	)
 	(junction
+		(at 134.62 85.09)
+		(diameter 0)
+		(color 0 0 0 0)
+	)
+	(junction
 		(at 74.93 166.37)
 		(diameter 0)
@@
 	(wire
 		(pts
-			(xy 134.62 80.01) (xy 138.43 80.01)
-		)
-		(stroke
-			(width 0)
-			(type default)
-		)
-	)
-	(wire
-		(pts
 			(xy 119.38 125.73) (xy 124.46 125.73)
 		)
@@
 	(wire
 		(pts
+			(xy 134.62 85.09) (xy 138.43 85.09)
+		)
+		(stroke
+			(width 0)
+			(type default)
+		)
+	)
+	(wire
+		(pts
 			(xy 146.05 116.84) (xy 147.32 116.84)
 		)
@@
 	(wire
 		(pts
-			(xy 134.62 80.01) (xy 134.62 96.52)
+			(xy 134.62 80.01) (xy 134.62 85.09)
 		)
 		(stroke
@@
 		(pts
 			(xy 123.19 114.3) (xy 124.46 114.3)
+		)
+		(stroke
+			(width 0)
+			(type default)
+		)
+	)
+	(wire
+		(pts
+			(xy 134.62 85.09) (xy 134.62 96.52)
 		)
 		(stroke
@@
 	(global_label "VCCP"
 		(shape passive)
-		(at 138.43 80.01 0)
+		(at 138.43 85.09 0)
 		(fields_autoplaced yes)
 		(effects
@@
 		)
 		(property "Intersheetrefs" "${INTERSHEET_REFS}"
-			(at 145.2025 80.01 0)
+			(at 145.2025 85.09 0)
 			(hide yes)
 			(show_name no)
@@
 	)
 	(symbol
-		(lib_id "power:GND")
+		(lib_id "power:GNDPWR")
 		(at 66.04 127 0)
 		(unit 1)
@@
 		)
 		(property "Value" "GND"
-			(at 66.04 132.08 0)
-			(show_name no)
-			(do_not_autoplace no)
-			(effects
-				(font
-					(size 1.27 1.27)
-				)
+			(at 68.58 128.0667 0)
+			(show_name no)
+			(do_not_autoplace no)
+			(effects
+				(font
+					(size 1.27 1.27)
+				)
+				(justify left)
 			)
 		)
 		(property "Footprint" ""
-			(at 66.04 127 0)
+			(at 66.04 128.27 0)
 			(hide yes)
 			(show_name no)
@@
 		)
 		(property "Datasheet" ""
-			(at 66.04 127 0)
-			(hide yes)
-			(show_name no)
-			(do_not_autoplace no)
-			(effects
-				(font
-					(size 1.27 1.27)
-				)
-			)
-		)
-		(property "Description" "Power symbol creates a global label with name \"GND\" , ground"
+			(at 66.04 128.27 0)
+			(hide yes)
+			(show_name no)
+			(do_not_autoplace no)
+			(effects
+				(font
+					(size 1.27 1.27)
+				)
+			)
+		)
+		(property "Description" "Power symbol creates a global label with name \"GNDPWR\" , global ground"
 			(at 66.04 127 0)
 			(hide yes)
@@
 	)
 	(symbol
-		(lib_id "power:GND")
+		(lib_id "power:GNDPWR")
 		(at 134.62 127 0)
 		(unit 1)
@@
 		)
 		(property "Value" "GND"
-			(at 134.62 132.08 0)
+			(at 134.493 130.81 0)
 			(show_name no)
 			(do_not_autoplace no)
@@
 		)
 		(property "Footprint" ""
+			(at 134.62 128.27 0)
+			(hide yes)
+			(show_name no)
+			(do_not_autoplace no)
+			(effects
+				(font
+					(size 1.27 1.27)
+				)
+			)
+		)
+		(property "Datasheet" ""
+			(at 134.62 128.27 0)
+			(hide yes)
+			(show_name no)
+			(do_not_autoplace no)
+			(effects
+				(font
+					(size 1.27 1.27)
+				)
+			)
+		)
+		(property "Description" "Power symbol creates a global label with name \"GNDPWR\" , global ground"
 			(at 134.62 127 0)
 			(hide yes)
@@
 			)
 		)
-		(property "Datasheet" ""
+		(property "Digikey Part Number" ""
 			(at 134.62 127 0)
 			(hide yes)
@@
 			)
 		)
-		(property "Description" "Power symbol creates a global label with name \"GND\" , ground"
+		(property "Digikey URL" ""
+			(at 134.62 127 0)
+			(hide yes)
+			(show_name no)
+			(do_not_autoplace no)
+			(effects
+				(font
+					(size 1.27 1.27)
+				)
+			)
+		)
+		(property "Manufacturer" ""
+			(at 134.62 127 0)
+			(hide yes)
+			(show_name no)
+			(do_not_autoplace no)
+			(effects
+				(font
+					(size 1.27 1.27)
+				)
+			)
+		)
+		(property "Manufacturer Part Number" ""
 			(at 134.62 127 0)
 			(hide yes)
@@
 	)
 	(symbol
-		(lib_id "power:GND")
+		(lib_id "power:GNDPWR")
 		(at 74.93 166.37 0)
 		(unit 1)
@@
 		)
 		(property "Value" "GND"
-			(at 74.93 171.45 0)
-			(show_name no)
-			(do_not_autoplace no)
-			(effects
-				(font
-					(size 1.27 1.27)
-				)
+			(at 77.47 167.4367 0)
+			(show_name no)
+			(do_not_autoplace no)
+			(effects
+				(font
+					(size 1.27 1.27)
+				)
+				(justify left)
 			)
 		)
 		(property "Footprint" ""
-			(at 74.93 166.37 0)
+			(at 74.93 167.64 0)
 			(hide yes)
 			(show_name no)
@@
 		)
 		(property "Datasheet" ""
-			(at 74.93 166.37 0)
-			(hide yes)
-			(show_name no)
-			(do_not_autoplace no)
-			(effects
-				(font
-					(size 1.27 1.27)
-				)
-			)
-		)
-		(property "Description" "Power symbol creates a global label with name \"GND\" , ground"
+			(at 74.93 167.64 0)
+			(hide yes)
+			(show_name no)
+			(do_not_autoplace no)
+			(effects
+				(font
+					(size 1.27 1.27)
+				)
+			)
+		)
+		(property "Description" "Power symbol creates a global label with name \"GNDPWR\" , global ground"
 			(at 74.93 166.37 0)
 			(hide yes)
@@
 	)
 	(symbol
-		(lib_id "power:GND")
+		(lib_id "power:GNDPWR")
 		(at 85.09 127 0)
 		(unit 1)
@@
 		)
 		(property "Value" "GND"
-			(at 85.09 132.08 0)
-			(show_name no)
-			(do_not_autoplace no)
-			(effects
-				(font
-					(size 1.27 1.27)
-				)
+			(at 87.63 128.0667 0)
+			(show_name no)
+			(do_not_autoplace no)
+			(effects
+				(font
+					(size 1.27 1.27)
+				)
+				(justify left)
 			)
 		)
 		(property "Footprint" ""
+			(at 85.09 128.27 0)
+			(hide yes)
+			(show_name no)
+			(do_not_autoplace no)
+			(effects
+				(font
+					(size 1.27 1.27)
+				)
+			)
+		)
+		(property "Datasheet" ""
+			(at 85.09 128.27 0)
+			(hide yes)
+			(show_name no)
+			(do_not_autoplace no)
+			(effects
+				(font
+					(size 1.27 1.27)
+				)
+			)
+		)
+		(property "Description" "Power symbol creates a global label with name \"GNDPWR\" , global ground"
 			(at 85.09 127 0)
 			(hide yes)
-			(show_name no)
-			(do_not_autoplace no)
-			(effects
-				(font
-					(size 1.27 1.27)
-				)
-			)
-		)
-		(property "Datasheet" ""
-			(at 85.09 127 0)
-			(hide yes)
-			(show_name no)
-			(do_not_autoplace no)
-			(effects
-				(font
-					(size 1.27 1.27)
-				)
-			)
-		)
-		(property "Description" "Power symbol creates a global label with name \"GND\" , ground"
-			(at 85.09 127 0)
-			(hide yes)

Commit message: fixes to schematic
Connections:
- net GND: now also C3.2; no longer C3.1
- net VCCP: now also C3.1; no longer C3.2
- net HS Driver renamed HI Driver
- net HI Driver: no longer C1.1
- net HS Return renamed HI Return
- net HI Return: now also C1.1
Other:
- moved on the sheet: C3
Changed lines of the file:
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@@
+	)
+	(junction
+		(at 85.09 156.21)
+		(diameter 0)
+		(color 0 0 0 0)
+	)
+	(junction
+		(at 85.09 114.3)
+		(diameter 0)
+		(color 0 0 0 0)
 	)
 	(junction
@@
 	)
 	(junction
-		(at 85.09 156.21)
+		(at 146.05 116.84)
 		(diameter 0)
 		(color 0 0 0 0)
 	)
 	(junction
-		(at 85.09 114.3)
+		(at 85.09 153.67)
 		(diameter 0)
 		(color 0 0 0 0)
 	)
 	(junction
-		(at 146.05 116.84)
+		(at 134.62 125.73)
+		(diameter 0)
+		(color 0 0 0 0)
+	)
+	(junction
+		(at 66.04 114.3)
+		(diameter 0)
+		(color 0 0 0 0)
+	)
+	(junction
+		(at 134.62 85.09)
 		(diameter 0)
 		(color 0 0 0 0)
@@
 	)
 	(junction
-		(at 85.09 153.67)
-		(diameter 0)
-		(color 0 0 0 0)
-	)
-	(junction
-		(at 134.62 125.73)
-		(diameter 0)
-		(color 0 0 0 0)
-	)
-	(junction
-		(at 66.04 114.3)
-		(diameter 0)
-		(color 0 0 0 0)
-	)
-	(junction
-		(at 134.62 85.09)
-		(diameter 0)
-		(color 0 0 0 0)
-	)
-	(junction
 		(at 74.93 166.37)
 		(diameter 0)
@@
 	(wire
 		(pts
-			(xy 119.38 125.73) (xy 124.46 125.73)
+			(xy 128.27 91.44) (xy 128.27 92.71)
 		)
 		(stroke
@@
 	(wire
 		(pts
-			(xy 129.54 125.73) (xy 134.62 125.73)
-		)
-		(stroke
-			(width 0)
-			(type default)
-		)
-	)
-	(wire
-		(pts
 			(xy 134.62 80.01) (xy 134.62 85.09)
 		)
@@
 	(wire
 		(pts
+			(xy 168.91 101.6) (xy 175.26 101.6)
+		)
+		(stroke
+			(width 0)
+			(type default)
+		)
+	)
+	(wire
+		(pts
 			(xy 134.62 125.73) (xy 134.62 127)
 		)
@@
 	(wire
 		(pts
-			(xy 175.26 101.6) (xy 168.91 101.6)
-		)
-		(stroke
-			(width 0)
-			(type default)
-		)
-	)
-	(wire
-		(pts
 			(xy 80.01 153.67) (xy 85.09 153.67)
 		)
@@
 	(wire
 		(pts
+			(xy 128.27 86.36) (xy 128.27 85.09)
+		)
+		(stroke
+			(width 0)
+			(type default)
+		)
+	)
+	(wire
+		(pts
 			(xy 66.04 102.87) (xy 66.04 105.41)
 		)
@@
 		(pts
 			(xy 168.91 107.95) (xy 168.91 106.68)
+		)
+		(stroke
+			(width 0)
+			(type default)
+		)
+	)
+	(wire
+		(pts
+			(xy 128.27 85.09) (xy 134.62 85.09)
 		)
 		(stroke
@@
 				)
 				(justify left)
-			)
-		)
-	)
-	(global_label "VCCP"
-		(shape passive)
-		(at 119.38 125.73 180)
-		(fields_autoplaced yes)
-		(effects
-			(font
-				(size 1.27 1.27)
-			)
-			(justify right)
-		)
-		(property "Intersheetrefs" "${INTERSHEET_REFS}"
-			(at 112.6075 125.73 0)
-			(hide yes)
-			(show_name no)
-			(do_not_autoplace no)
-			(effects
-				(font
-					(size 1.27 1.27)
-				)
-				(justify right)
 			)
 		)
@@
 		)
 	)
-	(hierarchical_label "HS Driver"
-		(shape input)
-		(at 175.26 101.6 0)
+	(hierarchical_label "HI Driver"
+		(shape output)
+		(at 154.94 104.14 0)
 		(effects
 			(font
@@
 		)
 	)
-	(hierarchical_label "HS Return"
+	(hierarchical_label "HI Return"
 		(shape input)
-		(at 154.94 104.14 0)
+		(at 175.26 101.6 0)
 		(effects
 			(font
@@
 				(path "/e994741c-7c7d-4124-9d00-43b883baa61d/c418867e-dc5c-4e54-b875-cab03a75b2d9"
 					(reference "TH1")
+					(unit 1)
+				)
+			)
+		)
+	)
+	(symbol
+		(lib_id "power:GNDPWR")
+		(at 128.27 92.71 0)
+		(unit 1)
+		(body_style 1)
+		(exclude_from_sim no)
+		(in_bom yes)
+		(on_board yes)
+		(in_pos_files yes)
+		(dnp no)
+		(fields_autoplaced yes)
+		(property "Reference" "#PWR04"
+			(at 128.27 99.06 0)
+			(hide yes)
+			(show_name no)
+			(do_not_autoplace no)
+			(effects
+				(font
+					(size 1.27 1.27)
+				)
+			)
+		)
+		(property "Value" "GND"
+			(at 128.143 96.52 0)
+			(show_name no)
+			(do_not_autoplace no)
+			(effects
+				(font
+					(size 1.27 1.27)
+				)
+			)
+		)
+		(property "Footprint" ""
+			(at 128.27 93.98 0)
+			(hide yes)
+			(show_name no)
+			(do_not_autoplace no)
+			(effects
+				(font
+					(size 1.27 1.27)
+				)
+			)
+		)
+		(property "Datasheet" ""
+			(at 128.27 93.98 0)
+			(hide yes)
+			(show_name no)
+			(do_not_autoplace no)
+			(effects
+				(font
+					(size 1.27 1.27)
+				)
+			)
+		)
+		(property "Description" "Power symbol creates a global label with name \"GNDPWR\" , global ground"
+			(at 128.27 92.71 0)
+			(hide yes)
+			(show_name no)
+			(do_not_autoplace no)
+			(effects
+				(font
+					(size 1.27 1.27)
+				)
+			)
+		)
+		(property "Digikey Part Number" ""
+			(at 128.27 92.71 0)
+			(hide yes)
+			(show_name no)
+			(do_not_autoplace no)
+			(effects
+				(font
+					(size 1.27 1.27)
+				)
+			)
+		)
+		(property "Digikey URL" ""
+			(at 128.27 92.71 0)
+			(hide yes)
+			(show_name no)
+			(do_not_autoplace no)
+			(effects
+				(font
+					(size 1.27 1.27)
+				)
+			)
+		)
+		(property "Manufacturer" ""
+			(at 128.27 92.71 0)
+			(hide yes)
+			(show_name no)
+			(do_not_autoplace no)
+			(effects
+				(font
+					(size 1.27 1.27)
+				)
+			)
+		)
+		(property "Manufacturer Part Number" ""
+			(at 128.27 92.71 0)
+			(hide yes)
+			(show_name no)
+			(do_not_autoplace no)
+			(effects
+				(font
+					(size 1.27 1.27)
+				)
+			)
+		)
+		(pin "1"
+		)
+		(instances
+			(project "llc-prototype"
+				(path "/e994741c-7c7d-4124-9d00-43b883baa61d/c418867e-dc5c-4e54-b875-cab03a75b2d9"
+					(reference "#PWR04")
 					(unit 1)
 				)
@@
 	(symbol
 		(lib_id "Device:C_Small")
-		(at 127 125.73 270)
+		(at 128.27 88.9 0)
 		(unit 1)
 		(body_style 1)
@@
 		(dnp no)
 		(property "Reference" "C3"
-			(at 127 129.286 90)
+			(at 123.698 87.884 0)
 			(show_name no)
 			(do_not_autoplace no)
@@
 		)
 		(property "Value" "2.2uF"
-			(at 126.746 131.826 90)
+			(at 123.952 90.678 0)
 			(show_name no)
 			(do_not_autoplace no)
@@
 		)
 		(property "Footprint" ""
-			(at 127 125.73 0)
+			(at 128.27 88.9 0)
 			(hide yes)
 			(show_name no)
@@
 		)
 		(property "Datasheet" "~"
-			(at 127 125.73 0)
+			(at 128.27 88.9 0)
 			(hide yes)
 			(show_name no)
@@
 		)
 		(property "Description" "Unpolarized capacitor, small symbol"
-			(at 127 125.73 0)
-			(hide yes)
-			(show_name no)
+			(at 128.27 88.9 0)
+			(hide yes)
+			(show_name no)

Commit message: update footprints to pcb editor
Parts:
- C1, C3: footprint (none) -> Capacitor_SMD:C_0603_1608Metric_Pad1.08x0.95mm_HandSolder
- TH1: footprint Resistor_SMD:R_0402_1005Metric_Pad0.72x0.64mm_HandSolder -> (none)
Connections:
- net VCCP: now also U1.12 (1); no longer U1.8 (VCCP)
Changed lines of the file:
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@@
 			)
 		)
-		(property "Footprint" "Resistor_SMD:R_0402_1005Metric_Pad0.72x0.64mm_HandSolder"
+		(property "Footprint" ""
 			(at 85.09 160.02 0)
 			(hide yes)
@@
 			)
 		)
-		(property "Footprint" ""
+		(property "Footprint" "Capacitor_SMD:C_0603_1608Metric_Pad1.08x0.95mm_HandSolder"
 			(at 168.91 104.14 0)
 			(hide yes)
@@
 			)
 		)
+		(pin "12"
+		)
+		(pin "7"
+		)
+		(pin "6"
+		)
+		(pin "15"
+		)
+		(pin "11"
+		)
+		(pin "4"
+		)
+		(pin "9"
+		)
+		(pin "1"
+		)
+		(pin "5"
+		)
+		(pin "3"
+		)
+		(pin "10"
+		)
 		(pin "8"
 		)
-		(pin "7"
-		)
-		(pin "6"
-		)
-		(pin "15"
-		)
-		(pin "11"
-		)
-		(pin "4"
-		)
-		(pin "9"
-		)
-		(pin "1"
-		)
-		(pin "5"
-		)
-		(pin "3"
-		)
-		(pin "10"
-		)
-		(pin "8"
-		)
 		(pin "14"
 		)
 		(pin "16"
+		)
+		(pin "13"
+		)
+		(pin "2"
 		)
 		(instances
@@
 			)
 		)
-		(property "Footprint" ""
+		(property "Footprint" "Capacitor_SMD:C_0603_1608Metric_Pad1.08x0.95mm_HandSolder"
 			(at 128.27 88.9 0)
 			(hide yes)

Commit message: added fuses
Connections:
- net GND renamed GNDPWR

Commit message: PCB work, added more caps
Parts:
- removed D3: D, symbol Device:D
- added C10: 4.7uF, Capacitor_SMD:C_0603_1608Metric_Pad1.08x0.95mm_HandSolder, symbol Device:C_Small
- added C11, C15: 100pF, Capacitor_SMD:C_0603_1608Metric_Pad1.08x0.95mm_HandSolder, symbol Device:C_Small
- added C12: 10nF, Capacitor_SMD:C_0603_1608Metric_Pad1.08x0.95mm_HandSolder, symbol Device:C_Small
- added C13: 330pF, Capacitor_SMD:C_0603_1608Metric_Pad1.08x0.95mm_HandSolder, symbol Device:C_Small
- added C14: 220pF, Capacitor_SMD:C_0603_1608Metric_Pad1.08x0.95mm_HandSolder, symbol Device:C_Small
- added D9: 1N5819HW-7-F, Diode_SMD:D_SOD-123, symbol Device:D
- added R23, R26: (no value), Resistor_SMD:R_0603_1608Metric_Pad0.98x0.95mm_HandSolder, symbol Device:R_Small_US
- added R6: 2.2, Resistor_SMD:R_0603_1608Metric_Pad0.98x0.95mm_HandSolder, symbol Device:R_Small_US
- C1: value C_Small -> 1.5uF
Connections:
- net BLK: now also C12.1
- net GNDPWR: now also C10.2, C11.2, C12.2, C13.2, C14.2, C15.2
- net HV: now also R23.1; no longer U1.1 (HV)
- net ISNS: now also C11.1
- net LL: now also C13.1
- net OVP/OTP: now also C15.1
- net TSET: now also C14.1
- net V5P: now also C10.1
- net VCCP: now also R6.2
- net at C1.2, U1.14 (HB): now also D9.1 (K)
- new net: R23.2, R26.1
- new net: R26.2, U1.1 (HV)
- new net: D9.2 (A), R6.1
Other:
- note removed: "OTP Trip at 85C OVP Trip at 110% of Vout"
- moved on the sheet: C1, C3, D1, R1, R11, R2, R3, R4, R5, TH1, U1

Commit message: pcb changes + fs-components update
Parts:
- U1: footprint Package_SO:SOIC-16_3.9x9.9mm_P1.27mm -> formula_slug_footprint_library:SOIC-16_3.9x9.9mm_P1.27mm_editedForLLC
Changed lines of the file:
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@@
 			)
 		)
-		(property "Footprint" "Package_SO:SOIC-16_3.9x9.9mm_P1.27mm"
+		(property "Footprint" "formula_slug_footprint_library:SOIC-16_3.9x9.9mm_P1.27mm_editedForLLC"
 			(at 136.398 67.31 0)
 			(hide yes)

Commit message: changed hb mosfet footprint
Changed lines of the file:
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@@
 		(property "Value" "1.5uF"
 			(at 172.72 93.9862 0)
+			(hide yes)
 			(show_name no)
 			(do_not_autoplace no)
