File: llc-prototype/llc-prototype.kicad_pcb (KiCad board)
At the start: 2 copper layers, 44 parts, among them Q1 MCTL011N20YH-TP, Q2 MCTL011N20YH-TP, Q3 NTMFS1D3N04XMT1G, Q4 NTMFS1D3N04XMT1G, U1 UCC256612DDBR, U2 UCC24624DR, U3 PC817, U4 TL431DBZ

Commit message: added fuses
Parts:
- removed R6: 8.06, Resistor_SMD:R_0603_1608Metric_Pad0.98x0.95mm_HandSolder
- added R22: 8.06, Resistor_SMD:R_0603_1608Metric_Pad0.98x0.95mm_HandSolder, F.Cu at (220.1, 39.0)
- moved C4 231.8 mm to (256.3, 60.9)
- moved U2 211.2 mm to (256.7, 21.1)
- moved U4 207.9 mm to (216.5, 86.5)
- moved C5 207.0 mm to (250.0, 20.6)
- moved R19 200.8 mm to (217.0, 111.2)
- moved R14 200.2 mm to (216.8, 106.0)
- moved R13 199.6 mm to (216.8, 101.8)
- moved C9 198.7 mm to (216.3, 92.1)
- moved R12 198.4 mm to (216.4, 97.3)
- moved R7 177.4 mm to (208.8, 39.4)
- moved U3 163.1 mm to (179.5, 98.5)
- moved Q4 162.2 mm to (223.4, 53.5), turned to 90 degrees
- moved R21 152.4 mm to (220.1, 37.5)
- moved D7 147.6 mm to (216.0, 37.5)
- moved Q3 144.6 mm to (204.7, 53.5), turned to 90 degrees
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Connections:
- C3 pad 2: GND -> GNDPWR
- D6 pad 1: unconnected-(D6-K-Pad1) -> VG1
- D6 pad 2: unconnected-(D6-A-Pad2) -> Net-(D6-A)
- D7 pad 1: unconnected-(D7-K-Pad1) -> VG2
- D7 pad 2: unconnected-(D7-A-Pad2) -> Net-(D7-A)
- Q3 pad 1: +Vout -> GND
- Q4 pad 1: +Vout -> GND
- R1 pad 2: GND -> GNDPWR
- R11 pad 2: GND -> GNDPWR
- R20 pad 1: unconnected-(R20-Pad1) -> Net-(D6-A)
- R20 pad 2: unconnected-(R20-Pad2) -> Net-(Q3-G)
- R21 pad 1: unconnected-(R21-Pad1) -> Net-(D7-A)
- R21 pad 2: unconnected-(R21-Pad2) -> Net-(Q4-G)
- R4 pad 2: GND -> GNDPWR
- R5 pad 2: GND -> GNDPWR
- TH1 pad 2: GND -> GNDPWR
- U1 pad 10: GND -> GNDPWR
Routing:
- net LL: track 0.00 -> 2.19 mm
- net TSET: track 0.00 -> 1.90 mm
Other:
- copper layers 2 -> 4

Commit message: PCB work, added more caps
Parts:
- removed C7: C, Capacitor_SMD:C_0603_1608Metric_Pad1.08x0.95mm_HandSolder
- added C10: 4.7uF, Capacitor_SMD:C_0603_1608Metric_Pad1.08x0.95mm_HandSolder, B.Cu at (106.0, 137.3)
- added C11: 100pF, Capacitor_SMD:C_0603_1608Metric_Pad1.08x0.95mm_HandSolder, B.Cu at (105.6, 134.0)
- added C12: 10nF, Capacitor_SMD:C_0603_1608Metric_Pad1.08x0.95mm_HandSolder, B.Cu at (99.1, 137.3)
- added C13: 330pF, Capacitor_SMD:C_0603_1608Metric_Pad1.08x0.95mm_HandSolder, B.Cu at (102.8, 137.3)
- added C14: 220pF, Capacitor_SMD:C_0603_1608Metric_Pad1.08x0.95mm_HandSolder, B.Cu at (104.3, 137.3)
- added C15: 100pF, Capacitor_SMD:C_0603_1608Metric_Pad1.08x0.95mm_HandSolder, B.Cu at (100.7, 137.3)
- added C16: C_Small, Capacitor_SMD:C_0603_1608Metric_Pad1.08x0.95mm_HandSolder, F.Cu at (131.5, 134.2)
- added C17: C_Small, Capacitor_SMD:C_0603_1608Metric_Pad1.08x0.95mm_HandSolder, F.Cu at (158.7, 96.2)
- added C18: C_Small, Capacitor_SMD:C_0603_1608Metric_Pad1.08x0.95mm_HandSolder, F.Cu at (159.1, 98.3)
- added C19: C_Small, Capacitor_SMD:C_0603_1608Metric_Pad1.08x0.95mm_HandSolder, F.Cu at (159.1, 102.0)
- added C20: C_Small, Capacitor_SMD:C_0603_1608Metric_Pad1.08x0.95mm_HandSolder, F.Cu at (158.8, 93.8)
- added C21: C_Small, Capacitor_SMD:C_0603_1608Metric_Pad1.08x0.95mm_HandSolder, F.Cu at (71.8, 144.2)
- added C22: C_Small, Capacitor_SMD:C_0603_1608Metric_Pad1.08x0.95mm_HandSolder, F.Cu at (72.0, 141.6)
- added C23: C_Small, Capacitor_SMD:C_0603_1608Metric_Pad1.08x0.95mm_HandSolder, F.Cu at (71.6, 137.4)
- added C24: C_Small, Capacitor_SMD:C_0603_1608Metric_Pad1.08x0.95mm_HandSolder, F.Cu at (72.0, 134.4)
- added C25: C_Small, Capacitor_SMD:C_0603_1608Metric_Pad1.08x0.95mm_HandSolder, F.Cu at (98.8, 84.5)
- added C26: C_Small, Capacitor_SMD:C_0603_1608Metric_Pad1.08x0.95mm_HandSolder, F.Cu at (106.4, 82.9)
- added C27: C_Small, Capacitor_SMD:C_0603_1608Metric_Pad1.08x0.95mm_HandSolder, F.Cu at (106.7, 85.7)
- added C28: C_Small, Capacitor_SMD:C_0603_1608Metric_Pad1.08x0.95mm_HandSolder, F.Cu at (106.7, 88.2)
- added C29: 1.5uF, Capacitor_SMD:C_0603_1608Metric_Pad1.08x0.95mm_HandSolder, F.Cu at (167.3, 108.7)
- added D9: 1N5819HW-7-F, Diode_SMD:D_SOD-123, F.Cu at (93.4, 135.8)
- added R23: ~, Resistor_SMD:R_0603_1608Metric_Pad0.98x0.95mm_HandSolder, F.Cu at (94.2, 142.9)
- added R24: R_Small_US, Resistor_SMD:R_0603_1608Metric_Pad0.98x0.95mm_HandSolder, F.Cu at (134.1, 131.6)
- added R25: 1200, Resistor_SMD:R_0603_1608Metric_Pad0.98x0.95mm_HandSolder, F.Cu at (134.8, 137.1)
- added R26: ~, Resistor_SMD:R_0603_1608Metric_Pad0.98x0.95mm_HandSolder, F.Cu at (92.6, 141.1)
- added R6: 2.2, Resistor_SMD:R_0603_1608Metric_Pad0.98x0.95mm_HandSolder, F.Cu at (92.7, 137.9)
- C1: value C_Small -> 1.5uF; moved to B.Cu
- C3, C5: moved to B.Cu
- C4, C6: value C -> C_Small
- moved U2 146.2 mm to (143.2, 113.4)
- moved C5 143.0 mm to (141.7, 114.0)
- moved R10 142.0 mm to (95.8, 142.9), turned to 90 degrees
- moved R8 140.3 mm to (98.4, 141.9)
- moved R9 136.9 mm to (98.3, 140.3), turned to 180 degrees
- moved C6 123.1 mm to (71.9, 131.1)
- moved R20 103.8 mm to (133.9, 109.7), turned to 180 degrees
- moved R7 103.8 mm to (133.9, 111.2), turned to 180 degrees
- moved R21 102.4 mm to (149.3, 111.5), turned to -90 degrees
- moved C4 102.4 mm to (158.5, 91.0)
- moved R22 102.3 mm to (147.8, 111.5), turned to -90 degrees
- moved D7 98.7 mm to (147.6, 108.6), turned to 180 degrees
- moved U4 98.5 mm to (128.7, 131.1), turned to 90 degrees
- moved D6 98.1 mm to (137.9, 109.7), turned to 180 degrees
- moved Q4 96.9 mm to (150.0, 116.8), turned to -90 degrees
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Connections:
- C9 pad 2: Net-(U4-REF) -> Net-(C9-Pad2)
- R12 pad 1: +Vout -> Net-(D8-K)
- R19 pad 1: +Vout -> Net-(R12-~-Pad2)
- U1 pad 1: +Vin -> Net-(U1-HV)
- U2 pad 7: VCCP -> +Vout
Routing:
- net TSET: track 1.90 -> 0.04 mm, vias 0 -> 1
- net LL: track 2.19 -> 0.35 mm, vias 0 -> 1
- net VCCP: track 0.00 -> 0.48 mm, vias 0 -> 1
- net Net-(D9-K): track 0.00 -> 0.41 mm, vias 0 -> 1
- net /LLC Controller/Gate Driver/HI Return: track 0.00 -> 0.41 mm, vias 0 -> 1
- net V5P: track 0.00 -> 0.39 mm, vias 0 -> 1
- net GNDPWR: track 0.00 -> 0.34 mm, vias 0 -> 1
- net /LLC Controller/Gate Driver/BLK: track 0.00 -> 0.33 mm, vias 0 -> 1
- net OVP/OTP: track 0.00 -> 0.18 mm, vias 0 -> 1
- net ISNS: track 0.00 -> 0.17 mm, vias 0 -> 1
Other:
- copper layers 4 -> 2
- board text added: "Credit Card Dimension Reference"

Commit message: pcb changes + fs-components update
Parts:
- C29: moved to B.Cu
- Q3, Q4: footprint Package_SO:ONSemi_SO-8FL_488AA -> formula_slug_footprint_library:ONSemi_SO-8FL_488AA_editedForLLC
- U1: footprint Package_SO:SOIC-16_3.9x9.9mm_P1.27mm -> formula_slug_footprint_library:SOIC-16_3.9x9.9mm_P1.27mm_editedForLLC
- moved C26 53.2 mm to (97.3, 135.3), turned to -90 degrees
- moved C27 51.3 mm to (93.8, 135.3), turned to -90 degrees
- moved C25 50.9 mm to (101.0, 135.3), turned to -90 degrees
- moved C28 49.9 mm to (90.0, 135.3), turned to -90 degrees
- moved D2 37.1 mm to (107.5, 134.4), turned to 0 degrees
- moved TH1 32.1 mm to (85.2, 121.9)
- moved R11 26.6 mm to (100.1, 124.6), turned to -90 degrees
- moved C29 22.2 mm to (145.7, 113.9), turned to -90 degrees
- moved R6 18.9 mm to (93.2, 119.1)
- moved D9 18.8 mm to (92.5, 117.1)
- moved R26 18.0 mm to (93.6, 123.2)
- moved R8 17.4 mm to (96.8, 124.6), turned to 90 degrees
- moved C1 17.2 mm to (97.6, 116.1)
- moved C3 17.2 mm to (102.7, 116.1)
- moved R1 17.2 mm to (105.0, 123.1)
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Routing:
- net V5P: track 0.39 -> 9.02 mm, vias 1 -> 0
- net Net-(U4-K): track 0.00 -> 8.18 mm
- net VCCP: track 0.48 -> 8.52 mm, vias 1 -> 0
- net VG1: track 0.00 -> 7.70 mm
- net LL: track 0.35 -> 7.45 mm, vias 1 -> 0
- net Net-(U4-REF): track 0.00 -> 7.07 mm
- net +Vout: track 0.00 -> 7.05 mm
- net VD2: track 0.00 -> 6.88 mm
- net Net-(D9-K): track 0.41 -> 6.02 mm, vias 1 -> 0
- net Net-(R12-~-Pad2): track 0.00 -> 5.58 mm
- net VG2: track 0.00 -> 5.05 mm
- net VD1: track 0.00 -> 4.78 mm
- net /LLC Controller/Gate Driver/BLK: track 0.33 -> 4.45 mm, vias 1 -> 0
- net TSET: track 0.04 -> 3.73 mm, vias 1 -> 0
- net Net-(Q3-G): track 0.00 -> 3.68 mm
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
Commit message: changed hb mosfet footprint
Parts:
- Q1, Q2: footprint Package_TO_SOT_SMD:Infineon_PG-HSOF-8-1_ThermalVias -> Package_TO_SOT_SMD:Infineon_PG-HSOF-8-1
- moved C10 1.50 mm to (105.9, 121.6), turned to -90 degrees
- moved C14 1.48 mm to (104.2, 121.6), turned to -90 degrees
- moved C13 1.47 mm to (102.6, 121.6), turned to -90 degrees
- moved C12 1.45 mm to (98.5, 121.6), turned to -90 degrees
- moved C15 1.45 mm to (100.2, 121.6), turned to -90 degrees
- moved C5 1.07 mm to (140.8, 113.5), turned to 90 degrees
- moved Q3 0.75 mm to (136.5, 116.2)
Routing:
- net VG1: track 7.70 -> 0.00 mm
- net V5P: track 9.02 -> 16.6 mm, vias 0 -> 1
- net GNDPWR: track 0.00 -> 6.28 mm, vias 0 -> 4
- net VD1: track 4.78 -> 0.00 mm
- net OVP/OTP: track 2.69 -> 6.97 mm, vias 0 -> 1
- net TSET: track 3.73 -> 7.62 mm, vias 0 -> 1
- net LL: track 7.45 -> 10.7 mm, vias 0 -> 1
- net /LLC Controller/Gate Driver/BLK: track 4.45 -> 7.67 mm, vias 0 -> 1
- net Net-(Q3-G): track 3.68 -> 1.50 mm
- net Net-(U2-REG): track 0.00 -> 1.74 mm, vias 0 -> 1
- net VD2: track 6.88 -> 8.61 mm, vias 0 -> 1
- net GND: vias 0 -> 3

Commit message: schematic
Parts:
- removed the C2 at (109.6, 112.5)
- removed D4: 1N5819HW-7-F, Diode_SMD:D_SOD-123
- removed the R5 at (106.9, 116.7)
- added C10: C_Small, Capacitor_SMD:C_1206_3216Metric_Pad1.33x1.80mm_HandSolder, F.Cu at (40.6, 98.2)
- added C16: C_Small, Capacitor_SMD:C_1206_3216Metric_Pad1.33x1.80mm_HandSolder, F.Cu at (40.6, 118.3)
- added C17: C_Small, Capacitor_SMD:C_1206_3216Metric_Pad1.33x1.80mm_HandSolder, F.Cu at (40.6, 121.7)
- added C18: C_Small, Capacitor_SMD:C_1206_3216Metric_Pad1.33x1.80mm_HandSolder, F.Cu at (40.6, 125.0)
- added C9: C_Small, Capacitor_SMD:C_1206_3216Metric_Pad1.33x1.80mm_HandSolder, F.Cu at (40.6, 94.8)
- added D1: 1N5819HW-7-F, Diode_SMD:D_SOD-123, F.Cu at (40.8, 135.9)
- added D3: 1N5819HW-7-F, Diode_SMD:D_SOD-123, F.Cu at (40.8, 142.7)
- added R8: 510, Resistor_SMD:R_0603_1608Metric_Pad0.98x0.95mm_HandSolder, F.Cu at (45.8, 135.5)
- C11, C15: value 100pF -> C_Small; footprint Capacitor_SMD:C_0603_1608Metric_Pad1.08x0.95mm_HandSolder -> Capacitor_SMD:C_1206_3216Metric_Pad1.33x1.80mm_HandSolder; moved to F.Cu
- C12: value 10nF -> C_Small; footprint Capacitor_SMD:C_0603_1608Metric_Pad1.08x0.95mm_HandSolder -> Capacitor_SMD:C_1206_3216Metric_Pad1.33x1.80mm_HandSolder; moved to F.Cu
- C13: value 330pF -> C_Small; footprint Capacitor_SMD:C_0603_1608Metric_Pad1.08x0.95mm_HandSolder -> Capacitor_SMD:C_1206_3216Metric_Pad1.33x1.80mm_HandSolder; moved to F.Cu
- C14: value 220pF -> C_Small; footprint Capacitor_SMD:C_0603_1608Metric_Pad1.08x0.95mm_HandSolder -> Capacitor_SMD:C_1206_3216Metric_Pad1.33x1.80mm_HandSolder; moved to F.Cu
- D7: value 1N5819HW-7-F -> 14V; footprint Diode_SMD:D_SOD-123 -> Diode_THT:D_DO-35_SOD27_P7.62mm_Horizontal
- R23: renamed from R11; value 29.4k -> ~
- R26: renamed from R6; value 2.2 -> ~
- TH1: value NTCS0402E3104JHT -> ~
- U1: renamed from U3; value PC817 -> PC817X2NSZ9F
- U2: renamed from U4; value TL431DBZ -> TL431IDBZT
- moved D7 110.9 mm to (38.9, 130.3)
- moved D6 104.9 mm to (40.8, 149.3), turned to 0 degrees
- moved D5 71.0 mm to (40.8, 146.0), turned to 0 degrees
- moved D2 66.8 mm to (40.8, 139.3)
- moved C11 66.3 mm to (40.6, 101.5), turned to 0 degrees
- moved C14 64.4 mm to (40.6, 111.6), turned to 0 degrees
- moved C13 63.4 mm to (40.6, 108.2), turned to 0 degrees
- moved C12 60.3 mm to (40.6, 104.9), turned to 0 degrees
- moved C15 59.9 mm to (40.6, 115.0), turned to 0 degrees
- moved Q2 0.37 mm to (106.9, 99.8)
- renumbered C24 to C1, C28 to C19, C23 to C2, C8 to C20, C9 to C21, C16 to C22, C20 to C23, C4 to C24, C17 to C25, C18 to C26, C19 to C27, C10 to C28, C3 to C29, C22 to C3, C1 to C30, C29 to C31, C5 to C32, C21 to C4, C6 to C5, C25 to C6, C26 to C7, C27 to C8, D9 to D8, R10 to R1, R19 to R10, R25 to R11, R24 to R12, R20 to R13, R7 to R14, R13 to R15, R14 to R16, R21 to R17, R22 to R18, R3 to R19, R8 to R2, R4 to R20, R2 to R21, R1 to R22, R23 to R24, R26 to R25, R9 to R3, R17 to R4, R15 to R5, R18 to R6, R16 to R7, R12 to R9, U1 to U3, U2 to U4
Connections:
- C11 pad 1: ISNS -> GNDPWR
- C11 pad 2: GNDPWR -> Net-(T1-OUT1A)
- C12 pad 1: /LLC Controller/Gate Driver/BLK -> GNDPWR
- C12 pad 2: GNDPWR -> Net-(T1-OUT1A)
- C13 pad 1: LL -> GNDPWR
- C13 pad 2: GNDPWR -> Net-(T1-OUT1A)
- C14 pad 1: TSET -> GNDPWR
- C14 pad 2: GNDPWR -> Net-(T1-OUT1A)
- C15 pad 1: OVP/OTP -> GNDPWR
- C15 pad 2: GNDPWR -> Net-(T1-OUT1A)
- C20 pad 2: ISNS -> Net-(C20-~-Pad2)
- D2 pad 1: VCCP -> /LLC Controller/Gate Driver/LO Driver
- D5 pad 1: /LLC Controller/Gate Driver/LO Driver -> VG1
- D6 pad 1: VG1 -> VG2
- D7 pad 1: VG2 -> VCCP
- D7 pad 2: Net-(D7-A) -> OVP/OTP
- R13 pad 1: Net-(D6-A) -> Net-(D5-A)
- R17 pad 1: Net-(D7-A) -> Net-(D6-A)
- R6 pad 1: Net-(D5-A) -> Net-(D2-A)
Routing:
- net V5P: track 16.6 -> 0.00 mm, vias 1 -> 0
- net LL: track 10.7 -> 0.00 mm, vias 1 -> 0
- net VD2: track 8.61 -> 0.00 mm, vias 1 -> 0
- net VCCP: track 8.52 -> 0.00 mm
- net Net-(U2-K): track 8.18 -> 0.00 mm
- net /LLC Controller/Gate Driver/BLK: track 7.67 -> 0.00 mm, vias 1 -> 0
- net TSET: track 7.62 -> 0.00 mm, vias 1 -> 0
- net Net-(U2-REF): track 7.07 -> 0.00 mm
- net +Vout: track 7.05 -> 0.00 mm
- net OVP/OTP: track 6.97 -> 0.00 mm, vias 1 -> 0
- net GNDPWR: track 6.28 -> 0.00 mm, vias 4 -> 0
- net Net-(D8-K): track 6.02 -> 0.00 mm
- net Net-(R10-Pad1): track 5.58 -> 0.00 mm
- net VG2: track 5.05 -> 0.00 mm
- net ISNS: track 3.50 -> 0.00 mm
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