File: llc-prototype/llc-prototype.kicad_sch (KiCad schematic)
At the start: 26 parts, among them J1 +HV, J2 -HV, J3 +LV, J4 -LV, Q1 NMOS, Q2 NMOS, Q3 NMOS, Q4 NMOS, T1 Transformer_SP_2S, U3 Optocoupler, U4 TL431DBZ

Commit message: fixed HV gnds
Connections:
- net +Vin: no longer Q1.1 (D)
- net GNDPWR: no longer Q2.3 (S)
- net LLC Controller/Gate Driver/HS Driver: no longer Q1.2 (G)
- net LLC Controller/Gate Driver/HS Return: no longer Q1.3 (S), Q2.1 (D)
- net LLC Controller/Gate Driver/LO Driver: no longer Q2.2 (G)
Other:
- note added: "apply gate drive tuning"
- moved on the sheet: Q1, Q2
Changed lines of the file:
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@@
 		)
 	)
+	(text "apply gate drive tuning\n"
+		(exclude_from_sim no)
+		(at 114.554 103.378 0)
+		(effects
+			(font
+				(size 1.27 1.27)
+			)
+		)
+	)
 	(text "drain voltage\nsense pins\n"
 		(exclude_from_sim no)
@@
 	(text "add info for both nmos\n"
 		(exclude_from_sim no)
-		(at 132.334 80.01 0)
+		(at 119.126 62.738 0)
 		(effects
 			(font
@@
 	)
 	(junction
-		(at 119.38 82.55)
-		(diameter 0)
-		(color 0 0 0 0)
-	)
-	(junction
 		(at 156.21 97.79)
 		(diameter 0)
@@
 	)
 	(junction
-		(at 119.38 97.79)
-		(diameter 0)
-		(color 0 0 0 0)
-	)
-	(junction
 		(at 243.84 140.97)
 		(diameter 0)
@@
 	(wire
 		(pts
-			(xy 110.49 74.93) (xy 111.76 74.93)
-		)
-		(stroke
-			(width 0)
-			(type default)
-		)
-	)
-	(wire
-		(pts
 			(xy 59.69 67.31) (xy 59.69 68.58)
 		)
@@
 	(wire
 		(pts
-			(xy 110.49 86.36) (xy 110.49 90.17)
-		)
-		(stroke
-			(width 0)
-			(type default)
-		)
-	)
-	(wire
-		(pts
-			(xy 119.38 80.01) (xy 119.38 82.55)
-		)
-		(stroke
-			(width 0)
-			(type default)
-		)
-	)
-	(wire
-		(pts
 			(xy 218.44 101.6) (xy 219.71 101.6)
 		)
@@
 	(wire
 		(pts
-			(xy 59.69 97.79) (xy 119.38 97.79)
-		)
-		(stroke
-			(width 0)
-			(type default)
-		)
-	)
-	(wire
-		(pts
 			(xy 195.58 66.04) (xy 201.93 66.04)
 		)
@@
 	(wire
 		(pts
-			(xy 119.38 97.79) (xy 119.38 95.25)
-		)
-		(stroke
-			(width 0)
-			(type default)
-		)
-	)
-	(wire
-		(pts
 			(xy 50.8 86.36) (xy 50.8 97.79)
 		)
@@
 	(wire
 		(pts
-			(xy 106.68 86.36) (xy 110.49 86.36)
-		)
-		(stroke
-			(width 0)
-			(type default)
-		)
-	)
-	(wire
-		(pts
 			(xy 59.69 67.31) (xy 76.2 67.31)
 		)
@@
 	(wire
 		(pts
-			(xy 119.38 97.79) (xy 135.89 97.79)
+			(xy 59.69 97.79) (xy 135.89 97.79)
 		)
 		(stroke
@@
 	(wire
 		(pts
-			(xy 106.68 82.55) (xy 119.38 82.55)
-		)
-		(stroke
-			(width 0)
-			(type default)
-		)
-	)
-	(wire
-		(pts
 			(xy 217.17 66.04) (xy 222.25 66.04)
 		)
@@
 	(wire
 		(pts
-			(xy 110.49 90.17) (xy 111.76 90.17)
-		)
-		(stroke
-			(width 0)
-			(type default)
-		)
-	)
-	(wire
-		(pts
 			(xy 226.06 151.13) (xy 243.84 151.13)
 		)
@@
 	(wire
 		(pts
-			(xy 119.38 82.55) (xy 140.97 82.55)
+			(xy 106.68 82.55) (xy 140.97 82.55)
 		)
 		(stroke
@@
 	(wire
 		(pts
-			(xy 119.38 82.55) (xy 119.38 85.09)
-		)
-		(stroke
-			(width 0)
-			(type default)
-		)
-	)
-	(wire
-		(pts
 			(xy 162.56 85.09) (xy 151.13 85.09)
 		)
@@
 	(wire
 		(pts
-			(xy 110.49 74.93) (xy 110.49 76.2)
-		)
-		(stroke
-			(width 0)
-			(type default)
-		)
-	)
-	(wire
-		(pts
 			(xy 50.8 67.31) (xy 59.69 67.31)
 		)
@@
 	(wire
 		(pts
-			(xy 119.38 69.85) (xy 119.38 67.31)
-		)
-		(stroke
-			(width 0)
-			(type default)
-		)
-	)
-	(wire
-		(pts
 			(xy 25.4 77.47) (xy 45.72 77.47)
 		)
@@
 	(wire
 		(pts
-			(xy 106.68 76.2) (xy 110.49 76.2)
-		)
-		(stroke
-			(width 0)
-			(type default)
-		)
-	)
-	(wire
-		(pts
 			(xy 250.19 92.71) (xy 250.19 93.98)
 		)
@@
 	(symbol
 		(lib_id "Simulation_SPICE:NMOS")
-		(at 116.84 90.17 0)
+		(at 125.73 90.17 0)
 		(unit 1)
 		(body_style 1)
@@
 		(fields_autoplaced yes)
 		(property "Reference" "Q2"
-			(at 123.19 88.8999 0)
+			(at 132.08 88.8999 0)
 			(show_name no)
 			(do_not_autoplace no)
@@
 		)
 		(property "Value" "NMOS"
-			(at 123.19 91.4399 0)
+			(at 132.08 91.4399 0)
 			(show_name no)
 			(do_not_autoplace no)
@@
 		)
 		(property "Footprint" ""
-			(at 121.92 87.63 0)
+			(at 130.81 87.63 0)
 			(hide yes)
 			(show_name no)
@@
 		)
 		(property "Datasheet" "https://ngspice.sourceforge.io/docs/ngspice-html-manual/manual.xhtml#cha_MOSFETs"
-			(at 116.84 102.87 0)
+			(at 125.73 102.87 0)
 			(hide yes)
 			(show_name no)
@@
 		)
 		(property "Description" "N-MOSFET transistor, drain/source/gate"
-			(at 116.84 90.17 0)
+			(at 125.73 90.17 0)
 			(hide yes)
 			(show_name no)
@@
 		)
 		(property "Sim.Device" "NMOS"
-			(at 116.84 107.315 0)
+			(at 125.73 107.315 0)
 			(hide yes)
 			(show_name no)
@@
 		)
 		(property "Sim.Type" "VDMOS"
-			(at 116.84 109.22 0)
+			(at 125.73 109.22 0)
 			(hide yes)
 			(show_name no)
@@
 		)
 		(property "Sim.Pins" "1=D 2=G 3=S"
-			(at 116.84 105.41 0)
+			(at 125.73 105.41 0)
 			(hide yes)
 			(show_name no)
@@
 	(symbol
 		(lib_id "Simulation_SPICE:NMOS")
-		(at 116.84 74.93 0)
+		(at 125.73 74.93 0)
 		(unit 1)
 		(body_style 1)
@@
 		(fields_autoplaced yes)
 		(property "Reference" "Q1"
-			(at 123.19 73.6599 0)
+			(at 132.08 73.6599 0)
 			(show_name no)
 			(do_not_autoplace no)
@@
 		)
 		(property "Value" "NMOS"
-			(at 123.19 76.1999 0)
+			(at 132.08 76.1999 0)
 			(show_name no)
 			(do_not_autoplace no)
@@
 		)
 		(property "Footprint" ""
-			(at 121.92 72.39 0)
+			(at 130.81 72.39 0)
 			(hide yes)
 			(show_name no)
@@
 		)
 		(property "Datasheet" "https://ngspice.sourceforge.io/docs/ngspice-html-manual/manual.xhtml#cha_MOSFETs"
-			(at 116.84 87.63 0)
+			(at 125.73 87.63 0)
 			(hide yes)
 			(show_name no)
@@
 		)
 		(property "Description" "N-MOSFET transistor, drain/source/gate"
-			(at 116.84 74.93 0)
+			(at 125.73 74.93 0)
 			(hide yes)
 			(show_name no)
@@
 		)
 		(property "Sim.Device" "NMOS"
-			(at 116.84 92.075 0)
+			(at 125.73 92.075 0)
 			(hide yes)
 			(show_name no)
@@
 		)
 		(property "Sim.Type" "VDMOS"
-			(at 116.84 93.98 0)
+			(at 125.73 93.98 0)
 			(hide yes)
 			(show_name no)
@@
 		)
 		(property "Sim.Pins" "1=D 2=G 3=S"
-			(at 116.84 90.17 0)
+			(at 125.73 90.17 0)
 			(hide yes)
 			(show_name no)

Commit message: fixes to schematic
Parts:
- added D4, D5: D, symbol Device:D
- added R15, R16, R17, R18: R_US, symbol Device:R_US
- Q1, Q2: value NMOS -> IRFB4227PBF; Digikey Part Number (none) -> 448-IRFB4227PBF-ND; Digikey URL (none) -> https://www.digikey.com/en/products/detail/infineon-technol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
- R12: value R_US -> 1200
- R13: value R_US -> 43.2k
- R14: value R_US -> 10k
- T1: footprint FS_4_Global_Footprint_Library:DIPS4064W80P508L5450H4090Q20N -> (none)
- U3: value Optocoupler -> PC817X2NSZ9F
Connections:
- net LLC Controller/Gate Driver/HS Return is gone; now on net LLC Controller/Gate Driver/HI Return: T1.5 (OUT1B)
- net +Vin: now also Q1.1 (D)
- net GNDPWR: now also Q2.3 (S)
- net LLC Controller/Gate Driver/LO Driver: now also D5.1 (K), R16.1
- net LLC Controller/Gate Driver/HI Return: now reaches Q2.1 (D)
- net LLC Controller/Gate Driver/HI Return: now also Q1.3 (S)
- net at Q2.2 (G): now also R16.2, R18.2
- net at Q1.2 (G): now also R15.2, R17.2
- new net: D5.2 (A), R18.1
- new net: D4.2 (A), R17.1
- new net LLC Controller/Gate Driver/HI Driver: D4.1 (K), R15.1
Other:
- sheet LLC Controller/Gate Driver ports: added HI Driver, HI Return; removed HS Driver, HS Return
- note removed: "Look into FOD817CSD optocoupler"
- note removed: "Vref: Configure Voltage Divider to program Shunt Regulator"
- moved on the sheet: C2, C4, C6, C7, C8, C9, D2, J1, J2, J3, J4, Q2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

Commit message: update footprints to pcb editor
Parts:
- removed C9: C, symbol Device:C
- removed U3: PC817X2NSZ9F, symbol Isolator:SFH617A-1
- added C9: C_Small, Capacitor_SMD:C_0603_1608Metric_Pad1.08x0.95mm_HandSolder, symbol Device:C_Small
- added D6, D7: 1N5819HW-7-F, Diode_SMD:D_SOD-123, symbol Device:D
- added R19: R_Small_US, Resistor_SMD:R_0603_1608Metric_Pad0.98x0.95mm_HandSolder, symbol Device:R_Small_US
- added R20, R21: 3.09, Resistor_SMD:R_0603_1608Metric_Pad0.98x0.95mm_HandSolder, symbol Device:R_US
- added U3: PC817, Package_DIP:DIP-4_W7.62mm, symbol Isolator:PC817
- C2, C4, C6, C7, C8: footprint (none) -> Capacitor_SMD:C_0603_1608Metric_Pad1.08x0.95mm_HandSolder
- D2, D4, D5: value D -> 1N5819HW-7-F; footprint (none) -> Diode_SMD:D_SOD-123
- Q1, Q2: value IRFB4227PBF -> MCTL011N20YH-TP; footprint (none) -> Package_TO_SOT_SMD:Infineon_PG-HSOF-8-1_ThermalVias; Digikey Part Number 448-IRFB4227PBF-ND -> (none); Digikey URL https://www.digikey.com/en/products/detail/infineon-technol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 -> (none)
- Q3, Q4: value NMOS -> NTMFS1D3N04XMT1G; footprint (none) -> Package_SO:ONSemi_SO-8FL_488AA
- R10: footprint Resistor_SMD:R_0201_0603Metric_Pad0.64x0.40mm_HandSolder -> Resistor_SMD:R_0603_1608Metric_Pad0.98x0.95mm_HandSolder
- R15, R16: value R_US -> 20.5; footprint (none) -> Resistor_SMD:R_0603_1608Metric_Pad0.98x0.95mm_HandSolder
- R17, R18: value R_US -> 10.5; footprint (none) -> Resistor_SMD:R_0603_1608Metric_Pad0.98x0.95mm_HandSolder
- R6, R7: value R -> 8.06
Connections:
- net +Vin: now also Q1.3 (D); no longer Q1.1 (D)
- net +Vout: now also Q3.1 (S), Q4.1 (S), R19.1; no longer Q3.3 (S), Q4.3 (S)
- net FB: now also U3.4
- net GNDPWR: now also Q2.2 (S), U3.3; no longer Q2.3 (S)
- net LLC Controller/Gate Driver/HI Return: now also Q1.2 (S), Q2.3 (D); no longer Q1.3 (S), Q2.1 (D)
- net VD1: now also Q3.5 (D); no longer Q3.1 (D)
- net VD2: now also Q4.5 (D); no longer Q4.1 (D)
- net at R13.2, R14.1, U4.2 (REF): now also C9.2
- net at R15.2, R17.2: now also Q1.1 (G); no longer Q1.2 (G)
- net at R7.2: now also Q3.4 (G); no longer Q3.2 (G)
- net at R6.2: now also Q4.4 (G); no longer Q4.2 (G)
- net at R12.2: now also U3.1
- net at U4.1 (K): now also C9.1, R19.2, U3.2
- net at R16.2, R18.2: now also Q2.1 (G); no longer Q2.2 (G)
Other:
- note added: "160uA of Current is supplied by UCC256612"
- note removed: "Current flows out of FB pin"
- note removed: "Used 2 Resistor in Series because of Max Working Voltage"
- note removed: "add info for both nmos"
- note removed: "apply gate drive tuning"
- note removed: "select smoothing cap"
- moved on the sheet: R13

Commit message: added fuses
Parts:
- removed R6: 8.06, Resistor_SMD:R_0603_1608Metric_Pad0.98x0.95mm_HandSolder, symbol Device:R_US
- added F1, F2: Fuse, symbol Device:Fuse
- added R22: 8.06, Resistor_SMD:R_0603_1608Metric_Pad0.98x0.95mm_HandSolder, symbol Device:R_US
Connections:
- net +Vin: now also F1.2; no longer J1.1 (Pin_1)
- net +Vout: now also T1.2 (PM), F2.1; no longer J3.1 (Pin_1), Q3.1 (S), Q4.1 (S)
- net GND: now also Q3.1 (S), Q4.1 (S); no longer T1.2 (PM)
- net VG1: now also D6.1 (K)
- net VG2: now also D7.1 (K), R22.1
- net at Q3.4 (G), R7.2: now also R20.2
- net at D7.2 (A): now also R21.1
- net at Q4.4 (G): now also R21.2, R22.2
- net at R20.1: now also D6.2 (A)
- new net: F1.1, J1.1 (Pin_1)
- new net: F2.2, J3.1 (Pin_1)
Other:
- note added: "Feedback"
- moved on the sheet: C2, C4, C6, C7, C8, C9, D2, D4, D5, D6, J1, J2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

Commit message: PCB work, added more caps
Parts:
- removed C4, C6, C7: C, Capacitor_SMD:C_0603_1608Metric_Pad1.08x0.95mm_HandSolder, symbol Device:C
- removed F1, F2: Fuse, symbol Device:Fuse
- added C16, C17, C18, C19, C20, C21, C22, C23, C24, C25, C26, C27, C28, C4, C6: C_Small, Capacitor_SMD:C_0603_1608Metric_Pad1.08x0.95mm_HandSolder, symbol Device:C_Small
- added D8: D_Zener, symbol Device:D_Zener
- added R24: R_Small_US, Resistor_SMD:R_0603_1608Metric_Pad0.98x0.95mm_HandSolder, symbol Device:R_Small_US
- added R25: 1200, Resistor_SMD:R_0603_1608Metric_Pad0.98x0.95mm_HandSolder, symbol Device:R_US
Connections:
- net +Vin: now also J1.1 (Pin_1), C21.1, C22.1, C23.1, C24.1, C6.1
- net +Vout: now also J3.1 (Pin_1), C17.1, C18.1, C19.1, C20.1, C4.1, R25.2; no longer R12.1, R19.1
- net GND: now also C17.2, C18.2, C19.2, C20.2, C4.2, D8.2 (A)
- net GNDPWR: now also C21.2, C22.2, C23.2, C24.2, C25.2, C26.2, C27.2, C28.2, C6.2
- net VCCP: now also C25.1, C26.1, C27.1, C28.1
- net at R13.2, R14.1, U4.2 (REF): now also C16.2, R24.2; no longer C9.2
- net at R12.2, U3.1: now also R19.1
- net at C9.1, R19.2, U3.2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: now also C16.1
- new net: C9.2, R24.1
- new net: D8.1 (K), R12.1, R25.1
Other:
- note removed: "Use Tertiary winding to supply VCCP - will also implement OVP"
- moved on the sheet: D2, J1, J2, J3, J4, R12, R13, R14, U3, U4

Commit message: pcb changes + fs-components update
Parts:
- Q3, Q4: footprint Package_SO:ONSemi_SO-8FL_488AA -> formula_slug_footprint_library:ONSemi_SO-8FL_488AA_editedForLLC
Changed lines of the file:
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@@
 	)
 	(junction
-		(at 298.45 139.7)
-		(diameter 0)
-		(color 0 0 0 0)
-	)
-	(junction
 		(at 76.2 118.11)
 		(diameter 0)
@@
 	)
 	(junction
+		(at 298.45 139.7)
+		(diameter 0)
+		(color 0 0 0 0)
+	)
+	(junction
 		(at 184.15 115.57)
 		(diameter 0)
@@
 	)
 	(symbol
-		(lib_name "NMOS_3")
-		(lib_id "Simulation_SPICE:NMOS")
-		(at 303.53 139.7 0)
-		(unit 1)
-		(body_style 1)
-		(exclude_from_sim no)
-		(in_bom yes)
-		(on_board yes)
-		(in_pos_files yes)
-		(dnp no)
-		(property "Reference" "Q4"
-			(at 308.356 144.018 0)
-			(show_name no)
-			(do_not_autoplace no)
-			(effects
-				(font
-					(size 1.27 1.27)
-				)
-				(justify left)
-			)
-		)
-		(property "Value" "NTMFS1D3N04XMT1G"
-			(at 308.356 146.558 0)
-			(show_name no)
-			(do_not_autoplace no)
-			(effects
-				(font
-					(size 1.27 1.27)
-				)
-				(justify left)
-			)
-		)
-		(property "Footprint" "Package_SO:ONSemi_SO-8FL_488AA"
-			(at 308.61 137.16 0)
-			(hide yes)
-			(show_name no)
-			(do_not_autoplace no)
-			(effects
-				(font
-					(size 1.27 1.27)
-				)
-			)
-		)
-		(property "Datasheet" "https://www.onsemi.com/download/data-sheet/pdf/ntmfs1d3n04xm-d.pdf"
-			(at 303.53 152.4 0)
-			(hide yes)
-			(show_name no)
-			(do_not_autoplace no)
-			(effects
-				(font
-					(size 1.27 1.27)
-				)
-			)
-		)
-		(property "Description" "N-MOSFET transistor, drain/source/gate"
-			(at 303.53 139.7 0)
-			(hide yes)
-			(show_name no)
-			(do_not_autoplace no)
-			(effects
-				(font
-					(size 1.27 1.27)
-				)
-			)
-		)
-		(property "Sim.Device" "NMOS"
-			(at 303.53 156.845 0)
-			(hide yes)
-			(show_name no)
-			(do_not_autoplace no)
-			(effects
-				(font
-					(size 1.27 1.27)
-				)
-			)
-		)
-		(property "Sim.Type" "VDMOS"
-			(at 303.53 158.75 0)
-			(hide yes)
-			(show_name no)
-			(do_not_autoplace no)
-			(effects
-				(font
-					(size 1.27 1.27)
-				)
-			)
-		)
-		(property "Sim.Pins" "1=D 2=G 3=S"
-			(at 303.53 154.94 0)
-			(hide yes)
-			(show_name no)
-			(do_not_autoplace no)
-			(effects
-				(font
-					(size 1.27 1.27)
-				)
-			)
-		)
-		(property "Digikey Part Number" ""
-			(at 303.53 139.7 0)
-			(hide yes)
-			(show_name no)
-			(do_not_autoplace no)
-			(effects
-				(font
-					(size 1.27 1.27)
-				)
-			)
-		)
-		(property "Digikey URL" ""
-			(at 303.53 139.7 0)
-			(hide yes)
-			(show_name no)
-			(do_not_autoplace no)
-			(effects
-				(font
-					(size 1.27 1.27)
-				)
-			)
-		)
-		(property "Manufacturer" ""
-			(at 303.53 139.7 0)
-			(hide yes)
-			(show_name no)
-			(do_not_autoplace no)
-			(effects
-				(font
-					(size 1.27 1.27)
-				)
-			)
-		)
-		(property "Manufacturer Part Number" ""
-			(at 303.53 139.7 0)
-			(hide yes)
-			(show_name no)
-			(do_not_autoplace no)
-			(effects
-				(font
-					(size 1.27 1.27)
-				)
-			)
-		)
-		(pin "5"
-		)
-		(pin "1"
-		)
-		(pin "4"
-		)
-		(instances
-			(project "llc-prototype"
-				(path "/e994741c-7c7d-4124-9d00-43b883baa61d"
-					(reference "Q4")
-					(unit 1)
-				)
-			)
-		)
-	)
-	(symbol
 		(lib_id "Device:C_Small")
 		(at 242.57 195.58 90)
@@
 			)
 		)
-		(property "Footprint" "Package_SO:ONSemi_SO-8FL_488AA"
+		(property "Footprint" "formula_slug_footprint_library:ONSemi_SO-8FL_488AA_editedForLLC"
 			(at 267.97 137.16 0)
 			(hide yes)
@@
 					(unit 1)
 				)
+			)
+		)
+	)
+	(symbol
+		(lib_name "NMOS_2")
+		(lib_id "Simulation_SPICE:NMOS")
+		(at 303.53 139.7 0)
+		(unit 1)
+		(body_style 1)
+		(exclude_from_sim no)
+		(in_bom yes)
+		(on_board yes)
+		(in_pos_files yes)
+		(dnp no)
+		(property "Reference" "Q4"
+			(at 308.356 144.018 0)
+			(show_name no)
+			(do_not_autoplace no)
+			(effects
+				(font
+					(size 1.27 1.27)
+				)
+				(justify left)
+			)
+		)
+		(property "Value" "NTMFS1D3N04XMT1G"
+			(at 308.356 146.558 0)
+			(show_name no)
+			(do_not_autoplace no)
+			(effects
+				(font
+					(size 1.27 1.27)
+				)
+				(justify left)
+			)
+		)
+		(property "Footprint" "formula_slug_footprint_library:ONSemi_SO-8FL_488AA_editedForLLC"
+			(at 308.61 137.16 0)
+			(hide yes)
+			(show_name no)
+			(do_not_autoplace no)
+			(effects
+				(font
+					(size 1.27 1.27)
+				)
+			)
+		)
+		(property "Datasheet" "https://www.onsemi.com/download/data-sheet/pdf/ntmfs1d3n04xm-d.pdf"
+			(at 303.53 152.4 0)
+			(hide yes)
+			(show_name no)
+			(do_not_autoplace no)
+			(effects
+				(font
+					(size 1.27 1.27)
+				)
+			)
+		)
+		(property "Description" "N-MOSFET transistor, drain/source/gate"
+			(at 303.53 139.7 0)
+			(hide yes)
+			(show_name no)
+			(do_not_autoplace no)
+			(effects
+				(font
+					(size 1.27 1.27)
+				)
+			)
+		)
+		(property "Sim.Device" "NMOS"
+			(at 303.53 156.845 0)
+			(hide yes)
+			(show_name no)
+			(do_not_autoplace no)
+			(effects
+				(font
+					(size 1.27 1.27)
+				)
+			)
+		)
+		(property "Sim.Type" "VDMOS"
+			(at 303.53 158.75 0)
+			(hide yes)
+			(show_name no)
+			(do_not_autoplace no)
+			(effects
+				(font
+					(size 1.27 1.27)
+				)
+			)
+		)
+		(property "Sim.Pins" "1=D 2=G 3=S"
+			(at 303.53 154.94 0)
+			(hide yes)
+			(show_name no)
+			(do_not_autoplace no)
+			(effects
+				(font
+					(size 1.27 1.27)
+				)
+			)
+		)
+		(property "Digikey Part Number" ""
+			(at 303.53 139.7 0)
+			(hide yes)
+			(show_name no)
+			(do_not_autoplace no)
+			(effects
+				(font
+					(size 1.27 1.27)
+				)
+			)
+		)
+		(property "Digikey URL" ""
+			(at 303.53 139.7 0)
+			(hide yes)
+			(show_name no)
+			(do_not_autoplace no)
+			(effects
+				(font
+					(size 1.27 1.27)
+				)
+			)
+		)
+		(property "Manufacturer" ""
+			(at 303.53 139.7 0)
+			(hide yes)
+			(show_name no)
+			(do_not_autoplace no)
+			(effects
+				(font
+					(size 1.27 1.27)
+				)
+			)
+		)
+		(property "Manufacturer Part Number" ""
+			(at 303.53 139.7 0)
+			(hide yes)
+			(show_name no)
+			(do_not_autoplace no)
+			(effects
+				(font
+					(size 1.27 1.27)
+				)
+			)
+		)
+		(pin "5"
+		)
+		(pin "1"
+		)
+		(pin "4"
+		)
+		(instances
+			(project "llc-prototype"
+				(path "/e994741c-7c7d-4124-9d00-43b883baa61d"
+					(reference "Q4")
+					(unit 1)
+				)

Commit message: changed hb mosfet footprint
Parts:
- Q1, Q2: footprint Package_TO_SOT_SMD:Infineon_PG-HSOF-8-1_ThermalVias -> Package_TO_SOT_SMD:Infineon_PG-HSOF-8-1
Changed lines of the file:
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@@
 			)
 		)
-		(property "Footprint" "Package_TO_SOT_SMD:Infineon_PG-HSOF-8-1_ThermalVias"
+		(property "Footprint" "Package_TO_SOT_SMD:Infineon_PG-HSOF-8-1"
 			(at 186.69 120.65 0)
 			(hide yes)
@@
 			)
 		)
-		(property "Footprint" "Package_TO_SOT_SMD:Infineon_PG-HSOF-8-1_ThermalVias"
+		(property "Footprint" "Package_TO_SOT_SMD:Infineon_PG-HSOF-8-1"
 			(at 186.69 106.68 0)
 			(hide yes)
