File: llc-prototype/llc-prototype.kicad_sch (KiCad schematic)
At the start: 52 parts, among them J1 +HV, J2 -HV, J3 +LV, J4 -LV, Q1 MCTL011N20YH-TP, Q2 MCTL011N20YH-TP, Q3 NTMFS1D3N04XMT1G, Q4 NTMFS1D3N04XMT1G, T1 Transformer_SP_2S, U3 PC817, U4 TL431DBZ

Commit message: schematic
Parts:
- removed C2: 1uF, Capacitor_SMD:C_0603_1608Metric_Pad1.08x0.95mm_HandSolder, symbol Device:C
- removed D4, D7: 1N5819HW-7-F, Diode_SMD:D_SOD-123, symbol Device:D
- removed R16: 20.5, Resistor_SMD:R_0603_1608Metric_Pad0.98x0.95mm_HandSolder, symbol Device:R_US
- removed R18: 10.5, Resistor_SMD:R_0603_1608Metric_Pad0.98x0.95mm_HandSolder, symbol Device:R_US
- added C10, C11, C12, C13, C14, C15, C16, C17, C18, C9: C_Small, Capacitor_SMD:C_1206_3216Metric_Pad1.33x1.80mm_HandSolder, symbol Device:C_Small
- added D1, D3: 1N5819HW-7-F, Diode_SMD:D_SOD-123, symbol Device:D
- added R2: 576k, Resistor_SMD:R_0603_1608Metric_Pad0.98x0.95mm_HandSolder, symbol Device:R_Small_US
- added R6: 10.5, Resistor_SMD:R_0603_1608Metric_Pad0.98x0.95mm_HandSolder, symbol Device:R_US
- added R7: 20.5, Resistor_SMD:R_0603_1608Metric_Pad0.98x0.95mm_HandSolder, symbol Device:R_US
- C20: renamed from C8; Digikey Part Number (none) -> 399-C0603C151J2GACTUCT-ND; Digikey URL (none) -> https://www.digikey.com/en/products/detail/kemet/C0603C151J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; Manufacturer (none) -> KEMET; Manufacturer Part Number (none) -> C0603C151J2GACTU
- D2, D5, D6: Digikey Part Number (none) -> 1N5819HW-FDICT-ND; Digikey URL (none) -> https://www.digikey.com/en/products/detail/diodes-incorpora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; Manufacturer (none) -> Diodes Incorporated; Manufacturer Part Number (none) -> 1N5819HW-7-F
- Q1, Q2: Digikey Part Number (none) -> 353-MCTL011N20YH-TPCT-ND; Digikey URL (none) -> https://www.digikey.com/en/products/detail/mcc-micro-commer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; Manufacturer (none) -> MCC (Micro Commercial Components); Manufacturer Part Number (none) -> MCTL011N20YH-TP
- R1: renamed from R10; Digikey Part Number (none) -> P576KHCT-ND; Digikey URL (none) -> https://www.digikey.com/en/products/detail/panasonic-indust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; Manufacturer (none) -> Panasonic Industry; Manufacturer Part Number (none) -> ERJ-3EKF5763V
- R3: renamed from R9; Digikey Part Number (none) -> 311-18KGRCT-ND; Digikey URL (none) -> https://www.digikey.com/en/products/detail/yageo/RC0603JR-0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; Manufacturer (none) -> YAGEO; Manufacturer Part Number (none) -> RC0603JR-0718KL
- R4: renamed from R17; Digikey Part Number (none) -> P10.5HCT-ND; Digikey URL (none) -> https://www.digikey.com/en/products/detail/panasonic-indust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; Manufacturer (none) -> Panasonic Industry; Manufacturer Part Number (none) -> ERJ-3EKF10R5V
- R5: renamed from R15; Digikey Part Number (none) -> 311-20.5HRCT-ND; Digikey URL (none) -> https://www.digikey.com/en/products/detail/yageo/RC0603FR-0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; Manufacturer (none) -> YAGEO; Manufacturer Part Number (none) -> RC0603FR-0720R5L
- R8: value 576k -> 510; DigiKey URL https://www.digikey.com/en/products/detail/panasonic-indust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 -> (none); Digikey Part Number (none) -> P510GCT-ND; Digikey URL (none) -> https://www.digikey.com/en/products/detail/panasonic-indust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; Manufacturer (none) -> Panasonic Industry; Manufacturer Part Number (none) -> ERJ-3GEYJ511V
- U1: renamed from U3; value PC817 -> PC817X2NSZ9F; Digikey Part Number (none) -> PC817X2NSZ9F-ND; Digikey URL (none) -> https://www.digikey.com/en/products/detail/sharp-socle-tech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; Manufacturer (none) -> SHARP/Socle Technology; Manufacturer Part Number (none) -> PC817X2NSZ9F
- U2: renamed from U4; value TL431DBZ -> TL431IDBZT; Digikey Part Number (none) -> 296-26719-1-ND; Digikey URL (none) -> https://www.digikey.com/en/products/detail/texas-instrument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; Manufacturer (none) -> Texas Instruments; Manufacturer Part Number (none) -> TL431IDBZT
- renumbered C24 to C1, C28 to C19, C23 to C2, C9 to C21, C16 to C22, C20 to C23, C4 to C24, C17 to C25, C18 to C26, C19 to C27, C22 to C3, C21 to C4, C6 to C5, C25 to C6, C26 to C7, C27 to C8, D8 to D4, R19 to R10, R25 to R11, R24 to R12, R20 to R13, R7 to R14, R13 to R15, R14 to R16, R21 to R17, R22 to R18, R12 to R9
Connections:
- net GNDPWR: now also C10.1, C11.1, C12.1, C13.1, C14.1, C15.1, C16.1, C17.1, C18.1, C9.1
- net ISNS: now also R8.2; no longer C20.2
- net LLC Controller/Gate Driver/BLK: now also R2.2; no longer R8.2
- net LLC Controller/Gate Driver/HI Driver: now also D1.1 (K)
- net LLC Controller/Gate Driver/LO Driver: now also D2.1 (K), R7.1; no longer D5.1 (K)
- net VCCP: now also D3.1 (K); no longer D2.1 (K)
- net VG1: now also D5.1 (K); no longer D6.1 (K)
- net VG2: now also D6.1 (K)
- net at R1.2: now also R2.1; no longer R8.1
- net at R4.1: now also D1.2 (A)
- net at Q2.1 (G): now also R6.2, R7.2
- net at C20.1, T1.4 (OUT1A): now also C10.2, C11.2, C12.2, C13.2, C14.2, C15.2, C16.2, C17.2, C18.2, C9.2
- net at R17.1: now also D6.2 (A)
- net at D5.2 (A): now also R13.1
- net at T1.7 (OUT2B): now also D3.2 (A); no longer D2.2 (A)
- new net: D2.2 (A), R6.1
- new net: C20.2, R8.1
Other:
- note added: "Lr = 1.1uH Lm = 6uH"
- note removed: "Lr = 1.126uH Lm = 6uH"
- moved on the sheet: R10
