File: strain-gauge-board/strain-gauge-board.kicad_sch (KiCad schematic)
At the start: 17 parts, among them U1 TLV172IDCK, U2 TLV172IDCK, U3 TLV172IDCK

Commit message: Layout help please
Parts:
- removed R1, R2, R3: R_45deg, symbol Device:R_45deg
- removed R4, R5, R6, R7: R, symbol Device:R
- removed U1, U2: TLV172IDCK, Package_TO_SOT_SMD:SOT-353_SC-70-5, symbol Amplifier_Operational:TLV172IDCK
Connections:
- net GND is gone; now on net +5V: R10.2, R11.2, R14.2
Other:
- note removed: "strain gauge"
- moved on the sheet: R10, R11, R12, R13, R14, R8, R9, U3

Commit message: more!
Parts:
- added R15, R18: R_US, symbol Device:R_US
Connections:
- net +5V: now also R15.1, R15.2, R18.2
Other:
- note added: "strain gauge"
