File: charging-board/charging-board.kicad_sch (KiCad schematic)
At the start: 53 parts, among them J1 Conn_02x13_Counter_Clockwise, J12 everything_connector, J13 FTSH-107-01-F-DV-K-P-TR, J2 Conn_01x04, J6 TSMP_to_HV, J7 TSMP_to_Banana Jacks, J8 J1772_Negotiation, SW1 Y97KT23B5NAFP, U1 AP63205WU, U2 ISO1044BD, U3 STM32G441KBTx, U7 MIC5504-3.3YM5, Y2 ECS-240-8-37B-CKY-TR

Commit message: added discharge relay
Parts:
- added J10: TSMP_to_Banana Jacks, Connector_Molex:Molex_Nano-Fit_105309-xx02_1x02_P2.50mm_Vertical, symbol Connector:Conn_01x02_Pin
- added J9: TSMP_to_HV, Connector_Molex:Molex_Nano-Fit_105309-xx02_1x02_P2.50mm_Vertical, symbol Connector:Conn_01x02_Pin
- added K1: Relay_SPDT, symbol Relay:Relay_SPDT
- added R14, R15: 5k, Resistor_THT:R_Axial_DIN0922_L20.0mm_D9.0mm_P25.40mm_Horizontal, symbol Device:R
- added R16: 25W, symbol Device:R
- added R4: 5K, symbol Device:R
Connections:
- net GND: now also R4.2
- net Shutdown_Acc_Out renamed IRs_Final
- net IRs_Final: now also K1.A2
- new net: J10.2 (Pin_2), R15.1
- new net: K1.12, R15.2
- new net: J9.1 (Pin_1), K1.11
- new net: J9.2 (Pin_2), R14.2, R16.1
- new net: K1.14, R16.2
- new net: J10.1 (Pin_1), R14.1
- new net: K1.A1, R4.1
Other:
- note added: "TSMPs and Shutdown Discharge"
- note removed: "IRs_Final"
- moved on the sheet: H1, H2

Commit message: switched to SPST relay
Parts:
- K1: value Relay_SPDT -> Relay_SPST_NO; footprint (none) -> formula_slug_footprint_library:RELAY_PR30-12V-450-1A-E; symbol Relay:Relay_SPDT -> Relay:Relay_SPST-NO
Connections:
- net at R15.2: now also J9.1 (Pin_1), K1.5; no longer K1.12
- net at R16.2: now also K1.8; no longer K1.14
Changed lines of the file:
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@@
 	)
 	(junction
+		(at 114.3 149.86)
+		(diameter 0)
+		(color 0 0 0 0)
+	)
+	(junction
 		(at 33.02 158.75)
 		(diameter 0)
@@
 	(wire
 		(pts
-			(xy 137.16 166.37) (xy 144.78 166.37)
-		)
-		(stroke
-			(width 0)
-			(type default)
-		)
-	)
-	(wire
-		(pts
 			(xy 165.1 30.48) (xy 168.91 30.48)
 		)
@@
 	(wire
 		(pts
-			(xy 144.78 149.86) (xy 149.86 149.86)
-		)
-		(stroke
-			(width 0)
-			(type default)
-		)
-	)
-	(wire
-		(pts
 			(xy 57.15 153.67) (xy 58.42 153.67)
 		)
@@
 	(wire
 		(pts
-			(xy 144.78 166.37) (xy 144.78 149.86)
-		)
-		(stroke
-			(width 0)
-			(type default)
-		)
-	)
-	(wire
-		(pts
 			(xy 31.75 44.45) (xy 35.56 44.45)
 		)
@@
 	(wire
 		(pts
+			(xy 114.3 149.86) (xy 149.86 149.86)
+		)
+		(stroke
+			(width 0)
+			(type default)
+		)
+	)
+	(wire
+		(pts
 			(xy 172.72 67.31) (xy 176.53 67.31)
 		)
@@
 	)
 	(symbol
-		(lib_id "Relay:Relay_SPDT")
+		(lib_id "Relay:Relay_SPST-NO")
 		(at 129.54 168.91 270)
 		(mirror x)
@@
 			)
 		)
-		(property "Value" "Relay_SPDT"
-			(at 118.618 169.164 90)
+		(property "Value" "Relay_SPST_NO"
+			(at 117.094 169.164 90)
 			(show_name no)
 			(do_not_autoplace no)
@@
 			)
 		)
-		(property "Footprint" ""
+		(property "Footprint" "formula_slug_footprint_library:RELAY_PR30-12V-450-1A-E"
 			(at 128.27 157.48 0)
 			(hide yes)
@@
 			)
 		)
-		(property "Description" "Relay SPDT, monostable, EN50005"
+		(property "Description" "Relay SPST, normally open, EN50005"
 			(at 129.54 168.91 0)
 			(hide yes)
@@
 			)
 		)
-		(pin "11"
+		(property "Digikey Part Number" ""
+			(at 129.54 168.91 0)
+			(hide yes)
+			(show_name no)
+			(do_not_autoplace no)
+			(effects
+				(font
+					(size 1.27 1.27)
+				)
+			)
 		)
-		(pin "14"
+		(property "Digikey URL" ""
+			(at 129.54 168.91 0)
+			(hide yes)
+			(show_name no)
+			(do_not_autoplace no)
+			(effects
+				(font
+					(size 1.27 1.27)
+				)
+			)
 		)
-		(pin "12"
+		(property "Manufacturer" ""
+			(at 129.54 168.91 0)
+			(hide yes)
+			(show_name no)
+			(do_not_autoplace no)
+			(effects
+				(font
+					(size 1.27 1.27)
+				)
+			)
+		)
+		(property "Manufacturer Part Number" ""
+			(at 129.54 168.91 0)
+			(hide yes)
+			(show_name no)
+			(do_not_autoplace no)
+			(effects
+				(font
+					(size 1.27 1.27)
+				)
+			)
+		)
+		(pin "8"
+		)
+		(pin "5"
 		)
 		(pin "A2"

Commit message: Just values
Parts:
- K1: value Relay_SPST_NO -> RELAY_PR30-12V-450-1A-E
Changed lines of the file:
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@@
 			)
 		)
-		(property "Value" "Relay_SPST_NO"
-			(at 117.094 169.164 90)
+		(property "Value" "RELAY_PR30-12V-450-1A-E"
+			(at 123.952 168.91 90)
 			(show_name no)
 			(do_not_autoplace no)
@@
 					(size 1.27 1.27)
 				)
+				(justify right)
 			)
 		)

Commit message: Removed duplicate TSMP circuit in schematic
Parts:
- removed J6: TSMP_to_HV, Connector_Molex:Molex_Nano-Fit_105309-xx02_1x02_P2.50mm_Vertical, symbol Connector:Conn_01x02_Pin
- removed J7: TSMP_to_Banana Jacks, Connector_Molex:Molex_Nano-Fit_105309-xx02_1x02_P2.50mm_Vertical, symbol Connector:Conn_01x02_Pin
- removed R5, R6: 5k, Resistor_THT:R_Axial_DIN0922_L20.0mm_D9.0mm_P25.40mm_Horizontal, symbol Device:R
- R4: footprint (none) -> Resistor_SMD:R_0603_1608Metric_Pad0.98x0.95mm_HandSolder
- renumbered R14 to R5, R15 to R6
Connections:
- net at J9.1 (Pin_1), R6.2: now also K1.13; no longer K1.5
- net at R16.2: now also K1.14; no longer K1.8
Other:
- note removed: "TSMPs"

Commit message: minor changes
Parts:
- removed R16: 25W, symbol Device:R
- added J3: Conn_01x07_Socket, Connector_FFC-FPC:Molex_200528-0070_1x07-1MP_P1.00mm_Horizontal, symbol Connector:Conn_01x07_Socket
- added J4: Discharge Resistor Nanofit Connector, Connector_Molex:Molex_Nano-Fit_105313-xx02_1x02_P2.50mm_Horizontal, symbol Connector:Conn_01x02_Socket
Connections:
- net +3V3: now also J3.1 (Pin_1)
- net +5V: now also J3.2 (Pin_2)
- net GND: now also J3.7 (Pin_7)
- net SPI.CLK: now also J3.4 (Pin_4)
- net SPI.CS: now also J3.3 (Pin_3)
- net SPI.MISO: now also J3.5 (Pin_5)
- net SPI.MOSI: now also J3.6 (Pin_6)
- net at J9.2 (Pin_2), R5.2: now also J4.1 (Pin_1)
- net at K1.14: now also J4.2 (Pin_2)
- net driver_power: no longer names the net of U3.30 (PB7)
Other:
- removed sheet screen-architecture
- note added: "Resistor must be <25W"
- note added: "SPI Connector to Screen Driver"
- moved on the sheet: H1, H2
