File: test-module-busbar-board/template.kicad_pcb (KiCad board)
At the start: 2 copper layers, 142.6 x 70.4 mm, 8 parts

Commit message: done
Parts:
- moved H2 160.9 mm to (190.8, 85.5)
- moved F2 149.5 mm to (196.0, 74.2)
- moved H4 45.7 mm to (68.3, 115.7)
- moved H3 44.1 mm to (68.3, 105.5)
- moved F3 40.0 mm to (71.5, 98.8), turned to 180 degrees
- moved H1 38.4 mm to (68.3, 65.5)
- moved F4 31.5 mm to (64.5, 98.8)
- moved F1 25.6 mm to (70.8, 55.5), turned to 180 degrees
Connections:
- H1 pad 1: (no net) -> /cell_2_fused
- H2 pad 1: (no net) -> /cell_1_fused
- H3 pad 1: (no net) -> /cell_0_fused
- H4 pad 1: (no net) -> /cell_0_minus_fused
Routing:
- net /cell_0_minus: track 0.00 -> 34.0 mm
- net /cell_0_minus_fused: track 0.00 -> 19.0 mm
- net /cell_1_fused: track 0.00 -> 11.8 mm
- net /cell_1_plus: track 0.00 -> 11.8 mm
- net /cell_0_fused: track 0.00 -> 10.2 mm
- net /cell_2_fused: track 0.00 -> 7.57 mm
- net /cell_2_plus: track 0.00 -> 3.75 mm
- net /cell_0_plus: track 0.00 -> 2.84 mm
