File: test-module-busbar-board/template.kicad_pcb (KiCad board)
At the start: 2 copper layers, 142.6 x 70.4 mm, 8 parts

Commit message: moved voltage tap
Parts:
- moved H2 3.00 mm to (193.8, 85.5)
Routing:
- net /cell_1_fused: track 11.8 -> 13.0 mm
Other:
- outline, holes or cut-outs redrawn
Changed lines of the file:
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@@
 	(footprint "formula_slug_footprint_library:24939"
 		(layer "F.Cu")
-		(at 190.775 85.45)
+		(at 193.775 85.45)
 		(property "Reference" "H2"
 			(at 4.575 0.15 0)
@@
 		(layer "Edge.Cuts")
 	)
-	(gr_circle
-		(center 190.7632 85.4752)
-		(end 192.8632 85.4752)
-		(stroke
-			(width 0.2)
-			(type default)
-		)
-		(fill no)
-		(layer "Edge.Cuts")
-	)
 	(gr_line
 		(start 192.706272 90.6949)
@@
 		(layer "User.1")
 	)
-	(gr_circle
-		(center 190.775 85.45)
-		(end 192.875 85.45)
+	(gr_line
+		(start 190.775 85.45)
+		(end 193.775 85.45)
 		(stroke
-			(width 0.005)
+			(width 0.1016)
 			(type solid)
 		)
-		(fill no)
 		(layer "User.1")
 	)
@@
 	(segment
 		(start 198.225 74.25)
-		(end 198.225 78)
+		(end 198.225 81)
 		(width 0.254)
 		(layer "F.Cu")
@@
 	)
 	(segment
-		(start 198.225 78)
-		(end 192.510832 83.714168)
+		(start 198.225 81)
+		(end 193.775 85.45)
 		(width 0.254)
 		(layer "F.Cu")
@@
 		(members "840feaf8-a0a4-4620-911b-05653ee67b5c")
 	)
-	(group ""
-		(members "03958cb6-b32f-4167-952d-321f6100df8b" "044738b2-46fd-4011-9fb8-9db0a0ff3492"
-			"04f88092-bc4d-42ec-ab09-29b07e8b292d" "0b149612-8f9c-4cd1-85ef-b6e637df22ac"
-			"0d400155-bee0-49de-a0dc-211132226e41" "0d7dc3d9-65e7-41fa-88f5-70db0279c659"
-			"1293c1c1-3d7b-4138-879f-14c71427c495" "18bf8217-7eff-4f24-b49b-28fa5605b6a3"
-			"1baa646e-938f-468c-a956-2fbf10347903" "1c714afd-f4c7-48c8-86d7-53b45543a77d"
-			"1c8ec656-6262-4ad5-a28f-9050bfb96e6f" "1dad1daf-0a7c-4dc7-b2c3-4a6ba66057e3"
-			"1f1ef52a-d0fc-4e48-8b21-4d6d7d1877eb" "20c488e9-37f2-43ac-8f67-17653c7a6d22"
-			"2320e303-2872-4f27-bd54-03ad8680b59c" "25e2dce8-eecf-411c-8e95-abc0a78175c1"
-			"2bfef294-56a7-45a5-87a9-436baa47c87b" "2c7eee7d-261f-452f-8886-6fa8c84151e5"
-			"2cffdedf-a7af-4df1-a0b1-150776a95f7b" "2dc423fc-73a6-4423-a12b-06fb56cca35d"
-			"2fd10fbf-69de-460c-bbbc-4aee00feb3f4" "2fe91940-79b8-488a-8c56-8cae0cc778bb"
-			"34b3ba5b-775f-4307-8548-d346290264a1" "36728cb0-3382-406b-b72b-3d4abbaf7f63"
-			"3da1aa90-e51a-4ebd-a9eb-419e3a2e165e" "3fe4d0e7-968b-4fbc-a8d5-ec2f8636c2aa"
-			"48aafe1e-a455-480d-8e2f-0b001946ab4f" "49af3596-2f48-4afa-96f5-cb481b679647"
-			"4c185e4a-165a-4c1b-b62f-fe9e290165d1" "4d5906f8-5ae0-4025-a76b-cd7fea72b84a"
-			"4d74c042-c5ca-497f-b8d1-83463a5e78ec" "4d8090c7-6f61-4d95-861a-a5a92721bccd"
-			"51cca778-579b-4e98-9370-9a381402846a" "559384a2-0dc6-4075-bb93-759361f2ba67"
-			"5c7f643f-98a8-47c6-bd5a-283d5c771b9e" "60bece42-acd0-4571-80a5-7c84ac722ce6"
-			"63554408-60f6-46fb-b8e9-856f863c4fa5" "673adb4d-0239-42c5-a36d-b39aeb8348f6"
-			"68fba486-057c-4ea6-8b25-96214a4f10ed" "694ef5cb-d379-47a1-b227-70ff85a4ccf5"
-			"6f9e457e-3139-4fde-83d9-e07c40e37bd8" "6fe440bb-b3e0-4d7d-aa9a-3d082f276127"
-			"73ffc45e-0b6b-4c2a-98e0-82c629e673dc" "7c3777f1-07e8-4a80-89f2-e1274fc90c4c"
-			"7d43d5b1-11fd-4bbd-abcb-fbc5b9cf5f0c" "831c395a-9826-4188-88cc-27eec7d28930"
-			"84f2f3dd-f692-4999-b9dc-5f1838b2c7ba" "85063ce6-5781-4c9c-909b-06f104461398"
-			"86408cfa-0d71-4c41-93df-11ea8499fac1" "8bccbd38-6595-47d5-8a89-97fb2d77ac54"
-			"8e00d3d2-13c3-478d-b450-d003899aa8d3" "8f636110-07b8-4e7c-8777-eefe5b78447e"
-			"93924009-52d6-4859-ac01-c3b9503b3a51" "94037d5e-6431-4c3e-845d-1245cbb075b3"
-			"94069fed-4463-45e7-a319-6dc76e9ecbac" "952408c0-f29a-42b8-91f5-d62e96e55e3a"
-			"9582ab75-d254-48e9-b69e-ffedb72534ad" "958bab7c-d80f-48be-9688-4d0937090c4e"
-			"96c69070-3f57-4992-9b00-223e8160c4f8" "970ed5a3-9808-459d-89a7-452e939cfae0"
-			"9984f41b-7afb-452d-9f5b-7dadb2dd1cbd" "9d49708e-69cb-4545-8314-de1257898a81"
-			"9e720a53-f6f8-41eb-9416-7cd60a6b781c" "9eb92097-6725-48bc-addd-b4c245826e69"
-			"a09d5f90-b250-4666-8f81-c0b05a6918c2" "a176c8e3-685e-41db-a656-eaa0836a6e1f"
-			"a34e3a71-ff09-436b-bee6-511550411cfd" "a3f91181-23d1-489c-9cf9-987225f888be"
-			"a52ce46f-6cdf-45a9-8c4a-6bf3a948bb5e" "a5974121-56d7-45b8-91cf-44cdb42c5e00"
-			"a5b7e978-4474-49f1-842f-e0ecda350d65" "a6115014-694a-476e-8fa6-c6b07069149d"
-			"a9c5a38c-7881-403e-8dac-ca875b0dc1e2" "ae354519-70f2-4519-9dff-f4ab984a1795"
-			"b0325cc7-9c47-4094-ae2b-ee13c3ec6c95" "b4c134f3-0b25-439f-af00-193b574543b3"
-			"b507a1cd-4bd8-48c6-9a5e-e21b1adb0b43" "b6791e39-08ac-4537-81df-21d3459e4543"
-			"b8fa0d57-f5a2-4bf9-a593-ea301b2bc584" "baeea880-8232-4f31-805e-8cd07f2e8717"
-			"bcbf584f-a062-4576-967b-062996f02b15" "be257dbf-60ff-4c50-b61d-7c84d58804da"
-			"bf212b64-620c-4fd7-90a0-e3409a73237f" "c0cf62f4-d375-4401-80fb-18f1d9e60c9b"
-			"c2f30d8c-7437-43cf-9cf3-b3a38cdf75c2" "c592ac96-f6ef-4b43-a72d-4d9e43e49bcd"
-			"c7f6df11-db42-4d7e-86cd-b8216ab045c1" "cae9f27e-42a2-45b5-ab84-70d29ac122b7"
-			"cb19ee7b-113a-467a-bfc9-314b174cfa07" "cd8ec693-a799-45a9-be3d-d021760daed8"
-			"d1467d7a-85b5-4543-abca-e4a23441e04b" "d350505a-35ea-4f92-8e4f-5bdcc17341fa"
-			"d414ee66-1abd-4b21-a659-1fd21159e3bd" "d6184179-cd33-4867-9414-726c70e0b04f"
-			"d7daf0e1-4069-48bb-a068-9b9c86bda313" "db2b6f6e-d42c-469c-aaf9-aaae5133adca"
-			"dd56ea71-b8cb-4cca-b9b9-0f8f07cb88ca" "df3331ee-01f8-4ed9-8c39-8df27d6ea6c3"
-			"e2583ae5-80a6-463d-b3f4-822d94bd0f30" "e2da0c20-63e6-4cab-9070-2b58bd4afe88"
-			"e2f982d6-5615-4cf0-9d51-fea42e1fcdde" "e40ef436-d62e-4864-955a-f350d32cb64b"
-			"e97e986d-daf5-42ca-ac34-3520170e8ab0" "e9f45b82-5e8e-4712-8530-bb75fa1597b8"
-			"ea3f24f0-7e6e-42b8-a774-0712890015ee" "eec4fd6a-823d-49e3-82a9-d07af52e398d"
-			"ef307607-6631-49dc-bf96-7f175a6e9169" "f08471f8-efae-4a21-a5df-07187da148f1"
-			"f0b3ca55-bbbd-4f83-8ad2-6337c42a2f49" "f272df28-0ff6-4d72-9bdd-10be4c42b573"
-			"f73da28d-d23b-414e-8826-bf10c1a87ee2" "ff280781-3dfb-4e3d-a857-cd0c1ed76a00"
-		)
-	)
 	(embedded_fonts no)
