File: temp-sense-board-flex-prototype-v.1/temp-sense-board-flex-prototype-v.1.kicad_sch (KiCad schematic)
At the start: 0 parts

Commit message: editing symbols and adding to library
Parts:
- added C1, C10, C11, C12, C2, C3, C4, C5, C6, C7, C8, C9: 1 uF, Capacitor_SMD:C_0603_1608Metric_Pad1.08x0.95mm_HandSolder, symbol Device:C
- added GHR-04V-S1, GHR-04V-S2, SM04B-GHS-TB1: Conn_01x04_Socket, symbol Connector:Conn_01x04_Socket
- added J2, J4: 512810598, FS_4_Footprint_Library:512810598, symbol Connector_Generic:Conn_01x05
- added U1, U10, U11, U12, U2, U3, U4, U5, U6, U7, U8, U9: TMP1075D, Package_SO:SO-8_3.9x4.9mm_P1.27mm, symbol Sensor_Temperature:TMP1075D
- added U13: DS18B20Z+, FS_4_Global_Footprint_Library:21-0041B_8_MXM, symbol 2026-01-10_01-54-57:DS18B20Z+
Connections:
- new net: J4.1 (Pin_1), U13.5 (GND)
- new net +5V: C1.1, C10.1, C11.1, C12.1, C2.1, C3.1, C4.1, C5.1, C6.1, C7.1, C8.1, C9.1, J2.5 (Pin_5), U1.8 (V+), U10.5 (A2), U10.8 (V+), U11.6 (A1), U11.8 (V+), U12.8 (V+), U2.7 (A0), U2.8 (V+), U3.6 (A1), U3.7 (A0), U3.8 (V+), U4.5 (A2), U4.6 (A1), U4.7 (A0), U4.8 (V+), U5.5 (A2), U5.7 (A0), U5.8 (V+), U6.8 (V+), U7.6 (A1), U7.8 (V+), U8.5 (A2), U8.6 (A1), U8.8 (V+), U9.8 (V+)
- new net ALERT: J2.4 (Pin_4), U1.3 (ALERT), U10.3 (ALERT), U11.3 (ALERT), U12.3 (ALERT), U2.3 (ALERT), U3.3 (ALERT), U4.3 (ALERT), U5.3 (ALERT), U6.3 (ALERT), U7.3 (ALERT), U8.3 (ALERT), U9.3 (ALERT)
- new net DQ: J4.5 (Pin_5), U13.4 (DQ)
- new net SCL: J2.2 (Pin_2), U1.2 (SCL), U10.2 (SCL), U11.2 (SCL), U12.2 (SCL), U12.7 (A0), U2.2 (SCL), U3.2 (SCL), U4.2 (SCL), U5.2 (SCL), U6.2 (SCL), U7.2 (SCL), U8.2 (SCL), U9.2 (SCL)
- new net SDA: J2.3 (Pin_3), U1.1 (SDA), U10.1 (SDA), U11.1 (SDA), U11.7 (A0), U12.1 (SDA), U2.1 (SDA), U3.1 (SDA), U4.1 (SDA), U5.1 (SDA), U6.1 (SDA), U6.6 (A1), U7.1 (SDA), U8.1 (SDA), U9.1 (SDA), U9.7 (A0)
- new net V-: C1.2, C10.2, C11.2, C12.2, C2.2, C3.2, C4.2, C5.2, C6.2, C7.2, C8.2, C9.2, J2.1 (Pin_1), U1.4 (GND), U1.5 (A2), U1.6 (A1), U1.7 (A0), U10.4 (GND), U10.6 (A1), U10.7 (A0), U11.4 (GND), U11.5 (A2), U12.4 (GND), U12.5 (A2), U12.6 (A1), U2.4 (GND), U2.5 (A2), U2.6 (A1), U3.4 (GND), U3.5 (A2), U4.4 (GND), U5.4 (GND), U5.6 (A1), U6.4 (GND), U6.5 (A2), U6.7 (A0), U7.4 (GND), U7.5 (A2), U7.7 (A0), U8.4 (GND), U8.7 (A0), U9.4 (GND), U9.5 (A2), U9.6 (A1)
- no-connect marks 0 -> 3

Commit message: Schematic done sans footprint assignments
i dont know what footprints to give to the imported connectors
Parts:
- removed C10, C11, C12, C4, C5, C6, C7, C8, C9: 1 uF, Capacitor_SMD:C_0603_1608Metric_Pad1.08x0.95mm_HandSolder, symbol Device:C
- removed GHR-04V-S1, GHR-04V-S2, SM04B-GHS-TB1: Conn_01x04_Socket, symbol Connector:Conn_01x04_Socket
- removed J4: 512810598, FS_4_Footprint_Library:512810598, symbol Connector_Generic:Conn_01x05
- removed U10, U11, U12, U4, U5, U6, U7, U8, U9: TMP1075D, Package_SO:SO-8_3.9x4.9mm_P1.27mm, symbol Sensor_Temperature:TMP1075D
- removed U13: DS18B20Z+, FS_4_Global_Footprint_Library:21-0041B_8_MXM, symbol 2026-01-10_01-54-57:DS18B20Z+
- added J10: 84952-5, symbol Connector_Generic:Conn_01x05
- added J11: 0015388040, symbol Connector_Generic:Conn_01x05
- added J8: GHR-04V-S1, symbol Connector_Generic:Conn_01x05
- added J9: SM04B-GHS-TB1, symbol Connector_Generic:Conn_01x05
Connections:
- net +5V: now also J10.5 (Pin_5), J11.5 (Pin_5), J8.5 (Pin_5), J9.5 (Pin_5)
- net ALERT: now also J10.4 (Pin_4), J11.4 (Pin_4), J8.4 (Pin_4), J9.4 (Pin_4)
- net SCL: now also J10.2 (Pin_2), J11.2 (Pin_2), J8.2 (Pin_2), J9.2 (Pin_2)
- net SDA: now also J10.3 (Pin_3), J11.3 (Pin_3), J8.3 (Pin_3), J9.3 (Pin_3)
- net V-: now also J10.1 (Pin_1), J11.1 (Pin_1), J8.1 (Pin_1), J9.1 (Pin_1)
- no-connect marks 3 -> 0
Other:
- moved on the sheet: J2, U1, U2, U3

Commit message: more connectors w footprints
Parts:
- J10: footprint (none) -> Connector_FFC-FPC:TE_1-84952-5_1x15-1MP_P1.0mm_Horizontal
- J8: Digikey URL https://www.jst-mfg.com/product/pdf/eng/eGH.pdf -> https://www.digikey.com/en/products/detail/jst-sales-americ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
- J9: footprint (none) -> Connector_JST:JST_GH_SM04B-GHS-TB_1x04-1MP_P1.25mm_Horizontal
Changed lines of the file:
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@@
 			)
 		)
-		(property "Footprint" ""
+		(property "Footprint" "Connector_FFC-FPC:TE_1-84952-5_1x15-1MP_P1.0mm_Horizontal"
 			(at 74.93 99.06 0)
 			(hide yes)
@@
 			)
 		)
-		(property "Footprint" ""
+		(property "Footprint" "Connector_JST:JST_GH_SM04B-GHS-TB_1x04-1MP_P1.25mm_Horizontal"
 			(at 74.93 115.57 0)
 			(hide yes)
@@
 			)
 		)
-		(property "Datasheet" ""
+		(property "Datasheet" "https://www.jst-mfg.com/product/pdf/eng/eGH.pdf"
 			(at 74.93 130.81 0)
 			(hide yes)
@@
 			)
 		)
-		(property "Digikey URL" "https://www.jst-mfg.com/product/pdf/eng/eGH.pdf"
+		(property "Digikey URL" "https://www.digikey.com/en/products/detail/jst-sales-america-inc/GHR-04V-S/807816?msockid=15685f35b86e654907ab4928b9226472"
 			(at 74.93 130.81 0)
 			(hide yes)

Commit message: schematic is finished; layout is not
-added footprints to fs library
-finalized schematic
-did a veeery rough layout not complete jiust here tonight
-yay eh someone give comments
Parts:
- removed J10: 84952-5, Connector_FFC-FPC:TE_1-84952-5_1x15-1MP_P1.0mm_Horizontal, symbol Connector_Generic:Conn_01x05
- removed J11: 0015388040, symbol Connector_Generic:Conn_01x05
- removed J2: 512810598, FS_4_Footprint_Library:512810598, symbol Connector_Generic:Conn_01x05
- removed J8: GHR-04V-S1, symbol Connector_Generic:Conn_01x05
- removed J9: SM04B-GHS-TB1, Connector_JST:JST_GH_SM04B-GHS-TB_1x04-1MP_P1.25mm_Horizontal, symbol Connector_Generic:Conn_01x05
- added J2: FH34SRJ-12S-0.5SH(50), formula_slug_footprint_library:CONN12x1_FH34SRJ-12S-0.5SH50_HIR, symbol Connector_Generic:Conn_01x12
- added J3: FH33-12S-0.5SH(10), formula_slug_footprint_library:CONN_FH33-12S-0.5SH10_HIR, symbol Connector_Generic:Conn_01x12
- added J4: 1-84953-2, formula_slug_footprint_library:CON12_SMT-RA_FCC-FPC2, symbol Connector_Generic:Conn_01x12
- added TP1, TP10, TP11, TP12, TP13, TP14, TP15, TP16, TP17, TP18, TP19, TP2, TP20, TP21, TP3, TP4, TP5, TP6, TP7, TP8, TP9: TestPoint, TestPoint:TestPoint_Pad_D1.0mm, symbol Connector:TestPoint
Connections:
- net +5V: now also J2.5 (Pin_5), J3.5 (Pin_5), J4.5 (Pin_5)
- net ALERT: now also J2.4 (Pin_4), J3.4 (Pin_4), J4.4 (Pin_4)
- net SCL: now also J2.2 (Pin_2), J3.2 (Pin_2), J4.2 (Pin_2)
- net SDA: now also J2.3 (Pin_3), J3.3 (Pin_3), J4.3 (Pin_3)
- net V-: now also J2.1 (Pin_1), J3.1 (Pin_1), J4.1 (Pin_1)
- new net: J4.6 (Pin_6), TP21.1
- new net: J2.10 (Pin_10), TP3.1
- new net: J3.12 (Pin_12), TP8.1
- new net: J2.8 (Pin_8), TP5.1
- new net: J4.10 (Pin_10), TP17.1
- new net: J4.11 (Pin_11), TP16.1
- new net: J4.12 (Pin_12), TP15.1
- new net: J4.7 (Pin_7), TP20.1
- new net: J4.8 (Pin_8), TP19.1
- new net: J4.9 (Pin_9), TP18.1
- new net: J3.10 (Pin_10), TP10.1
- new net: J3.11 (Pin_11), TP9.1
- new net: J3.6 (Pin_6), TP14.1
- new net: J3.7 (Pin_7), TP13.1
- new net: J3.8 (Pin_8), TP12.1
- new net: J3.9 (Pin_9), TP11.1
- new net: J2.6 (Pin_6), TP7.1
- new net: J2.9 (Pin_9), TP4.1
- new net: J2.11 (Pin_11), TP2.1
- new net: J2.12 (Pin_12), TP1.1
- new net: J2.7 (Pin_7), TP6.1

Commit message: first trace thing done
Parts:
- J4: footprint formula_slug_footprint_library:CON12_SMT-RA_FCC-FPC2 -> formula_slug_footprint_library:FPC-12PIN-CABLE-1mm-0.71mm
Changed lines of the file:
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@@
 			)
 		)
-		(property "Footprint" "formula_slug_footprint_library:CON12_SMT-RA_FCC-FPC2"
+		(property "Footprint" "formula_slug_footprint_library:FPC-12PIN-CABLE-1mm-0.71mm"
 			(at 63.5 124.46 0)
 			(hide yes)

Commit message: more!
Parts:
- J2: footprint formula_slug_footprint_library:CONN12x1_FH34SRJ-12S-0.5SH50_HIR -> formula_slug_footprint_library:FPC_12-CABLE-0.5mm-0.3mm
- J3: value FH33-12S-0.5SH(10) -> FH12-12S-1SH(55); footprint formula_slug_footprint_library:CONN_FH33-12S-0.5SH10_HIR -> formula_slug_footprint_library:FPC-12PIN-CABLE-1mm-0.65mm; Digikey URL https://www.digikey.com/en/products/detail/hirose-electric-co-ltd/FH33-12S-0-5SH-10/1305325 -> https://www.digikey.com/en/products/detail/hirose-electric-co-ltd/FH12-12S-1SH-55/3873256
Changed lines of the file:
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@@
 			)
 		)
-		(property "Value" "FH33-12S-0.5SH(10)"
+		(property "Value" "FH12-12S-1SH(55)"
 			(at 49.53 93.98 0)
 			(show_name no)
@@
 			)
 		)
-		(property "Footprint" "formula_slug_footprint_library:CONN_FH33-12S-0.5SH10_HIR"
+		(property "Footprint" "formula_slug_footprint_library:FPC-12PIN-CABLE-1mm-0.65mm"
 			(at 63.5 91.44 0)
 			(hide yes)
@@
 			)
 		)
-		(property "Datasheet" "https://www.hirose.com/product/document?clcode=CL0580-1304-0-10&productname=FH33-10S-0.5SH(10)&series=FH33&documenttype=Catalog&lang=en&documentid=D49357_en"
+		(property "Datasheet" "https://www.lcsc.com/datasheet/C5148307.pdf"
 			(at 63.5 91.44 0)
 			(hide yes)
@@
 			)
 		)
-		(property "Digikey URL" "https://www.digikey.com/en/products/detail/hirose-electric-co-ltd/FH33-12S-0-5SH-10/1305325"
+		(property "Digikey URL" "https://www.digikey.com/en/products/detail/hirose-electric-co-ltd/FH12-12S-1SH-55/3873256"
 			(at 63.5 91.44 0)
 			(hide yes)
@@
 			)
 		)
-		(property "Footprint" "formula_slug_footprint_library:CONN12x1_FH34SRJ-12S-0.5SH50_HIR"
+		(property "Footprint" "formula_slug_footprint_library:FPC_12-CABLE-0.5mm-0.3mm"
 			(at 68.58 57.15 0)
 			(hide yes)

Commit message: FH34SRJ-12S-0.5SH(50) footprint made
Parts:
- added J5: FH34SRJ-12S-0.5SH(50), formula_slug_footprint_library:FPC_12-CABLE-0.5mm-0.3mm, symbol Connector_Generic:Conn_01x12
- added J6: FH12-12S-1SH(55), formula_slug_footprint_library:FPC-12PIN-CABLE-1mm-0.65mm, symbol Connector_Generic:Conn_01x12
- added J7: 1-84953-2, formula_slug_footprint_library:FPC-12PIN-CABLE-1mm-0.71mm, symbol Connector_Generic:Conn_01x12
- added TP22, TP23, TP24, TP25, TP26, TP27, TP28, TP29, TP30, TP31, TP32, TP33, TP34, TP35, TP36, TP37, TP38, TP39, TP40, TP41, TP42, TP43, TP44, TP45, TP46, TP47, TP48, TP49, TP50, TP51, TP52, TP53, TP54, TP55, TP56, TP57: TestPoint, TestPoint:TestPoint_Pad_D1.0mm, symbol Connector:TestPoint
- J2: footprint formula_slug_footprint_library:FPC_12-CABLE-0.5mm-0.3mm -> formula_slug_footprint_library:CONN12x1_FH34SRJ-12S-0.5SH50_HIR
- J3: footprint formula_slug_footprint_library:FPC-12PIN-CABLE-1mm-0.65mm -> (none)
- J4: footprint formula_slug_footprint_library:FPC-12PIN-CABLE-1mm-0.71mm -> formula_slug_footprint_library:TE_84952-5
Connections:
- new net: J7.4 (Pin_4), TP54.1
- new net: J7.8 (Pin_8), TP40.1
- new net: J6.2 (Pin_2), TP51.1
- new net: J5.5 (Pin_5), TP43.1
- new net: J6.3 (Pin_3), TP50.1
- new net: J6.9 (Pin_9), TP32.1
- new net: J6.8 (Pin_8), TP33.1
- new net: J6.10 (Pin_10), TP31.1
- new net: J7.11 (Pin_11), TP37.1
- new net: J5.8 (Pin_8), TP26.1
- new net: J7.1 (Pin_1), TP57.1
- new net: J7.10 (Pin_10), TP38.1
- new net: J7.12 (Pin_12), TP36.1
- new net: J7.2 (Pin_2), TP56.1
- new net: J7.3 (Pin_3), TP55.1
- new net: J7.5 (Pin_5), TP53.1
- new net: J7.6 (Pin_6), TP42.1
- new net: J7.7 (Pin_7), TP41.1
- new net: J7.9 (Pin_9), TP39.1
- new net: J6.6 (Pin_6), TP35.1
- new net: J6.5 (Pin_5), TP48.1
- new net: J5.9 (Pin_9), TP25.1
- new net: J5.11 (Pin_11), TP23.1
- new net: J6.1 (Pin_1), TP52.1
- new net: J6.11 (Pin_11), TP30.1
- new net: J6.12 (Pin_12), TP29.1
- new net: J6.4 (Pin_4), TP49.1
- new net: J6.7 (Pin_7), TP34.1
- new net: J5.1 (Pin_1), TP47.1
- new net: J5.10 (Pin_10), TP24.1
- new net: J5.12 (Pin_12), TP22.1
- new net: J5.2 (Pin_2), TP46.1
- new net: J5.3 (Pin_3), TP45.1
- new net: J5.4 (Pin_4), TP44.1
- new net: J5.6 (Pin_6), TP28.1
- new net: J5.7 (Pin_7), TP27.1
Other:
- note added: "2 layer board"
- note added: "cable footprints on left"
- note added: "connector footprints on right"
- note added: "right now cable footrpings"
- moved on the sheet: J2, J3, J4, TP1, TP10, TP11, TP12, TP13, TP14, TP15, TP16, TP17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

Commit message: schematic finished??
Parts:
- added C4, C5, C6: 1 uF, Capacitor_SMD:C_0603_1608Metric_Pad1.08x0.95mm_HandSolder, symbol Device:C
- added R1, R2, R3: 5k, Resistor_SMD:R_0201_0603Metric, symbol Device:R
- added U4, U5, U6: TMP1075D, Package_SO:SO-8_3.9x4.9mm_P1.27mm, symbol Sensor_Temperature:TMP1075D
- J3: footprint (none) -> formula_slug_footprint_library:FH12-12S-1SH_55_
Connections:
- net +5V: now also C4.1, C5.1, C6.1, R1.1, R2.1, R3.1, U4.8 (V+), U5.7 (A0), U5.8 (V+), U6.7 (A0), U6.8 (V+)
- net ALERT: now also R1.2, U4.3 (ALERT), U5.3 (ALERT), U6.3 (ALERT)
- net SCL: now also R2.2, U4.2 (SCL), U5.2 (SCL), U6.2 (SCL)
- net SDA: now also R3.2, U4.1 (SDA), U5.1 (SDA), U6.1 (SDA)
- net V-: now also C4.2, C5.2, C6.2, U4.4 (GND), U4.5 (A2), U4.6 (A1), U4.7 (A0), U5.4 (GND), U5.5 (A2), U5.6 (A1), U6.4 (GND), U6.5 (A2), U6.6 (A1)
Other:
- note removed: "right now cable footrpings"
- moved on the sheet: J2, J3, J4, J5, J6, J7, TP1, TP10, TP11, TP12, TP13, TP14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
