File: temp-sense-board-flex-prototype-v.1/temp-sense-board-flex-prototype-v.1.kicad_pcb (KiCad board)
At the start: 2 copper layers, 3.5 x 13 mm, 34 parts, among them J2 FH34SRJ-12S-0.5SH(50), J3 FH33-12S-0.5SH(10), J4 1-84953-2, U1 TMP1075D, U2 TMP1075D, U3 TMP1075D

Commit message: Layout help please
Parts:
- moved C3 36.9 mm to (161.3, 48.3), turned to -90 degrees
- moved U1 29.0 mm to (115.6, 48.3)
- moved U3 28.5 mm to (152.4, 48.3)
- moved C1 22.9 mm to (123.2, 48.3), turned to -90 degrees
- moved TP19 21.6 mm to (151.1, 68.6)
- moved TP16 20.1 mm to (139.7, 71.1)
- moved TP15 18.0 mm to (139.7, 67.3)
- moved C2 17.8 mm to (142.2, 48.3), turned to -90 degrees
- moved TP18 17.6 mm to (146.1, 72.4)
- moved TP21 17.1 mm to (154.9, 68.6)
- moved TP17 16.6 mm to (146.1, 68.6)
- moved J4 13.7 mm to (152.4, 62.2)
- moved TP20 13.1 mm to (152.4, 72.4)
- moved TP3 11.5 mm to (149.9, 92.7)
- moved TP1 10.2 mm to (144.8, 91.4)
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Other:
- board size 3.5 x 13 mm -> 76.2 x 12.7 mm

Commit message: changing footprints, changing whole design, its something
Parts:
- moved J2 136.2 mm to (25.3, 42.1)
- moved TP10 135.6 mm to (276.9, 66.0)
- moved TP11 135.6 mm to (280.7, 66.0)
- moved TP13 135.6 mm to (288.3, 68.6)
- moved TP8 135.6 mm to (269.2, 59.7)
- moved TP12 135.6 mm to (283.2, 66.0)
- moved TP14 135.6 mm to (287.0, 64.8)
- moved TP9 135.6 mm to (271.8, 64.8)
- moved J3 134.0 mm to (280.7, 59.7)
- moved J4 115.4 mm to (47.0, 15.2)
- moved REF** 114.4 mm to (143.5, 75.2)
- moved TP21 111.5 mm to (47.0, 40.6)
- moved TP19 110.0 mm to (44.5, 41.9)
- moved TP20 109.4 mm to (47.0, 43.2)
- moved REF** 109.3 mm to (142.2, 45.0)
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Routing:
- net Net-(J4-Pin_8): track 0.00 -> 88.2 mm
- net Net-(J2-Pin_10): track 0.00 -> 87.7 mm
- net Net-(J4-Pin_12): track 0.00 -> 87.6 mm
- net Net-(J2-Pin_9): track 0.00 -> 87.3 mm
- net Net-(J4-Pin_10): track 0.00 -> 84.3 mm
- net Net-(J4-Pin_6): track 0.00 -> 82.5 mm
- net Net-(J4-Pin_7): track 0.00 -> 81.3 mm
- net Net-(J4-Pin_11): track 0.00 -> 81.3 mm
- net Net-(J2-Pin_8): track 0.00 -> 80.5 mm
- net Net-(J4-Pin_9): track 0.00 -> 80.0 mm
- net Net-(J2-Pin_7): track 0.00 -> 76.2 mm
- net Net-(J2-Pin_6): track 0.00 -> 73.7 mm
- net Net-(J2-Pin_12): track 0.00 -> 0.66 mm
Other:
- board size 76.2 x 12.7 mm -> 135.9 x 88.9 mm

Commit message: first trace thing done
Parts:
- removed the REF** at (142.2, 45.0)
- removed the REF** at (143.5, 75.2)
- J4: footprint formula_slug_footprint_library:CON12_SMT-RA_FCC-FPC2 -> formula_slug_footprint_library:FPC-12PIN-CABLE-1mm-0.71mm
- moved J2 124.6 mm to (144.8, 77.5), turned to -90 degrees
- moved J4 106.4 mm to (149.8, 42.6), turned to 90 degrees
- turned U1 to 0 degrees
- turned U2 to 0 degrees
- turned U3 to 0 degrees
Routing:
- net +5V: track 0.00 -> 54.6 mm
- net V-: track 0.00 -> 22.0 mm
- net /ALERT: track 0.00 -> 21.5 mm
- net /SDA: track 0.00 -> 16.5 mm
- net /SCL: track 0.00 -> 16.3 mm
- net Net-(J2-Pin_9): track 87.3 -> 85.7 mm
- net Net-(J2-Pin_10): track 87.7 -> 86.3 mm

Commit message: more!
Parts:
- removed REF**: FPC_5, FPC_5
- removed REF**: FPC_13, formula_slug_footprint_library:FPC_13
- J2: footprint formula_slug_footprint_library:CONN12x1_FH34SRJ-12S-0.5SH50_HIR -> formula_slug_footprint_library:FPC_12-CABLE-0.5mm-0.3mm
- J3: value FH33-12S-0.5SH(10) -> FH12-12S-1SH(55); footprint formula_slug_footprint_library:CONN_FH33-12S-0.5SH10_HIR -> formula_slug_footprint_library:FPC-12PIN-CABLE-1mm-0.65mm
- moved J3 237.2 mm to (47.4, 102.5), turned to -90 degrees
- moved TP14 125.2 mm to (166.4, 98.6), turned to 90 degrees
- moved TP8 121.8 mm to (161.4, 116.3), turned to 90 degrees
- moved TP13 121.5 mm to (170.3, 97.3), turned to 90 degrees
- moved TP12 121.1 mm to (167.7, 102.4), turned to 90 degrees
- moved TP11 119.5 mm to (167.7, 104.9), turned to 90 degrees
- moved TP10 117.2 mm to (167.7, 108.7), turned to 90 degrees
- moved TP9 116.2 mm to (166.4, 113.8), turned to 90 degrees
- moved J2 6.13 mm to (149.9, 74.0)
- moved C3 1.75 mm to (167.6, 85.9)
- moved U3 1.75 mm to (167.6, 77.0)
Other:
- board size 135.9 x 88.9 mm -> 134.7 x 88.9 mm

Commit message: FH34SRJ-12S-0.5SH(50) footprint made
Parts:
- moved J4 106.7 mm to (43.1, 45.0)
- moved J2 104.3 mm to (45.5, 74.9)
- moved TP15 89.5 mm to (132.8, 34.3)
- moved TP17 89.5 mm to (132.8, 30.5)
- moved TP19 89.5 mm to (132.8, 27.9)
- moved TP16 89.5 mm to (135.4, 35.6)
- moved TP18 89.5 mm to (135.4, 33.0)
- moved TP20 89.5 mm to (135.4, 29.2)
- moved TP21 89.5 mm to (135.4, 26.7)
- moved TP1 86.1 mm to (131.3, 64.5)
- moved TP2 86.1 mm to (131.3, 67.1)
- moved TP7 86.1 mm to (141.5, 64.5)
- moved TP3 86.1 mm to (135.1, 64.5)
- moved TP4 86.1 mm to (135.1, 68.3)
- moved TP5 86.1 mm to (138.9, 64.5)
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Routing:
- net Net-(J4-Pin_8): track 88.2 -> 0.00 mm
- net Net-(J4-Pin_12): track 87.6 -> 0.00 mm
- net Net-(J4-Pin_10): track 84.3 -> 0.00 mm
- net Net-(J2-Pin_9): track 85.7 -> 1.60 mm
- net Net-(J2-Pin_10): track 86.3 -> 3.22 mm
- net Net-(J4-Pin_6): track 82.5 -> 0.00 mm
- net Net-(J4-Pin_7): track 81.3 -> 0.00 mm
- net Net-(J4-Pin_11): track 81.3 -> 0.00 mm
- net Net-(J4-Pin_9): track 80.0 -> 0.00 mm
- net Net-(J2-Pin_8): track 80.5 -> 1.80 mm
- net Net-(J2-Pin_7): track 76.2 -> 0.00 mm
- net Net-(J2-Pin_6): track 73.7 -> 0.00 mm
Other:
- board size 134.7 x 88.9 mm -> 134.7 x 89.8 mm

Commit message: outline added and layout started
Parts:
- removed J3: FH12-12S-1SH(55), formula_slug_footprint_library:FPC-12PIN-CABLE-1mm-0.65mm
- removed TP10, TP11, TP12, TP13, TP14, TP8, TP9: TestPoint, TestPoint:TestPoint_Pad_D1.0mm
- added J5: FH34SRJ-12S-0.5SH(50), formula_slug_footprint_library:FPC_12-CABLE-0.5mm-0.3mm, F.Cu at (51.9, 57.4)
- added J6: FH12-12S-1SH(55), formula_slug_footprint_library:FPC-12PIN-CABLE-1mm-0.65mm, F.Cu at (49.7, 105.9)
- added J7: 1-84953-2, formula_slug_footprint_library:FPC-12PIN-CABLE-1mm-0.71mm, F.Cu at (49.9, 79.8)
- added TP22: TestPoint, TestPoint:TestPoint_Pad_D1.0mm, F.Cu at (104.9, 56.1)
- added TP23: TestPoint, TestPoint:TestPoint_Pad_D1.0mm, F.Cu at (114.8, 58.4)
- added TP24: TestPoint, TestPoint:TestPoint_Pad_D1.0mm, F.Cu at (112.3, 56.1)
- added TP25: TestPoint, TestPoint:TestPoint_Pad_D1.0mm, F.Cu at (137.7, 57.9)
- added TP26: TestPoint, TestPoint:TestPoint_Pad_D1.0mm, F.Cu at (132.3, 57.9)
- added TP27: TestPoint, TestPoint:TestPoint_Pad_D1.0mm, F.Cu at (127.3, 55.1)
- added TP28: TestPoint, TestPoint:TestPoint_Pad_D1.0mm, F.Cu at (108.2, 59.2)
- added TP29: TestPoint, TestPoint:TestPoint_Pad_D1.0mm, F.Cu at (103.4, 101.6)
- added TP30: TestPoint, TestPoint:TestPoint_Pad_D1.0mm, F.Cu at (109.2, 107.7)
- added TP31: TestPoint, TestPoint:TestPoint_Pad_D1.0mm, F.Cu at (109.5, 104.1)
- added TP32: TestPoint, TestPoint:TestPoint_Pad_D1.0mm, F.Cu at (133.9, 103.4)
- added TP33: TestPoint, TestPoint:TestPoint_Pad_D1.0mm, F.Cu at (127.5, 107.4)
- added TP34: TestPoint, TestPoint:TestPoint_Pad_D1.0mm, F.Cu at (98.6, 104.4)
- added TP35: TestPoint, TestPoint:TestPoint_Pad_D1.0mm, F.Cu at (102.4, 108.0)
- added TP36: TestPoint, TestPoint:TestPoint_Pad_D1.0mm, F.Cu at (128.8, 76.7)
- added TP37: TestPoint, TestPoint:TestPoint_Pad_D1.0mm, F.Cu at (95.8, 81.0)
- added TP38: TestPoint, TestPoint:TestPoint_Pad_D1.0mm, F.Cu at (139.4, 80.5)
- added TP39: TestPoint, TestPoint:TestPoint_Pad_D1.0mm, F.Cu at (134.4, 78.0)
- added TP40: TestPoint, TestPoint:TestPoint_Pad_D1.0mm, F.Cu at (104.1, 80.8)
- added TP41: TestPoint, TestPoint:TestPoint_Pad_D1.0mm, F.Cu at (112.5, 82.3)
- added TP42: TestPoint, TestPoint:TestPoint_Pad_D1.0mm, F.Cu at (131.3, 82.0)
- added TP43: TestPoint, TestPoint:TestPoint_Pad_D1.0mm, F.Cu at (118.6, 56.1)
- added TP44: TestPoint, TestPoint:TestPoint_Pad_D1.0mm, F.Cu at (136.7, 55.9)
- added TP45: TestPoint, TestPoint:TestPoint_Pad_D1.0mm, F.Cu at (123.4, 57.9)
- added TP46: TestPoint, TestPoint:TestPoint_Pad_D1.0mm, F.Cu at (101.3, 57.9)
- added TP47: TestPoint, TestPoint:TestPoint_Pad_D1.0mm, F.Cu at (97.0, 56.6)
- added TP48: TestPoint, TestPoint:TestPoint_Pad_D1.0mm, F.Cu at (119.1, 105.4)
- added TP49: TestPoint, TestPoint:TestPoint_Pad_D1.0mm, F.Cu at (117.6, 110.2)
- added TP50: TestPoint, TestPoint:TestPoint_Pad_D1.0mm, F.Cu at (133.9, 107.7)
- added TP51: TestPoint, TestPoint:TestPoint_Pad_D1.0mm, F.Cu at (115.8, 101.3)
- added TP52: TestPoint, TestPoint:TestPoint_Pad_D1.0mm, F.Cu at (95.2, 108.7)
- added TP53: TestPoint, TestPoint:TestPoint_Pad_D1.0mm, F.Cu at (118.9, 76.7)
- added TP54: TestPoint, TestPoint:TestPoint_Pad_D1.0mm, F.Cu at (119.9, 84.1)
- added TP55: TestPoint, TestPoint:TestPoint_Pad_D1.0mm, F.Cu at (126.2, 84.1)
- added TP56: TestPoint, TestPoint:TestPoint_Pad_D1.0mm, F.Cu at (139.2, 84.1)
- added TP57: TestPoint, TestPoint:TestPoint_Pad_D1.0mm, F.Cu at (135.4, 83.8)
- J2: footprint formula_slug_footprint_library:FPC_12-CABLE-0.5mm-0.3mm -> formula_slug_footprint_library:CONN12x1_FH34SRJ-12S-0.5SH50_HIR
- J4: footprint formula_slug_footprint_library:FPC-12PIN-CABLE-1mm-0.71mm -> formula_slug_footprint_library:TE_84952-5
- moved J4 136.1 mm to (174.2, 81.8)
- moved J2 131.1 mm to (175.7, 58.9)
- moved TP19 82.8 mm to (191.0, 86.9), turned to 180 degrees
- moved TP21 81.2 mm to (188.5, 88.1), turned to 180 degrees
- moved TP17 79.3 mm to (191.0, 84.3), turned to 180 degrees
- moved TP20 77.4 mm to (188.5, 85.6), turned to 180 degrees
- moved TP15 74.3 mm to (191.0, 80.5), turned to 180 degrees
- moved TP18 72.1 mm to (188.5, 81.8), turned to 180 degrees
- moved TP16 68.8 mm to (188.5, 79.2), turned to 180 degrees
- moved TP2 56.5 mm to (187.7, 63.8), turned to 90 degrees
- moved TP4 54.5 mm to (189.0, 59.9), turned to 90 degrees
- moved TP1 53.9 mm to (185.2, 63.8), turned to 90 degrees
- moved TP6 51.5 mm to (189.0, 56.1), turned to 90 degrees
- moved TP3 50.2 mm to (185.2, 59.9), turned to 90 degrees
- moved TP5 47.0 mm to (185.2, 56.1), turned to 90 degrees
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Routing:
- net +5V: track 54.6 -> 1.27 mm
- net V-: track 22.0 -> 0.00 mm
- net /ALERT: track 21.5 -> 0.00 mm
- net /SDA: track 16.5 -> 0.00 mm
- net /SCL: track 16.3 -> 0.00 mm
Other:
- board size 134.7 x 89.8 mm -> 144.4 x 111.8 mm

Commit message: schematic finished??
Parts:
- added C4: 1 uF, Capacitor_SMD:C_0603_1608Metric_Pad1.08x0.95mm_HandSolder, F.Cu at (186.9, 41.9)
- added C5: 1 uF, Capacitor_SMD:C_0603_1608Metric_Pad1.08x0.95mm_HandSolder, F.Cu at (167.4, 79.8)
- added C6: 1 uF, Capacitor_SMD:C_0603_1608Metric_Pad1.08x0.95mm_HandSolder, F.Cu at (189.0, 102.4)
- added J3: FH12-12S-1SH(55), formula_slug_footprint_library:FH12-12S-1SH_55_, F.Cu at (175.6, 107.4)
- added R1: 5k, Resistor_SMD:R_0201_0603Metric, F.Cu at (179.8, 49.5)
- added R2: 5k, Resistor_SMD:R_0201_0603Metric, F.Cu at (180.1, 72.6)
- added R3: 5k, Resistor_SMD:R_0201_0603Metric, F.Cu at (180.6, 96.3)
- added TP10: TestPoint, TestPoint:TestPoint_Pad_D1.0mm, F.Cu at (185.7, 126.2)
- added TP11: TestPoint, TestPoint:TestPoint_Pad_D1.0mm, F.Cu at (185.7, 129.3)
- added TP12: TestPoint, TestPoint:TestPoint_Pad_D1.0mm, F.Cu at (188.7, 120.1)
- added TP13: TestPoint, TestPoint:TestPoint_Pad_D1.0mm, F.Cu at (188.7, 123.2)
- added TP14: TestPoint, TestPoint:TestPoint_Pad_D1.0mm, F.Cu at (188.7, 126.2)
- added TP8: TestPoint, TestPoint:TestPoint_Pad_D1.0mm, F.Cu at (185.7, 120.1)
- added TP9: TestPoint, TestPoint:TestPoint_Pad_D1.0mm, F.Cu at (185.7, 123.2)
- added U4: TMP1075D, Package_SO:SO-8_3.9x4.9mm_P1.27mm, F.Cu at (168.0, 85.6)
- added U5: TMP1075D, Package_SO:SO-8_3.9x4.9mm_P1.27mm, F.Cu at (188.0, 108.5)
- added U6: TMP1075D, Package_SO:SO-8_3.9x4.9mm_P1.27mm, F.Cu at (168.1, 126.2)
- moved U2 41.0 mm to (188.0, 47.5), turned to 90 degrees
- moved U3 34.9 mm to (148.1, 128.8), turned to 90 degrees
- moved C2 31.7 mm to (167.4, 120.1), turned to 0 degrees
- moved C3 20.7 mm to (149.3, 121.7), turned to 0 degrees
- moved C1 17.6 mm to (147.3, 61.5), turned to 0 degrees
- moved U1 16.0 mm to (148.0, 67.9), turned to 90 degrees
Routing:
- net +5V: track 1.27 -> 0.00 mm
Other:
- board size 144.4 x 111.8 mm -> 144.4 x 133.8 mm

Commit message: more
Parts:
- added H1: MountingHole_Pad, MountingHole:MountingHole_3.2mm_M3_Pad, F.Cu at (134.1, 149.9)
- moved TP34 49.7 mm to (147.1, 115.3)
- moved TP52 49.6 mm to (142.2, 124.7)
- moved TP37 46.1 mm to (140.2, 68.8)
- moved TP29 45.2 mm to (147.1, 113.3)
- moved TP47 45.0 mm to (140.2, 43.9)
- moved TP40 43.2 mm to (143.8, 98.0)
- moved TP35 43.2 mm to (143.3, 121.9)
- moved TP46 42.5 mm to (143.3, 51.1)
- moved TP22 41.4 mm to (146.1, 51.3)
- moved TP28 39.4 mm to (146.1, 48.3)
- moved TP31 37.3 mm to (143.5, 119.4)
- moved TP30 35.1 mm to (143.8, 113.8)
- moved TP23 34.2 mm to (146.6, 45.7)
- moved TP24 32.0 mm to (143.3, 48.3)
- moved TP41 31.7 mm to (143.5, 88.9)
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Routing:
- net +5V: track 0.00 -> 21.5 mm
- net V-: track 0.00 -> 17.9 mm
- net Net-(J2-Pin_10): track 3.22 -> 0.00 mm
- net Net-(J2-Pin_8): track 1.80 -> 0.00 mm
- net Net-(J2-Pin_9): track 1.60 -> 0.00 mm
