File: temp-sense-board-flex-prototype-v.1/temp-sense-board-flex-prototype-v.1.kicad_pcb (KiCad board)
At the start: 2 copper layers, 144.4 x 133.8 mm, 79 parts, among them J2 FH34SRJ-12S-0.5SH(50), J3 FH12-12S-1SH(55), J4 1-84953-2, J5 FH34SRJ-12S-0.5SH(50), J6 FH12-12S-1SH(55), J7 1-84953-2, U1 TMP1075D, U2 TMP1075D, U3 TMP1075D, U4 TMP1075D, U5 TMP1075D, U6 TMP1075D

Commit message: Mounting holes, auxillary board connectors, starting layout with finalized connectors?
Parts:
- removed J2: FH34SRJ-12S-0.5SH(50), formula_slug_footprint_library:CONN12x1_FH34SRJ-12S-0.5SH50_HIR
- removed J3: FH12-12S-1SH(55), formula_slug_footprint_library:FH12-12S-1SH_55_
- removed J4: 1-84953-2, formula_slug_footprint_library:TE_84952-5
- removed TP22, TP23, TP24, TP25, TP26, TP27, TP28, TP29, TP30, TP31, TP32, TP33, TP34, TP35, TP36, TP37, TP38, TP39, TP4, TP40, TP41, TP42, TP43, TP44, TP45, TP46, TP47, TP48, TP49, TP5, TP50, TP51, TP52, TP53, TP54, TP55, TP56, TP57, TP6, TP7: TestPoint, TestPoint:TestPoint_Pad_D1.0mm
- added H2: MountingHole_Pad, MountingHole:MountingHole_3.2mm_M3_Pad, F.Cu at (154.2, 26.4)
- added H3: MountingHole_Pad, MountingHole:MountingHole_3.2mm_M3_Pad, F.Cu at (174.0, 149.9)
- added H4: MountingHole_Pad, MountingHole:MountingHole_3.2mm_M3_Pad, F.Cu at (184.2, 149.9)
- moved J7 25.9 mm to (50.4, 106.2)
- moved J6 25.4 mm to (50.2, 80.8)
- moved J5 1.87 mm to (50.0, 57.9), turned to 90 degrees
- moved U5 0.25 mm to (188.2, 108.5)
- moved U4 0.15 mm to (167.9, 85.6)
- moved U1 0.07 mm to (148.0, 67.8)
Connections:
- H1 pad 1: unconnected-(H1-Pad1) -> /v1
- J5 pad 1: Net-(J5-Pin_1) -> V-
- J5 pad 2: Net-(J5-Pin_2) -> /SCL
- J5 pad 3: Net-(J5-Pin_3) -> /SDA
- J5 pad 4: Net-(J5-Pin_4) -> /ALERT
- J5 pad 5: Net-(J5-Pin_5) -> +5V
- J5 pad 6: Net-(J5-Pin_6) -> /v3
- J5 pad 7: Net-(J5-Pin_7) -> /v2
- J5 pad 8: Net-(J5-Pin_8) -> /v1
- J5 pad 9: Net-(J5-Pin_9) -> /v0
- J6 pad 1: Net-(J6-Pin_1) -> V-
- J6 pad 2: Net-(J6-Pin_2) -> /SCL
- J6 pad 3: Net-(J6-Pin_3) -> /SDA
- J6 pad 4: Net-(J6-Pin_4) -> /ALERT
- J6 pad 5: Net-(J6-Pin_5) -> +5V
- J7 pad 1: Net-(J7-Pin_1) -> V-
- J7 pad 2: Net-(J7-Pin_2) -> /SCL
- J7 pad 3: Net-(J7-Pin_3) -> /SDA
- J7 pad 4: Net-(J7-Pin_4) -> /ALERT
- J7 pad 5: Net-(J7-Pin_5) -> +5V
- R1 pad 2: /ALERT -> /SDA
- R3 pad 2: /SDA -> /ALERT
- TP1 pad 1: Net-(J2-Pin_12) -> Net-(J5-Pin_12)
- TP10 pad 1: Net-(J3-Pin_10) -> Net-(J6-Pin_10)
- TP11 pad 1: Net-(J3-Pin_9) -> Net-(J6-Pin_9)
- TP12 pad 1: Net-(J3-Pin_8) -> Net-(J6-Pin_8)
- TP13 pad 1: Net-(J3-Pin_7) -> Net-(J6-Pin_7)
- TP14 pad 1: Net-(J3-Pin_6) -> Net-(J6-Pin_6)
- TP15 pad 1: Net-(J4-Pin_12) -> Net-(J7-Pin_12)
- TP16 pad 1: Net-(J4-Pin_11) -> Net-(J7-Pin_11)
- TP17 pad 1: Net-(J4-Pin_10) -> Net-(J7-Pin_10)
- TP18 pad 1: Net-(J4-Pin_9) -> Net-(J7-Pin_9)
- TP19 pad 1: Net-(J4-Pin_8) -> Net-(J7-Pin_8)
- TP2 pad 1: Net-(J2-Pin_11) -> Net-(J5-Pin_11)
- TP20 pad 1: Net-(J4-Pin_7) -> Net-(J7-Pin_7)
- TP21 pad 1: Net-(J4-Pin_6) -> Net-(J7-Pin_6)
- TP3 pad 1: Net-(J2-Pin_10) -> Net-(J5-Pin_10)
- TP8 pad 1: Net-(J3-Pin_12) -> Net-(J6-Pin_12)
- TP9 pad 1: Net-(J3-Pin_11) -> Net-(J6-Pin_11)
Routing:
- net /SCL: track 0.00 -> 135.9 mm
- net V-: track 17.9 -> 14.2 mm
- net +5V: track 21.5 -> 18.1 mm
- net Net-(J2-Pin_12): track 0.66 -> 0.00 mm
Other:
- outline, holes or cut-outs redrawn

Commit message: fixed connector glitch, unincluded alert pin, layed out traces, updated schematic
Parts:
- removed TP12, TP13, TP14, TP19, TP20, TP21: TestPoint, TestPoint:TestPoint_Pad_D1.0mm
- added TP4: TestPoint, TestPoint:TestPoint_Pad_D1.0mm, F.Cu at (192.8, 121.4)
- moved R3 41.6 mm to (148.7, 122.9)
- moved R2 33.8 mm to (146.4, 74.7)
- moved J7 25.8 mm to (49.9, 80.3)
- moved J6 25.2 mm to (50.2, 106.0)
- moved R1 9.76 mm to (185.2, 41.4), turned to 180 degrees
- moved U6 0.25 mm to (167.9, 126.2)
- moved U3 0.13 mm to (148.0, 128.7)
- moved H1 0.07 mm to (134.1, 149.9)
Connections:
- J5 pad 4: /ALERT -> +5V
- J5 pad 5: +5V -> /v3
- J5 pad 6: /v3 -> /v2
- J5 pad 7: /v2 -> /v1
- J5 pad 8: /v1 -> /v0
- J5 pad 9: /v0 -> Net-(J5-Pin_9)
- J6 pad 4: /ALERT -> +5V
- J6 pad 5: +5V -> /v3
- J6 pad 6: Net-(J6-Pin_6) -> /v2
- J6 pad 7: Net-(J6-Pin_7) -> /v1
- J6 pad 8: Net-(J6-Pin_8) -> /v0
- J7 pad 4: /ALERT -> +5V
- J7 pad 5: +5V -> /v3
- J7 pad 6: Net-(J7-Pin_6) -> /v2
- J7 pad 7: Net-(J7-Pin_7) -> /v1
- J7 pad 8: Net-(J7-Pin_8) -> /v0
- R3 pad 2: /ALERT -> unconnected-(R3-Pad2)
- U1 pad 3: /ALERT -> unconnected-(U1-ALERT-Pad3)
- U2 pad 3: /ALERT -> unconnected-(U2-ALERT-Pad3)
- U3 pad 3: /ALERT -> unconnected-(U3-ALERT-Pad3)
- U4 pad 3: /ALERT -> unconnected-(U4-ALERT-Pad3)
- U5 pad 3: /ALERT -> unconnected-(U5-ALERT-Pad3)
- U6 pad 3: /ALERT -> unconnected-(U6-ALERT-Pad3)
Routing:
- net /SDA: track 0.00 -> 585.6 mm, vias 0 -> 10
- net /SCL: track 135.9 -> 455.6 mm, vias 0 -> 2
- net +5V: track 18.1 -> 223.8 mm
- net V-: track 14.2 -> 206.4 mm, vias 0 -> 2
Other:
- outline, holes or cut-outs redrawn

Commit message: added voltage tap net class, changed edgecuts for connector and tem sensors, other things in my list trust
Parts:
- moved J7 0.29 mm to (50.2, 80.3)
- moved U4 0.21 mm to (168.1, 85.6)
Routing:
- net /SDA: track 585.6 -> 14.3 mm, vias 10 -> 0
- net /SCL: track 455.6 -> 0.00 mm, vias 2 -> 0
- net +5V: track 223.8 -> 12.4 mm
- net V-: track 206.4 -> 6.93 mm, vias 2 -> 0
- net /v2: track 0.00 -> 8.42 mm
- net /v0: track 0.00 -> 7.81 mm
- net Net-(J7-Pin_9): track 0.00 -> 6.77 mm
Other:
- outline, holes or cut-outs redrawn

Commit message: locked component placement yay
Parts:
- moved J5 0.24 mm to (50.2, 57.9)
- moved U6 0.21 mm to (168.1, 126.2)
- moved J6 0.17 mm to (50.3, 106.0)
- moved U2 0.17 mm to (188.1, 47.5)
- moved U1 0.14 mm to (148.1, 67.8)
- moved U3 0.14 mm to (148.1, 128.7)
- moved U5 0.10 mm to (188.1, 108.4)
Routing:
- net /SDA: track 14.3 -> 0.00 mm
- net +5V: track 12.4 -> 3.41 mm
- net V-: track 6.93 -> 3.32 mm
Other:
- outline, holes or cut-outs redrawn

Commit message: test module TSB - save everything before changing mounting holes
Parts:
- J5: footprint formula_slug_footprint_library:FPC_12-CABLE-0.5mm-0.3mm -> formula_slug_footprint_library:FPC-12PIN-CABLE-P0.5mm-W0.3mm
- J6: footprint formula_slug_footprint_library:FPC-12PIN-CABLE-1mm-0.65mm -> formula_slug_footprint_library:FPC-12PIN-CABLE-P1mm-W0.65mm
- J7: footprint formula_slug_footprint_library:FPC-12PIN-CABLE-1mm-0.71mm -> formula_slug_footprint_library:FPC-12PIN-CABLE-P1mm-W0.71mm
- moved TP1 5.49 mm to (192.0, 57.8)
- moved TP2 5.49 mm to (192.0, 55.5)
- moved TP3 5.49 mm to (192.3, 60.1)
- moved R2 2.27 mm to (147.0, 72.5)
- moved J7 0.10 mm to (50.3, 80.3)
- moved J5 0.06 mm to (50.3, 57.9)
Routing:
- net /v2: track 8.42 -> 0.00 mm
- net /v0: track 7.81 -> 7.01 mm

Commit message: finish mounting points, start routing!
Parts:
- removed R3: 5k, Resistor_SMD:R_0201_0603Metric
- R1, R2: footprint Resistor_SMD:R_0201_0603Metric -> Resistor_SMD:R_0603_1608Metric
- moved R1 68.6 mm to (184.5, 110.0), turned to -90 degrees
- moved R2 51.0 mm to (184.5, 107.0), turned to -90 degrees
- moved C3 2.45 mm to (148.5, 124.0)
- moved C5 1.69 mm to (167.5, 81.0)
- moved C2 1.42 mm to (168.0, 121.5)
- moved C1 1.39 mm to (147.5, 63.0)
- moved C6 0.90 mm to (188.1, 103.5)
- moved C4 0.62 mm to (188.1, 42.5)
- moved H4 0.18 mm to (184.3, 149.9)
- moved H3 0.18 mm to (174.2, 149.9)
- moved H2 0.11 mm to (154.1, 26.3)
- moved H1 0.10 mm to (134.1, 149.9)
Routing:
- net V-: track 3.32 -> 318.7 mm, vias 0 -> 10
- net +5V: track 3.41 -> 300.7 mm, vias 0 -> 5
- net /SCL: track 0.00 -> 278.4 mm, vias 0 -> 10
- net /SDA: track 0.00 -> 269.1 mm, vias 0 -> 4
- net /v2: track 0.00 -> 199.4 mm, vias 0 -> 4
- net /v0: track 7.01 -> 205.0 mm, vias 0 -> 2
- net /v1: track 0.00 -> 186.0 mm, vias 0 -> 2
- net /v3: track 0.00 -> 127.9 mm
Other:
- outline, holes or cut-outs redrawn

Commit message: finish temp sense prototype flex board; make auxiliary-test-board
Parts:
- J6: moved to B.Cu
- moved TP4 57.4 mm to (193.0, 64.0), turned to 90 degrees
- moved TP10 35.6 mm to (193.0, 96.0)
- moved TP8 34.5 mm to (193.0, 90.0)
- moved TP11 30.0 mm to (193.0, 99.0)
- moved TP9 24.6 mm to (193.0, 93.0)
- moved TP15 6.24 mm to (193.0, 72.5)
- moved TP17 5.58 mm to (193.0, 78.5)
- moved TP1 2.96 mm to (193.0, 55.0)
- moved TP2 2.69 mm to (193.0, 58.0)
- moved TP3 1.19 mm to (193.0, 61.0)
- moved TP16 0.49 mm to (193.0, 75.5)
- moved TP18 0.22 mm to (193.0, 81.5)
- turned J6 to -90 degrees
Routing:
- net V-: track 318.7 -> 559.4 mm, vias 10 -> 14
- net /SCL: track 278.4 -> 507.1 mm, vias 10 -> 12
- net /v3: track 127.9 -> 356.3 mm, vias 0 -> 4
- net /SDA: track 269.1 -> 491.5 mm, vias 4 -> 5
- net +5V: track 300.7 -> 518.3 mm, vias 5 -> 8
- net /v0: track 205.0 -> 390.4 mm, vias 2 -> 5
- net /v1: track 186.0 -> 368.5 mm, vias 2 -> 5
- net /v2: track 199.4 -> 379.6 mm, vias 4 -> 7
- net Net-(J6-Pin_12): track 0.00 -> 149.9 mm, vias 0 -> 3
- net Net-(J6-Pin_11): track 0.00 -> 148.2 mm, vias 0 -> 3
- net Net-(J5-Pin_9): track 0.00 -> 146.8 mm, vias 0 -> 2
- net Net-(J6-Pin_10): track 0.00 -> 146.6 mm, vias 0 -> 3
- net Net-(J5-Pin_10): track 0.00 -> 146.1 mm, vias 0 -> 2
- net Net-(J5-Pin_11): track 0.00 -> 145.5 mm, vias 0 -> 2
- net Net-(J5-Pin_12): track 0.00 -> 144.9 mm, vias 0 -> 2
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Other:
- board text added: "Stiffener"
- board text added: "Total Thickness: 0.3mm"
