File: iso-vi-pcb/ISO VI PCB .kicad_sch (KiCad schematic)
At the start: 14 parts, among them U1 STM32F405RGTx, U2 ADS124S08IPBSR, U3 SN65HVD230, U4 LMR36510ADDA

Commit message: UPDATE 2: SN65HVD230 WIRING COMPLETE
Wire SN65HVD230 CAN transceiver

- Connect U3 D to STM32 CAN1_TX (PA12).
- Connect U3 R to STM32 CAN1_RX (PA11).
- Connect U3 VCC to 3.3 V and GND to ground.
- Ground RS to set the transceiver to high-speed mode.
- Add a 100 nF bypass capacitor across 3.3 V and ground.
- Add CAN_H and CAN_L net labels to the bus pins.
- Mark Vref as not connected.
Parts:
- added C10, C13, C14, C15, C16, C18, C20: 100nF, symbol Device:C
- added C11, C12: 2.2uF, symbol Device:C
- added C17: 4.7uF, symbol Device:C
- added C19: 1uF, symbol Device:C
- added R3: 100kΩ, symbol Device:R
Connections:
- net +3.3V: now also U1.1 (VBAT), U1.13 (VDDA), U3.3 (VCC), C10.1, C13.1, C14.1, C15.1, C16.1, C17.1, C18.1, C19.1
- net GND: now also U1.12 (VSSA), U1.18 (VSS), U1.63 (VSS), U3.2 (GND), U3.8 (Rs), C10.2, C11.2, C12.2, C13.2, C14.2, C15.2, C16.2, C17.2, C18.2, C19.2, C20.2, R3.1
- net CAN1_TX: now reaches U3.1 (D)
- net CAN1_TX: now also U1.45 (PA12)
- net CAN1_RX: now reaches U3.4 (R)
- net CAN1_RX: now also U1.44 (PA11)
- net CAN_L: now reaches U3.6 (CANL)
- net CAN_H: now reaches U3.7 (CANH)
- net at U1.31 (VCAP_1): now also C11.1
- net SWDIO: now reaches U1.46 (PA13)
- net at U1.47 (VCAP_2): now also C12.1
- net SWCLK: now reaches U1.49 (PA14)
- net at U1.60 (BOOT0): now also R3.2
- net NRST: now reaches U1.7 (NRST)
- net NRST: now also C20.1
- no-connect marks 0 -> 1
Other:
- moved on the sheet: U2

Commit message: UPDATE 3: ADS124S08 INPUT MAPPING
Map six assumed peak-hold outputs to the ADC

- Connect PH_OUT1 to U2 AIN0 (pin 7).
- Connect PH_OUT2 to U2 AIN1 (pin 6).
- Connect PH_OUT3 to U2 AIN2 (pin 5).
- Connect PH_OUT4 to U2 AIN3 (pin 4).
- Connect PH_OUT5 to U2 AIN4 (pin 3) and PH_OUT6 to U2 AIN5 (pin 2).
- Connect U2 AINCOM (pin 1) to GND for the assumed single-ended inputs; remove the NC markers from these pins.
- Document the assumed conditioned positive 0–2.5 V peak outputs; raw 0–5 V sensor signals must not connect directly to the ADC.
- Export a netlist to confirm the pin mappings; sensor connectors and peak-hold circuits are still absent, and ADC/STM32 grounds remain shared, so the board is not galvanically isolated.
Parts:
- added C21: 330nF, Capacitor_SMD:C_0603_1608Metric_Pad1.08x0.95mm_HandSolder, symbol Device:C
- added C22, C23: 100nF, Capacitor_SMD:C_0603_1608Metric_Pad1.08x0.95mm_HandSolder, symbol Device:C
- added C24, C25: 10pF, Capacitor_SMD:C_0603_1608Metric_Pad1.08x0.95mm_HandSolder, symbol Device:C
- added C26: 1uF, Capacitor_SMD:C_0805_2012Metric_Pad1.18x1.45mm_HandSolder, symbol Device:C
- added D1: D, symbol Device:D
- added J1: ZX-XH2.54-4PZZ, Connector_JST:JST_XH_B4B-XH-A_1x04_P2.50mm_Vertical, symbol Connector:Conn_01x04_Pin
- added J2: Conn_01x03_Pin, Connector_JST:JST_XH_B3B-XH-A_1x03_P2.50mm_Vertical, symbol Connector:Conn_01x03_Pin
- added J3, J4, J5, J6, J7, J8: Conn_01x02, symbol Connector_Generic:Conn_01x02
- added U10, U5, U6, U7, U8, U9: TLV9064, symbol Amplifier_Operational:TLV9064
- added Y1: 16MHz, Crystal:Crystal_SMD_3225-4Pin_3.2x2.5mm_HandSoldering, symbol Device:Crystal_GND24
- C1: footprint (none) -> Capacitor_SMD:C_1206_3216Metric_Pad1.33x1.80mm_HandSolder
- C10, C13, C14, C15, C16, C18, C20, C3, C6: footprint (none) -> Capacitor_SMD:C_0603_1608Metric_Pad1.08x0.95mm_HandSolder
- C11, C12, C17, C19, C5: footprint (none) -> Capacitor_SMD:C_0805_2012Metric_Pad1.18x1.45mm_HandSolder
- C7, C8, C9: footprint (none) -> Capacitor_SMD:C_1210_3225Metric_Pad1.33x2.70mm_HandSolder
- L1: footprint (none) -> Inductor_SMD:L_Bourns-SRR1005
- R1, R2, R3: footprint (none) -> Resistor_SMD:R_0603_1608Metric_Pad0.98x0.95mm_HandSolder
- U2: footprint PBS0032A_N -> Package_QFP:TQFP-32_5x5mm_P0.5mm
Connections:
- net +3.3V: now also U1.19 (VDD), U1.32 (VDD), U1.48 (VDD), U1.64 (VDD), U2.15 (IOVDD), U2.16 (DVDD), U2.18 (RESET_N), U2.26 (AVDD), C21.1, C22.1, C23.1, J1.1 (Pin_1)
- net GND: now also U2.1 (AINCOM), U2.14 (DGND), U2.17 (CLK), U2.24 (REFCOM), U2.27 (AVSS), U2.28 (AVSS-SW), U2.8 (START_SYNC), C21.2, C22.2, C23.2, C24.2, C25.2, C26.2, J1.2 (Pin_2), J2.3 (Pin_3), Y1.2 (G), Y1.4 (G); no longer U4.4 (PG)
- net ADC_MOSI: now reaches U2.10 (DIN)
- net ADC_MOSI: now also U1.23 (PA7)
- net ADC_SCLK: now reaches U2.11 (SCLK)
- net ADC_SCLK: now also U1.21 (PA5)
- net ADC_MISO: now reaches U2.12 (DOUT_DRDY_N)
- net ADC_MISO: now also U1.22 (PA6)
- net ADC_DRDY_N: now reaches U2.13 (DRDY_N)
- net ADC_DRDY_N: now also U1.26 (PB0)
- net PH_OUT6: now reaches U2.2 (AIN5)
- net at U2.23 (REFOUT): now also C26.1
- net PH_OUT5: now reaches U2.3 (AIN4)
- net PH_OUT4: now reaches U2.4 (AIN3)
- net PH_OUT3: now reaches U2.5 (AIN2)
- net PH_OUT2: now reaches U2.6 (AIN1)
- net PH_OUT1: now reaches U2.7 (AIN0)
- net ADC_CS_N: now reaches U2.9 (CS_N)
- net ADC_CS_N: now also U1.20 (PA4)
- net HSE_IN: now reaches U1.5 (PH0)
- net HSE_IN: now also C25.1, Y1.3
- net HSE_OUT: now reaches U1.6 (PH1)
- net HSE_OUT: now also C24.1, Y1.1
- net CAN_H: no longer names the net of U3.7 (CANH)
- net CAN_H: now also J2.1 (Pin_1)
- net CAN_L: no longer names the net of U3.6 (CANL)
- net CAN_L: now also J2.2 (Pin_2)
- net SWCLK: no longer names the net of U1.49 (PA14)
- net SWCLK: now also J1.3 (Pin_3)
- net SWDIO: no longer names the net of U1.46 (PA13)
- net SWDIO: now also J1.4 (Pin_4)
- no-connect marks 1 -> 51
Other:
- moved on the sheet: U2, U3
