File: strain-gauges/tripple-strain-gauge/adc-chip.kicad_sch (KiCad schematic)
At the start: 6 parts, among them U2 MCP3564R-E/ST

Commit message: added caps to ground for 3V3 and 12V; changed strain gauge and op amp to 3V3_A; changed ADC DVDD to 3v3
Parts:
- renumbered C9 to C10, C10 to C11
Connections:
- net +3V3: now also U2.20 (DVDD)
- net +3.3VA renamed +3V3_A
- net +3V3_A: no longer U2.20 (DVDD)
Changed lines of the file:
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@@
+		)
+	)
+	(rectangle
+		(start 15.24 19.304)
+		(end 154.686 67.818)
+		(stroke
+			(width 0)
+			(type default)
+		)
+		(fill
+			(type none)
 		)
 	)
@@
 		)
 	)
-	(polyline
-		(pts
-			(xy 155.702 77.724) (xy 155.702 19.812)
-		)
-		(stroke
-			(width 0)
-			(type default)
-		)
-	)
 	(wire
 		(pts
@@
 		)
 	)
-	(polyline
-		(pts
-			(xy 155.702 19.304) (xy 15.24 19.304)
-		)
-		(stroke
-			(width 0)
-			(type default)
-		)
-	)
 	(wire
 		(pts
@@
 		)
 	)
-	(polyline
-		(pts
-			(xy 15.24 19.304) (xy 15.24 77.216)
-		)
-		(stroke
-			(width 0)
-			(type default)
-		)
-	)
 	(wire
 		(pts
 			(xy 189.23 40.64) (xy 172.72 40.64)
-		)
-		(stroke
-			(width 0)
-			(type default)
-		)
-	)
-	(polyline
-		(pts
-			(xy 15.24 77.216) (xy 155.702 77.216)
 		)
 		(stroke
@@
 		(dnp no)
 		(fields_autoplaced yes)
-		(property "Reference" "C9"
+		(property "Reference" "C10"
 			(at 193.04 35.5599 0)
 			(show_name no)
@@
 			(project "tripple-strain-gauge"
 				(path "/e994741c-7c7d-4124-9d00-43b883baa61d/9081ec08-249e-44b2-aa2e-ebca62a73fcf"
-					(reference "C9")
+					(reference "C10")
 					(unit 1)
 				)
@@
 	)
 	(symbol
+		(lib_id "power:+3V3")
+		(at 135.89 34.29 0)
+		(unit 1)
+		(body_style 1)
+		(exclude_from_sim no)
+		(in_bom yes)
+		(on_board yes)
+		(in_pos_files yes)
+		(dnp no)
+		(fields_autoplaced yes)
+		(property "Reference" "#PWR038"
+			(at 135.89 38.1 0)
+			(hide yes)
+			(show_name no)
+			(do_not_autoplace no)
+			(effects
+				(font
+					(size 1.27 1.27)
+				)
+			)
+		)
+		(property "Value" "+3V3"
+			(at 135.89 29.21 0)
+			(show_name no)
+			(do_not_autoplace no)
+			(effects
+				(font
+					(size 1.27 1.27)
+				)
+			)
+		)
+		(property "Footprint" "Package_DFN_QFN:Diodes_UDFN3810-9_TYPE_B"
+			(at 135.89 34.29 0)
+			(hide yes)
+			(show_name no)
+			(do_not_autoplace no)
+			(effects
+				(font
+					(size 1.27 1.27)
+				)
+			)
+		)
+		(property "Datasheet" ""
+			(at 135.89 34.29 0)
+			(hide yes)
+			(show_name no)
+			(do_not_autoplace no)
+			(effects
+				(font
+					(size 1.27 1.27)
+				)
+			)
+		)
+		(property "Description" "Power symbol creates a global label with name \"+3V3\""
+			(at 135.89 34.29 0)
+			(hide yes)
+			(show_name no)
+			(do_not_autoplace no)
+			(effects
+				(font
+					(size 1.27 1.27)
+				)
+			)
+		)
+		(pin "1"
+		)
+		(instances
+			(project "tripple-strain-gauge"
+				(path "/e994741c-7c7d-4124-9d00-43b883baa61d/9081ec08-249e-44b2-aa2e-ebca62a73fcf"
+					(reference "#PWR038")
+					(unit 1)
+				)
+			)
+		)
+	)
+	(symbol
 		(lib_id "power:GND")
 		(at 172.72 41.91 0)
@@
 		(in_pos_files yes)
 		(dnp no)
-		(property "Reference" "#PWR033"
+		(property "Reference" "#PWR030"
 			(at 172.72 48.26 0)
 			(hide yes)
@@
 			(project "tripple-strain-gauge"
 				(path "/e994741c-7c7d-4124-9d00-43b883baa61d/9081ec08-249e-44b2-aa2e-ebca62a73fcf"
-					(reference "#PWR033")
+					(reference "#PWR030")
 					(unit 1)
 				)
@@
 		(in_pos_files yes)
 		(dnp no)
-		(property "Reference" "#PWR032"
+		(property "Reference" "#PWR028"
 			(at 142.24 41.91 0)
 			(hide yes)
@@
 			(project "tripple-strain-gauge"
 				(path "/e994741c-7c7d-4124-9d00-43b883baa61d/9081ec08-249e-44b2-aa2e-ebca62a73fcf"
-					(reference "#PWR032")
+					(reference "#PWR028")
 					(unit 1)
 				)
@@
 		(dnp no)
 		(fields_autoplaced yes)
-		(property "Reference" "#PWR034"
+		(property "Reference" "#PWR025"
 			(at 54.61 39.37 0)
 			(hide yes)
@@
 			)
 		)
-		(property "Value" "+3.3VA"
+		(property "Value" "+3V3_A"
 			(at 54.61 30.48 0)
 			(show_name no)
@@
 			(project "tripple-strain-gauge"
 				(path "/e994741c-7c7d-4124-9d00-43b883baa61d/9081ec08-249e-44b2-aa2e-ebca62a73fcf"
-					(reference "#PWR034")
+					(reference "#PWR025")
 					(unit 1)
 				)
@@
 		(dnp no)
 		(fields_autoplaced yes)
-		(property "Reference" "C10"
+		(property "Reference" "C11"
 			(at 204.47 35.5599 0)
 			(show_name no)
@@
 			(project "tripple-strain-gauge"
 				(path "/e994741c-7c7d-4124-9d00-43b883baa61d/9081ec08-249e-44b2-aa2e-ebca62a73fcf"
-					(reference "C10")
+					(reference "C11")
 					(unit 1)
 				)
@@
 		(dnp no)
 		(fields_autoplaced yes)
-		(property "Reference" "#PWR029"
+		(property "Reference" "#PWR031"
 			(at 214.63 35.56 0)
 			(hide yes)
@@
 			)
 		)
-		(property "Value" "+3.3VA"
+		(property "Value" "+3V3_A"
 			(at 214.63 26.67 0)
 			(show_name no)
@@
 			(project "tripple-strain-gauge"
 				(path "/e994741c-7c7d-4124-9d00-43b883baa61d/9081ec08-249e-44b2-aa2e-ebca62a73fcf"
-					(reference "#PWR029")
-					(unit 1)
-				)
-			)
-		)
-	)
-	(symbol
-		(lib_id "power:+3.3VA")
-		(at 135.89 34.29 0)
-		(mirror y)
-		(unit 1)
-		(body_style 1)
-		(exclude_from_sim no)
-		(in_bom yes)
-		(on_board yes)
-		(in_pos_files yes)
-		(dnp no)
-		(fields_autoplaced yes)
-		(property "Reference" "#PWR028"
-			(at 135.89 38.1 0)
-			(hide yes)
-			(show_name no)
-			(do_not_autoplace no)
-			(effects
-				(font
-					(size 1.27 1.27)
-				)
-			)
-		)
-		(property "Value" "+3.3VA"
-			(at 135.89 29.21 0)
-			(show_name no)
-			(do_not_autoplace no)
-			(effects
-				(font
-					(size 1.27 1.27)
-				)
-			)
-		)
-		(property "Footprint" "TSSOP20_ST_MCH"
-			(at 135.89 34.29 0)
-			(hide yes)
-			(show_name no)
-			(do_not_autoplace no)
-			(effects
-				(font
-					(size 1.27 1.27)
-				)
-			)
-		)
-		(property "Datasheet" ""
-			(at 135.89 34.29 0)
-			(hide yes)
-			(show_name no)
-			(do_not_autoplace no)
-			(effects
-				(font
-					(size 1.27 1.27)
-				)
-			)
-		)
-		(property "Description" "Power symbol creates a global label with name \"+3.3VA\""
-			(at 135.89 34.29 0)
-			(hide yes)
-			(show_name no)
-			(do_not_autoplace no)
-			(effects
-				(font
-					(size 1.27 1.27)
-				)
-			)
-		)
-		(pin "1"
-		)
-		(instances
-			(project "tripple-strain-gauge"
-				(path "/e994741c-7c7d-4124-9d00-43b883baa61d/9081ec08-249e-44b2-aa2e-ebca62a73fcf"
-					(reference "#PWR028")
+					(reference "#PWR031")
 					(unit 1)
 				)
@@
 		(in_pos_files yes)
 		(dnp no)
-		(property "Reference" "#PWR031"
+		(property "Reference" "#PWR026"
 			(at 58.42 44.45 0)
 			(hide yes)
@@
 			(project "tripple-strain-gauge"
 				(path "/e994741c-7c7d-4124-9d00-43b883baa61d/9081ec08-249e-44b2-aa2e-ebca62a73fcf"
-					(reference "#PWR031")
+					(reference "#PWR026")
 					(unit 1)
 				)
@@
 		(dnp no)
 		(fields_autoplaced yes)
-		(property "Reference" "#PWR08"
+		(property "Reference" "#PWR029"
 			(at 172.72 35.56 0)
 			(hide yes)
@@
 			(project "tripple-strain-gauge"
 				(path "/e994741c-7c7d-4124-9d00-43b883baa61d/9081ec08-249e-44b2-aa2e-ebca62a73fcf"
-					(reference "#PWR08")
+					(reference "#PWR029")
 					(unit 1)
 				)
