File: strain-gauges/tripple-strain-gauge/tripple-strain-gauge.kicad_sch (KiCad schematic)
At the start: 29 parts, among them IC1 TSV914IDT, J1 Conn_01x07, J2 Conn_01x07, U1 LDK320AM33R

Commit message: added caps to ground for 3V3 and 12V; changed strain gauge and op amp to 3V3_A; changed ADC DVDD to 3v3
Parts:
- added C5, C6: 10nF, Capacitor_SMD:C_0603_1608Metric_Pad1.08x0.95mm_HandSolder, symbol Device:C
- renumbered C5 to C4, C6 to C9, J2 to J1, J1 to J2, JP3 to JP2, JP2 to JP3, R13 to R10, R14 to R11, R8 to R5, R7 to R6, R10 to R7, R12 to R8, R11 to R9
Connections:
- net +12V: now also C5.1
- net +3V3: now also C6.1; no longer C1.1, IC1.4 (VCC+), R1.1, S1.2, S2.2, S3.2, S4.2
- net GND: now also C5.2, C6.2
- net Center_Buffered: now reaches IC1.6 (IN2-), IC1.7 (OUT2), JP1.2, R4.1
- net Reference_Buffered: now reaches IC1.1 (OUT1), IC1.2 (IN1-), R5.2
- net Left_Buffered: now reaches IC1.13 (IN4-), IC1.14 (OUT4), JP2.2, R8.1
- net Right_Buffered: now reaches IC1.8 (OUT3), IC1.9 (IN3-), JP3.2, R9.1
- new net +3V3_A: C1.1, IC1.4 (VCC+), R1.1, S1.2, S2.2, S3.2, S4.2
Other:
- moved on the sheet: C7, C9, JP2, JP3, R8, R9
