File: strain-gauges/tripple-strain-gauge/tripple-strain-gauge.kicad_pcb (KiCad board)
At the start: 2 copper layers, 223 x 50 mm, 35 parts, among them IC1 TSV914IDT, J1 Conn_01x07, J2 Conn_01x07, U1 LDK320AM33R, U2 MCP3564R-E/ST

Commit message: added stiffener area with text for JLCPCB engineers regarding stiffener
Other:
- board text added: "3M tessa8854 Stiffener Area"
Changed lines of the file:
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@@
 		(layer "F.Fab")
+	)
+	(gr_text "3M tessa8854 Stiffener Area"
+		(at 212.06 27.97 0)
+		(layer "User.1")
+		(effects
+			(font
+				(size 1.016 1.016)
+				(thickness 0.1524)
+			)
+			(justify left bottom)
+		)
 	)
 	(segment
@@
 		(net "SPI_CS")
 	)
+	(zone
+		(layer "User.1")
+		(name "3M tessa8854 Stiffener Area")
+		(hatch edge 0.5)
+		(connect_pads
+			(clearance 0)
+		)
+		(min_thickness 0.25)
+		(keepout
+			(tracks allowed)
+			(vias allowed)
+			(pads allowed)
+			(copperpour allowed)
+			(footprints allowed)
+		)
+		(placement
+			(enabled no)
+			(sheetname "/")
+		)
+		(fill
+			(thermal_gap 0.5)
+			(thermal_bridge_width 0.5)
+			(island_removal_mode 0)
+		)
+		(polygon
+			(pts
+				(xy 212.06 27.97) (xy 240.06 27.97) (xy 240.06 52.97) (xy 212.06 52.97)
+			)
+		)
+	)
 	(embedded_fonts no)

Commit message: rounded corners and fixed a few small other issues
Parts:
- moved J1 0.57 mm to (222.4, 29.9)
Routing:
- net Right_Gauge_Unbuffered: track 34.6 -> 33.0 mm
Other:
- outline, holes or cut-outs redrawn

Commit message: added caps to ground for 3V3 and 12V; changed strain gauge and op amp to 3V3_A; changed ADC DVDD to 3v3
Parts:
- added C5: 10nF, Capacitor_SMD:C_0603_1608Metric_Pad1.08x0.95mm_HandSolder, F.Cu at (218.1, 29.9)
- added C6: 10nF, Capacitor_SMD:C_0603_1608Metric_Pad1.08x0.95mm_HandSolder, F.Cu at (219.9, 51.2)
- renumbered C9 to C10, C10 to C11, C5 to C4, C6 to C9, J2 to J1, J1 to J2, JP3 to JP2, JP2 to JP3, R13 to R10, R14 to R11, R8 to R5, R7 to R6, R10 to R7, R12 to R8, R11 to R9
Connections:
- net Net-(IC1-IN1-) renamed /Reference_Buffered
- net Net-(IC1-IN2-) renamed /Center_Buffered
- net Net-(IC1-IN3-) renamed /Right_Buffered
- net Net-(IC1-IN4-) renamed /Left_Buffered
- C1 pad 1: +3V3 -> +3V3_A
- C10 pad 1: +3.3VA -> +3V3_A
- C11 pad 1: +3.3VA -> +3V3_A
- FB1 pad 2: +3.3VA -> +3V3_A
- IC1 pad 4: +3V3 -> +3V3_A
- R1 pad 1: +3V3 -> +3V3_A
- S1 pad 2: +3V3 -> +3V3_A
- S2 pad 2: +3V3 -> +3V3_A
- S3 pad 2: +3V3 -> +3V3_A
- S4 pad 2: +3V3 -> +3V3_A
- U2 pad 1: +3.3VA -> +3V3_A
- U2 pad 20: +3.3VA -> +3V3
- U2 pad 4: +3.3VA -> +3V3_A
Routing:
- net +3V3_A: track 0.00 -> 161.5 mm, vias 0 -> 4
- net +3V3: track 149.7 -> 49.2 mm, vias 5 -> 3
- net +3.3VA: track 15.6 -> 0.00 mm
- net GND: track 115.6 -> 122.5 mm
- net +12V: track 12.2 -> 15.5 mm
- net Reference_Gauge: track 42.4 -> 41.8 mm
