File: vectornav-imu/vectornav-imu.kicad_sch (KiCad schematic)
At the start: 28 parts, among them J1 M80-4201042, J2 CAN_INTERFACE, J3 SWD_PROGRAMMING, J4 REGULATED_5V_INPUT, SW1 SW_Push, SW2 SW_Push, U1 TCAN332, U2 STM32G431CBTx, U3 TLV75533PDBV

Commit message: update the jits
Parts:
- removed C11, C4, C6, C7: 100nF, symbol Device:C
- removed C14, C8: 1uF, symbol Device:C
- removed C15: 2.2uF, symbol Device:C
- removed J2: CAN_INTERFACE, symbol Connector_Generic:Conn_01x03
- removed J3: SWD_PROGRAMMING, symbol Connector_Generic:Conn_01x05
- removed J4: REGULATED_5V_INPUT, symbol Connector_Generic:Conn_01x02
- removed R2, R4: 10k, symbol Device:R
- removed R3: 1k, symbol Device:R
- removed SW2: SW_Push, symbol Switch:SW_Push
- removed U1: TCAN332, symbol Interface_CAN_LIN:TCAN332
- removed U2: STM32G431CBTx, Package_QFP:LQFP-48_7x7mm_P0.5mm, symbol MCU_ST_STM32G4:STM32G431CBTx
- removed U3: TLV75533PDBV, Package_TO_SOT_SMD:SOT-23-5, symbol Regulator_Linear:TLV75533PDBV
- added C11: 100nF, Capacitor_SMD:C_0603_1608Metric_Pad1.08x0.95mm_HandSolder, symbol Device:C_Small
- added C21, C22, C23, C24: 10uF, Capacitor_SMD:C_0805_2012Metric_Pad1.18x1.45mm_HandSolder, symbol Device:C
- added C25: 47uF, Capacitor_SMD:C_0805_2012Metric_Pad1.18x1.45mm_HandSolder, symbol Device:C
- added J2: FTSH-107-01-F-DV-K-P-TR, Connector_PinHeader_1.27mm:PinHeader_2x07_P1.27mm_Vertical_SMD, symbol Connector_Generic:Conn_02x07_Odd_Even
- added J3: Conn_01x04, Connector_PinSocket_2.54mm:PinSocket_1x04_P2.54mm_Vertical, symbol Connector_Generic:Conn_01x04
- added JP1: Force_en, Jumper:SolderJumper-2_P1.3mm_Open_Pad1.0x1.5mm, symbol Jumper:SolderJumper_2_Open
- added L3: 4.7uF, Inductor_SMD:L_Bourns_SRP5030T, symbol Device:L
- added Q1: AO3401A, Package_TO_SOT_SMD:SOT-23, symbol Transistor_FET:AO3401A
- added Q2: AO3400A, Package_TO_SOT_SMD:SOT-23, symbol Transistor_FET:AO3400A
- added R2: 221k, Resistor_SMD:R_0603_1608Metric_Pad0.98x0.95mm_HandSolder, symbol Device:R_Small
- added R3: 32.4k, Resistor_SMD:R_0603_1608Metric_Pad0.98x0.95mm_HandSolder, symbol Device:R_Small
- added R4: 56.2k, Resistor_SMD:R_0603_1608Metric_Pad0.98x0.95mm_HandSolder, symbol Device:R_Small
- added R5, R7: 10k, Resistor_SMD:R_0603_1608Metric_Pad0.98x0.95mm_HandSolder, symbol Device:R_Small
- added R6: 2.2k, Resistor_SMD:R_0603_1608Metric_Pad0.98x0.95mm_HandSolder, symbol Device:R_Small
- added U1: STM32G441KBTx, Package_QFP:LQFP-32_7x7mm_P0.8mm, symbol MCU_ST_STM32G4:STM32G441KBTx
- added U2: ISO1044BD, Package_SO:SOIC-8_3.9x4.9mm_P1.27mm, symbol Interface_CAN_LIN:ISO1044BD
- added U3: AP62300TWU, Package_TO_SOT_SMD:TSOT-23-6, symbol Regulator_Switching:AP62300TWU
- added U4: MIC5504-3.3YM5, Package_TO_SOT_SMD:SOT-23-5, symbol Regulator_Linear:MIC5504-3.3YM5
- added Y1: ECS-240-8-37B-CKY-TR, Crystal:Crystal_SMD_2016-4Pin_2.0x1.6mm, symbol Device:Crystal_GND24
- C1, C2: value 100nF -> 6.8pF; footprint (none) -> Capacitor_SMD:C_0603_1608Metric_Pad1.08x0.95mm_HandSolder; Digi PN (none) -> 311-3874-1-ND; Digi URL (none) -> https://www.digikey.com/en/products/detail/yageo/CC0603DRNP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; MFG (none) -> Yageo; MFG PN (none) -> CC0603DRNPO9BN6R8
- C10: value 1uF -> 100nF; footprint (none) -> Capacitor_SMD:C_0603_1608Metric_Pad1.08x0.95mm_HandSolder; Digi PN (none) -> 311-1140-1-ND; MFG (none) -> Yageo; MFG PN (none) -> CC0805KRX7R9BB104
- C12: value 10uF -> 1uF; footprint (none) -> Capacitor_SMD:C_0805_2012Metric_Pad1.18x1.45mm_HandSolder; Manufacturer (none) -> Samsung Electro-Mechanics; PN (none) -> CL21B105KBFNNNE
- C13: value 100nF -> 1uF; footprint (none) -> Capacitor_SMD:C_0805_2012Metric_Pad1.18x1.45mm_HandSolder; Manufacturer (none) -> Samsung Electro-Mechanics; PN (none) -> CL21B105KBFNNNE
- C3: footprint (none) -> Capacitor_SMD:C_0603_1608Metric_Pad1.08x0.95mm_HandSolder; Digi PN (none) -> 311-1344-1-ND; Digi URL (none) -> https://www.digikey.com/en/products/detail/yageo/CC0603KRX7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; MFG (none) -> Yageo; MFG PN (none) -> CC0603KRX7R9BB104
- C5: value 4.7uF -> 100nF; footprint (none) -> Capacitor_SMD:C_0603_1608Metric_Pad1.08x0.95mm_HandSolder; Digi PN (none) -> 311-1344-1-ND; Digi URL (none) -> https://www.digikey.com/en/products/detail/yageo/CC0603KRX7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; MFG (none) -> Yageo; MFG PN (none) -> CC0603KRX7R9BB104
- C9: footprint (none) -> Capacitor_SMD:C_0603_1608Metric_Pad1.08x0.95mm_HandSolder; Digi PN (none) -> 311-1140-1-ND; MFG (none) -> Yageo; MFG PN (none) -> CC0805KRX7R9BB104
- J1: footprint (none) -> formula_slug_footprint_library:HARWIN_M80-4201042
- R1: footprint (none) -> Resistor_SMD:R_0603_1608Metric_Pad0.98x0.95mm_HandSolder; Digi PN (none) -> 311-10KLDCT-ND; Digi URL (none) -> https://www.digikey.com/en/products/detail/yageo/AC0603FR-0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; MFG (none) -> Yageo; MFG PN (none) -> AC0603FR-0710KL
- SW1: value SW_Push -> Y97KT23B5NAFP; footprint (none) -> Button_Switch_SMD:SW_SPST_PTS647_Sx38; Digi PN (none) -> 108-Y97KT23B5NAFPCT-ND; Digi URL (none) -> https://www.digikey.com/en/products/detail/c-k/y97kt23b5naf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; MFG (none) -> C&K; MFG PN (none) -> Y97KT23B5NAFP
Connections:
- net MCU_NRST is gone; now on net GND: C13.1, R1.2, SW1.1
- net +3V3: now also C13.2, C5.2, J2.3 (Pin_3), U1.1 (VDD), U1.15 (VDDA), U1.17 (VDD), U2.1 (VCC1), U4.5 (VOUT); no longer C1.1, C10.1, C2.1, C3.1, C5.1, R1.1
- net +5V: now also C10.1, C12.2, C24.2, C25.2, JP1.1 (A), L3.2, Q1.2 (S), R4.1, R6.1, U2.8 (VCC2), U4.1 (VIN), U4.3 (EN); no longer C12.1, J1.1 (Pin_1)
- net BOOT0: now also R1.1, U1.31 (PB8)
- net CAN_RX: now also U1.21 (PA11), U2.3 (RXD)
- net CAN_TX: now also U1.22 (PA12), U2.2 (TXD)
- net GND: now also C12.1, C3.1, C5.1, C21.1, C22.1, C23.1, C24.1, C25.1, J2.11 (Pin_11), J2.5 (Pin_5), J2.7 (Pin_7), J3.1 (Pin_1), Q2.2 (S), R3.2, R7.2, U1.14 (VSSA), U1.16 (VSS), U1.32 (VSS), U2.4 (GND1), U2.7 (GND2), U3.1 (GND), U4.2 (GND), Y1.2, Y1.4; no longer C12.2, C13.2, C3.2, C5.2, SW1.2
- net VN_RX: now also U1.19 (PA9)
- net VN_TX: now also U1.20 (PA10)
- net SYNC_OUT: now reaches J1.4 (Pin_4)
- net SYNC_OUT: now also U1.29 (PB6)
- new net: C11.2, L3.1, U3.2 (SW)
- new net: R5.2, U3.4 (FB)
- new net: R2.2, R3.1, U3.5 (EN)
- new net: C11.1, U3.6 (BST)
- new net: R4.2, R5.1
- new net: Q1.1 (G), Q2.3 (D), R6.2
- new net +12V: C21.2, C22.2, C23.2, J3.4 (Pin_4), R2.1, U3.3 (IN)
- new net CANH: J3.3 (Pin_3), U2.6 (CANH)
- new net CANL: J3.2 (Pin_2), U2.5 (CANL)
- new net NRST: C3.2, J2.12 (Pin_12), SW1.2, U1.4 (PG10)
- new net OSC_IN: C1.1, U1.2 (PF0), Y1.3
- new net OSC_OUT: C2.1, U1.3 (PF1), Y1.1
- new net STLINK_SWCLK: J2.6 (Pin_6), U1.24 (PA14)
- new net STLINK_SWDIO: J2.4 (Pin_4), U1.23 (PA13)
- new net STLINK_SWO: J2.8 (Pin_8), U1.26 (PB3)
- new net SW_5V: J1.1 (Pin_1), JP1.2 (B), Q1.3 (D)
- new net VCP_UART_RX: J2.13 (Pin_13), U1.8 (PA3)
- new net VCP_UART_TX: J2.14 (Pin_14), U1.7 (PA2)
- new net VN_EN: Q2.1 (G), R7.1, U1.28 (PB5)
- no-connect marks 33 -> 8
Other:
- note added: "24MHz"
- note added: "Decoupling 100nF capacitors need to be placed as close to respective Vdd/Vss as possible. Note that VSS contains all VSS mcu pins for each VDD/VSS pair."
- note added: "ST-Link Programming/Debugging Connector"
- note added: "STM32G441KBTx MCU"
- moved on the sheet: J1
