File: auxiliary-test-board/auxiliary-test-board.kicad_sch (KiCad schematic)
At the start: 0 parts

Commit message: Mounting holes, auxillary board connectors, starting layout with finalized connectors?
Parts:
- added J2: FH34SRJ-12S-0.5SH(50), formula_slug_footprint_library:CONN12x1_FH34SRJ-12S-0.5SH50_HIR, symbol Connector_Generic:Conn_01x12
- added J3: FH12-12S-1SH(55), formula_slug_footprint_library:FH12-12S-1SH_55_, symbol Connector_Generic:Conn_01x12
- added J4: 1-84953-2, formula_slug_footprint_library:TE_84952-5, symbol Connector_Generic:Conn_01x12

Commit message: finish temp sense prototype flex board; make auxiliary-test-board
Parts:
- added J1: Conn_01x12, Connector_PinHeader_2.54mm:PinHeader_1x12_P2.54mm_Vertical, symbol Connector_Generic:Conn_01x12
- J4: footprint formula_slug_footprint_library:TE_84952-5 -> Connector_FFC-FPC:TE_1-84953-2_1x12-1MP_P1.0mm_Horizontal
Connections:
- net V-: now reaches J2.1 (Pin_1)
- net V-: now also J3.1 (Pin_1), J4.1 (Pin_1), J1.12 (Pin_12)
- net TP2: now reaches J2.10 (Pin_10)
- net TP2: now also J3.10 (Pin_10), J4.10 (Pin_10), J1.3 (Pin_3)
- net TP1: now reaches J2.11 (Pin_11)
- net TP1: now also J3.11 (Pin_11), J4.11 (Pin_11), J1.2 (Pin_2)
- net TP0: now reaches J2.12 (Pin_12)
- net TP0: now also J3.12 (Pin_12), J4.12 (Pin_12), J1.1 (Pin_1)
- net SCL: now reaches J2.2 (Pin_2)
- net SCL: now also J3.2 (Pin_2), J4.2 (Pin_2), J1.11 (Pin_11)
- net SDA: now reaches J2.3 (Pin_3)
- net SDA: now also J3.3 (Pin_3), J4.3 (Pin_3), J1.10 (Pin_10)
- net +5V: now reaches J2.4 (Pin_4)
- net +5V: now also J3.4 (Pin_4), J4.4 (Pin_4), J1.9 (Pin_9)
- net v3: now reaches J2.5 (Pin_5)
- net v3: now also J3.5 (Pin_5), J4.5 (Pin_5), J1.8 (Pin_8)
- net v2: now reaches J2.6 (Pin_6)
- net v2: now also J3.6 (Pin_6), J4.6 (Pin_6), J1.7 (Pin_7)
- net v1: now reaches J2.7 (Pin_7)
- net v1: now also J3.7 (Pin_7), J4.7 (Pin_7), J1.6 (Pin_6)
- net v0: now reaches J2.8 (Pin_8)
- net v0: now also J3.8 (Pin_8), J4.8 (Pin_8), J1.5 (Pin_5)
- net TP3: now reaches J2.9 (Pin_9)
- net TP3: now also J3.9 (Pin_9), J4.9 (Pin_9), J1.4 (Pin_4)
Other:
- moved on the sheet: J3, J4
