File: strain-gauges/amplifier-board/AmpliferBoard/AmpliferBoard.kicad_sch (KiCad schematic)
At the start: 17 parts, among them J1 Conn_01x07, U1 MCP3564R-E/ST

Commit message: AmpBoard Schematic adjustments
Parts:
- removed TP1, TP2, TP3, TP4, TP5, TP6, TP7: TestPoint, TestPoint:TestPoint_Pad_1.0x1.0mm, symbol Connector:TestPoint
- added J2: Conn_01x07, symbol Connector_Generic:Conn_01x07
- C1: value 10nF -> 1nF
- R2: value V_Gauge -> A_Gauge
Connections:
- net +3V3_A is gone; now on net +3V3: FB1.2
Other:
- moved on the sheet: FB1, J1

Commit message: Upload Prototype Projects
Completed FPC Type B.
Changed to design:
Each FPC Gauge will now have its own bridge on the gauge itself. They will output a differential voltage that connects to the main amplifier board that is standalone.
Parts:
- added C2: 10uF, Capacitor_SMD:C_0402_1005Metric, symbol Device:C
- added C3: 100nF, Capacitor_SMD:C_0402_1005Metric, symbol Device:C
- added C4, C5, C6: 1nF, Capacitor_SMD:C_0402_1005Metric, symbol Device:C
- added R10, R15, R16, R21, R22, R9: 100, Resistor_SMD:R_0402_1005Metric, symbol Device:R
- added R11: A_Gauge, Connector_PinHeader_2.54mm:PinHeader_1x03_P2.54mm_Vertical_SMD_Pin1Left, symbol Device:R
- added R12, R14, R18, R20, R24, R8: 350, Resistor_SMD:R_0402_1005Metric, symbol Device:R
- added R13: R_Gauge, symbol Device:R
- added R17, R23: A_Gauge, symbol Device:R
- added R19: R_Gauge, Connector_PinHeader_2.54mm:PinHeader_1x03_P2.54mm_Vertical_SMD_Pin1Left, symbol Device:R
- added R7: R_Gauge, Connector_PinHeader_2.54mm:PinHeader_1x03_P2.54mm_Vertical, symbol Device:R
- added U2: LDK320AM33R, symbol formula_slug_symbol_library:LDK320AM33R
- FB1: value FerriteBead -> FCM 1608KF-601T03; footprint (none) -> Inductor_SMD:L_0603_1608Metric_Pad1.05x0.95mm_HandSolder; Digikey Part Number (none) -> 4816-FCM1608KF-601T03CT-ND; Digikey URL (none) -> https://mm.digikey.com/Volume0/opasdata/d220001/medias/docu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; Manufacturer (none) -> TAI-TECH Advanced Electronics Co., Ltd.
- J1: value Conn_01x07 -> Out Conn; footprint (none) -> Connector_PinHeader_2.54mm:PinHeader_1x07_P2.54mm_Vertical
- J2: value Conn_01x07 -> Input Conn; footprint (none) -> Connector_PinHeader_2.54mm:PinHeader_1x07_P2.54mm_Vertical
- R1: footprint TestPoint:TestPoint_Pad_1.0x1.0mm -> Connector_PinHeader_2.54mm:PinHeader_1x03_P2.54mm_Vertical_SMD_Pin1Left
- R2: footprint TestPoint:TestPoint_Pad_1.0x1.0mm -> (none)
- U1: footprint TSSOP20_ST_MCH -> formula_slug_footprint_library:MCP3564R-EST
Connections:
- net +3V3: now also J2.6 (Pin_6)
- net ADC_CS: now also J2.1 (Pin_1)
- net GND: now also J2.7 (Pin_7), C2.2, C3.2, R12.2, R14.2, R18.2, R20.2, R24.2, R8.2
- net SPI_DRDY: now also J2.5 (Pin_5)
- net SPI_MISO: now also J2.4 (Pin_4)
- net SPI_MOSI: now also J2.3 (Pin_3)
- net SPI_SCK: now also J2.2 (Pin_2)
- net Bridge3B_Out: now reaches U1.10 (CH5)
- net Bridge3B_Out: now also C5.2, R16.2
- net Bridge4B_Out: now reaches U1.11 (CH6)
- net Bridge4B_Out: now also C6.2, R22.2
- net Bridge4A_Out: now reaches U1.12 (CH7)
- net Bridge4A_Out: now also C6.1, R21.2
- net Bridge2A_Out: now reaches U1.7 (CH2)
- net Bridge2A_Out: now also C4.1, R9.2
- net Bridge2B_Out: now reaches U1.8 (CH3)
- net Bridge2B_Out: now also C4.2, R10.2
- net Bridge3A_Out: now reaches U1.9 (CH4)
- net Bridge3A_Out: now also C5.1, R15.2
- net 3V3_Filtered renamed +3V3_A
- net +3V3_A: now also C2.1, C3.1, R11.1, R13.1, R17.1, R19.1, R23.1, R7.1
- net BRIDGE_N: no longer names the net of R1.2, R3.1, R6.1
- net BRIDGE_P: no longer names the net of R2.2, R4.1, R5.1
- net Hori_Out renamed Bridge1A_Out
- net Vert_Out renamed Bridge1B_Out
- new net: R19.2, R20.1, R21.1
- new net: R16.1, R17.2, R18.1
- new net: R13.2, R14.1, R15.1
- new net: R7.2, R8.1, R9.1
- new net: R22.1, R23.2, R24.1
- new net: R10.1, R11.2, R12.1
Other:
- moved on the sheet: FB1, R3, R4
