File: strain-gauges/single-strain-gauge/FPCSingleGaugeTypeB/FPCSingleGaugeTypeB.kicad_sch (KiCad schematic)
At the start: 8 parts, among them J3 Conn_01x04

Commit message: Finish Amp Board
Main connection point to fpc gauges
Parts:
- J3: footprint (none) -> Connector_PinHeader_2.54mm:PinHeader_1x04_P2.54mm_Vertical
