File: strain-gauges/single-strain-gauge/FPCSingleGaugeTypeB/FPCSingleGaugeTypeB.kicad_pcb (KiCad board)
At the start: 4 copper layers, 43 x 49.5 mm, 6 parts, among them J3 Conn_01x04

Commit message: Fix DRC and Setup Errors
Routing:
- net GND: track 0.00 -> 14.0 mm, vias 0 -> 3
