File: strain-gauges/amplifier-board/AmpBoardTypeB/AmpBoardTypeB.kicad_sch (KiCad schematic)
At the start: 35 parts, among them J1 Out Conn, J2 Input Conn, U1 MCP3564R-E/ST, U2 LDK320AM33R

Commit message: Last minute changes
Parts:
- removed C1, C4, C5, C6: 1nF, Capacitor_SMD:C_0402_1005Metric, symbol Device:C
- removed R1, R19: R_Gauge, Connector_PinHeader_2.54mm:PinHeader_1x03_P2.54mm_Vertical_SMD_Pin1Left, symbol Device:R
- removed R10, R15, R16, R21, R22, R5, R6, R9: 100, Resistor_SMD:R_0402_1005Metric, symbol Device:R
- removed R11: A_Gauge, Connector_PinHeader_2.54mm:PinHeader_1x03_P2.54mm_Vertical_SMD_Pin1Left, symbol Device:R
- removed R12, R14, R18, R20, R24, R3, R4, R8: 350, Resistor_SMD:R_0402_1005Metric, symbol Device:R
- removed R13: R_Gauge, symbol Device:R
- removed R17, R2, R23: A_Gauge, symbol Device:R
- removed R7: R_Gauge, Connector_PinHeader_2.54mm:PinHeader_1x03_P2.54mm_Vertical, symbol Device:R
- removed U2: LDK320AM33R, symbol formula_slug_symbol_library:LDK320AM33R
- added J3, J4, J5, J6: Conn_01x04, Connector_PinHeader_2.54mm:PinHeader_1x04_P2.54mm_Vertical, symbol Connector_Generic:Conn_01x04
Connections:
- net +3V3_A: now also J3.2 (Pin_2), J4.2 (Pin_2), J5.2 (Pin_2), J6.2 (Pin_2)
- net Bridge1A_Out: now also J3.3 (Pin_3)
- net Bridge1B_Out: now also J3.4 (Pin_4)
- net Bridge2A_Out: now also J4.3 (Pin_3)
- net Bridge2B_Out: now also J4.4 (Pin_4)
- net Bridge3A_Out: now also J5.3 (Pin_3)
- net Bridge3B_Out: now also J5.4 (Pin_4)
- net Bridge4A_Out: now also J6.4 (Pin_4)
- net Bridge4B_Out: now also J6.3 (Pin_3)
- net GND: now also J3.1 (Pin_1), J4.1 (Pin_1), J5.1 (Pin_1), J6.1 (Pin_1)
Other:
- note removed: "Wheatstone Half Bridge"
