File: rt-simulator-interface/rt-simulator-interface.kicad_sch (KiCad schematic)
At the start: 0 parts

Commit message: Added NUCLEO-G491RE symbol
Created NUCLEO-G491RE symbol
Added NUCLEO-G491RE symbol to main schematic sheet
Parts:
- added U1: (no value), Module:ST_Morpho_Connector_144_STLink, symbol Symbol:NUCLEO-G491RE
Changed lines of the file:
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@@
+		)
+	)
+	(symbol
+		(lib_id "Symbol:NUCLEO-G491RE")
+		(at 74.93 73.66 0)
+		(unit 1)
+		(body_style 1)
+		(exclude_from_sim no)
+		(in_bom yes)
+		(on_board yes)
+		(in_pos_files yes)
+		(dnp no)
+		(fields_autoplaced yes)
+		(property "Reference" "U1"
+			(at 74.93 43.18 0)
+			(show_name no)
+			(do_not_autoplace no)
+			(effects
+				(font
+					(size 1.27 1.27)
+				)
+			)
+		)
+		(property "Value" ""
+			(at 74.93 73.66 0)
+			(show_name no)
+			(do_not_autoplace no)
+			(effects
+				(font
+					(size 1.27 1.27)
+				)
+			)
+		)
+		(property "Footprint" "Module:ST_Morpho_Connector_144_STLink"
+			(at 74.93 73.66 0)
+			(hide yes)
+			(show_name no)
+			(do_not_autoplace no)
+			(effects
+				(font
+					(size 1.27 1.27)
+				)
+			)
+		)
+		(property "Datasheet" ""
+			(at 74.93 73.66 0)
+			(hide yes)
+			(show_name no)
+			(do_not_autoplace no)
+			(effects
+				(font
+					(size 1.27 1.27)
+				)
+			)
+		)
+		(property "Description" ""
+			(at 74.93 73.66 0)
+			(hide yes)
+			(show_name no)
+			(do_not_autoplace no)
+			(effects
+				(font
+					(size 1.27 1.27)
+				)
+			)
+		)
+		(pin "CN7_4"
+		)
+		(pin "CN7_5"
+		)
+		(pin "CN7_13"
+		)
+		(pin "CN7_2"
+		)
+		(pin "CN7_6"
+		)
+		(pin "CN7_3"
+		)
+		(pin "CN7_14"
+		)
+		(pin "CN7_11"
+		)
+		(pin "CN7_12"
+		)
+		(pin "CN7_10"
+		)
+		(pin "CN7_8"
+		)
+		(pin "CN7_7"
+		)
+		(pin "CN7_1"
+		)
+		(pin "CN7_9"
+		)
+		(pin "CN10_37"
+		)
+		(pin "CN10_34"
+		)
+		(pin "CN10_38"
+		)
+		(pin "CN10_36"
+		)
+		(pin "CN10_33"
+		)
+		(pin "CN10_35"
+		)
+		(pin "CN10_32"
+		)
+		(pin "CN10_31"
+		)
+		(pin "CN10_30"
+		)
+		(pin "CN7_21"
+		)
+		(pin "CN7_22"
+		)
+		(pin "CN7_37"
+		)
+		(pin "CN7_16"
+		)
+		(pin "CN7_19"
+		)
+		(pin "CN7_35"
+		)
+		(pin "CN7_36"
+		)
+		(pin "CN7_28"
+		)
+		(pin "CN7_30"
+		)
+		(pin "CN7_18"
+		)
+		(pin "CN7_29"
+		)
+		(pin "CN7_38"
+		)
+		(pin "CN7_26"
+		)
+		(pin "CN7_34"
+		)
+		(pin "CN10_2"
+		)
+		(pin "CN7_27"
+		)
+		(pin "CN10_1"
+		)
+		(pin "CN7_32"
+		)
+		(pin "CN10_7"
+		)
+		(pin "CN7_23"
+		)
+		(pin "CN10_5"
+		)
+		(pin "CN10_6"
+		)
+		(pin "CN7_15"
+		)
+		(pin "CN7_24"
+		)
+		(pin "CN10_8"
+		)
+		(pin "CN7_31"
+		)
+		(pin "CN7_33"
+		)
+		(pin "CN10_3"
+		)
+		(pin "CN7_20"
+		)
+		(pin "CN10_4"
+		)
+		(pin "CN7_25"
+		)
+		(pin "CN7_17"
+		)
+		(pin "CN10_14"
+		)
+		(pin "CN10_22"
+		)
+		(pin "CN10_15"
+		)
+		(pin "CN10_19"
+		)
+		(pin "CN10_28"
+		)
+		(pin "CN10_29"
+		)
+		(pin "CN10_12"
+		)
+		(pin "CN10_17"
+		)
+		(pin "CN10_23"
+		)
+		(pin "CN10_9"
+		)
+		(pin "CN10_13"
+		)
+		(pin "CN10_18"
+		)
+		(pin "CN10_16"
+		)
+		(pin "CN10_21"
+		)
+		(pin "CN10_10"
+		)
+		(pin "CN10_25"
+		)
+		(pin "CN10_26"
+		)
+		(pin "CN10_24"
+		)
+		(pin "CN10_20"
+		)
+		(pin "CN10_11"
+		)
+		(pin "CN10_27"
+		)
+		(instances
+			(project "rt-simulator-interface"
+				(path "/e994741c-7c7d-4124-9d00-43b883baa61d"
+					(reference "U1")
+					(unit 1)
+				)
+			)
 		)
 	)
